File: hardware/kicad/1_Connectors.kicad_sch (KiCad schematic)
At the start: 27 parts, among them CN12 5017, CN13 B4B-PH-K-S(LF)(SN), Q68 CSD17577Q5A, U155 MT9700-N, U156 150uF, U181 LM5050MKX-1/NOPB, U81 DS1021-2x13SF11-B

Commit message: sub modules
Other:
- added sheet Connectors 12V JST (29_Connectors-12V-JST.kicad_sch)
- added sheet Connectors 5V JST (34_Connectors-5v-JST.kicad_sch)
- added sheet Connectors ESC (20_Connectors-ESC.kicad_sch)
- added sheet Connectors Wire To Board (32_Connectors-wire-to-board.kicad_sch)
