File: hardware/kicad/30_Microcontroller extra.kicad_sch (KiCad schematic)
At the start: 15 parts, among them U183 Teensy4.0, U191 CH343P

Commit message: sub modules
Parts:
- U183: footprint teensy:Teensy40 -> teensy:Teensy41
