File: hardware/kicad/untitled.kicad_sch (KiCad schematic)
At the start: 1 part

Commit message: netties and better sheet nesting for servo connectors
Parts:
- removed H7: MountingHoles_and_outline_mikroeclick4_stm32f7, 5v rail sm-easyedapro:stm32f7MikroeClick4Model, symbol 5v rail sm-easyedapro:MountingHoles_and_outline_mikroeclick4_stm32f7
Changed lines of the file:
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@@
 	(generator_version "9.0")
 	(paper "A4")
-	(symbol
-		(lib_id "5v rail sm-easyedapro:MountingHoles_and_outline_mikroeclick4_stm32f7")
-		(at 74.93 81.28 0)
-		(unit 1)
-		(exclude_from_sim no)
-		(in_bom no)
-		(on_board yes)
-		(dnp no)
-		(fields_autoplaced yes)
-		(property "Reference" "H7"
-			(at 93.98 74.9299 0)
-			(effects
-				(font
-					(size 1.27 1.27)
-				)
-				(justify left)
-			)
-		)
-		(property "Value" "MountingHoles_and_outline_mikroeclick4_stm32f7"
-			(at 93.98 77.4699 0)
-			(effects
-				(font
-					(size 1.27 1.27)
-				)
-				(justify left)
-			)
-		)
-		(property "Footprint" "5v rail sm-easyedapro:stm32f7MikroeClick4Model"
-			(at 74.93 81.28 0)
-			(effects
-				(font
-					(size 1.27 1.27)
-				)
-				(hide yes)
-			)
-		)
-		(property "Datasheet" "~"
-			(at 74.93 81.28 0)
-			(effects
-				(font
-					(size 1.27 1.27)
-				)
-				(hide yes)
-			)
-		)
-		(property "Description" "Mounting Hole without connection"
-			(at 83.058 84.328 0)
-			(effects
-				(font
-					(size 1.27 1.27)
-				)
-				(hide yes)
-			)
-		)
-		(instances
-			(project ""
-				(path "/3f85abf4-0b95-4c4a-b7e9-06f59ca1ea3d/59bb4b63-0f85-41ba-9593-c1b306c47470"
-					(reference "H7")
-					(unit 1)
-				)
-			)
-		)
-	)
 )
