File: hardware/kicad/12v_LTM8055_BUCK.kicad_sch (KiCad schematic)
At the start: 23 parts, among them U44 MCP4725A0T-E/CH, U47 LTM8055IY_PBF, U48 68uF

Commit message: starting erc check
Parts:
- C51, C52, C58: footprint Capacitor_SMD:C_0805_2012Metric -> 5v rail sm-easyedapro:C0805
- C53, C54, C55, C57: footprint Capacitor_SMD:C_0603_1608Metric -> 5v rail sm-easyedapro:C0603
- H2: footprint Connector_PinHeader_2.54mm:PinHeader_2x01_P2.54mm_Vertical -> 5v rail sm-easyedapro:HDR-TH_2P-P2.54-V-M
- R106, R109, R110, R111: footprint Resistor_SMD:R_0603_1608Metric -> 5v rail sm-easyedapro:R0603
- R112: footprint Resistor_SMD:R_2512_6332Metric -> 5v rail sm-easyedapro:R2512
- U44: footprint Package_TO_SOT_SMD:SOT-23-6 -> 5v rail sm-easyedapro:SOT-23-6_L2.9-W1.6-P0.95-LS2.8-BL
Changed lines of the file:
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@@
 			)
 		)
-		(property "Footprint" "Capacitor_SMD:C_0805_2012Metric"
+		(property "Footprint" "5v rail sm-easyedapro:C0805"
 			(at 30.48 91.44 0)
 			(effects
@@
 			)
 		)
-		(property "Footprint" "Connector_PinHeader_2.54mm:PinHeader_2x01_P2.54mm_Vertical"
+		(property "Footprint" "5v rail sm-easyedapro:HDR-TH_2P-P2.54-V-M"
 			(at 77.47 85.09 0)
 			(effects
@@
 			)
 		)
-		(property "Description" ""
+		(property "Description" "Power symbol creates a global label with name \"GND\" , ground"
 			(at 95.25 110.49 0)
 			(effects
@@
 			)
 		)
-		(property "Footprint" "Capacitor_SMD:C_0603_1608Metric"
+		(property "Footprint" "5v rail sm-easyedapro:C0603"
 			(at 95.25 104.14 0)
 			(effects
@@
 			)
 		)
-		(property "Footprint" "Resistor_SMD:R_0603_1608Metric"
+		(property "Footprint" "5v rail sm-easyedapro:R0603"
 			(at 120.65 105.41 0)
 			(effects
@@
 			)
 		)
-		(property "Footprint" "Resistor_SMD:R_0603_1608Metric"
+		(property "Footprint" "5v rail sm-easyedapro:R0603"
 			(at 227.33 74.93 0)
 			(effects
@@
 			)
 		)
-		(property "Description" ""
+		(property "Description" "Power symbol creates a global label with name \"GND\" , ground"
 			(at 180.34 144.78 0)
 			(effects
@@
 			)
 		)
-		(property "Footprint" "Resistor_SMD:R_0603_1608Metric"
+		(property "Footprint" "5v rail sm-easyedapro:R0603"
 			(at 227.33 90.17 0)
 			(effects
@@
 			)
 		)
-		(property "Footprint" "Capacitor_SMD:C_0805_2012Metric"
+		(property "Footprint" "5v rail sm-easyedapro:C0805"
 			(at 43.18 91.44 0)
 			(effects
@@
 			)
 		)
-		(property "Description" ""
+		(property "Description" "Power symbol creates a global label with name \"GND\" , ground"
 			(at 106.68 162.56 0)
 			(effects
@@
 			)
 		)
-		(property "Description" ""
+		(property "Description" "Power symbol creates a global label with name \"GND\" , ground"
 			(at 72.39 168.91 0)
 			(effects
@@
 			)
 		)
-		(property "Footprint" "Resistor_SMD:R_2512_6332Metric"
+		(property "Footprint" "5v rail sm-easyedapro:R2512"
 			(at 257.81 66.04 0)
 			(effects
@@
 			)
 		)
-		(property "Footprint" "Capacitor_SMD:C_0603_1608Metric"
+		(property "Footprint" "5v rail sm-easyedapro:C0603"
 			(at 80.01 156.21 0)
 			(effects
@@
 			)
 		)
-		(property "Description" ""
+		(property "Description" "Power symbol creates a global label with name \"GND\" , ground"
 			(at 200.66 106.68 0)
 			(effects
@@
 			)
 		)
-		(property "Footprint" "Capacitor_SMD:C_0603_1608Metric"
+		(property "Footprint" "5v rail sm-easyedapro:C0603"
 			(at 64.77 156.21 0)
 			(effects
@@
 			)
 		)
-		(property "Footprint" "Resistor_SMD:R_0603_1608Metric"
+		(property "Footprint" "5v rail sm-easyedapro:R0603"
 			(at 54.61 92.71 0)
 			(effects
@@
 			)
 		)
-		(property "Description" ""
+		(property "Description" "Power symbol creates a global label with name \"GND\" , ground"
 			(at 238.76 105.41 0)
 			(effects
@@
 			)
 		)
-		(property "Description" "Power-5V"
+		(property "Description" "Power symbol creates a global label with name \"+3V3\""
 			(at 64.77 142.24 0)
 			(effects
@@
 			)
 		)
-		(property "Footprint" "Capacitor_SMD:C_0603_1608Metric"
+		(property "Footprint" "5v rail sm-easyedapro:C0603"
 			(at 180.34 134.62 0)
 			(effects
@@
 			)
 		)
-		(property "Footprint" "Capacitor_SMD:C_0805_2012Metric"
+		(property "Footprint" "5v rail sm-easyedapro:C0805"
 			(at 238.76 82.55 0)
 			(effects
@@
 			)
 		)
-		(property "Footprint" "Package_TO_SOT_SMD:SOT-23-6"
+		(property "Footprint" "5v rail sm-easyedapro:SOT-23-6_L2.9-W1.6-P0.95-LS2.8-BL"
 			(at 106.68 144.78 0)
 			(effects
@@
 			)
 		)
-		(property "Datasheet" ""
+		(property "Datasheet" "~"
 			(at 166.37 124.46 0)
 			(effects
@@
 			)
 		)
-		(property "Description" ""
+		(property "Description" "Jumper, 2-pole, closed/bridged"
 			(at 166.37 124.46 0)
 			(effects
@@
 			)
 		)
-		(property "Description" ""
+		(property "Description" "Power symbol creates a global label with name \"GND\" , ground"
 			(at 120.65 120.65 0)
 			(effects
@@
 			)
 		)
-		(property "Description" ""
+		(property "Description" "Power symbol creates a global label with name \"GND\" , ground"
 			(at 30.48 119.38 0)
 			(effects

Commit message: more fixes
Parts:
- removed R106: 100kΩ, 5v rail sm-easyedapro:R0603, symbol 5v rail sm-easyedapro:FRC0603J104 TS
- added R1401: 100k, Resistor_SMD:R_0402_1005Metric, symbol Device:R
Connections:
- net EN: now also R1401.1
- net GND: now also R1401.2
Changed lines of the file:
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@@
 	(wire
 		(pts
-			(xy 54.61 114.3) (xy 54.61 97.79)
+			(xy 54.61 114.3) (xy 54.61 95.25)
 		)
 		(stroke
@@
 	)
 	(symbol
-		(lib_id "5v rail sm-easyedapro:CC0603KRX7R9BB104")
-		(at 64.77 156.21 90)
+		(lib_id "Device:R")
+		(at 54.61 91.44 0)
 		(unit 1)
 		(exclude_from_sim no)
@@
 		(on_board yes)
 		(dnp no)
-		(property "Reference" "C53"
-			(at 68.58 156.21 90)
-			(effects
-				(font
-					(size 1.27 1.27)
-				)
-				(justify right top)
-			)
-		)
-		(property "Value" "100nF"
-			(at 68.58 158.75 90)
-			(effects
-				(font
-					(size 1.27 1.27)
-				)
-				(justify right top)
-			)
-		)
-		(property "Footprint" "5v rail sm-easyedapro:C0603"
-			(at 64.77 156.21 0)
-			(effects
-				(font
-					(size 1.27 1.27)
-				)
-				(hide yes)
-			)
-		)
-		(property "Datasheet" "https://atta.szlcsc.com/upload/public/pdf/source/20180910/C282072_33301C7F631E79921B82A8DAC6BCC5B3.pdf"
-			(at 64.77 156.21 0)
-			(effects
-				(font
-					(size 1.27 1.27)
-				)
-				(hide yes)
-			)
-		)
-		(property "Description" "Capacitance:100nF Tolerance:±10% Tolerance:±10% Voltage Rating:50V Temperature Coefficient:X7R"
-			(at 64.77 156.21 0)
-			(effects
-				(font
-					(size 1.27 1.27)
-				)
-				(hide yes)
-			)
-		)
-		(property "Manufacturer Part" "CC0603KRX7R9BB104"
-			(at 64.77 156.21 0)
+		(fields_autoplaced yes)
+		(property "Reference" "R1401"
+			(at 57.15 90.1699 0)
 			(effects
 				(font
 					(size 1.27 1.27)
 				)
-				(hide yes)
+				(justify left)
 			)
 		)
-		(property "Manufacturer" "YAGEO(国巨)"
-			(at 64.77 156.21 0)
+		(property "Value" "100k"
+			(at 57.15 92.7099 0)
 			(effects
 				(font
 					(size 1.27 1.27)
 				)
-				(hide yes)
+				(justify left)
 			)
 		)
-		(property "Supplier Part" "C14663"
-			(at 64.77 156.21 0)
+		(property "Footprint" "Resistor_SMD:R_0402_1005Metric"
+			(at 52.832 91.44 90)
 			(effects
 				(font
@@
 			)
 		)
-		(property "Supplier" "LCSC"
-			(at 64.77 156.21 0)
+		(property "Datasheet" "~"
+			(at 54.61 91.44 0)
 			(effects
 				(font
@@
 			)
 		)
-		(property "LCSC Part Name" "100nF ±10% 50V"
-			(at 64.77 156.21 0)
+		(property "Description" "Resistor"
+			(at 54.61 91.44 0)
 			(effects
 				(font
@@
 		)
 		(instances
-			(project "svea_powerboard_rev3"
+			(project ""
 				(path "/3f85abf4-0b95-4c4a-b7e9-06f59ca1ea3d/5c2e021f-c2d4-49e2-8c36-9a64f1f12001/535c4b9d-dd70-4891-8336-b5700298b4d1"
-					(reference "C53")
+					(reference "R1401")
 					(unit 1)
 				)
@@
 	)
 	(symbol
-		(lib_id "5v rail sm-easyedapro:FRC0603J104 TS")
-		(at 54.61 92.71 90)
+		(lib_id "5v rail sm-easyedapro:CC0603KRX7R9BB104")
+		(at 64.77 156.21 90)
 		(unit 1)
 		(exclude_from_sim no)
@@
 		(on_board yes)
 		(dnp no)
-		(property "Reference" "R106"
-			(at 57.15 92.71 90)
+		(property "Reference" "C53"
+			(at 68.58 156.21 90)
 			(effects
 				(font
@@
 			)
 		)
-		(property "Value" "100kΩ"
-			(at 57.15 95.25 90)
+		(property "Value" "100nF"
+			(at 68.58 158.75 90)
 			(effects
 				(font
@@
 			)
 		)
-		(property "Footprint" "5v rail sm-easyedapro:R0603"
-			(at 54.61 92.71 0)
+		(property "Footprint" "5v rail sm-easyedapro:C0603"
+			(at 64.77 156.21 0)
 			(effects
 				(font
@@
 			)
 		)
-		(property "Datasheet" ""
-			(at 54.61 92.71 0)
+		(property "Datasheet" "https://atta.szlcsc.com/upload/public/pdf/source/20180910/C282072_33301C7F631E79921B82A8DAC6BCC5B3.pdf"
+			(at 64.77 156.21 0)
 			(effects
 				(font
@@
 			)
 		)
-		(property "Description" "Type:Thick Film Resistor Resistance:100kΩ Tolerance:±5% Tolerance:±5% Power(Watts):100mW Voltage-Supply(Max):75V Temperature Coefficient:±100ppm/°C Temperature Coefficient:±100ppm/°C Operating Temperature:-55°C~+155°C Operating Temperature:-55°C~+155°C"
-			(at 54.61 92.71 0)
+		(property "Description" "Capacitance:100nF Tolerance:±10% Tolerance:±10% Voltage Rating:50V Temperature Coefficient:X7R"
+			(at 64.77 156.21 0)
 			(effects
 				(font
@@
 			)
 		)
-		(property "Manufacturer Part" "FRC0603J104 TS"
-			(at 54.61 92.71 0)
+		(property "Manufacturer Part" "CC0603KRX7R9BB104"
+			(at 64.77 156.21 0)
 			(effects
 				(font
@@
 			)
 		)
-		(property "Manufacturer" "FOJAN(富捷)"
-			(at 54.61 92.71 0)
+		(property "Manufacturer" "YAGEO(国巨)"
+			(at 64.77 156.21 0)
 			(effects
 				(font
@@
 			)
 		)
-		(property "Supplier Part" "C2907088"
-			(at 54.61 92.71 0)
+		(property "Supplier Part" "C14663"
+			(at 64.77 156.21 0)
 			(effects
 				(font
@@
 		)
 		(property "Supplier" "LCSC"
-			(at 54.61 92.71 0)
+			(at 64.77 156.21 0)
 			(effects
 				(font
@@
 			)
 		)
-		(property "LCSC Part Name" "100kΩ ±5% 100mW 厚膜电阻"
-			(at 54.61 92.71 0)
+		(property "LCSC Part Name" "100nF ±10% 50V"
+			(at 64.77 156.21 0)
 			(effects
 				(font
@@
 			(project "svea_powerboard_rev3"
 				(path "/3f85abf4-0b95-4c4a-b7e9-06f59ca1ea3d/5c2e021f-c2d4-49e2-8c36-9a64f1f12001/535c4b9d-dd70-4891-8336-b5700298b4d1"
-					(reference "R106")
+					(reference "C53")
 					(unit 1)
 				)

Commit message: more updates
Parts:
- removed C50: 100uF, 5v rail sm-easyedapro:CAP-SMD_BD6.3-L6.6-W6.6-LS7.6-RD, symbol 5v rail sm-easyedapro:RVT1H101M0607
- removed C51, C52: 4.7uF, 5v rail sm-easyedapro:C0805, symbol 5v rail sm-easyedapro:CL21A475KBQNNNE
- removed C58: 22uF, 5v rail sm-easyedapro:C0805, symbol 5v rail sm-easyedapro:CL21A226MAQNNNE
- removed C59: 47uF, 5v rail sm-easyedapro:CAP-SMD_BD6.3-L6.6-W6.6-LS7.6-FD, symbol 5v rail sm-easyedapro:RVT1H470M0607
- removed C60: 470uF, 5v rail sm-easyedapro:CAP-SMD_BD10.0-L10.3-W10.3-LS11.0-R-RD, symbol 5v rail sm-easyedapro:RVT1V471M1010-C72519
- removed R110: 100kΩ, 5v rail sm-easyedapro:R0603, symbol 5v rail sm-easyedapro:0603WAF1003T5E
- removed R111: 11kΩ, 5v rail sm-easyedapro:R0603, symbol 5v rail sm-easyedapro:FRC0603F1102TS
- removed U48: 68uF, 5v rail sm-easyedapro:CAP-SMD_BD6.3-L6.6-W6.6-LS7.4-FD, symbol 5v rail sm-easyedapro:RVT1E680M0605
- added C1401, C1402: 4.7u, Capacitor_SMD:C_1210_3225Metric, symbol Device:C
- added C1403: 22uF, Capacitor_SMD:C_0805_2012Metric, symbol Device:C
- added R1402: 100k, Resistor_SMD:R_0402_1005Metric, symbol Device:R
- added R1403: 11k, Resistor_SMD:R_0402_1005Metric, symbol Device:R
- added SWITCHTODATASHEETERCOMMENDED1401: 68uF, 5v rail sm-easyedapro:CAP-SMD_BD6.3-L6.6-W6.6-LS7.4-FD, symbol 5v rail sm-easyedapro:RVT1E680M0605
Connections:
- net GND: now also C1401.2, C1402.2, C1403.2, R1403.2, SWITCHTODATASHEETERCOMMENDED1401.2
- net IN: now also C1401.1, C1402.1
- net OUT: now also C1403.1, SWITCHTODATASHEETERCOMMENDED1401.1
- net at U47.J1 (FB): now also R1402.2, R1403.1
- net at R112.1, U47.A1 (VOUT), U47.A2 (VOUT)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: now also R1402.1

Commit message: almost done 12v buck
Parts:
- removed C55: 220nF, 5v rail sm-easyedapro:C0603, symbol 5v rail sm-easyedapro:CL10B224KB8NNNC
- added C1404: 220nF, Capacitor_SMD:C_0402_1005Metric, symbol Device:C
Connections:
- net GND: now also C1404.2
- net OUT: no longer C1403.1, SWITCHTODATASHEETERCOMMENDED1401.1
- net at U47.K1 (SS): now also C1404.1
- net at R112.1, R1402.1, U47.A1 (VOUT)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: now also C1403.1, SWITCHTODATASHEETERCOMMENDED1401.1
Other:
- moved on the sheet: C1403, SWITCHTODATASHEETERCOMMENDED1401
Changed lines of the file:
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@@
 	(text "7.5ms"
 		(exclude_from_sim no)
-		(at 98.806 102.616 0)
+		(at 99.06 100.838 0)
 		(effects
 			(font
@@
 	(wire
 		(pts
-			(xy 238.76 87.63) (xy 238.76 99.06)
+			(xy 238.76 83.82) (xy 238.76 99.06)
 		)
 		(stroke
@@
 	(wire
 		(pts
-			(xy 238.76 66.04) (xy 238.76 77.47)
+			(xy 238.76 66.04) (xy 238.76 76.2)
 		)
 		(stroke
@@
 	)
 	(symbol
-		(lib_id "5v rail sm-easyedapro:CL10B224KB8NNNC")
-		(at 95.25 104.14 90)
-		(unit 1)
-		(exclude_from_sim no)
-		(in_bom yes)
-		(on_board yes)
-		(dnp no)
-		(property "Reference" "C55"
-			(at 99.06 105.41 90)
-			(effects
-				(font
-					(size 1.27 1.27)
-				)
-				(justify right top)
-			)
-		)
-		(property "Value" "220nF"
-			(at 99.06 107.95 90)
-			(effects
-				(font
-					(size 1.27 1.27)
-				)
-				(justify right top)
-			)
-		)
-		(property "Footprint" "5v rail sm-easyedapro:C0603"
-			(at 95.25 104.14 0)
-			(effects
-				(font
-					(size 1.27 1.27)
-				)
-				(hide yes)
-			)
-		)
-		(property "Datasheet" "https://item.szlcsc.com/datasheet/CL10B224KB8NNNC/65773.html"
-			(at 95.25 104.14 0)
-			(effects
-				(font
-					(size 1.27 1.27)
-				)
-				(hide yes)
-			)
-		)
-		(property "Description" "Capacitance:220nF Tolerance:±10% Tolerance:±10% Voltage Rating:50V Temperature Coefficient:X7R"
-			(at 95.25 104.14 0)
-			(effects
-				(font
-					(size 1.27 1.27)
-				)
-				(hide yes)
-			)
-		)
-		(property "Manufacturer Part" "CL10B224KB8NNNC"
-			(at 95.25 104.14 0)
-			(effects
-				(font
-					(size 1.27 1.27)
-				)
-				(hide yes)
-			)
-		)
-		(property "Manufacturer" "SAMSUNG(三星)"
-			(at 95.25 104.14 0)
-			(effects
-				(font
-					(size 1.27 1.27)
-				)
-				(hide yes)
-			)
-		)
-		(property "Supplier Part" "C64705"
-			(at 95.25 104.14 0)
-			(effects
-				(font
-					(size 1.27 1.27)
-				)
-				(hide yes)
-			)
-		)
-		(property "Supplier" "LCSC"
-			(at 95.25 104.14 0)
-			(effects
-				(font
-					(size 1.27 1.27)
-				)
-				(hide yes)
-			)
-		)
-		(property "LCSC Part Name" "220nF ±10% 50V"
-			(at 95.25 104.14 0)
-			(effects
-				(font
-					(size 1.27 1.27)
-				)
-				(hide yes)
-			)
-		)
-		(pin "1"
-		)
-		(pin "2"
-		)
-		(instances
-			(project "svea_powerboard_rev3"
-				(path "/3f85abf4-0b95-4c4a-b7e9-06f59ca1ea3d/5c2e021f-c2d4-49e2-8c36-9a64f1f12001/535c4b9d-dd70-4891-8336-b5700298b4d1"
-					(reference "C55")
-					(unit 1)
-				)
-			)
-		)
-	)
-	(symbol
 		(lib_id "Device:NetTie_2")
 		(at 261.62 57.15 0)
@@
 	(symbol
 		(lib_id "5v rail sm-easyedapro:RVT1E680M0605")
-		(at 276.86 81.28 270)
+		(at 250.19 82.55 270)
 		(unit 1)
 		(exclude_from_sim no)
@@
 		(fields_autoplaced yes)
 		(property "Reference" "SWITCHTODATASHEETERCOMMENDED1401"
-			(at 279.4 81.2799 90)
+			(at 252.73 82.5499 90)
 			(effects
 				(font
@@
 		)
 		(property "Value" "68uF"
-			(at 276.86 81.28 0)
+			(at 250.19 82.55 0)
 			(effects
 				(font
@@
 		)
 		(property "Footprint" "5v rail sm-easyedapro:CAP-SMD_BD6.3-L6.6-W6.6-LS7.4-FD"
-			(at 276.86 81.28 0)
+			(at 250.19 82.55 0)
 			(effects
 				(font
@@
 		)
 		(property "Datasheet" ""
-			(at 276.86 81.28 0)
+			(at 250.19 82.55 0)
 			(effects
 				(font
@@
 		)
 		(property "Description" "Capacitance:68uF Tolerance:±20% Tolerance:±20% Voltage Rating:25V Ripple Current:55mA@120Hz Diameter:6.3mm Height - Seated (Max):5.4mm Lifetime:2000hrs@105°C Operating Temperature:-40°C~+105°C Operating Temperature:-40°C~+105°C"
-			(at 276.86 81.28 0)
+			(at 250.19 82.55 0)
 			(effects
 				(font
@@
 		)
 		(property "Manufacturer Part" "RVT1E680M0605"
-			(at 276.86 81.28 0)
+			(at 250.19 82.55 0)
 			(effects
 				(font
@@
 		)
 		(property "Manufacturer" "ROQANG(容强)"
-			(at 276.86 81.28 0)
+			(at 250.19 82.55 0)
 			(effects
 				(font
@@
 		)
 		(property "Supplier Part" "C7436903"
-			(at 276.86 81.28 0)
+			(at 250.19 82.55 0)
 			(effects
 				(font
@@
 		)
 		(property "Supplier" "LCSC"
-			(at 276.86 81.28 0)
+			(at 250.19 82.55 0)
 			(effects
 				(font
@@
 		)
 		(property "LCSC Part Name" "68uF ±20% 25V"
-			(at 276.86 81.28 0)
+			(at 250.19 82.55 0)
 			(effects
 				(font
@@
 		)
 		(instances
-			(project ""
+			(project "svea_powerboard_rev3"
 				(path "/3f85abf4-0b95-4c4a-b7e9-06f59ca1ea3d/5c2e021f-c2d4-49e2-8c36-9a64f1f12001/535c4b9d-dd70-4891-8336-b5700298b4d1"
 					(reference "SWITCHTODATASHEETERCOMMENDED1401")
@@
 	)
 	(symbol
+		(lib_id "Device:C")
+		(at 95.25 104.14 0)
+		(unit 1)
+		(exclude_from_sim no)
+		(in_bom yes)
+		(on_board yes)
+		(dnp no)
+		(fields_autoplaced yes)
+		(property "Reference" "C1404"
+			(at 99.06 102.8699 0)
+			(effects
+				(font
+					(size 1.27 1.27)
+				)
+				(justify left)
+			)
+		)
+		(property "Value" "220nF"
+			(at 99.06 105.4099 0)
+			(effects
+				(font
+					(size 1.27 1.27)
+				)
+				(justify left)
+			)
+		)
+		(property "Footprint" "Capacitor_SMD:C_0402_1005Metric"
+			(at 96.2152 107.95 0)
+			(effects
+				(font
+					(size 1.27 1.27)
+				)
+				(hide yes)
+			)
+		)
+		(property "Datasheet" "~"
+			(at 95.25 104.14 0)
+			(effects
+				(font
+					(size 1.27 1.27)
+				)
+				(hide yes)
+			)
+		)
+		(property "Description" "Unpolarized capacitor"
+			(at 95.25 104.14 0)
+			(effects
+				(font
+					(size 1.27 1.27)
+				)
+				(hide yes)
+			)
+		)
+		(pin "1"
+		)
+		(pin "2"
+		)
+		(instances
+			(project ""
+				(path "/3f85abf4-0b95-4c4a-b7e9-06f59ca1ea3d/5c2e021f-c2d4-49e2-8c36-9a64f1f12001/535c4b9d-dd70-4891-8336-b5700298b4d1"
+					(reference "C1404")
+					(unit 1)
+				)
+			)
+		)
+	)
+	(symbol
 		(lib_id "power:GND")
 		(at 72.39 168.91 0)
@@
 	(symbol
 		(lib_id "Device:C")
-		(at 266.7 82.55 0)
+		(at 238.76 80.01 0)
 		(unit 1)
 		(exclude_from_sim no)
@@
 		(fields_autoplaced yes)
 		(property "Reference" "C1403"
-			(at 270.51 81.2799 0)
+			(at 242.57 78.7399 0)
 			(effects
 				(font
@@
 		)
 		(property "Value" "22uF"
-			(at 270.51 83.8199 0)
+			(at 242.57 81.2799 0)
 			(effects
 				(font
@@
 		)
 		(property "Footprint" "Capacitor_SMD:C_0805_2012Metric"
-			(at 267.6652 86.36 0)
+			(at 239.7252 83.82 0)
 			(effects
 				(font
@@
 		)
 		(property "Datasheet" "~"
-			(at 266.7 82.55 0)
+			(at 238.76 80.01 0)
 			(effects
 				(font
@@
 		)
 		(property "Description" "Unpolarized capacitor"
-			(at 266.7 82.55 0)
+			(at 238.76 80.01 0)
 			(effects
 				(font
@@
 		)
 		(instances
-			(project ""
+			(project "svea_powerboard_rev3"
 				(path "/3f85abf4-0b95-4c4a-b7e9-06f59ca1ea3d/5c2e021f-c2d4-49e2-8c36-9a64f1f12001/535c4b9d-dd70-4891-8336-b5700298b4d1"
 					(reference "C1403")

Commit message: even more almost done
Parts:
- removed R108: 0, Resistor_SMD:R_0603_1608Metric, symbol Device:R
- removed R109: 36.5kΩ, 5v rail sm-easyedapro:R0603, symbol 5v rail sm-easyedapro:FRC0603F3652TS
- added NT1401: NetTie_2, 5v rail sm-easyedapro:NetTie-2_SMD_Pad0.3mm, symbol Device:NetTie_2
- added R1404: 7mΩ, 5v rail sm-easyedapro:R2512, symbol 5v rail sm-easyedapro:JER2512F3R007
- added R1405: 36.5kΩ, Resistor_SMD:R_0402_1005Metric, symbol Device:R
Connections:
- net GND: now also R1405.2
- net IN: now also NT1401.1, R1404.1; no longer U47.F10 (SVIN), U47.F11 (SVIN), U47.G10 (VIN), U47.G11 (VIN), U47.H10 (VIN), U47.H11 (VIN), U47.J10 (VIN), U47.J11 (VIN), U47.K10 (VIN), U47.K11 (VIN), U47.L10 (VIN), U47.L11 (VIN)
- net at U47.H1 (RT): now also R1405.1
- net at U47.L9 (IIN): now also NT1401.2
- new net 12vbuckvintochip: R1404.2, U47.F10 (SVIN), U47.F11 (SVIN), U47.G10 (VIN), U47.G11 (VIN), U47.H10 (VIN), U47.H11 (VIN), U47.J10 (VIN), U47.J11 (VIN), U47.K10 (VIN), U47.K11 (VIN), U47.L10 (VIN), U47.L11 (VIN)
Other:
- note added: "7.1A"
- note added: "Reverse current protection, when current is less than 0.83A mode is switched to prevent reverse current"

Commit message: about to land
Parts:
- removed C53, C57: 100nF, 5v rail sm-easyedapro:C0603, symbol 5v rail sm-easyedapro:CC0603KRX7R9BB104
- removed C54: 1uF, 5v rail sm-easyedapro:C0603, symbol 5v rail sm-easyedapro:CL10B105KB8NQNC
- removed U46: ~, Jumper:SolderJumper-2_P1.3mm_Bridged_Pad1.0x1.5mm, symbol Jumper:Jumper_2_Bridged
- added C1405, C1406: 100nF, Capacitor_SMD:C_0402_1005Metric, symbol Device:C
- added C1407: 1uF, Capacitor_SMD:C_0603_1608Metric, symbol Device:C
Connections:
- net +3V3: now also C1406.1, C1407.1
- net GND: now also C1405.2, C1406.2, C1407.2
- net at U47.F1 (LL): now also U47.G2 (MODE), C1405.1

Commit message: various updates
Parts:
- removed C1401, C1402: 4.7u, Capacitor_SMD:C_1210_3225Metric, symbol Device:C
- removed C1403: 22uF, Capacitor_SMD:C_0805_2012Metric, symbol Device:C
- removed SWITCHTODATASHEETERCOMMENDED1401: 68uF, 5v rail sm-easyedapro:CAP-SMD_BD6.3-L6.6-W6.6-LS7.4-FD, symbol 5v rail sm-easyedapro:RVT1E680M0605
- added C1401, C1403: CL32B475KBUYNNE, JLCImport:CL32B475KBUYNNE, symbol JLCImport:CL32B475KBUYNNE
- added C1408: TPSC686M016R0200, JLCImport:TPSC686M016R0200, symbol JLCImport:TPSC686M016R0200
- added C1409: CL21A226MAYNNNE, JLCImport:CL21A226MAYNNNE, symbol JLCImport:CL21A226MAYNNNE
- added JP1401: Jumper_2_Bridged, PCM_SparkFun-Jumper:Jumper_2_NC_Trace, symbol Jumper:Jumper_2_Bridged
Connections:
- net 12vbuckvintochip: now also C1401.2, C1403.2, JP1401.1 (A)
- net GND: now also C1401.1, C1403.1, C1408.2, C1409.1
- net at R112.1, R1402.1, U47.A1 (VOUT)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: now also C1408.1, C1409.2
- net at NT1401.2, U47.L9 (IIN): now also JP1401.2 (B)
Other:
- moved on the sheet: R1404
