File: hardware/kicad/12v_LTM8055_BUCK.kicad_sch (KiCad schematic)
At the start: 21 parts, among them U44 MCP4725A0T-E/CH, U47 LTM8055IY_PBF

Commit message: various updates
Other:
- moved on the sheet: R1404
Changed lines of the file:
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@@
 	(wire
 		(pts
-			(xy 16.51 66.04) (xy 19.05 66.04)
+			(xy 3.81 66.04) (xy 6.35 66.04)
 		)
 		(stroke
@@
 	(wire
 		(pts
-			(xy 29.21 66.04) (xy 30.48 66.04)
+			(xy 16.51 66.04) (xy 30.48 66.04)
 		)
 		(stroke
@@
 	(hierarchical_label "IN"
 		(shape input)
-		(at 16.51 66.04 180)
+		(at 3.81 66.04 180)
 		(effects
 			(font
@@
 	(symbol
 		(lib_id "5v rail sm-easyedapro:JER2512F3R007")
-		(at 24.13 66.04 0)
+		(at 11.43 66.04 0)
 		(unit 1)
 		(exclude_from_sim no)
@@
 		(dnp no)
 		(property "Reference" "R1404"
-			(at 21.59 64.77 0)
+			(at 8.89 64.77 0)
 			(effects
 				(font
@@
 		)
 		(property "Value" "7mΩ"
-			(at 21.59 69.85 0)
+			(at 8.89 69.85 0)
 			(effects
 				(font
@@
 		)
 		(property "Footprint" "5v rail sm-easyedapro:R2512"
-			(at 24.13 66.04 0)
+			(at 11.43 66.04 0)
 			(effects
 				(font
@@
 		)
 		(property "Datasheet" "https://item.szlcsc.com/datasheet/JER2512F3R007/51553032.html"
-			(at 24.13 66.04 0)
+			(at 11.43 66.04 0)
 			(effects
 				(font
@@
 		)
 		(property "Description" "Type:Current Sense Resistor Resistance:7mΩ Tolerance:±1% Tolerance:±1% Power(Watts):3W Temperature Coefficient:±50ppm/°C Temperature Coefficient:±50ppm/°C"
-			(at 24.13 66.04 0)
+			(at 11.43 66.04 0)
 			(effects
 				(font
@@
 		)
 		(property "Manufacturer Part" "JER2512F3R007"
-			(at 24.13 66.04 0)
+			(at 11.43 66.04 0)
 			(effects
 				(font
@@
 		)
 		(property "Manufacturer" "JIERR(捷而瑞)"
-			(at 24.13 66.04 0)
+			(at 11.43 66.04 0)
 			(effects
 				(font
@@
 		)
 		(property "Supplier Part" "C49164689"
-			(at 24.13 66.04 0)
+			(at 11.43 66.04 0)
 			(effects
 				(font
@@
 		)
 		(property "Supplier" "LCSC"
-			(at 24.13 66.04 0)
+			(at 11.43 66.04 0)
 			(effects
 				(font
@@
 		)
 		(property "LCSC Part Name" "7mΩ 3W 2512 ±1%"
-			(at 24.13 66.04 0)
-			(effects
-				(font
+			(at 11.43 66.04 0)
+			(effects
+				(font
