File: hardware/kicad/4_Charging-Buck.kicad_sch (KiCad schematic)
At the start: 39 parts, among them Q1 L2N7002SLLT1G, Q2 ME50P06-G, U29 RVT1H680M0607, U30 CN3722, U31 15uH

Commit message: switches charging buck fet to something with lower gate capacitance
Parts:
- removed Q2: ME50P06-G, Package_TO_SOT_SMD:TO-252-2, symbol 5v rail sm-easyedapro:ME50P06
- removed R84: 0Ω, Resistor_SMD:R_0603_1608Metric, symbol 5v rail sm-easyedapro:0603WAF0000T5E
- added C601: 10uF, Capacitor_SMD:C_1206_3216Metric, symbol Device:C
- added NT601: NetTie_2, 5v rail sm-easyedapro:NetTie-2_SMD_Pad0.2mm, symbol Device:NetTie_2
- added Q602: AO4459, JLCImport:AO4459, symbol JLCImport:AO4459
Connections:
- net GND: now also C601.2, NT601.1
- net IN: now also Q602.1 (S), Q602.2 (S), Q602.3 (S)
- net OUT: now also C601.1
- net at C28.1, C29.2, C30.1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: now also NT601.2
- net at U30.16 (DRV): now also Q602.4 (G)
- net at D11.1, D11.2: now also Q602.5 (D), Q602.6 (D), Q602.7 (D), Q602.8 (D)

Commit message: new location for "wago" connector
Parts:
- U31: footprint (none) -> JLCImport:XAL1010-153MED
Changed lines of the file:
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@@
 			)
 		)
-		(property "Footprint" ""
+		(property "Footprint" "JLCImport:XAL1010-153MED"
 			(at 232.41 74.93 0)
 			(effects

Commit message: starting erc check
Parts:
- C23, C24, C25: footprint 5v rail sm-easyedapro:C0402 -> 5v rail sm-easyedapro:C0603
- C28: footprint Capacitor_SMD:C_0402_1005Metric -> 5v rail sm-easyedapro:C0402
- D11, D12: footprint JLCImport:SBR8U60P5-13 -> 5v rail sm-easyedapro:POWERDI-5_L5.4-W4.0-LS6.5-RD
- LED6: footprint JLCImport:PSC-1608U50GC-G4 -> 5v rail sm-easyedapro:LED0603-RD_GREEN
- LED7: footprint JLCImport:19-217UYOC_S3112_TR8 -> 5v rail sm-easyedapro:LED0603-RD
- R75, R76, R78, R83, R88, R89: footprint Resistor_SMD:R_0603_1608Metric -> 5v rail sm-easyedapro:R0603
- R77: footprint Resistor_SMD:R_0603_1608Metric -> 5v rail sm-easyedapro:R0402; LCSC Part Name 1kΩ ±1% 50mW 厚膜电阻 -> 1kΩ ±1% 62.5mW 厚膜电阻; Manufacturer Part 0201WMF1001TEE -> 0402WGF1001TCE; Supplier Part C270365 -> C11702
- R79: footprint Resistor_SMD:R_0402_1005Metric -> 5v rail sm-easyedapro:R0402; LCSC Part Name 1kΩ ±1% 50mW 厚膜电阻 -> 1kΩ ±1% 62.5mW 厚膜电阻; Manufacturer Part 0201WMF1001TEE -> 0402WGF1001TCE; Supplier Part C270365 -> C11702
- R81, R85: footprint Resistor_SMD:R_0603_1608Metric -> 5v rail sm-easyedapro:R0402
- R86: footprint JLCImport:PE2512FKE7W0R06L -> 5v rail sm-easyedapro:R2512
- R87: footprint JLCImport:PE2512FKE7W0R06L -> 5v rail sm-easyedapro:R2512; LCSC Part Name -- -> 薄膜电阻 60mΩ ±1% 2W; Manufacturer -- -> YAGEO(国巨); Manufacturer Part -- -> PE2512FKE7W0R06L; Supplier -- -> LCSC; Supplier Part -- -> C875732
- U30: footprint Package_SO:TSSOP-16_4.4x5mm_P0.65mm -> 5v rail sm-easyedapro:TSSOP-16_L5.0-W4.4-P0.65-LS6.4-BL
- U31: footprint JLCImport:XAL1010-153MED -> 5v rail sm-easyedapro:IND-SMD_2P-L11.3-W10.0-XAL1010-153MED
Changed lines of the file:
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@@
 			)
 		)
-		(property "Footprint" "Resistor_SMD:R_0603_1608Metric"
+		(property "Footprint" "5v rail sm-easyedapro:R0603"
 			(at 270.51 111.76 0)
 			(effects
@@
 			)
 		)
-		(property "Footprint" "Resistor_SMD:R_0603_1608Metric"
+		(property "Footprint" "5v rail sm-easyedapro:R0603"
 			(at 60.96 96.52 0)
 			(effects
@@
 			)
 		)
-		(property "Footprint" "Resistor_SMD:R_0402_1005Metric"
+		(property "Footprint" "5v rail sm-easyedapro:R0402"
 			(at 121.92 12.7 0)
 			(effects
@@
 			)
 		)
-		(property "Datasheet" "https://item.szlcsc.com/datasheet/0201WMF1001TEE/259895.html"
+		(property "Datasheet" "https://item.szlcsc.com/datasheet/0402WGF1001TCE/12256.html"
 			(at 121.92 12.7 0)
 			(effects
@@
 			)
 		)
-		(property "Description" "Type:Thick Film Resistor Resistance:1kΩ Tolerance:±1% Tolerance:±1% Power(Watts):50mW Voltage-Supply(Max):25V Temperature Coefficient:±200ppm/℃ Temperature Coefficient:±200ppm/℃ Operating Temperature:-55℃~+155℃ Operating Temperature:-55℃~+155℃"
+		(property "Description" "Type:Thick Film Resistor Resistance:1kΩ Tolerance:±1% Tolerance:±1% Power(Watts):62.5mW Voltage-Supply(Max):50V Temperature Coefficient:±100ppm/°C Temperature Coefficient:±100ppm/°C Operating Temperature:-55°C~+155°C Operating Temperature:-55°C~+155°C"
 			(at 121.92 12.7 90)
 			(effects
@@
 			)
 		)
-		(property "Manufacturer Part" "0201WMF1001TEE"
+		(property "Manufacturer Part" "0402WGF1001TCE"
 			(at 121.92 12.7 0)
 			(effects
@@
 			)
 		)
-		(property "Supplier Part" "C270365"
+		(property "Supplier Part" "C11702"
 			(at 121.92 12.7 0)
 			(effects
@@
 			)
 		)
-		(property "LCSC Part Name" "1kΩ ±1% 50mW 厚膜电阻"
+		(property "LCSC Part Name" "1kΩ ±1% 62.5mW 厚膜电阻"
 			(at 121.92 12.7 0)
 			(effects
@@
 			)
 		)
-		(property "Footprint" "JLCImport:SBR8U60P5-13"
+		(property "Footprint" "5v rail sm-easyedapro:POWERDI-5_L5.4-W4.0-LS6.5-RD"
 			(at 217.17 86.36 0)
 			(effects
@@
 			)
 		)
-		(property "Footprint" "Capacitor_SMD:C_0402_1005Metric"
+		(property "Footprint" "5v rail sm-easyedapro:C0402"
 			(at 167.64 130.81 0)
 			(effects
@@
 			)
 		)
-		(property "Footprint" "Package_SO:TSSOP-16_4.4x5mm_P0.65mm"
+		(property "Footprint" "5v rail sm-easyedapro:TSSOP-16_L5.0-W4.4-P0.65-LS6.4-BL"
 			(at 181.61 110.49 0)
 			(effects
@@
 			)
 		)
-		(property "Description" ""
+		(property "Description" "Power symbol creates a global label with name \"GND\" , ground"
 			(at 29.21 93.98 0)
 			(effects
@@
 			)
 		)
-		(property "Footprint" "JLCImport:XAL1010-153MED"
+		(property "Footprint" "5v rail sm-easyedapro:IND-SMD_2P-L11.3-W10.0-XAL1010-153MED"
 			(at 232.41 74.93 0)
 			(effects
@@
 			)
 		)
-		(property "Footprint" "Resistor_SMD:R_0603_1608Metric"
+		(property "Footprint" "5v rail sm-easyedapro:R0402"
 			(at 73.66 12.7 0)
 			(effects
@@
 			)
 		)
-		(property "Datasheet" "https://item.szlcsc.com/datasheet/0201WMF1001TEE/259895.html"
+		(property "Datasheet" "https://item.szlcsc.com/datasheet/0402WGF1001TCE/12256.html"
 			(at 73.66 12.7 0)
 			(effects
@@
 			)
 		)
-		(property "Description" "Type:Thick Film Resistor Resistance:1kΩ Tolerance:±1% Tolerance:±1% Power(Watts):50mW Voltage-Supply(Max):25V Temperature Coefficient:±200ppm/℃ Temperature Coefficient:±200ppm/℃ Operating Temperature:-55℃~+155℃ Operating Temperature:-55℃~+155℃"
+		(property "Description" "Type:Thick Film Resistor Resistance:1kΩ Tolerance:±1% Tolerance:±1% Power(Watts):62.5mW Voltage-Supply(Max):50V Temperature Coefficient:±100ppm/°C Temperature Coefficient:±100ppm/°C Operating Temperature:-55°C~+155°C Operating Temperature:-55°C~+155°C"
 			(at 73.66 12.7 90)
 			(effects
@@
 			)
 		)
-		(property "Manufacturer Part" "0201WMF1001TEE"
+		(property "Manufacturer Part" "0402WGF1001TCE"
 			(at 73.66 12.7 0)
 			(effects
@@
 			)
 		)
-		(property "Supplier Part" "C270365"
+		(property "Supplier Part" "C11702"
 			(at 73.66 12.7 0)
 			(effects
@@
 			)
 		)
-		(property "LCSC Part Name" "1kΩ ±1% 50mW 厚膜电阻"
+		(property "LCSC Part Name" "1kΩ ±1% 62.5mW 厚膜电阻"
 			(at 73.66 12.7 0)
 			(effects
@@
 			)
 		)
-		(property "Footprint" "JLCImport:PSC-1608U50GC-G4"
+		(property "Footprint" "5v rail sm-easyedapro:LED0603-RD_GREEN"
 			(at 73.66 30.48 0)
 			(effects
@@
 			)
 		)
-		(property "Footprint" "JLCImport:SBR8U60P5-13"
+		(property "Footprint" "5v rail sm-easyedapro:POWERDI-5_L5.4-W4.0-LS6.5-RD"
 			(at 191.77 74.93 0)
 			(effects
@@
 			)
 		)
-		(property "Footprint" "Resistor_SMD:R_0603_1608Metric"
+		(property "Footprint" "5v rail sm-easyedapro:R0603"
 			(at 270.51 121.92 0)
 			(effects
@@
 			)
 		)
-		(property "Footprint" "Resistor_SMD:R_0603_1608Metric"
+		(property "Footprint" "5v rail sm-easyedapro:R0603"
 			(at 154.94 130.81 0)
 			(effects
@@
 			)
 		)
-		(property "Footprint" "Resistor_SMD:R_0603_1608Metric"
+		(property "Footprint" "5v rail sm-easyedapro:R0402"
 			(at 198.12 125.73 0)
 			(effects
@@
 			)
 		)
-		(property "Description" ""
+		(property "Description" "Power symbol creates a global label with name \"GND\" , ground"
 			(at 158.75 31.75 0)
 			(effects
@@
 			)
 		)
-		(property "Footprint" "Resistor_SMD:R_0603_1608Metric"
+		(property "Footprint" "5v rail sm-easyedapro:R0402"
 			(at 135.89 166.37 0)
 			(effects
@@
 			)
 		)
-		(property "Footprint" "JLCImport:PE2512FKE7W0R06L"
+		(property "Footprint" "5v rail sm-easyedapro:R2512"
 			(at 264.16 74.93 0)
 			(effects
@@
 			)
 		)
-		(property "Footprint" "Resistor_SMD:R_0603_1608Metric"
+		(property "Footprint" "5v rail sm-easyedapro:R0603"
 			(at 60.96 135.89 0)
 			(effects
@@
 			)
 		)
-		(property "Description" ""
+		(property "Description" "Power symbol creates a global label with name \"GND\" , ground"
 			(at 288.29 92.71 0)
 			(effects
@@
 			)
 		)
-		(property "Footprint" "5v rail sm-easyedapro:C0402"
+		(property "Footprint" "5v rail sm-easyedapro:C0603"
 			(at 41.91 81.28 0)
 			(effects
@@
 			)
 		)
-		(property "Footprint" "5v rail sm-easyedapro:C0402"
+		(property "Footprint" "5v rail sm-easyedapro:C0603"
 			(at 80.01 30.48 0)
 			(effects
@@
 			)
 		)
-		(property "Description" ""
+		(property "Description" "Power symbol creates a global label with name \"GND\" , ground"
 			(at 270.51 127 0)
 			(effects
@@
 			)
 		)
-		(property "Description" ""
+		(property "Description" "Power symbol creates a global label with name \"GND\" , ground"
 			(at 111.76 184.15 0)
 			(effects
@@
 			)
 		)
-		(property "Description" ""
+		(property "Description" "Power symbol creates a global label with name \"GND\" , ground"
 			(at 217.17 97.79 0)
 			(effects
@@
 			)
 		)
-		(property "Description" ""
+		(property "Description" "Power symbol creates a global label with name \"GND\" , ground"
 			(at 31.75 31.75 0)
 			(effects
@@
 			)
 		)
-		(property "Description" "Power-5V"
+		(property "Description" "Power symbol creates a global label with name \"+3V3\""
 			(at 97.79 1.27 0)
 			(effects
@@
 			)
 		)
-		(property "Footprint" "JLCImport:PE2512FKE7W0R06L"
+		(property "Footprint" "5v rail sm-easyedapro:R2512"
 			(at 264.16 83.82 0)
 			(effects
@@
 			)
 		)
-		(property "Datasheet" "--"
+		(property "Datasheet" "https://atta.szlcsc.com/upload/public/pdf/source/20211020/C6103334F76DC954DA6F525702694423.pdf"
 			(at 264.16 83.82 0)
 			(effects
@@
 			)
 		)
-		(property "Description" "--"
+		(property "Description" "Type:Thin Film Resistor Resistance: Tolerance:±1% Tolerance:±1% Power(Watts): Temperature Coefficient:±50ppm/°C Temperature Coefficient:±50ppm/°C Operating Temperature Range:-55°C~+170°C Operating Temperature Range:-55°C~+170°C"
 			(at 264.16 83.82 0)
 			(effects
@@
 			)
 		)
-		(property "Manufacturer Part" "--"
+		(property "Manufacturer Part" "PE2512FKE7W0R06L"
 			(at 264.16 83.82 0)
 			(effects
@@
 			)
 		)
-		(property "Manufacturer" "--"
+		(property "Manufacturer" "YAGEO(国巨)"
 			(at 264.16 83.82 0)
 			(effects
@@
 			)
 		)
-		(property "Supplier Part" "--"
+		(property "Supplier Part" "C875732"
 			(at 264.16 83.82 0)
 			(effects
@@
 			)
 		)
-		(property "Supplier" "--"
+		(property "Supplier" "LCSC"
 			(at 264.16 83.82 0)
 			(effects
@@
 			)
 		)
-		(property "LCSC Part Name" "--"
+		(property "LCSC Part Name" "薄膜电阻 60mΩ ±1% 2W"
 			(at 264.16 83.82 0)
 			(effects
@@
 			)
 		)
-		(property "Footprint" "JLCImport:19-217UYOC_S3112_TR8"
+		(property "Footprint" "5v rail sm-easyedapro:LED0603-RD"
 			(at 121.92 30.48 0)
 			(effects
@@
 			)
 		)
-		(property "Footprint" "Resistor_SMD:R_0603_1608Metric"
+		(property "Footprint" "5v rail sm-easyedapro:R0603"
 			(at 100.33 172.72 0)
 			(effects
@@
 			)
 		)
-		(property "Footprint" "5v rail sm-easyedapro:C0402"
+		(property "Footprint" "5v rail sm-easyedapro:C0603"
 			(at 114.3 30.48 0)
 			(effects

Commit message: Update KiCad schematic components and footprints
Make sweeping updates to the KiCad project: major edits to hardware/kicad/4_Charging-Buck.kicad_sch replacing and reconfiguring many symbols (resistor/capacitor/LED swaps), updating values, footprints, datasheets, manufacturer/supplier/LCSC metadata, and symbol graphics/pin positions. Added JLCImport 3D model files (UWT1H221MNL1GS.step/.wrl) and a footprint module (UWT1H221MNL1GS.kicad_mod), and updated hardware/kicad/JLCImport.kicad_sym. Also updated PCB and project files (svea_powerboard_rev3.kicad_pcb, .kicad_pro) to reflect the part/footprint changes. These changes align schematic symbols with chosen replacement parts and include associated 3D/footprint assets for BOM/PCB integration.
Parts:
- removed C26: 100nF, 5v rail sm-easyedapro:C0402, symbol 5v rail sm-easyedapro:0402B104K500NT
- removed C28: 470pF, 5v rail sm-easyedapro:C0402, symbol 5v rail sm-easyedapro:CC0402JRNPO9BN471
- removed C29: 220nF, 5v rail sm-easyedapro:C0603, symbol 5v rail sm-easyedapro:TCC0603X7R224K500CT
- removed C30: 100nF, 5v rail sm-easyedapro:C0402, symbol 5v rail sm-easyedapro:CL05B104KB54PNC
- removed C31: 2pF, 5v rail sm-easyedapro:C0402, symbol 5v rail sm-easyedapro:CC0402BRNPO9BN2R0
- removed R75, R78: 100kΩ, 5v rail sm-easyedapro:R0603, symbol 5v rail sm-easyedapro:0603WAF1003T5E
- removed R76: 5.76kΩ, 5v rail sm-easyedapro:R0603, symbol 5v rail sm-easyedapro:FRC0603F5761TS
- removed R81: 10kΩ, 5v rail sm-easyedapro:R0402, symbol 5v rail sm-easyedapro:0402WGF1002TCE
- removed R83: 1MΩ, 5v rail sm-easyedapro:R0603, symbol 5v rail sm-easyedapro:0603WAF1004T5E
- removed R85: 120Ω, 5v rail sm-easyedapro:R0402, symbol 5v rail sm-easyedapro:0402WGF1200TCE
- removed R88: 105kΩ, 5v rail sm-easyedapro:R0603, symbol 5v rail sm-easyedapro:FRC0603F1053TS
- removed R89: 24.9kΩ, 5v rail sm-easyedapro:R0603, symbol 5v rail sm-easyedapro:FRC0603F2492TS
- removed U29: RVT1H680M0607, JLCImport:RVT1H680M0607, symbol JLCImport:RVT1H680M0607
- added C602: UWT1H221MNL1GS, JLCImport:UWT1H221MNL1GS, symbol JLCImport:UWT1H221MNL1GS
- added C603: 470pF, Capacitor_SMD:C_0402_1005Metric, symbol Device:C
- added C604: 220nF, Capacitor_SMD:C_0402_1005Metric, symbol Device:C
- added C605, C606: 100nF, Capacitor_SMD:C_0402_1005Metric, symbol Device:C
- added C607: 2pF, Capacitor_SMD:C_0402_1005Metric, symbol Device:C
- added R601: 1M, Resistor_SMD:R_0402_1005Metric, symbol Device:R
- added R602: 120, Resistor_SMD:R_0402_1005Metric, symbol Device:R
- added R603: 10k, Resistor_SMD:R_0402_1005Metric, symbol Device:R
- added R604, R606: 100k, Resistor_SMD:R_0402_1005Metric, symbol Device:R
- added R605: 5.76k, Resistor_SMD:R_0402_1005Metric, symbol Device:R
- added R607: 105k, Resistor_SMD:R_0402_1005Metric, symbol Device:R
- added R608: 24.9k, Resistor_SMD:R_0402_1005Metric, symbol Device:R
Connections:
- net #EN: now also R604.1
- net GND: now also C602.2, R603.2, R604.2, R605.2, R608.2
- net IN: now also C602.1, C606.1, R606.1
- net OUT: now also C607.1, R607.1
- net at U30.10 (FB): now also C607.2, R607.2, R608.1
- net at U30.7 (MPPT): now also R605.1, R606.2
- net at NT601.2, U30.3 (GND): now also C603.2, C604.2, C605.2, R601.2
- net at U30.8 (COM1): now also C603.1, R601.1
- net at U30.1 (VG): now also C606.2
- net at U30.11 (COM3): now also C605.1
- net at Q1.3 (D), U30.6 (TEMP): now also R603.1
- net at U30.9 (COM2): now also R602.1
- new net: C604.1, R602.2

Commit message: Adjust 5V rail routing and add vias
Small footprint position tweaks (R269, R268, R19) and a local reroute of the 5V rail: multiple track segments were added/modified, segment endpoints adjusted, and several vias added to connect layers. UUIDs for tracks/segments/vias were updated to reflect the new geometry. Changes affect multiple nets and inner-layer segments to correct routing and improve connectivity around the revised footprints.
Other:
- note removed: "hacky way of disabling the charging circuit default always on"
Changed lines of the file:
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@@
-		)
-	)
-	(text "hacky way of disabling the charging circuit\ndefault always on"
-		(exclude_from_sim no)
-		(at 119.38 186.436 0)
-		(effects
-			(font
-				(size 1.27 1.27)
-			)
-			(justify left bottom)
 		)
 	)

Commit message: removed redundant charg indi caps
Parts:
- removed C22, C27: 100nF, 5v rail sm-easyedapro:C0402, symbol 5v rail sm-easyedapro:CL05B104KB54PNC
- removed C24, C25: 100nF, 5v rail sm-easyedapro:C0603, symbol 5v rail sm-easyedapro:CC0603KRX7R9BB104
- added C608: 100nF, Capacitor_SMD:C_0402_1005Metric, symbol Device:C
Connections:
- net GND: now also C608.2
- net IN: now also C608.1

Commit message: starting to route charger
Connections:
- net Charger/CN3072/CHG-ACTIVE: no longer LED6.1 (K), R73.2, R74.2, U30.5 (DONE#)
- net Charger/CN3072/CHG-DONE: no longer LED7.1 (-), R80.2, R82.1, U30.4 (CHRG#)
- net GND: no longer Q1.2 (S), R603.2, R604.2
- net at C603.2, C604.2, C605.2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: now also Q1.2 (S), R603.2, R604.2
- new net: LED7.1 (-), R80.2, R82.1, U30.4 (CHRG#)
- new net: LED6.1 (K), R73.2, R74.2, U30.5 (DONE#)
Other:
- moved on the sheet: Q1, R603, R604

Commit message: update
Parts:
- added NT602: NetTie_2, 5v rail sm-easyedapro:NetTie-2_SMD_Pad0.3mm, symbol Device:NetTie_2
- NT601: footprint 5v rail sm-easyedapro:NetTie-2_SMD_Pad0.2mm -> 5v rail sm-easyedapro:NetTie-2_SMD_Pad0.3mm
Connections:
- net OUT: now also NT602.2; no longer U30.14 (BAT)
- new net: NT602.1, U30.14 (BAT)
Changed lines of the file:
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@@
 	)
 	(junction
-		(at 265.43 106.68)
-		(diameter 0)
-		(color 0 0 0 0)
-	)
-	(junction
 		(at 128.27 90.17)
 		(diameter 0)
@@
 	)
 	(junction
+		(at 278.13 74.93)
+		(diameter 0)
+		(color 0 0 0 0)
+	)
+	(junction
 		(at 246.38 74.93)
 		(diameter 0)
@@
 	(wire
 		(pts
-			(xy 58.42 39.37) (xy 73.6346 39.37)
+			(xy 246.38 74.93) (xy 246.38 109.22)
 		)
 		(stroke
@@
 	(wire
 		(pts
-			(xy 184.15 72.39) (xy 179.07 72.39)
+			(xy 58.42 39.37) (xy 73.6346 39.37)
 		)
 		(stroke
@@
 	(wire
 		(pts
-			(xy 3.81 88.9) (xy 3.81 86.36)
+			(xy 184.15 72.39) (xy 179.07 72.39)
 		)
 		(stroke
@@
 	(wire
 		(pts
-			(xy 121.92 35.56) (xy 121.92 39.37)
+			(xy 3.81 88.9) (xy 3.81 86.36)
 		)
 		(stroke
@@
 	(wire
 		(pts
-			(xy 246.38 109.22) (xy 246.38 74.93)
+			(xy 121.92 35.56) (xy 121.92 39.37)
 		)
 		(stroke
@@
 	(wire
 		(pts
-			(xy 271.78 74.93) (xy 283.21 74.93)
+			(xy 271.78 74.93) (xy 278.13 74.93)
 		)
 		(stroke
@@
 	(wire
 		(pts
+			(xy 278.13 93.98) (xy 278.13 91.44)
+		)
+		(stroke
+			(width 0)
+			(type default)
+		)
+	)
+	(wire
+		(pts
 			(xy 161.29 143.51) (xy 198.12 143.51)
 		)
@@
 	(wire
 		(pts
+			(xy 278.13 74.93) (xy 283.21 74.93)
+		)
+		(stroke
+			(width 0)
+			(type default)
+		)
+	)
+	(wire
+		(pts
 			(xy 121.92 5.08) (xy 97.79 5.08)
 		)
@@
 	(wire
 		(pts
+			(xy 193.04 106.68) (xy 260.35 106.68)
+		)
+		(stroke
+			(width 0)
+			(type default)
+		)
+	)
+	(wire
+		(pts
 			(xy 8.89 74.93) (xy 16.51 74.93)
 		)
@@
 	(wire
 		(pts
+			(xy 278.13 74.93) (xy 278.13 86.36)
+		)
+		(stroke
+			(width 0)
+			(type default)
+		)
+	)
+	(wire
+		(pts
 			(xy 156.21 74.93) (xy 157.48 74.93)
 		)
@@
 	(wire
 		(pts
+			(xy 260.35 93.98) (xy 278.13 93.98)
+		)
+		(stroke
+			(width 0)
+			(type default)
+		)
+	)
+	(wire
+		(pts
+			(xy 260.35 106.68) (xy 260.35 93.98)
+		)
+		(stroke
+			(width 0)
+			(type default)
+		)
+	)
+	(wire
+		(pts
 			(xy 58.42 5.08) (xy 58.42 8.89)
 		)
@@
 	(wire
 		(pts
-			(xy 283.21 106.68) (xy 283.21 74.93)
+			(xy 283.21 74.93) (xy 283.21 106.68)
 		)
 		(stroke
@@
 	(wire
 		(pts
-			(xy 193.04 106.68) (xy 265.43 106.68)
-		)
-		(stroke
-			(width 0)
-			(type default)
-		)
-	)
-	(wire
-		(pts
 			(xy 199.39 104.14) (xy 199.39 95.25)
 		)
@@
 	)
 	(symbol
+		(lib_id "Device:NetTie_2")
+		(at 278.13 88.9 270)
+		(mirror x)
+		(unit 1)
+		(exclude_from_sim no)
+		(in_bom no)
+		(on_board yes)
+		(dnp no)
+		(property "Reference" "NT602"
+			(at 276.86 87.6299 90)
+			(effects
+				(font
+					(size 1.27 1.27)
+				)
+				(justify right)
+			)
+		)
+		(property "Value" "NetTie_2"
+			(at 276.86 90.1699 90)
+			(effects
+				(font
+					(size 1.27 1.27)
+				)
+				(justify right)
+			)
+		)
+		(property "Footprint" "5v rail sm-easyedapro:NetTie-2_SMD_Pad0.3mm"
+			(at 278.13 88.9 0)
+			(effects
+				(font
+					(size 1.27 1.27)
+				)
+				(hide yes)
+			)
+		)
+		(property "Datasheet" "~"
+			(at 278.13 88.9 0)
+			(effects
+				(font
+					(size 1.27 1.27)
+				)
+				(hide yes)
+			)
+		)
+		(property "Description" "Net tie, 2 pins"
+			(at 278.13 88.9 0)
+			(effects
+				(font
+					(size 1.27 1.27)
+				)
+				(hide yes)
+			)
+		)
+		(pin "1"
+		)
+		(pin "2"
+		)
+		(instances
+			(project "svea_powerboard_rev3"
+				(path "/3f85abf4-0b95-4c4a-b7e9-06f59ca1ea3d/5c2e021f-c2d4-49e2-8c36-9a64f1f12001/31f44477-0097-4e02-b6ff-5111b8556cfe"
+					(reference "NT602")
+					(unit 1)
+				)
+			)
+		)
+	)
+	(symbol
 		(lib_id "Device:C")
 		(at 283.21 113.03 0)
@@
 			)
 		)
-		(property "Footprint" "5v rail sm-easyedapro:NetTie-2_SMD_Pad0.2mm"
+		(property "Footprint" "5v rail sm-easyedapro:NetTie-2_SMD_Pad0.3mm"
 			(at 161.29 153.67 0)
 			(effects
