File: hardware/kicad/LED-NETWORK.kicad_sch (KiCad schematic)
At the start: 1 part

Commit message: removed uselss text
Parts:
- LED3: footprint JLCImport:XL-1608UBC-04 -> LED_SMD:LED_0603_1608Metric
Changed lines of the file:
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@@
 			)
 		)
-		(property "Footprint" "JLCImport:XL-1608UBC-04"
+		(property "Footprint" "LED_SMD:LED_0603_1608Metric"
 			(at 74.93 63.5 0)
 			(effects
