File: hardware/kicad/5vrail.kicad_sch (KiCad schematic)
At the start: 13 parts, among them Q12 L2N7002SLLT1G, U74 TPSM33625RDNR

Commit message: starting erc check
Parts:
- C100, C101: footprint Capacitor_SMD:C_1206_3216Metric -> 5v rail sm-easyedapro:C1206
- C96, C99: footprint Capacitor_SMD:C_0603_1608Metric -> 5v rail sm-easyedapro:C0603
- C97: footprint Capacitor_SMD:C_0805_2012Metric -> 5v rail sm-easyedapro:C0805
- Q12: footprint Package_TO_SOT_SMD:SOT-23 -> 5v rail sm-easyedapro:SOT-23-3_L3.0-W1.7-P0.95-LS2.9-BR
- R155, R156, R157, R158, R159: footprint Resistor_SMD:R_0603_1608Metric -> 5v rail sm-easyedapro:R0603
Changed lines of the file:
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@@
 			)
 		)
-		(property "Footprint" "Capacitor_SMD:C_1206_3216Metric"
+		(property "Footprint" "5v rail sm-easyedapro:C1206"
 			(at 212.09 67.31 0)
 			(effects
@@
 			)
 		)
-		(property "Footprint" "Resistor_SMD:R_0603_1608Metric"
+		(property "Footprint" "5v rail sm-easyedapro:R0603"
 			(at 111.76 119.38 0)
 			(effects
@@
 			)
 		)
-		(property "Footprint" "Package_TO_SOT_SMD:SOT-23"
+		(property "Footprint" "5v rail sm-easyedapro:SOT-23-3_L3.0-W1.7-P0.95-LS2.9-BR"
 			(at 121.92 109.22 0)
 			(effects
@@
 			)
 		)
-		(property "Description" ""
+		(property "Description" "Power symbol creates a global label with name \"GND\" , ground"
 			(at 212.09 78.74 0)
 			(effects
@@
 			)
 		)
-		(property "Footprint" "Capacitor_SMD:C_0603_1608Metric"
+		(property "Footprint" "5v rail sm-easyedapro:C0603"
 			(at 49.53 93.98 0)
 			(effects
@@
 			)
 		)
-		(property "Footprint" "Resistor_SMD:R_0603_1608Metric"
+		(property "Footprint" "5v rail sm-easyedapro:R0603"
 			(at 180.34 71.12 0)
 			(effects
@@
 			)
 		)
-		(property "Footprint" "Capacitor_SMD:C_0603_1608Metric"
+		(property "Footprint" "5v rail sm-easyedapro:C0603"
 			(at 157.48 99.06 0)
 			(effects
@@
 			)
 		)
-		(property "Description" ""
+		(property "Description" "Power symbol creates a global label with name \"GND\" , ground"
 			(at 180.34 119.38 0)
 			(effects
@@
 			)
 		)
-		(property "Description" ""
+		(property "Description" "Power symbol creates a global label with name \"GND\" , ground"
 			(at 121.92 129.54 0)
 			(effects
@@
 			)
 		)
-		(property "Footprint" "Resistor_SMD:R_0603_1608Metric"
+		(property "Footprint" "5v rail sm-easyedapro:R0603"
 			(at 162.56 77.47 0)
 			(effects
@@
 			)
 		)
-		(property "Footprint" "Resistor_SMD:R_0603_1608Metric"
+		(property "Footprint" "5v rail sm-easyedapro:R0603"
 			(at 114.3 82.55 0)
 			(effects
@@
 			)
 		)
-		(property "Footprint" "Capacitor_SMD:C_1206_3216Metric"
+		(property "Footprint" "5v rail sm-easyedapro:C1206"
 			(at 198.12 67.31 0)
 			(effects
@@
 			)
 		)
-		(property "Footprint" "Capacitor_SMD:C_0805_2012Metric"
+		(property "Footprint" "5v rail sm-easyedapro:C0805"
 			(at 64.77 93.98 0)
 			(effects
@@
 			)
 		)
-		(property "Description" ""
+		(property "Description" "Power symbol creates a global label with name \"GND\" , ground"
 			(at 64.77 110.49 0)
 			(effects
@@
 			)
 		)
-		(property "Footprint" "Resistor_SMD:R_0603_1608Metric"
+		(property "Footprint" "5v rail sm-easyedapro:R0603"
 			(at 180.34 95.25 0)
 			(effects

Commit message: various updates
Parts:
- removed R155, R156: 100kΩ, 5v rail sm-easyedapro:R0603, symbol 5v rail sm-easyedapro:FRC0603J104 TS
- removed R157: 15.8kΩ, 5v rail sm-easyedapro:R0603, symbol 5v rail sm-easyedapro:FRC0603F1582TS
- removed R158: 40.2kΩ, 5v rail sm-easyedapro:R0603, symbol 5v rail sm-easyedapro:RC0603FR-0740K2L
- removed R159: 10kΩ, 5v rail sm-easyedapro:R0603, symbol 5v rail sm-easyedapro:0603WAF1002T5E
- added R2701: 40.2kΩ, Resistor_SMD:R_0402_1005Metric, symbol Device:R
- added R2702: 10kΩ, Resistor_SMD:R_0402_1005Metric, symbol Device:R
- added R2703: 15.8k, Resistor_SMD:R_0402_1005Metric, symbol Device:R
- added R2704, R2705: 100k, Resistor_SMD:R_0402_1005Metric, symbol Device:R
Connections:
- net #EN: now also R2705.2
- net 5V-OUT: now also R2701.1
- net GND: now also R2702.2, R2703.2, R2705.1
- net VCC: now also R2704.1
- net at U74.11 (RT): now also R2703.1
- net at Q12.3 (D), U74.2 (EN): now also R2704.2
- net at U74.9 (FB): now also R2701.2, R2702.1
Other:
- note added: "2.5A variant"

Commit message: various updates
Parts:
- removed C100, C101: 22uF, 5v rail sm-easyedapro:C1206, symbol 5v rail sm-easyedapro:CL31A226KAHNNNE
- removed C97: 4.7uF, 5v rail sm-easyedapro:C0805, symbol 5v rail sm-easyedapro:CL21A475KBQNNNE
- added C2701, C2702: CL32B475KBUYNNE, JLCImport:CL32B475KBUYNNE, symbol JLCImport:CL32B475KBUYNNE
- added C2703, C2704: CL32B226KAJNNNE, JLCImport:CL32B226KAJNNNE, symbol JLCImport:CL32B226KAJNNNE
- added C2705: 22pF, Capacitor_SMD:C_0402_1005Metric_Pad0.74x0.62mm_HandSolder, symbol Device:C
Connections:
- net 5V-OUT: now also C2703.2, C2704.2, C2705.1
- net GND: now also C2701.2, C2702.2, C2703.1, C2704.1
- net VCC: now also C2701.1, C2702.1
- net at R2701.2, R2702.1, U74.9 (FB): now also C2705.2
Other:
- moved on the sheet: R2704

Commit message: update
Parts:
- added NT2701: NetTie_2, 5v rail sm-easyedapro:NetTie-2_SMD_Pad0.3mm, symbol Device:NetTie_2
Connections:
- net 5V-OUT: now also NT2701.2; no longer C2705.1, R2701.1
- new net: C2705.1, NT2701.1, R2701.1
Other:
- moved on the sheet: C2705, R2701
Changed lines of the file:
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@@
+	)
+	(junction
+		(at 187.96 68.58)
+		(diameter 0)
+		(color 0 0 0 0)
 	)
 	(junction
@@
 	)
 	(junction
-		(at 194.31 59.69)
-		(diameter 0)
-		(color 0 0 0 0)
-	)
-	(junction
-		(at 180.34 59.69)
-		(diameter 0)
-		(color 0 0 0 0)
-	)
-	(junction
 		(at 180.34 116.84)
 		(diameter 0)
@@
 	)
 	(junction
+		(at 187.96 59.69)
+		(diameter 0)
+		(color 0 0 0 0)
+	)
+	(junction
 		(at 64.77 104.14)
 		(diameter 0)
@@
 	(wire
 		(pts
-			(xy 194.31 59.69) (xy 194.31 66.04)
-		)
-		(stroke
-			(width 0)
-			(type default)
-		)
-	)
-	(wire
-		(pts
 			(xy 111.76 124.46) (xy 111.76 127)
 		)
@@
 	(wire
 		(pts
-			(xy 180.34 66.04) (xy 180.34 59.69)
+			(xy 187.96 68.58) (xy 187.96 67.31)
 		)
 		(stroke
@@
 	(wire
 		(pts
-			(xy 180.34 59.69) (xy 194.31 59.69)
-		)
-		(stroke
-			(width 0)
-			(type default)
-		)
-	)
-	(wire
-		(pts
 			(xy 111.76 116.84) (xy 111.76 109.22)
 		)
@@
 	(wire
 		(pts
+			(xy 180.34 68.58) (xy 180.34 69.85)
+		)
+		(stroke
+			(width 0)
+			(type default)
+		)
+	)
+	(wire
+		(pts
 			(xy 157.48 85.09) (xy 149.86 85.09)
 		)
@@
 	(wire
 		(pts
-			(xy 194.31 73.66) (xy 194.31 82.55)
+			(xy 194.31 77.47) (xy 194.31 82.55)
 		)
 		(stroke
@@
 	(wire
 		(pts
-			(xy 180.34 90.17) (xy 180.34 82.55)
+			(xy 194.31 69.85) (xy 194.31 68.58)
+		)
+		(stroke
+			(width 0)
+			(type default)
+		)
+	)
+	(wire
+		(pts
+			(xy 187.96 62.23) (xy 187.96 59.69)
 		)
 		(stroke
@@
 	(wire
 		(pts
-			(xy 194.31 59.69) (xy 222.25 59.69)
+			(xy 194.31 68.58) (xy 187.96 68.58)
 		)
 		(stroke
@@
 	(wire
 		(pts
-			(xy 180.34 73.66) (xy 180.34 82.55)
-		)
-		(stroke
-			(width 0)
-			(type default)
-		)
-	)
-	(wire
-		(pts
-			(xy 83.82 59.69) (xy 180.34 59.69)
+			(xy 180.34 77.47) (xy 180.34 82.55)
+		)
+		(stroke
+			(width 0)
+			(type default)
+		)
+	)
+	(wire
+		(pts
+			(xy 83.82 59.69) (xy 187.96 59.69)
 		)
 		(stroke
@@
 	(wire
 		(pts
+			(xy 187.96 59.69) (xy 222.25 59.69)
+		)
+		(stroke
+			(width 0)
+			(type default)
+		)
+	)
+	(wire
+		(pts
 			(xy 64.77 104.14) (xy 49.53 104.14)
 		)
@@
 	(wire
 		(pts
+			(xy 187.96 68.58) (xy 180.34 68.58)
+		)
+		(stroke
+			(width 0)
+			(type default)
+		)
+	)
+	(wire
+		(pts
 			(xy 158.75 77.47) (xy 149.86 77.47)
 		)
@@
 	(wire
 		(pts
+			(xy 180.34 82.55) (xy 180.34 90.17)
+		)
+		(stroke
+			(width 0)
+			(type default)
+		)
+	)
+	(wire
+		(pts
 			(xy 237.49 58.42) (xy 237.49 59.69)
 		)
@@
 			(width 0)
 			(type default)
+		)
+	)
+	(label "5V buck rail"
+		(at 212.09 59.69 0)
+		(effects
+			(font
+				(size 1.27 1.27)
+			)
+			(justify left bottom)
 		)
 	)
@@
 	)
 	(symbol
+		(lib_id "Device:NetTie_2")
+		(at 187.96 64.77 90)
+		(unit 1)
+		(exclude_from_sim no)
+		(in_bom no)
+		(on_board yes)
+		(dnp no)
+		(fields_autoplaced yes)
+		(property "Reference" "NT2701"
+			(at 189.23 63.4999 90)
+			(effects
+				(font
+					(size 1.27 1.27)
+				)
+				(justify right)
+				(hide yes)
+			)
+		)
+		(property "Value" "NetTie_2"
+			(at 189.23 66.0399 90)
+			(effects
+				(font
+					(size 1.27 1.27)
+				)
+				(justify right)
+				(hide yes)
+			)
+		)
+		(property "Footprint" "5v rail sm-easyedapro:NetTie-2_SMD_Pad0.3mm"
+			(at 187.96 64.77 0)
+			(effects
+				(font
+					(size 1.27 1.27)
+				)
+				(hide yes)
+			)
+		)
+		(property "Datasheet" "~"
+			(at 187.96 64.77 0)
+			(effects
+				(font
+					(size 1.27 1.27)
+				)
+				(hide yes)
+			)
+		)
+		(property "Description" "Net tie, 2 pins"
+			(at 187.96 64.77 0)
+			(effects
+				(font
+					(size 1.27 1.27)
+				)
+				(hide yes)
+			)
+		)
+		(pin "1"
+		)
+		(pin "2"
+		)
+		(instances
+			(project ""
+				(path "/3f85abf4-0b95-4c4a-b7e9-06f59ca1ea3d/5c2e021f-c2d4-49e2-8c36-9a64f1f12001/de8125f2-04ec-46c6-89d6-d0b5e89f6023"
+					(reference "NT2701")
+					(unit 1)
+				)
+			)
+		)
+	)
+	(symbol
 		(lib_id "JLCImport:CL32B226KAJNNNE")
 		(at 237.49 68.58 0)
@@
 	(symbol
 		(lib_id "Device:C")
-		(at 194.31 69.85 0)
+		(at 194.31 73.66 0)
 		(unit 1)
 		(exclude_from_sim no)
@@
 		(fields_autoplaced yes)
 		(property "Reference" "C2705"
-			(at 198.12 68.5799 0)
+			(at 198.12 72.3899 0)
 			(effects
 				(font
@@
 		)
 		(property "Value" "22pF"
-			(at 198.12 71.1199 0)
+			(at 198.12 74.9299 0)
 			(effects
 				(font
@@
 		)
 		(property "Footprint" "Capacitor_SMD:C_0402_1005Metric_Pad0.74x0.62mm_HandSolder"
-			(at 195.2752 73.66 0)
+			(at 195.2752 77.47 0)
 			(effects
 				(font
@@
 		)
 		(property "Datasheet" "~"
-			(at 194.31 69.85 0)
+			(at 194.31 73.66 0)
 			(effects
 				(font
@@
 		)
 		(property "Description" "Unpolarized capacitor"
-			(at 194.31 69.85 0)
+			(at 194.31 73.66 0)
 			(effects
 				(font
@@
 		)
 		(property "note" "feedforward cap, can tune if unstable see 8.2.2.7 in datasheet"
-			(at 194.31 69.85 0)
+			(at 194.31 73.66 0)
 			(effects
 				(font
@@
 	(symbol
 		(lib_id "Device:R")
-		(at 180.34 69.85 0)
+		(at 180.34 73.66 0)
 		(unit 1)
 		(exclude_from_sim no)
@@
 		(fields_autoplaced yes)
 		(property "Reference" "R2701"
-			(at 182.88 68.5799 0)
+			(at 182.88 72.3899 0)
 			(effects
 				(font
@@
 		)
 		(property "Value" "40.2kΩ"
-			(at 182.88 71.1199 0)
+			(at 182.88 74.9299 0)
 			(effects
 				(font
@@
 		)
 		(property "Footprint" "Resistor_SMD:R_0402_1005Metric"
-			(at 178.562 69.85 90)
+			(at 178.562 73.66 90)
 			(effects
 				(font
@@
 		)
 		(property "Datasheet" "~"
-			(at 180.34 69.85 0)
+			(at 180.34 73.66 0)
 			(effects
 				(font
@@
 		)
 		(property "Description" "Resistor"
-			(at 180.34 69.85 0)
-			(effects
-				(font
+			(at 180.34 73.66 0)
+			(effects
+				(font

Commit message: updating symbols to use kicad footprints where possible
Parts:
- C96, C99: footprint 5v rail sm-easyedapro:C0603 -> Capacitor_SMD:C_0603_1608Metric
Changed lines of the file:
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@@
 			)
 		)
-		(property "Footprint" "5v rail sm-easyedapro:C0603"
+		(property "Footprint" "Capacitor_SMD:C_0603_1608Metric"
 			(at 49.53 93.98 0)
 			(effects
@@
 			)
 		)
-		(property "Footprint" "5v rail sm-easyedapro:C0603"
+		(property "Footprint" "Capacitor_SMD:C_0603_1608Metric"
 			(at 157.48 99.06 0)
 			(effects

Commit message: updates
Parts:
- removed U74: TPSM33625RDNR, 5v rail sm-easyedapro:QFN-11_L4.5-W3.5-P0.50-TL_TPSM365R6FRDNR, symbol 5v rail sm-easyedapro:TPSM33625RDNR
- added U2701: TPSM33625RDNR, JLCImport:TPSM33625RDNR, symbol JLCImport:TPSM33625RDNR
Connections:
- net 5V-OUT: now also U2701.4 (VOUT)
- net GND: now also U2701.10 (GND)
- net Power/5V-Buck/PGOOD: now also U2701.1 (PGOOD)
- net VCC: now also U2701.3 (VIN)
- net at C2705.2, R2701.2, R2702.1: now also U2701.9 (FB)
- net at Q12.3 (D), R2704.2: now also U2701.2 (EN)
- net at R2703.1: now also U2701.11 (RT)
- net at C99.2: now also U2701.8 (VCC)
Changed lines of the file:
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@@
 	(text "2.5A variant"
 		(exclude_from_sim no)
-		(at 144.018 72.898 0)
+		(at 138.684 66.04 0)
 		(effects
 			(font
@@
 	)
 	(symbol
-		(lib_id "5v rail sm-easyedapro:TPSM33625RDNR")
-		(at 138.43 83.82 0)
-		(unit 1)
-		(exclude_from_sim no)
-		(in_bom yes)
-		(on_board yes)
-		(dnp no)
-		(property "Reference" "U74"
-			(at 129.54 74.93 0)
-			(effects
-				(font
-					(size 1.27 1.27)
-				)
-				(justify left bottom)
-			)
-		)
-		(property "Value" "TPSM33625RDNR"
-			(at 129.54 95.25 0)
-			(effects
-				(font
-					(size 1.27 1.27)
-				)
-				(justify left bottom)
-			)
-		)
-		(property "Footprint" "5v rail sm-easyedapro:QFN-11_L4.5-W3.5-P0.50-TL_TPSM365R6FRDNR"
-			(at 138.43 83.82 0)
-			(effects
-				(font
-					(size 1.27 1.27)
-				)
-				(hide yes)
-			)
-		)
-		(property "Datasheet" "https://item.szlcsc.com/datasheet/TPSM33625RDNR/8040204.html"
-			(at 138.43 83.82 0)
-			(effects
-				(font
-					(size 1.27 1.27)
-				)
-				(hide yes)
-			)
-		)
-		(property "Description" "Function:Buck Number of Outputs:1 Voltage - Supply:3V~36V Voltage - Supply:3V~36V Output Voltage Accuracy:±1% Output Voltage Accuracy:±1% Output Voltage:1V~15V Output Voltage:1V~15V Output Current(Max):2.5A Output Current(Max):2.5A Conversion Efficiency:8"
-			(at 138.43 83.82 0)
-			(effects
-				(font
-					(size 1.27 1.27)
-				)
-				(hide yes)
-			)
-		)
-		(property "Manufacturer Part" "TPSM33625RDNR"
-			(at 138.43 83.82 0)
-			(effects
-				(font
-					(size 1.27 1.27)
-				)
-				(hide yes)
-			)
-		)
-		(property "Manufacturer" "TI(德州仪器)"
-			(at 138.43 83.82 0)
-			(effects
-				(font
-					(size 1.27 1.27)
-				)
-				(hide yes)
-			)
-		)
-		(property "Supplier Part" "C7073593"
-			(at 138.43 83.82 0)
-			(effects
-				(font
-					(size 1.27 1.27)
-				)
-				(hide yes)
-			)
-		)
-		(property "Supplier" "LCSC"
-			(at 138.43 83.82 0)
-			(effects
-				(font
-					(size 1.27 1.27)
-				)
-				(hide yes)
-			)
-		)
-		(property "LCSC Part Name" "3V至36V输入、1V至15V输出同步降压转换器电源模块"
-			(at 138.43 83.82 0)
-			(effects
-				(font
-					(size 1.27 1.27)
-				)
-				(hide yes)
-			)
-		)
-		(pin "2"
-		)
-		(pin "3"
-		)
-		(pin "4"
-		)
-		(pin "1"
-		)
-		(pin "5"
-		)
-		(pin "11"
-		)
-		(pin "10"
-		)
-		(pin "9"
-		)
-		(pin "8"
-		)
-		(pin "7"
-		)
-		(pin "6"
-		)
-		(instances
-			(project "svea_powerboard_rev3"
-				(path "/3f85abf4-0b95-4c4a-b7e9-06f59ca1ea3d/5c2e021f-c2d4-49e2-8c36-9a64f1f12001/de8125f2-04ec-46c6-89d6-d0b5e89f6023"
-					(reference "U74")
-					(unit 1)
-				)
-			)
-		)
-	)
-	(symbol
 		(lib_id "Device:R")
 		(at 111.76 120.65 180)
@@
 					(unit 1)
 				)
+			)
+		)
+	)
+	(symbol
+		(lib_id "JLCImport:TPSM33625RDNR")
+		(at 138.43 83.82 0)
+		(unit 1)
+		(exclude_from_sim no)
+		(in_bom yes)
+		(on_board yes)
+		(dnp no)
+		(fields_autoplaced yes)
+		(property "Reference" "U2701"
+			(at 138.43 69.85 0)
+			(effects
+				(font
+					(size 1.27 1.27)
+				)
+			)
+		)
+		(property "Value" "TPSM33625RDNR"
+			(at 138.43 72.39 0)
+			(effects
+				(font
+					(size 1.27 1.27)
+				)
+			)
+		)
+		(property "Footprint" "JLCImport:TPSM33625RDNR"
+			(at 138.43 83.82 0)
+			(effects
+				(font
+					(size 1.27 1.27)
+				)
+				(hide yes)
+			)
+		)
+		(property "Datasheet" "https://wmsc.lcsc.com/wmsc/upload/file/pdf/v2/lcsc/2309210041_Texas-Instruments-TPSM33625RDNR_C7073593.pdf"
+			(at 138.43 83.82 0)
+			(effects
+				(font
+					(size 1.27 1.27)
+				)
+				(hide yes)
+			)
+		)
+		(property "Description" "-40℃~+105℃ 1 1.5uA 1V~15V 2.5A 2mm 3.5mm 3V~36V 4.5mm 88% Buck Short Circuit Protection、Overheat protection、Over Current Protection ±1% QFN-11 DC-DC Power Modules ROHS"
+			(at 138.43 83.82 0)
+			(effects
+				(font
+					(size 1.27 1.27)
+				)
+				(hide yes)
+			)
+		)
+		(property "LCSC" "C7073593"
+			(at 138.43 83.82 0)
+			(effects
+				(font
+					(size 1.27 1.27)
+				)
+				(hide yes)
+			)
+		)
+		(property "Manufacturer" "Texas Instruments"
+			(at 138.43 83.82 0)
+			(effects
+				(font
+					(size 1.27 1.27)
+				)
+				(hide yes)
+			)
+		)
+		(property "Manufacturer Part" "TPSM33625RDNR"
+			(at 138.43 83.82 0)
+			(effects
+				(font
+					(size 1.27 1.27)
+				)
+				(hide yes)
+			)
+		)
+		(pin "6"
+		)
+		(pin "9"
+		)
+		(pin "1"
+		)
+		(pin "7"
+		)
+		(pin "8"
+		)
+		(pin "10"
+		)
+		(pin "3"
+		)
+		(pin "2"
+		)
+		(pin "11"
+		)
+		(pin "5"
+		)
+		(pin "4"
+		)
+		(instances
+			(project ""
+				(path "/3f85abf4-0b95-4c4a-b7e9-06f59ca1ea3d/5c2e021f-c2d4-49e2-8c36-9a64f1f12001/de8125f2-04ec-46c6-89d6-d0b5e89f6023"
+					(reference "U2701")
+					(unit 1)
+				)

Commit message: more fixes
Parts:
- U2701: footprint JLCImport:TPSM33625RDNR -> 5v rail sm-easyedapro:QFN-11_L4.5-W3.5-P0.50-TL_TPSM365R6FRDNR
Changed lines of the file:
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@@
 			)
 		)
-		(property "Footprint" "JLCImport:TPSM33625RDNR"
+		(property "Footprint" "5v rail sm-easyedapro:QFN-11_L4.5-W3.5-P0.50-TL_TPSM365R6FRDNR"
 			(at 138.43 83.82 0)
 			(effects
