File: hardware/kicad/21_Microcontroller-Interface.kicad_sch (KiCad schematic)
At the start: 24 parts, among them Q17 L2N7002SLLT1G, Q18 L2N7002SLLT1G, Q19 SI2309A, U49 TPS3700DDCR

Commit message: forgot to add jumpstart
Parts:
- removed H8: PZ254V-11-02P, Connector_PinHeader_2.54mm:PinHeader_2x01_P2.54mm_Vertical, symbol 5v rail sm-easyedapro:PZ254V-11-02P
- removed R121, R122: 4.7kΩ, Resistor_SMD:R_0603_1608Metric, symbol 5v rail sm-easyedapro:0603WAF4701T5E
- removed R123, R124: 2.2kΩ, Resistor_SMD:R_0603_1608Metric, symbol 5v rail sm-easyedapro:0603WAF2201T5E
- added JP3602: Jumper_2_Open, PCM_SparkFun-Jumper:Jumper_2_NO, symbol Jumper:Jumper_2_Open
Connections:
- net GND: now also JP3602.1 (A)
- net at BMS_Bypass_5V_SW1.1, C103.1, Q17.2 (S)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: now also JP3602.2 (B)
- net BAT+ renamed in
- net VCC-KICKSTART renamed out
Other:
- note added: "tie close to bat connector"

Commit message: almost done with kickstart
Parts:
- removed C103: 100nF, Capacitor_SMD:C_0603_1608Metric, symbol 5v rail sm-easyedapro:CC0603KRX7R9BB104
- removed Q17: L2N7002SLLT1G, Package_TO_SOT_SMD:SOT-23, symbol 5v rail sm-easyedapro:L2N7002SLLT1G
- removed R113: 309kΩ, Resistor_SMD:R_0603_1608Metric, symbol 5v rail sm-easyedapro:FRC0603F3093TS
- removed R114, R116: 10kΩ, Resistor_SMD:R_0603_1608Metric, symbol 5v rail sm-easyedapro:FRC0603F1002TS
- removed R115: 232kΩ, Resistor_SMD:R_0603_1608Metric, symbol 5v rail sm-easyedapro:0603WAF2323T5E
- removed R117, R118, R119: 100kΩ, Resistor_SMD:R_0603_1608Metric, symbol 5v rail sm-easyedapro:FRC0603J104 TS
- removed R120: 1kΩ, Resistor_SMD:R_0603_1608Metric, symbol 5v rail sm-easyedapro:FRC0603F1001TS
- added C3601, C3602, C3603: 100n, Capacitor_SMD:C_0402_1005Metric, symbol Device:C
- added R3601, R3603: 100k, Resistor_SMD:R_0402_1005Metric, symbol Device:R
- added R3602: 1k, Resistor_SMD:R_0402_1005Metric, symbol Device:R
- added R3609, R3610: 10k, Resistor_SMD:R_0402_1005Metric, symbol Device:R
- added R3611: 309k, Resistor_SMD:R_0402_1005Metric, symbol Device:R
- added R3612: 232k, Resistor_SMD:R_0402_1005Metric, symbol Device:R
- renumbered BMS_Bypass_5V_SW1 to BMS_Bypass_5V_SW3601, D27 to D3601, D28 to D3602, F5 to F3601, F6 to F3602, JP3602 to JP3601, NT22 to NT3601, Q18 to Q3602, Q19 to Q3603, U49 to U3601
Connections:
- net at BMS_Bypass_5V_SW3601.1, JP3601.2 (B), Q3602.3 (D): now also C3601.2, R3601.1
- net at BMS_Bypass_5V_SW3601.2: now also C3601.1, R3602.2
- net at D3601.2, F3602.2, U3601.5 (VDD): now also R3611.1, R3612.1
- net at U3601.4 (INB-): now also C3602.1, R3609.1, R3611.2
- net at U3601.3 (INA+): now also C3603.1, R3610.1, R3612.2
- net at D3602.2 (A), Q3603.1 (G): now also R3602.1, R3603.2
- net at D3601.1, D3602.1 (K), Q3603.2 (S): now also R3603.1
- net at Q3602.1 (G), U3601.1 (OUTA), U3601.6 (OUTB): now also R3601.2
- net at NT3601.2, U3601.2 (GND): now also C3603.2, R3610.2
- new net: C3602.2, R3609.2
Other:
- moved on the sheet: NT3601

Commit message: switched to ideal diode for 5v
Changed lines of the file:
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@@
 	)
 	(hierarchical_label "out"
-		(shape input)
+		(shape output)
 		(at 307.34 102.87 0)
 		(effects

Commit message: updates
Parts:
- removed BMS_Bypass_5V_SW3601: ~, 5v rail sm-easyedapro:SW-SMD_L3.9-W3.0-P4.45, symbol 5v rail sm-easyedapro:TS-1088-AR02016
- added SW2: TC-6615-5-260G, JLCImport:TC-6615-5-260G, symbol JLCImport:TC-6615-5-260G
Connections:
- net GND: now also SW2.3, SW2.4
- net at C3601.2, JP3601.2 (B), Q3602.3 (D)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: now also SW2.2
- net at C3601.1, R3602.2: now also SW2.1
Changed lines of the file:
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@@
 	(wire
 		(pts
-			(xy 273.05 157.48) (xy 273.05 153.67)
+			(xy 273.05 157.48) (xy 273.05 147.32)
 		)
 		(stroke
@@
 	(wire
 		(pts
-			(xy 273.05 133.35) (xy 273.05 138.43)
+			(xy 273.05 133.35) (xy 273.05 137.16)
 		)
 		(stroke
@@
 	)
 	(symbol
-		(lib_id "5v rail sm-easyedapro:TS-1088-AR02016")
-		(at 273.05 146.05 90)
+		(lib_id "power:GND")
+		(at 270.51 147.32 0)
 		(unit 1)
 		(exclude_from_sim no)
@@
 		(on_board yes)
 		(dnp no)
-		(property "Reference" "BMS_Bypass_5V_SW3601"
-			(at 275.59 143.51 90)
-			(effects
-				(font
-					(size 1.27 1.27)
-				)
-				(justify right top)
-			)
-		)
-		(property "Value" "~"
-			(at 273.05 146.05 0)
-			(effects
-				(font
-					(size 1.27 1.27)
-				)
-			)
-		)
-		(property "Footprint" "5v rail sm-easyedapro:SW-SMD_L3.9-W3.0-P4.45"
-			(at 273.05 146.05 0)
-			(effects
-				(font
-					(size 1.27 1.27)
-				)
-				(hide yes)
-			)
-		)
-		(property "Datasheet" "https://atta.szlcsc.com/upload/public/pdf/source/20200810/C720475_60D09DD6C54279ADDB2DC25100F1CC11.pdf"
-			(at 273.05 146.05 0)
-			(effects
-				(font
-					(size 1.27 1.27)
-				)
-				(hide yes)
-			)
-		)
-		(property "Description" "Circuit:SPST Actuator Style:Round Button Operating Force:160gf Mounting Style:Brick nogging Switch Length:4mm Switch Width:3mm Switch Height:2mm Strike Gundam:不带 Contact Current:50mA Voltage Rating (DC):12V Insulation Resistance:100MΩ Actuator/Cap Color:B"
-			(at 273.05 146.05 0)
-			(effects
-				(font
-					(size 1.27 1.27)
-				)
-				(hide yes)
-			)
-		)
-		(property "Manufacturer Part" "TS-1088-AR02016"
-			(at 273.05 146.05 0)
-			(effects
-				(font
-					(size 1.27 1.27)
-				)
-				(hide yes)
-			)
-		)
-		(property "Manufacturer" "XUNPU(讯普)"
-			(at 273.05 146.05 0)
-			(effects
-				(font
-					(size 1.27 1.27)
-				)
-				(hide yes)
-			)
-		)
-		(property "Supplier Part" "C720477"
-			(at 273.05 146.05 0)
-			(effects
-				(font
-					(size 1.27 1.27)
-				)
-				(hide yes)
-			)
-		)
-		(property "Supplier" "LCSC"
-			(at 273.05 146.05 0)
-			(effects
-				(font
-					(size 1.27 1.27)
-				)
-				(hide yes)
-			)
-		)
-		(property "LCSC Part Name" "4*3*2mm 立贴 轻触开关"
-			(at 273.05 146.05 0)
+		(fields_autoplaced yes)
+		(property "Reference" "#PWR04501"
+			(at 270.51 153.67 0)
+			(effects
+				(font
+					(size 1.27 1.27)
+				)
+				(hide yes)
+			)
+		)
+		(property "Value" "GND"
+			(at 270.51 152.4 0)
+			(effects
+				(font
+					(size 1.27 1.27)
+				)
+			)
+		)
+		(property "Footprint" ""
+			(at 270.51 147.32 0)
+			(effects
+				(font
+					(size 1.27 1.27)
+				)
+				(hide yes)
+			)
+		)
+		(property "Datasheet" ""
+			(at 270.51 147.32 0)
+			(effects
+				(font
+					(size 1.27 1.27)
+				)
+				(hide yes)
+			)
+		)
+		(property "Description" "Power symbol creates a global label with name \"GND\" , ground"
+			(at 270.51 147.32 0)
 			(effects
 				(font
@@
 		)
 		(pin "1"
-		)
-		(pin "2"
 		)
 		(instances
 			(project "svea_powerboard_rev3"
 				(path "/3f85abf4-0b95-4c4a-b7e9-06f59ca1ea3d/5c2e021f-c2d4-49e2-8c36-9a64f1f12001/044ae6eb-f416-4b68-9d75-784bdd14fca8"
-					(reference "BMS_Bypass_5V_SW3601")
+					(reference "#PWR04501")
 					(unit 1)
 				)
@@
 	)
 	(symbol
+		(lib_id "power:GND")
+		(at 270.51 137.16 180)
+		(unit 1)
+		(exclude_from_sim no)
+		(in_bom yes)
+		(on_board yes)
+		(dnp no)
+		(fields_autoplaced yes)
+		(property "Reference" "#PWR04502"
+			(at 270.51 130.81 0)
+			(effects
+				(font
+					(size 1.27 1.27)
+				)
+				(hide yes)
+			)
+		)
+		(property "Value" "GND"
+			(at 270.51 132.08 0)
+			(effects
+				(font
+					(size 1.27 1.27)
+				)
+			)
+		)
+		(property "Footprint" ""
+			(at 270.51 137.16 0)
+			(effects
+				(font
+					(size 1.27 1.27)
+				)
+				(hide yes)
+			)
+		)
+		(property "Datasheet" ""
+			(at 270.51 137.16 0)
+			(effects
+				(font
+					(size 1.27 1.27)
+				)
+				(hide yes)
+			)
+		)
+		(property "Description" "Power symbol creates a global label with name \"GND\" , ground"
+			(at 270.51 137.16 0)
+			(effects
+				(font
+					(size 1.27 1.27)
+				)
+				(hide yes)
+			)
+		)
+		(pin "1"
+		)
+		(instances
+			(project "svea_powerboard_rev3"
+				(path "/3f85abf4-0b95-4c4a-b7e9-06f59ca1ea3d/5c2e021f-c2d4-49e2-8c36-9a64f1f12001/044ae6eb-f416-4b68-9d75-784bdd14fca8"
+					(reference "#PWR04502")
+					(unit 1)
+				)
+			)
+		)
+	)
+	(symbol
 		(lib_id "Device:R")
 		(at 156.21 177.8 0)
@@
 					(unit 1)
 				)
+			)
+		)
+	)
+	(symbol
+		(lib_id "JLCImport:TC-6615-5-260G")
+		(at 273.05 142.24 270)
+		(unit 1)
+		(exclude_from_sim no)
+		(in_bom yes)
+		(on_board yes)
+		(dnp no)
+		(property "Reference" "SW2"
+			(at 276.352 142.24 0)
+			(effects
+				(font
+					(size 1.27 1.27)
+				)
+			)
+		)
+		(property "Value" "TC-6615-5-260G"
+			(at 276.86 142.24 0)
+			(effects
+				(font
+					(size 1.27 1.27)
+				)
+				(hide yes)
+			)
+		)
+		(property "Footprint" "JLCImport:TC-6615-5-260G"
+			(at 273.05 142.24 0)
+			(effects
+				(font
+					(size 1.27 1.27)
+				)
+				(hide yes)
+			)
+		)
+		(property "Datasheet" "https://item.szlcsc.com/763338.html?ref=editor&logined=true"
+			(at 273.05 142.24 0)
+			(effects
+				(font
+					(size 1.27 1.27)
+				)
+				(hide yes)
+			)
+		)
+		(property "Description" ""
+			(at 273.05 142.24 0)
+			(effects
+				(font
+					(size 1.27 1.27)
+				)
+				(hide yes)
+			)
+		)
+		(property "LCSC" "C2845270"
+			(at 273.05 142.24 0)
+			(effects
+				(font
+					(size 1.27 1.27)
+				)
+				(hide yes)
+			)
+		)
+		(property "Manufacturer" "HCTL(华灿天禄)"
+			(at 273.05 142.24 0)
+			(effects
+				(font
+					(size 1.27 1.27)
+				)
+				(hide yes)
+			)
+		)
+		(property "Manufacturer Part" "TC-6615-5-260G"
+			(at 273.05 142.24 0)
+			(effects
+				(font
+					(size 1.27 1.27)
+				)
+				(hide yes)
+			)
+		)
+		(pin "4"
+		)
+		(pin "2"
+		)
+		(pin "3"
+		)
+		(pin "1"
+		)
+		(instances
+			(project "svea_powerboard_rev3"
+				(path "/3f85abf4-0b95-4c4a-b7e9-06f59ca1ea3d/5c2e021f-c2d4-49e2-8c36-9a64f1f12001/044ae6eb-f416-4b68-9d75-784bdd14fca8"
+					(reference "SW2")
+					(unit 1)
+				)

Commit message: updated more footprints
Parts:
- JP3601: footprint PCM_SparkFun-Jumper:Jumper_2_NO -> Jumper:SolderJumper-2_P1.3mm_Open_TrianglePad1.0x1.5mm
Changed lines of the file:
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@@
 			)
 		)
-		(property "Footprint" "PCM_SparkFun-Jumper:Jumper_2_NO"
+		(property "Footprint" "Jumper:SolderJumper-2_P1.3mm_Open_TrianglePad1.0x1.5mm"
 			(at 303.53 167.64 0)
 			(effects

Commit message: various erc fixes
Parts:
- removed JP3601: Jumper_2_Open, Jumper:SolderJumper-2_P1.3mm_Open_TrianglePad1.0x1.5mm, symbol Jumper:Jumper_2_Open
- added JP3601: SolderJumper_2_Open, Jumper:SolderJumper-2_P1.3mm_Open_TrianglePad1.0x1.5mm, symbol Jumper:SolderJumper_2_Open
Connections:
- net GND: now also JP3601.1 (A)
- net at C3601.2, Q3602.3 (D), R3601.1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: now also JP3601.2 (B)
Changed lines of the file:
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@@
+	(wire
+		(pts
+			(xy 303.53 157.48) (xy 303.53 163.83)
+		)
+		(stroke
+			(width 0)
+			(type default)
+		)
+	)
 	(wire
 		(pts
@@
 	(wire
 		(pts
-			(xy 303.53 179.07) (xy 303.53 172.72)
+			(xy 303.53 179.07) (xy 303.53 171.45)
 		)
 		(stroke
@@
 		(pts
 			(xy 179.07 189.23) (xy 179.07 191.77)
-		)
-		(stroke
-			(width 0)
-			(type default)
-		)
-	)
-	(wire
-		(pts
-			(xy 303.53 157.48) (xy 303.53 162.56)
 		)
 		(stroke
@@
 	)
 	(symbol
+		(lib_id "Jumper:SolderJumper_2_Open")
+		(at 303.53 167.64 90)
+		(unit 1)
+		(exclude_from_sim no)
+		(in_bom no)
+		(on_board yes)
+		(dnp no)
+		(fields_autoplaced yes)
+		(property "Reference" "JP3601"
+			(at 306.07 166.3699 90)
+			(effects
+				(font
+					(size 1.27 1.27)
+				)
+				(justify right)
+				(hide yes)
+			)
+		)
+		(property "Value" "SolderJumper_2_Open"
+			(at 306.07 168.9099 90)
+			(effects
+				(font
+					(size 1.27 1.27)
+				)
+				(justify right)
+				(hide yes)
+			)
+		)
+		(property "Footprint" "Jumper:SolderJumper-2_P1.3mm_Open_TrianglePad1.0x1.5mm"
+			(at 303.53 167.64 0)
+			(effects
+				(font
+					(size 1.27 1.27)
+				)
+				(hide yes)
+			)
+		)
+		(property "Datasheet" "~"
+			(at 303.53 167.64 0)
+			(effects
+				(font
+					(size 1.27 1.27)
+				)
+				(hide yes)
+			)
+		)
+		(property "Description" "Solder Jumper, 2-pole, open"
+			(at 303.53 167.64 0)
+			(effects
+				(font
+					(size 1.27 1.27)
+				)
+				(hide yes)
+			)
+		)
+		(pin "2"
+		)
+		(pin "1"
+		)
+		(instances
+			(project "svea_powerboard_rev3"
+				(path "/3f85abf4-0b95-4c4a-b7e9-06f59ca1ea3d/5c2e021f-c2d4-49e2-8c36-9a64f1f12001/044ae6eb-f416-4b68-9d75-784bdd14fca8"
+					(reference "JP3601")
+					(unit 1)
+				)
+			)
+		)
+	)
+	(symbol
 		(lib_id "Device:R")
 		(at 280.67 125.73 0)
@@
 					(unit 1)
 				)
-			)
-		)
-	)
-	(symbol
-		(lib_id "Jumper:Jumper_2_Open")
-		(at 303.53 167.64 90)
-		(unit 1)
-		(exclude_from_sim no)
-		(in_bom yes)
-		(on_board yes)
-		(dnp no)
-		(fields_autoplaced yes)
-		(property "Reference" "JP3601"
-			(at 304.8 166.3699 90)
-			(effects
-				(font
-					(size 1.27 1.27)
-				)
-				(justify right)
-			)
-		)
-		(property "Value" "Jumper_2_Open"
-			(at 304.8 168.9099 90)
-			(effects
-				(font
-					(size 1.27 1.27)
-				)
-				(justify right)
-			)
-		)
-		(property "Footprint" "Jumper:SolderJumper-2_P1.3mm_Open_TrianglePad1.0x1.5mm"
-			(at 303.53 167.64 0)
-			(effects
-				(font
-					(size 1.27 1.27)
-				)
-				(hide yes)
-			)
-		)
-		(property "Datasheet" "~"
-			(at 303.53 167.64 0)
-			(effects
-				(font
-					(size 1.27 1.27)
-				)
-				(hide yes)
-			)
-		)
-		(property "Description" "Jumper, 2-pole, open"
-			(at 303.53 167.64 0)
-			(effects
-				(font
-					(size 1.27 1.27)
-				)
-				(hide yes)
-			)
-		)
-		(pin "1"
-		)
-		(pin "2"
-		)
-		(instances
-			(project ""
-				(path "/3f85abf4-0b95-4c4a-b7e9-06f59ca1ea3d/5c2e021f-c2d4-49e2-8c36-9a64f1f12001/044ae6eb-f416-4b68-9d75-784bdd14fca8"
-					(reference "JP3601")
-					(unit 1)
-				)

Commit message: various updates
Parts:
- D3601, D3602: footprint Diode_SMD:SOD-123 -> Diode_SMD:D_SOD-123
Connections:
- net in renamed IN
- net out renamed OUT
Changed lines of the file:
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@@
 		)
 	)
-	(hierarchical_label "in"
+	(hierarchical_label "IN"
 		(shape input)
 		(at 128.27 102.87 180)
@@
 		)
 	)
-	(hierarchical_label "out"
+	(hierarchical_label "OUT"
 		(shape output)
 		(at 307.34 102.87 0)
@@
 			)
 		)
-		(property "Footprint" "Diode_SMD:SOD-123"
+		(property "Footprint" "Diode_SMD:D_SOD-123"
 			(at 207.01 102.87 0)
 			(effects
@@
 			)
 		)
-		(property "Footprint" "Diode_SMD:SOD-123"
+		(property "Footprint" "Diode_SMD:D_SOD-123"
 			(at 255.27 109.22 0)
 			(effects
