File: hardware/kicad/27_Microcontroller-PIN-IC.kicad_sch (KiCad schematic)
At the start: 19 parts, among them U50 PCAL6524HEAZ

Commit message: exported to schematic
Parts:
- C104: LCSC (none) -> C1600541
Changed lines of the file:
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@@
+			)
+		)
+		(property "LCSC" "C1600541"
+			(at 227.33 52.07 0)
+			(effects
+				(font
+					(size 1.27 1.27)
+				)
+				(hide yes)
 			)
 		)
