File: hardware/kicad/IDEAL_OR_LM73100.kicad_sch (KiCad schematic)
At the start: 10 parts, among them Q19 L2N7002SLLT1G, U70 LM73100RPWR

Commit message: updating symbols to use kicad footprints where possible
Parts:
- C137: footprint 5v rail sm-easyedapro:C0603 -> Capacitor_SMD:C_0603_1608Metric
- D39: footprint 5v rail sm-easyedapro:SMA_L4.3-W2.6-LS5.2-RD -> Diode_SMD:D_SMA
Changed lines of the file:
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@@
 			)
 		)
-		(property "Footprint" "5v rail sm-easyedapro:C0603"
+		(property "Footprint" "Capacitor_SMD:C_0603_1608Metric"
 			(at 184.15 68.58 0)
 			(effects
@@
 			)
 		)
-		(property "Footprint" "5v rail sm-easyedapro:SMA_L4.3-W2.6-LS5.2-RD"
+		(property "Footprint" "Diode_SMD:D_SMA"
 			(at 196.85 68.58 0)
 			(effects

Commit message: switched some more
Parts:
- D39: footprint Diode_SMD:D_SMA -> Diode_SMD:SMA
Changed lines of the file:
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@@
 			)
 		)
-		(property "Footprint" "Diode_SMD:D_SMA"
+		(property "Footprint" "Diode_SMD:SMA"
 			(at 196.85 68.58 0)
 			(effects

Commit message: exported to schematic
Parts:
- U70: LCSC C3210761 -> C22371533
Changed lines of the file:
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@@
 			)
 		)
-		(property "LCSC" "C3210761"
+		(property "LCSC" "C22371533"
 			(at 135.89 68.58 0)
 			(effects
