File: hardware/kicad/INA226_SINGLE_CURR_SENSOR.kicad_sch (KiCad schematic)
At the start: 5 parts, among them U72 INA226AIDGSR

Commit message: servo current sensor also done
Changed lines of the file:
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@@
 	)
 	(junction
-		(at 163.83 81.28)
+		(at 151.13 76.2)
 		(diameter 0)
 		(color 0 0 0 0)
@@
 	(wire
 		(pts
+			(xy 151.13 76.2) (xy 147.32 76.2)
+		)
+		(stroke
+			(width 0)
+			(type default)
+		)
+	)
+	(wire
+		(pts
+			(xy 147.32 81.28) (xy 151.13 81.28)
+		)
+		(stroke
+			(width 0)
+			(type default)
+		)
+	)
+	(wire
+		(pts
 			(xy 147.32 83.82) (xy 151.13 83.82)
 		)
@@
 	(wire
 		(pts
-			(xy 163.83 81.28) (xy 163.83 76.2)
-		)
-		(stroke
-			(width 0)
-			(type default)
-		)
-	)
-	(wire
-		(pts
 			(xy 200.66 86.36) (xy 194.31 86.36)
 		)
@@
 	(wire
 		(pts
-			(xy 172.72 78.74) (xy 147.32 78.74)
+			(xy 147.32 78.74) (xy 172.72 78.74)
 		)
 		(stroke
@@
 	(wire
 		(pts
+			(xy 151.13 81.28) (xy 151.13 76.2)
+		)
+		(stroke
+			(width 0)
+			(type default)
+		)
+	)
+	(wire
+		(pts
 			(xy 194.31 86.36) (xy 194.31 83.82)
 		)
@@
 	(wire
 		(pts
-			(xy 177.8 81.28) (xy 181.61 81.28)
+			(xy 177.8 76.2) (xy 181.61 76.2)
 		)
 		(stroke
@@
 	(wire
 		(pts
-			(xy 172.72 81.28) (xy 163.83 81.28)
-		)
-		(stroke
-			(width 0)
-			(type default)
-		)
-	)
-	(wire
-		(pts
-			(xy 147.32 81.28) (xy 163.83 81.28)
-		)
-		(stroke
-			(width 0)
-			(type default)
-		)
-	)
-	(wire
-		(pts
 			(xy 151.13 83.82) (xy 151.13 91.44)
 		)
@@
 	(wire
 		(pts
-			(xy 163.83 76.2) (xy 147.32 76.2)
+			(xy 151.13 76.2) (xy 172.72 76.2)
 		)
 		(stroke
@@
 	)
 	(label "VIN_P"
-		(at 166.37 81.28 0)
+		(at 166.37 76.2 0)
 		(effects
 			(font
@@
 	(hierarchical_label "VIN+"
 		(shape input)
-		(at 181.61 81.28 0)
+		(at 181.61 76.2 0)
 		(effects
 			(font
@@
 	(symbol
 		(lib_id "Device:NetTie_2")
-		(at 175.26 81.28 180)
+		(at 175.26 76.2 180)
 		(unit 1)
 		(exclude_from_sim no)
@@
 		(fields_autoplaced yes)
 		(property "Reference" "NT19"
-			(at 173.9899 80.01 90)
+			(at 173.9899 74.93 90)
 			(effects
 				(font
@@
 		)
 		(property "Value" "NetTie_2"
-			(at 176.5299 80.01 90)
+			(at 176.5299 74.93 90)
 			(effects
 				(font
@@
 		)
 		(property "Footprint" "5v rail sm-easyedapro:NetTie-2_SMD_Pad0.2mm"
-			(at 175.26 81.28 0)
+			(at 175.26 76.2 0)
 			(effects
 				(font
@@
 		)
 		(property "Datasheet" "~"
-			(at 175.26 81.28 0)
+			(at 175.26 76.2 0)
 			(effects
 				(font
@@
 		)
 		(property "Description" "Net tie, 2 pins"
-			(at 175.26 81.28 0)
-			(effects
-				(font
+			(at 175.26 76.2 0)
+			(effects
+				(font

Commit message: starting erc check
Parts:
- C89, C90: footprint Capacitor_SMD:C_0603_1608Metric -> 5v rail sm-easyedapro:C0603
- U72: footprint Package_SO:MSOP-10_3x3mm_P0.5mm -> 5v rail sm-easyedapro:MSOP-10_L3.0-W3.0-P0.50-LS5.0-BL
Changed lines of the file:
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@@
 			)
 		)
-		(property "Description" "Power-5V"
+		(property "Description" "Power symbol creates a global label with name \"+3V3\""
 			(at 194.31 83.82 0)
 			(effects
@@
 			)
 		)
-		(property "Description" ""
+		(property "Description" "Power symbol creates a global label with name \"GND\" , ground"
 			(at 151.13 91.44 0)
 			(effects
@@
 			)
 		)
-		(property "Footprint" "Capacitor_SMD:C_0603_1608Metric"
+		(property "Footprint" "5v rail sm-easyedapro:C0603"
 			(at 200.66 93.98 0)
 			(effects
@@
 			)
 		)
-		(property "Description" ""
+		(property "Description" "Power symbol creates a global label with name \"GND\" , ground"
 			(at 194.31 104.14 0)
 			(effects
@@
 			)
 		)
-		(property "Footprint" "Package_SO:MSOP-10_3x3mm_P0.5mm"
+		(property "Footprint" "5v rail sm-easyedapro:MSOP-10_L3.0-W3.0-P0.50-LS5.0-BL"
 			(at 134.62 81.28 0)
 			(effects
@@
 			)
 		)
-		(property "Footprint" "Capacitor_SMD:C_0603_1608Metric"
+		(property "Footprint" "5v rail sm-easyedapro:C0603"
 			(at 187.96 93.98 0)
 			(effects

Commit message: updating symbols to use kicad footprints where possible
Parts:
- C89, C90: footprint 5v rail sm-easyedapro:C0603 -> Capacitor_SMD:C_0603_1608Metric
- U72: footprint 5v rail sm-easyedapro:MSOP-10_L3.0-W3.0-P0.50-LS5.0-BL -> Package_SO:VSSOP-10_3x3mm_P0.5mm
Changed lines of the file:
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@@
 			)
 		)
-		(property "Footprint" "5v rail sm-easyedapro:C0603"
+		(property "Footprint" "Capacitor_SMD:C_0603_1608Metric"
 			(at 200.66 93.98 0)
 			(effects
@@
 			)
 		)
-		(property "Footprint" "5v rail sm-easyedapro:MSOP-10_L3.0-W3.0-P0.50-LS5.0-BL"
+		(property "Footprint" "Package_SO:VSSOP-10_3x3mm_P0.5mm"
 			(at 134.62 81.28 0)
 			(effects
@@
 			)
 		)
-		(property "Footprint" "5v rail sm-easyedapro:C0603"
+		(property "Footprint" "Capacitor_SMD:C_0603_1608Metric"
 			(at 187.96 93.98 0)
 			(effects

Commit message: updated more footprints
Parts:
- U72: footprint Package_SO:VSSOP-10_3x3mm_P0.5mm -> Package_SO:VSSOP-10_3.0x3.0mm_P0.5mm
Changed lines of the file:
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@@
 			)
 		)
-		(property "Footprint" "Package_SO:VSSOP-10_3x3mm_P0.5mm"
+		(property "Footprint" "Package_SO:VSSOP-10_3.0x3.0mm_P0.5mm"
 			(at 134.62 81.28 0)
 			(effects

Commit message: update
Parts:
- U72: footprint Package_SO:VSSOP-10_3.0x3.0mm_P0.5mm -> Package_SO:VSSOP-10_3x3mm_P0.5mm
Changed lines of the file:
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@@
 			)
 		)
-		(property "Footprint" "Package_SO:VSSOP-10_3.0x3.0mm_P0.5mm"
+		(property "Footprint" "Package_SO:VSSOP-10_3x3mm_P0.5mm"
 			(at 134.62 81.28 0)
 			(effects

Commit message: fixing inconsistencies in value convention
Parts:
- C89: value 1uF -> 1u
- C90: value 100nF -> 100n
Changed lines of the file:
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@@
 			)
 		)
-		(property "Value" "100nF"
+		(property "Value" "100n"
 			(at 204.47 96.52 90)
 			(effects
@@
 			)
 		)
-		(property "Value" "1uF"
+		(property "Value" "1u"
 			(at 191.77 96.52 90)
 			(effects

Commit message: exported to schematic
Parts:
- C89: LCSC (none) -> C5199872
- C90: LCSC (none) -> C14663
- U72: LCSC (none) -> C49851
Changed lines of the file:
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@@
+			)
+		)
+		(property "LCSC" "C14663"
+			(at 204.47 93.98 0)
+			(effects
+				(font
+					(size 1.27 1.27)
+				)
+				(hide yes)
 			)
 		)
@@
 			)
 		)
+		(property "LCSC" "C49851"
+			(at 127 73.152 0)
+			(effects
+				(font
+					(size 1.27 1.27)
+				)
+				(hide yes)
+			)
+		)
 		(pin "7"
 		)
@@
 			(effects
 				(font
+					(size 1.27 1.27)
+				)
+				(hide yes)
+			)
+		)
+		(property "LCSC" "C5199872"
+			(at 191.77 93.98 0)
+			(effects
+				(font
