File: hardware/kicad/JST-VH-12V-PIN.kicad_sch (KiCad schematic)
At the start: 5 parts, among them U41 VH3_96-2P_WZ

Commit message: starting erc check
Parts:
- C44: footprint Capacitor_SMD:C_0805_2012Metric -> 5v rail sm-easyedapro:C0805
- C45: footprint Capacitor_SMD:C_0603_1608Metric -> 5v rail sm-easyedapro:C0603
- D13: footprint Diode_SMD:SOD-123FL -> 5v rail sm-easyedapro:SOD-123FL_L2.8-W1.8-LS3.6-RD
- R103: footprint Resistor_SMD:R_2512_6332Metric -> 5v rail sm-easyedapro:R2512
Changed lines of the file:
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@@
 			)
 		)
-		(property "Footprint" "Diode_SMD:SOD-123FL"
+		(property "Footprint" "5v rail sm-easyedapro:SOD-123FL_L2.8-W1.8-LS3.6-RD"
 			(at 152.4 96.52 0)
 			(effects
@@
 			)
 		)
-		(property "Footprint" "Capacitor_SMD:C_0603_1608Metric"
+		(property "Footprint" "5v rail sm-easyedapro:C0603"
 			(at 139.7 96.52 0)
 			(effects
@@
 			)
 		)
-		(property "Footprint" "Capacitor_SMD:C_0805_2012Metric"
+		(property "Footprint" "5v rail sm-easyedapro:C0805"
 			(at 128.27 96.52 0)
 			(effects
@@
 			)
 		)
-		(property "Footprint" "Resistor_SMD:R_2512_6332Metric"
+		(property "Footprint" "5v rail sm-easyedapro:R2512"
 			(at 160.02 91.44 0)
 			(effects

Commit message: flipped spots for 12v ports
Parts:
- renumbered C44 to C403, C45 to C404, D13 to D402, R103 to R402, U41 to U401
Changed lines of the file:
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@@
 		(on_board yes)
 		(dnp no)
-		(property "Reference" "U41"
+		(property "Reference" "U401"
 			(at 97.79 105.41 0)
 			(effects
@@
 		(instances
 			(project "svea_powerboard_rev3"
-				(path "/3f85abf4-0b95-4c4a-b7e9-06f59ca1ea3d/5c2e021f-c2d4-49e2-8c36-9a64f1f12001/03241f80-3125-4f5b-a1a0-add76ba31aaa"
-					(reference "U41")
+				(path "/3f85abf4-0b95-4c4a-b7e9-06f59ca1ea3d/5c2e021f-c2d4-49e2-8c36-9a64f1f12001/26d23ec5-4653-42e2-9dd5-fc2659d8ed77"
+					(reference "U401")
+					(unit 1)
+				)
+				(path "/3f85abf4-0b95-4c4a-b7e9-06f59ca1ea3d/5c2e021f-c2d4-49e2-8c36-9a64f1f12001/323d2f5c-e7b4-423e-bfab-5a31f4298708"
+					(reference "U501")
 					(unit 1)
 				)
 				(path "/3f85abf4-0b95-4c4a-b7e9-06f59ca1ea3d/5c2e021f-c2d4-49e2-8c36-9a64f1f12001/782118f9-6c0b-4f5a-9c3b-1e5b8fc1f0ac"
 					(reference "U42")
-					(unit 1)
-				)
-				(path "/3f85abf4-0b95-4c4a-b7e9-06f59ca1ea3d/5c2e021f-c2d4-49e2-8c36-9a64f1f12001/beb9ceef-df3a-4e22-8974-012ce1407a41"
-					(reference "U43")
 					(unit 1)
 				)
@@
 		(on_board yes)
 		(dnp no)
-		(property "Reference" "D13"
+		(property "Reference" "D402"
 			(at 154.94 97.79 90)
 			(effects
@@
 		(instances
 			(project "svea_powerboard_rev3"
-				(path "/3f85abf4-0b95-4c4a-b7e9-06f59ca1ea3d/5c2e021f-c2d4-49e2-8c36-9a64f1f12001/03241f80-3125-4f5b-a1a0-add76ba31aaa"
-					(reference "D13")
+				(path "/3f85abf4-0b95-4c4a-b7e9-06f59ca1ea3d/5c2e021f-c2d4-49e2-8c36-9a64f1f12001/26d23ec5-4653-42e2-9dd5-fc2659d8ed77"
+					(reference "D402")
+					(unit 1)
+				)
+				(path "/3f85abf4-0b95-4c4a-b7e9-06f59ca1ea3d/5c2e021f-c2d4-49e2-8c36-9a64f1f12001/323d2f5c-e7b4-423e-bfab-5a31f4298708"
+					(reference "D501")
 					(unit 1)
 				)
 				(path "/3f85abf4-0b95-4c4a-b7e9-06f59ca1ea3d/5c2e021f-c2d4-49e2-8c36-9a64f1f12001/782118f9-6c0b-4f5a-9c3b-1e5b8fc1f0ac"
 					(reference "D14")
-					(unit 1)
-				)
-				(path "/3f85abf4-0b95-4c4a-b7e9-06f59ca1ea3d/5c2e021f-c2d4-49e2-8c36-9a64f1f12001/beb9ceef-df3a-4e22-8974-012ce1407a41"
-					(reference "D15")
 					(unit 1)
 				)
@@
 		(on_board yes)
 		(dnp no)
-		(property "Reference" "C45"
+		(property "Reference" "C404"
 			(at 143.51 96.52 90)
 			(effects
@@
 		(instances
 			(project "svea_powerboard_rev3"
-				(path "/3f85abf4-0b95-4c4a-b7e9-06f59ca1ea3d/5c2e021f-c2d4-49e2-8c36-9a64f1f12001/03241f80-3125-4f5b-a1a0-add76ba31aaa"
-					(reference "C45")
+				(path "/3f85abf4-0b95-4c4a-b7e9-06f59ca1ea3d/5c2e021f-c2d4-49e2-8c36-9a64f1f12001/26d23ec5-4653-42e2-9dd5-fc2659d8ed77"
+					(reference "C404")
+					(unit 1)
+				)
+				(path "/3f85abf4-0b95-4c4a-b7e9-06f59ca1ea3d/5c2e021f-c2d4-49e2-8c36-9a64f1f12001/323d2f5c-e7b4-423e-bfab-5a31f4298708"
+					(reference "C502")
 					(unit 1)
 				)
 				(path "/3f85abf4-0b95-4c4a-b7e9-06f59ca1ea3d/5c2e021f-c2d4-49e2-8c36-9a64f1f12001/782118f9-6c0b-4f5a-9c3b-1e5b8fc1f0ac"
 					(reference "C47")
-					(unit 1)
-				)
-				(path "/3f85abf4-0b95-4c4a-b7e9-06f59ca1ea3d/5c2e021f-c2d4-49e2-8c36-9a64f1f12001/beb9ceef-df3a-4e22-8974-012ce1407a41"
-					(reference "C49")
 					(unit 1)
 				)
@@
 		(on_board yes)
 		(dnp no)
-		(property "Reference" "C44"
+		(property "Reference" "C403"
 			(at 132.08 96.52 90)
 			(effects
@@
 		(instances
 			(project "svea_powerboard_rev3"
-				(path "/3f85abf4-0b95-4c4a-b7e9-06f59ca1ea3d/5c2e021f-c2d4-49e2-8c36-9a64f1f12001/03241f80-3125-4f5b-a1a0-add76ba31aaa"
-					(reference "C44")
+				(path "/3f85abf4-0b95-4c4a-b7e9-06f59ca1ea3d/5c2e021f-c2d4-49e2-8c36-9a64f1f12001/26d23ec5-4653-42e2-9dd5-fc2659d8ed77"
+					(reference "C403")
+					(unit 1)
+				)
+				(path "/3f85abf4-0b95-4c4a-b7e9-06f59ca1ea3d/5c2e021f-c2d4-49e2-8c36-9a64f1f12001/323d2f5c-e7b4-423e-bfab-5a31f4298708"
+					(reference "C501")
 					(unit 1)
 				)
 				(path "/3f85abf4-0b95-4c4a-b7e9-06f59ca1ea3d/5c2e021f-c2d4-49e2-8c36-9a64f1f12001/782118f9-6c0b-4f5a-9c3b-1e5b8fc1f0ac"
 					(reference "C46")
-					(unit 1)
-				)
-				(path "/3f85abf4-0b95-4c4a-b7e9-06f59ca1ea3d/5c2e021f-c2d4-49e2-8c36-9a64f1f12001/beb9ceef-df3a-4e22-8974-012ce1407a41"
-					(reference "C48")
 					(unit 1)
 				)
@@
 		(on_board yes)
 		(dnp no)
-		(property "Reference" "R103"
+		(property "Reference" "R402"
 			(at 162.56 93.218 0)
 			(effects
@@
 		(instances
 			(project "svea_powerboard_rev3"
-				(path "/3f85abf4-0b95-4c4a-b7e9-06f59ca1ea3d/5c2e021f-c2d4-49e2-8c36-9a64f1f12001/03241f80-3125-4f5b-a1a0-add76ba31aaa"
-					(reference "R103")
+				(path "/3f85abf4-0b95-4c4a-b7e9-06f59ca1ea3d/5c2e021f-c2d4-49e2-8c36-9a64f1f12001/26d23ec5-4653-42e2-9dd5-fc2659d8ed77"
+					(reference "R402")
+					(unit 1)
+				)
+				(path "/3f85abf4-0b95-4c4a-b7e9-06f59ca1ea3d/5c2e021f-c2d4-49e2-8c36-9a64f1f12001/323d2f5c-e7b4-423e-bfab-5a31f4298708"
+					(reference "R501")
 					(unit 1)
 				)
@@
 					(unit 1)
 				)
-				(path "/3f85abf4-0b95-4c4a-b7e9-06f59ca1ea3d/5c2e021f-c2d4-49e2-8c36-9a64f1f12001/beb9ceef-df3a-4e22-8974-012ce1407a41"
-					(reference "R105")
-					(unit 1)
-				)

Commit message: updating symbols to use kicad footprints where possible
Parts:
- C403: footprint 5v rail sm-easyedapro:C0805 -> Capacitor_SMD:C_0805_2012Metric
- C404: footprint 5v rail sm-easyedapro:C0603 -> Capacitor_SMD:C_0603_1608Metric
- R402: footprint 5v rail sm-easyedapro:R2512 -> Resistor_SMD:R_2512_6332Metric
Changed lines of the file:
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@@
 			)
 		)
-		(property "Footprint" "5v rail sm-easyedapro:C0603"
+		(property "Footprint" "Capacitor_SMD:C_0603_1608Metric"
 			(at 139.7 96.52 0)
 			(effects
@@
 			)
 		)
-		(property "Footprint" "5v rail sm-easyedapro:C0805"
+		(property "Footprint" "Capacitor_SMD:C_0805_2012Metric"
 			(at 128.27 96.52 0)
 			(effects
@@
 			)
 		)
-		(property "Footprint" "5v rail sm-easyedapro:R2512"
+		(property "Footprint" "Resistor_SMD:R_2512_6332Metric"
 			(at 160.02 91.44 0)
 			(effects

Commit message: switched some more
Parts:
- D402: footprint 5v rail sm-easyedapro:SOD-123FL_L2.8-W1.8-LS3.6-RD -> Diode_SMD:SOD-123FL
Changed lines of the file:
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@@
 			)
 		)
-		(property "Footprint" "5v rail sm-easyedapro:SOD-123FL_L2.8-W1.8-LS3.6-RD"
+		(property "Footprint" "Diode_SMD:SOD-123FL"
 			(at 152.4 96.52 0)
 			(effects

Commit message: update
Parts:
- D402: footprint Diode_SMD:SOD-123FL -> 5v rail sm-easyedapro:SOD-123FL_L2.8-W1.8-LS3.6-RD
Changed lines of the file:
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@@
 			)
 		)
-		(property "Footprint" "Diode_SMD:SOD-123FL"
+		(property "Footprint" "5v rail sm-easyedapro:SOD-123FL_L2.8-W1.8-LS3.6-RD"
 			(at 152.4 96.52 0)
 			(effects

Commit message: fixing inconsistencies in value convention
Parts:
- C403: value 10uF -> 10u
- C404: value 100nF -> 100n
- R402: value 16mΩ -> 16m
Changed lines of the file:
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@@
 			)
 		)
-		(property "Value" "100nF"
+		(property "Value" "100n"
 			(at 143.51 99.06 90)
 			(effects
@@
 			)
 		)
-		(property "Value" "10uF"
+		(property "Value" "10u"
 			(at 132.08 99.06 90)
 			(effects
@@
 			)
 		)
-		(property "Value" "16mΩ"
+		(property "Value" "16m"
 			(at 163.068 88.392 0)
 			(effects

Commit message: exported to schematic
Parts:
- C403: LCSC (none) -> C440198
- C404: LCSC (none) -> C14663
- D402: LCSC (none) -> C353315
- R402: LCSC (none) -> C5775686
Changed lines of the file:
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@@
+			)
+		)
+		(property "LCSC" "C353315"
+			(at 154.94 97.79 0)
+			(effects
+				(font
+					(size 1.27 1.27)
+				)
+				(hide yes)
 			)
 		)
@@
 			)
 		)
+		(property "LCSC" "C14663"
+			(at 143.51 96.52 0)
+			(effects
+				(font
+					(size 1.27 1.27)
+				)
+				(hide yes)
+			)
+		)
 		(pin "2"
 		)
@@
 			)
 		)
+		(property "LCSC" "C440198"
+			(at 132.08 96.52 0)
+			(effects
+				(font
+					(size 1.27 1.27)
+				)
+				(hide yes)
+			)
+		)
 		(pin "1"
 		)
@@
 			(effects
 				(font
+					(size 1.27 1.27)
+				)
+				(hide yes)
+			)
+		)
+		(property "LCSC" "C5775686"
+			(at 162.56 93.218 0)
+			(effects
+				(font
