File: hardware/kicad/TPS16630RGER_CHARGING_EFUSE.kicad_sch (KiCad schematic)
At the start: 16 parts, among them U62 TPS16630RGER

Commit message: updates
Parts:
- D17: footprint Diode_SMD:SMB -> Diode_SMD:D_SMB
- D35: footprint Diode_SMD:SMA -> Diode_SMD:D_SMA
Connections:
- net GND: now also U62.20 (N.C), U62.21 (N.C), U62.22 (N.C)
Changed lines of the file:
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@@
+	)
+	(junction
+		(at 186.69 82.55)
+		(diameter 0)
+		(color 0 0 0 0)
 	)
 	(junction
@@
 	)
 	(junction
+		(at 186.69 90.17)
+		(diameter 0)
+		(color 0 0 0 0)
+	)
+	(junction
 		(at 135.89 80.01)
 		(diameter 0)
@@
 	)
 	(junction
+		(at 186.69 87.63)
+		(diameter 0)
+		(color 0 0 0 0)
+	)
+	(junction
 		(at 73.66 97.79)
 		(diameter 0)
@@
 	(junction
 		(at 161.29 80.01)
+		(diameter 0)
+		(color 0 0 0 0)
+	)
+	(junction
+		(at 186.69 85.09)
 		(diameter 0)
 		(color 0 0 0 0)
@@
 	(wire
 		(pts
+			(xy 186.69 90.17) (xy 186.69 92.71)
+		)
+		(stroke
+			(width 0)
+			(type default)
+		)
+	)
+	(wire
+		(pts
 			(xy 63.5 97.79) (xy 73.66 97.79)
 		)
@@
 	(wire
 		(pts
-			(xy 186.69 82.55) (xy 186.69 92.71)
+			(xy 186.69 87.63) (xy 186.69 90.17)
+		)
+		(stroke
+			(width 0)
+			(type default)
+		)
+	)
+	(wire
+		(pts
+			(xy 186.69 82.55) (xy 186.69 85.09)
 		)
 		(stroke
@@
 		(pts
 			(xy 236.22 107.95) (xy 236.22 106.68)
+		)
+		(stroke
+			(width 0)
+			(type default)
+		)
+	)
+	(wire
+		(pts
+			(xy 186.69 85.09) (xy 186.69 87.63)
 		)
 		(stroke
@@
 			)
 		)
-		(property "Footprint" "Diode_SMD:SMA"
+		(property "Footprint" "Diode_SMD:D_SMA"
 			(at 266.7 101.6 0)
 			(effects
@@
 			)
 		)
-		(property "Footprint" "Diode_SMD:SMB"
+		(property "Footprint" "Diode_SMD:D_SMB"
 			(at 236.22 101.6 0)
 			(effects

Commit message: updates
Parts:
- R1908: value 19.1Ω -> 19.1kΩ
Changed lines of the file:
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@@
 			)
 		)
-		(property "Value" "19.1Ω"
+		(property "Value" "19.1kΩ"
 			(at 220.98 142.2399 0)
 			(effects

Commit message: various erc fixes
Parts:
- removed U60: ~, Jumper:SolderJumper-2_P1.3mm_Bridged_Pad1.0x1.5mm, symbol Jumper:Jumper_2_Bridged
- added JP1901: SolderJumper_2_Bridged, Jumper:SolderJumper-2_P1.3mm_Bridged_Pad1.0x1.5mm, symbol Jumper:SolderJumper_2_Bridged
- U62: footprint 5v rail sm-easyedapro:VFQFPN-24_L4.0-W4.0-P0.50-BL-EP2.8 -> Package_DFN_QFN:QFN-24-1EP_4x4mm_P0.5mm_EP2.8x2.8mm
Connections:
- net GND: now also JP1901.1 (A)
- net at R1902.1, R1903.2: now also JP1901.2 (B)
Changed lines of the file:
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@@
 	(wire
 		(pts
-			(xy 66.04 139.7) (xy 66.04 143.51)
+			(xy 66.04 139.7) (xy 66.04 144.78)
 		)
 		(stroke
@@
 	(wire
 		(pts
-			(xy 66.04 157.48) (xy 66.04 153.67)
+			(xy 66.04 157.48) (xy 66.04 152.4)
 		)
 		(stroke
@@
 	)
 	(symbol
+		(lib_id "Jumper:SolderJumper_2_Bridged")
+		(at 66.04 148.59 90)
+		(unit 1)
+		(exclude_from_sim no)
+		(in_bom no)
+		(on_board yes)
+		(dnp no)
+		(fields_autoplaced yes)
+		(property "Reference" "JP1901"
+			(at 68.58 147.3199 90)
+			(effects
+				(font
+					(size 1.27 1.27)
+				)
+				(justify right)
+				(hide yes)
+			)
+		)
+		(property "Value" "SolderJumper_2_Bridged"
+			(at 68.58 149.8599 90)
+			(effects
+				(font
+					(size 1.27 1.27)
+				)
+				(justify right)
+				(hide yes)
+			)
+		)
+		(property "Footprint" "Jumper:SolderJumper-2_P1.3mm_Bridged_Pad1.0x1.5mm"
+			(at 66.04 148.59 0)
+			(effects
+				(font
+					(size 1.27 1.27)
+				)
+				(hide yes)
+			)
+		)
+		(property "Datasheet" "~"
+			(at 66.04 148.59 0)
+			(effects
+				(font
+					(size 1.27 1.27)
+				)
+				(hide yes)
+			)
+		)
+		(property "Description" "Solder Jumper, 2-pole, closed/bridged"
+			(at 66.04 148.59 0)
+			(effects
+				(font
+					(size 1.27 1.27)
+				)
+				(hide yes)
+			)
+		)
+		(pin "2"
+		)
+		(pin "1"
+		)
+		(instances
+			(project "svea_powerboard_rev3"
+				(path "/3f85abf4-0b95-4c4a-b7e9-06f59ca1ea3d/5c2e021f-c2d4-49e2-8c36-9a64f1f12001/edbb302e-07de-47c0-9e17-f5f094cbde02"
+					(reference "JP1901")
+					(unit 1)
+				)
+			)
+		)
+	)
+	(symbol
 		(lib_id "Device:R")
 		(at 127 118.11 90)
@@
 	)
 	(symbol
-		(lib_id "Jumper:Jumper_2_Bridged")
-		(at 66.04 148.59 90)
-		(unit 1)
-		(exclude_from_sim no)
-		(in_bom yes)
-		(on_board yes)
-		(dnp no)
-		(property "Reference" "U60"
-			(at 67.31 149.86 90)
-			(effects
-				(font
-					(size 1.27 1.27)
-				)
-				(justify right top)
-				(hide yes)
-			)
-		)
-		(property "Value" "~"
-			(at 66.04 148.59 0)
-			(effects
-				(font
-					(size 1.27 1.27)
-				)
-			)
-		)
-		(property "Footprint" "Jumper:SolderJumper-2_P1.3mm_Bridged_Pad1.0x1.5mm"
-			(at 66.04 148.59 0)
-			(effects
-				(font
-					(size 1.27 1.27)
-				)
-				(hide yes)
-			)
-		)
-		(property "Datasheet" "~"
-			(at 66.04 148.59 0)
-			(effects
-				(font
-					(size 1.27 1.27)
-				)
-				(hide yes)
-			)
-		)
-		(property "Description" "Jumper, 2-pole, closed/bridged"
-			(at 66.04 148.59 0)
-			(effects
-				(font
-					(size 1.27 1.27)
-				)
-				(hide yes)
-			)
-		)
-		(pin "1"
-		)
-		(pin "2"
-		)
-		(instances
-			(project "svea_powerboard_rev3"
-				(path "/3f85abf4-0b95-4c4a-b7e9-06f59ca1ea3d/5c2e021f-c2d4-49e2-8c36-9a64f1f12001/edbb302e-07de-47c0-9e17-f5f094cbde02"
-					(reference "U60")
-					(unit 1)
-				)
-			)
-		)
-	)
-	(symbol
 		(lib_id "Device:R")
 		(at 73.66 148.59 180)
@@
 			)
 		)
-		(property "Footprint" "5v rail sm-easyedapro:VFQFPN-24_L4.0-W4.0-P0.50-BL-EP2.8"
+		(property "Footprint" "Package_DFN_QFN:QFN-24-1EP_4x4mm_P0.5mm_EP2.8x2.8mm"
 			(at 175.26 93.98 0)
 			(effects

Commit message: various updates
Parts:
- D36: footprint Diode_SMD:SMB -> Diode_SMD:D_SMB
Changed lines of the file:
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@@
 			)
 		)
-		(property "Footprint" "Diode_SMD:SMB"
+		(property "Footprint" "Diode_SMD:D_SMB"
 			(at 87.63 68.58 0)
 			(effects

Commit message: update
Changed lines of the file:
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@@
+	)
+	(junction
+		(at 160.02 143.51)
+		(diameter 0)
+		(color 0 0 0 0)
 	)
 	(junction
@@
 	)
 	(junction
-		(at 147.32 144.78)
-		(diameter 0)
-		(color 0 0 0 0)
-	)
-	(junction
 		(at 251.46 95.25)
 		(diameter 0)
@@
 	)
 	(junction
-		(at 160.02 144.78)
-		(diameter 0)
-		(color 0 0 0 0)
-	)
-	(junction
 		(at 69.85 157.48)
 		(diameter 0)
@@
 	)
 	(junction
-		(at 147.32 144.7546)
+		(at 147.32 143.51)
 		(diameter 0)
 		(color 0 0 0 0)
@@
 	(wire
 		(pts
-			(xy 160.02 144.78) (xy 147.32 144.78)
+			(xy 160.02 143.51) (xy 147.32 143.51)
 		)
 		(stroke
@@
 	(wire
 		(pts
-			(xy 147.32 153.67) (xy 147.32 144.78)
-		)
-		(stroke
-			(width 0)
-			(type default)
-		)
-	)
-	(wire
-		(pts
-			(xy 87.63 97.79) (xy 87.63 144.7546)
+			(xy 87.63 97.79) (xy 87.63 143.51)
 		)
 		(stroke
@@
 	(wire
 		(pts
-			(xy 147.32 144.78) (xy 147.32 144.7546)
-		)
-		(stroke
-			(width 0)
-			(type default)
-		)
-	)
-	(wire
-		(pts
 			(xy 125.73 74.93) (xy 114.3 74.93)
 		)
@@
 	(wire
 		(pts
+			(xy 147.32 143.51) (xy 147.32 129.54)
+		)
+		(stroke
+			(width 0)
+			(type default)
+		)
+	)
+	(wire
+		(pts
 			(xy 218.44 130.81) (xy 229.87 130.81)
 		)
@@
 	(wire
 		(pts
-			(xy 190.5 144.78) (xy 160.02 144.78)
+			(xy 190.5 143.51) (xy 160.02 143.51)
 		)
 		(stroke
@@
 	(wire
 		(pts
-			(xy 87.63 144.7546) (xy 147.32 144.7546)
-		)
-		(stroke
-			(width 0)
-			(type default)
-		)
-	)
-	(wire
-		(pts
-			(xy 147.32 144.7546) (xy 147.32 129.54)
+			(xy 87.63 143.51) (xy 147.32 143.51)
+		)
+		(stroke
+			(width 0)
+			(type default)
+		)
+	)
+	(wire
+		(pts
+			(xy 147.32 143.51) (xy 147.32 153.67)
 		)
 		(stroke
@@
 	(wire
 		(pts
-			(xy 190.5 77.47) (xy 190.5 144.78)
+			(xy 190.5 77.47) (xy 190.5 143.51)
 		)
 		(stroke
@@
 	(wire
 		(pts
-			(xy 160.02 105.41) (xy 160.02 144.78)
+			(xy 160.02 105.41) (xy 160.02 143.51)
 		)
 		(stroke
@@
 			(table_cell "MODE Pin Configuration "
 				(exclude_from_sim no)
-				(at 160.274 129.286 0)
+				(at 161.798 146.558 0)
 				(size 6.858 4.572)
 				(margins 0.9525 0.9525 0.9525 0.9525)
@@
 			(table_cell "Power Limiting, Over Current fault and Thermal Shutdown Operation"
 				(exclude_from_sim no)
-				(at 167.132 129.286 0)
+				(at 168.656 146.558 0)
 				(size 22.606 4.572)
 				(margins 0.9525 0.9525 0.9525 0.9525)
@@
 			(table_cell "Open"
 				(exclude_from_sim no)
-				(at 160.274 133.858 0)
+				(at 161.798 151.13 0)
 				(size 6.858 6.096)
 				(margins 0.9525 0.9525 0.9525 0.9525)
@@
 			(table_cell "Active Current limiting for a maximum duration of tCL_PLIM(dly). There after Latches OFF.\n\nLatch reset by toggling SHDN or UVLO low to high or power cycle"
 				(exclude_from_sim no)
-				(at 167.132 133.858 0)
+				(at 168.656 151.13 0)
 				(size 22.606 6.096)
 				(margins 0.9525 0.9525 0.9525 0.9525)
@@
 			(table_cell "Shorted to GND "
 				(exclude_from_sim no)
-				(at 160.274 139.954 0)
+				(at 161.798 157.226 0)
 				(size 6.858 3.81)
 				(margins 0.9525 0.9525 0.9525 0.9525)
@@
 			(table_cell "delay of t(TSD_retry).\nActive current limiting for a maximum duration of tCL_PLIM(dly). There after auto-retries after a"
 				(exclude_from_sim no)
-				(at 167.132 139.954 0)
+				(at 168.656 157.226 0)
 				(size 22.606 3.81)
 				(margins 0.9525 0.9525 0.9525 0.9525)

Commit message: fixes
Parts:
- U62: footprint Package_DFN_QFN:QFN-24-1EP_4x4mm_P0.5mm_EP2.8x2.8mm -> Package_DFN_QFN:Texas_RGE0024H_VQFN-24-1EP_4x4mm_P0.5mm_EP2.7x2.7mm
Changed lines of the file:
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@@
 			)
 		)
-		(property "Footprint" "Package_DFN_QFN:QFN-24-1EP_4x4mm_P0.5mm_EP2.8x2.8mm"
+		(property "Footprint" "Package_DFN_QFN:Texas_RGE0024H_VQFN-24-1EP_4x4mm_P0.5mm_EP2.7x2.7mm"
 			(at 175.26 93.98 0)
 			(effects

Commit message: fixing inconsistencies in value convention
Parts:
- C16: value 1uF -> 1u
- C74: value 100nF -> 100n
- C75: value 22nF -> 22n
- R1902: value 3.92kΩ -> 3.92k
- R1903: value 1.58kΩ -> 1.58k
- R1904: value 442kΩ -> 442k
- R1905: value 11kΩ -> 11k
- R1906: value 20kΩ -> 20k
- R1908: value 19.1kΩ -> 19.1k
- U62: footprint Package_DFN_QFN:Texas_RGE0024H_VQFN-24-1EP_4x4mm_P0.5mm_EP2.7x2.7mm -> JLCImport:TPS16630RGER
Changed lines of the file:
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@@
 			)
 		)
-		(property "Value" "20kΩ"
+		(property "Value" "20k"
 			(at 116.84 83.8199 0)
 			(effects
@@
 			)
 		)
-		(property "Value" "11kΩ"
+		(property "Value" "11k"
 			(at 116.84 69.8499 0)
 			(effects
@@
 			)
 		)
-		(property "Value" "100nF"
+		(property "Value" "100n"
 			(at 76.708 70.612 90)
 			(effects
@@
 			)
 		)
-		(property "Value" "1.58kΩ"
+		(property "Value" "1.58k"
 			(at 76.2 149.8599 0)
 			(effects
@@
 			)
 		)
-		(property "Value" "22nF"
+		(property "Value" "22n"
 			(at 138.43 127 90)
 			(effects
@@
 			)
 		)
-		(property "Value" "3.92kΩ"
+		(property "Value" "3.92k"
 			(at 72.39 132.0799 0)
 			(effects
@@
 			)
 		)
-		(property "Value" "442kΩ"
+		(property "Value" "442k"
 			(at 116.84 55.8799 0)
 			(effects
@@
 			)
 		)
-		(property "Value" "1uF"
+		(property "Value" "1u"
 			(at 58.674 69.85 90)
 			(effects
@@
 			)
 		)
-		(property "Value" "19.1kΩ"
+		(property "Value" "19.1k"
 			(at 220.98 142.2399 0)
 			(effects
@@
 			)
 		)
-		(property "Footprint" "Package_DFN_QFN:Texas_RGE0024H_VQFN-24-1EP_4x4mm_P0.5mm_EP2.7x2.7mm"
+		(property "Footprint" "JLCImport:TPS16630RGER"
 			(at 175.26 93.98 0)
 			(effects

Commit message: exported to schematic
Parts:
- C16: LCSC (none) -> C5199872
- C74: LCSC (none) -> C14663
- C75: LCSC (none) -> C21122
- R1901, R1907: LCSC (none) -> C25741
- R1902: LCSC (none) -> C2960797
- R1903: LCSC (none) -> C2974011
- R1904: LCSC (none) -> C49654384
- R1905: LCSC (none) -> C2909313
- R1906: LCSC (none) -> C25765
- R1908: LCSC (none) -> C2998158
- U62: LCSC (none) -> C1850279
Changed lines of the file:
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@@
+			)
+		)
+		(property "LCSC" "C25741"
+			(at 127 111.76 0)
+			(effects
+				(font
+					(size 1.27 1.27)
+				)
+				(hide yes)
 			)
 		)
@@
 			)
 		)
+		(property "LCSC" "C25765"
+			(at 116.84 81.2799 0)
+			(effects
+				(font
+					(size 1.27 1.27)
+				)
+				(hide yes)
+			)
+		)
 		(pin "1"
 		)
@@
 			)
 		)
+		(property "LCSC" "C2909313"
+			(at 116.84 67.3099 0)
+			(effects
+				(font
+					(size 1.27 1.27)
+				)
+				(hide yes)
+			)
+		)
 		(pin "1"
 		)
@@
 			)
 		)
+		(property "LCSC" "C14663"
+			(at 76.708 68.58 0)
+			(effects
+				(font
+					(size 1.27 1.27)
+				)
+				(hide yes)
+			)
+		)
 		(pin "1"
 		)
@@
 			)
 		)
+		(property "LCSC" "C2974011"
+			(at 76.2 147.3199 0)
+			(effects
+				(font
+					(size 1.27 1.27)
+				)
+				(hide yes)
+			)
+		)
 		(pin "1"
 		)
@@
 		(property "LCSC Part Name" "22nF ±20% 50V"
 			(at 147.32 124.46 0)
+			(effects
+				(font
+					(size 1.27 1.27)
+				)
+				(hide yes)
+			)
+		)
+		(property "LCSC" "C21122"
+			(at 138.43 124.46 0)
 			(effects
 				(font
@@
 			)
 		)
+		(property "LCSC" "C2960797"
+			(at 72.39 129.5399 0)
+			(effects
+				(font
+					(size 1.27 1.27)
+				)
+				(hide yes)
+			)
+		)
 		(pin "1"
 		)
@@
 			)
 		)
+		(property "LCSC" "C49654384"
+			(at 116.84 53.3399 0)
+			(effects
+				(font
+					(size 1.27 1.27)
+				)
+				(hide yes)
+			)
+		)
 		(pin "1"
 		)
@@
 			)
 		)
+		(property "LCSC" "C5199872"
+			(at 56.642 67.818 0)
+			(effects
+				(font
+					(size 1.27 1.27)
+				)
+				(hide yes)
+			)
+		)
 		(pin "2"
 		)
@@
 			)
 		)
+		(property "LCSC" "C25741"
+			(at 220.98 121.9199 0)
+			(effects
+				(font
+					(size 1.27 1.27)
+				)
+				(hide yes)
+			)
+		)
 		(pin "1"
 		)
@@
 			)
 		)
+		(property "LCSC" "C2998158"
+			(at 220.98 139.6999 0)
+			(effects
+				(font
+					(size 1.27 1.27)
+				)
+				(hide yes)
+			)
+		)
 		(pin "1"
 		)
@@
 			(effects
 				(font
+					(size 1.27 1.27)
+				)
+				(hide yes)
+			)
+		)
+		(property "LCSC" "C1850279"
+			(at 166.37 74.93 0)
+			(effects
+				(font
