File: hardware/kicad/ioexpandermcu.kicad_sch (KiCad schematic)
At the start: 10 parts, among them J10 PINHD_1x8_Male, J11 PINHD_1x8_Male, J12 PINHD_1x8_Male, U301 EXB2HV102JV, U302 EXB2HV102JV, U303 EXB2HV102JV, U90 PCAL6524HEAZ

Commit message: update
Parts:
- removed J10, J11, J12: PINHD_1x8_Male, Connector_PinHeader_2.54mm:PinHeader_1x08_P2.54mm_Vertical, symbol PCM_SL_Pin_Headers:PINHD_1x8_Male
- added J301, J302, J303, J304, J305, J306, J307, J308, J309, J310, J311, J312, J313, J314, J315, J316, J317, J318, J319, J320, J321, J322, J339, J340: PINHD_1x1_Male, Connector_PinHeader_2.54mm:PinHeader_1x01_P2.54mm_Vertical, symbol PCM_SL_Pin_Headers:PINHD_1x1_Male
Connections:
- net P0_0: now also J301.1
- net P0_1: now also J302.1
- net P0_2: now also J303.1
- net P0_3: now also J304.1
- net P0_4: now also J305.1
- net P0_5: now also J306.1
- net P0_6: now also J307.1
- net P0_7: now also J308.1
- net P1_0: now also J309.1
- net P1_1: now also J310.1
- net P1_2: now also J311.1
- net P1_3: now also J312.1
- net P1_4: now also J313.1
- net P1_5: now also J314.1
- net P1_6: now also J315.1
- net P1_7: now also J316.1
- net P2_0: now also J340.1
- net P2_1: now also J339.1
- net P2_2: now also J322.1
- net P2_3: now also J321.1
- net P2_4: now also J320.1
- net P2_5: now also J319.1
- net P2_6: now also J318.1
- net P2_7: now also J317.1

Commit message: update
Parts:
- removed J301, J302, J303, J304, J305, J306, J307, J308, J309, J310, J311, J312, J313, J314, J315, J316, J317, J318, J319, J320, J321, J322, J339, J340: PINHD_1x1_Male, Connector_PinHeader_2.54mm:PinHeader_1x01_P2.54mm_Vertical, symbol PCM_SL_Pin_Headers:PINHD_1x1_Male

Commit message: updating symbols to use kicad footprints where possible
Parts:
- removed U90: PCAL6524HEAZ, 5v rail sm-easyedapro:HQFN-32_L5.0-W5.0-P0.50-BL-EP3.0, symbol 5v rail sm-easyedapro:PCAL6524HEAZ
- added U304: PCAL6524HEAZ, Package_CSP:LFCSP-32-1EP_5x5mm_P0.5mm_EP3.6x3.6mm, symbol JLCImport:PCAL6524HEAZ
- C142: footprint 5v rail sm-easyedapro:C0603 -> Capacitor_SMD:C_0603_1608Metric
- R268, R269: footprint 5v rail sm-easyedapro:R0402 -> Resistor_SMD:R_0402_1005Metric
- U301, U302, U303: footprint JLCImport:EXB2HV102JV -> Resistor_SMD:R_Array_Convex_8x0602
Connections:
- net +3V3: now also U304.27 (VDD(P)), U304.31 (VDD(I2C-bus))
- net ADDR: now also U304.26 (ADDR)
- net GND: now also U304.25 (VSS), U304.33 (EP)
- net INT#: now also U304.32 (INT#)
- net SCL_SLOW: now also U304.29 (SCL)
- net SDA_SLOW: now also U304.30 (SDA)
- net at U303.1: now also U304.24 (P2_7)
- net at U303.2: now also U304.23 (P2_6)
- net at U303.3: now also U304.22 (P2_5)
- net at U303.4: now also U304.21 (P2_4)
- net at U303.5: now also U304.20 (P2_3)
- net at U303.6: now also U304.19 (P2_2)
- net at U303.7: now also U304.18 (P2_1)
- net at U303.8: now also U304.17 (P2_0)
- net at R269.1: now also U304.28 (RESET#)
- net at U301.16: now also U304.1 (P0_0)
- net at U302.15: now also U304.10 (P1_1)
- net at U302.14: now also U304.11 (P1_2)
- net at U302.13: now also U304.12 (P1_3)
- net at U302.12: now also U304.13 (P1_4)
- net at U302.11: now also U304.14 (P1_5)
- net at U302.10: now also U304.15 (P1_6)
- net at U302.9: now also U304.16 (P1_7)
- net at U301.15: now also U304.2 (P0_1)
- net at U301.14: now also U304.3 (P0_2)
- net at U301.13: now also U304.4 (P0_3)
- net at U301.12: now also U304.5 (P0_4)
- net at U301.11: now also U304.6 (P0_5)
- net at U301.10: now also U304.7 (P0_6)
- net at U301.9: now also U304.8 (P0_7)
- net at U302.16: now also U304.9 (P1_0)
Changed lines of the file:
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@@
 			)
 		)
-		(property "Footprint" "JLCImport:EXB2HV102JV"
+		(property "Footprint" "Resistor_SMD:R_Array_Convex_8x0602"
 			(at 176.53 106.68 0)
 			(effects
@@
 			)
 		)
-		(property "Footprint" "5v rail sm-easyedapro:C0603"
+		(property "Footprint" "Capacitor_SMD:C_0603_1608Metric"
 			(at 207.01 73.66 0)
 			(effects
@@
 			)
 		)
-		(property "Footprint" "5v rail sm-easyedapro:R0402"
+		(property "Footprint" "Resistor_SMD:R_0402_1005Metric"
 			(at 189.23 68.58 0)
 			(effects
@@
 	)
 	(symbol
-		(lib_id "5v rail sm-easyedapro:PCAL6524HEAZ")
+		(lib_id "JLCImport:PCAL6524HEAZ")
 		(at 121.92 99.06 0)
 		(unit 1)
@@
 		(dnp no)
 		(fields_autoplaced yes)
-		(property "Reference" "U90"
-			(at 106.68 71.12 0)
-			(effects
-				(font
-					(size 1.27 1.27)
-				)
-				(justify left bottom)
+		(property "Reference" "U304"
+			(at 121.92 68.58 0)
+			(effects
+				(font
+					(size 1.27 1.27)
+				)
 			)
 		)
 		(property "Value" "PCAL6524HEAZ"
-			(at 106.68 121.92 0)
-			(effects
-				(font
-					(size 1.27 1.27)
-				)
-				(justify left bottom)
-			)
-		)
-		(property "Footprint" "5v rail sm-easyedapro:HQFN-32_L5.0-W5.0-P0.50-BL-EP3.0"
+			(at 121.92 71.12 0)
+			(effects
+				(font
+					(size 1.27 1.27)
+				)
+			)
+		)
+		(property "Footprint" "Package_CSP:LFCSP-32-1EP_5x5mm_P0.5mm_EP3.6x3.6mm"
 			(at 121.92 99.06 0)
 			(effects
@@
 			)
 		)
-		(property "Datasheet" "https://www.nxp.com/docs/en/data-sheet/PCAL6524DS.pdf"
+		(property "Datasheet" "https://cn.bing.com/search?q=datasheet： PCAL6524HEHP"
 			(at 121.92 99.06 0)
 			(effects
@@
 			)
 		)
-		(property "Description" "Interface:I2C；SMBus Number of I/O:24 Interrupt Output:Interrupt Output Output Type:Open Drain；Push-Pull Voltage - Supply:1.65V~5.5V；800mV~3.6V Voltage - Supply:1.65V~5.5V；800mV~3.6V Current - Output Low(IOL):25mA Clock Frequency:1MHz Operating Temperature"
+		(property "Description" "-40℃~+85℃ 1MHz 24 25mA 2uA 4 800mV~3.6V、1.65V~5.5V I2C、SMBus Interrupt Output Push-Pull、Open Drain Reset function、Cascading and address extension、Input anti-jitter、Built-in LED driver、IO level configurable HUQFN-32-EP(5x5) I/O Expanders ROHS"
+			(at 121.92 99.06 0)
+			(effects
+				(font
+					(size 1.27 1.27)
+				)
+				(hide yes)
+			)
+		)
+		(property "LCSC" "C3000497"
+			(at 121.92 99.06 0)
+			(effects
+				(font
+					(size 1.27 1.27)
+				)
+				(hide yes)
+			)
+		)
+		(property "Manufacturer" "NXP Semicon"
 			(at 121.92 99.06 0)
 			(effects
@@
 			)
 		)
-		(property "Manufacturer" "NXP(恩智浦)"
-			(at 121.92 99.06 0)
-			(effects
-				(font
-					(size 1.27 1.27)
-				)
-				(hide yes)
-			)
-		)
-		(property "Supplier Part" "C3000497"
-			(at 121.92 99.06 0)
-			(effects
-				(font
-					(size 1.27 1.27)
-				)
-				(hide yes)
-			)
-		)
-		(property "Supplier" "LCSC"
-			(at 121.92 99.06 0)
-			(effects
-				(font
-					(size 1.27 1.27)
-				)
-				(hide yes)
-			)
-		)
-		(property "LCSC Part Name" "具备灵活I/O特性、中断输出和复位功能的超低压转换24位Fm+ I²C总线/SMBus I/O扩展器"
-			(at 121.92 99.06 0)
-			(effects
-				(font
-					(size 1.27 1.27)
-				)
-				(hide yes)
-			)
+		(pin "7"
+		)
+		(pin "8"
+		)
+		(pin "4"
 		)
 		(pin "1"
@@
 		(pin "2"
 		)
+		(pin "5"
+		)
 		(pin "3"
 		)
-		(pin "4"
-		)
-		(pin "5"
-		)
 		(pin "6"
 		)
-		(pin "7"
-		)
-		(pin "8"
+		(pin "24"
+		)
+		(pin "23"
+		)
+		(pin "27"
+		)
+		(pin "13"
+		)
+		(pin "12"
+		)
+		(pin "14"
+		)
+		(pin "11"
+		)
+		(pin "29"
+		)
+		(pin "28"
+		)
+		(pin "25"
+		)
+		(pin "26"
+		)
+		(pin "15"
+		)
+		(pin "31"
+		)
+		(pin "32"
+		)
+		(pin "33"
+		)
+		(pin "16"
+		)
+		(pin "30"
+		)
+		(pin "10"
 		)
 		(pin "9"
 		)
-		(pin "10"
-		)
-		(pin "11"
-		)
-		(pin "12"
-		)
-		(pin "13"
-		)
-		(pin "14"
-		)
-		(pin "15"
-		)
-		(pin "16"
-		)
-		(pin "33"
-		)
-		(pin "32"
-		)
-		(pin "31"
-		)
-		(pin "30"
-		)
-		(pin "29"
-		)
-		(pin "28"
-		)
-		(pin "27"
-		)
-		(pin "26"
-		)
-		(pin "25"
-		)
-		(pin "24"
-		)
-		(pin "23"
-		)
 		(pin "22"
 		)
@@
 		)
 		(instances
-			(project "svea_powerboard_rev3"
+			(project ""
 				(path "/3f85abf4-0b95-4c4a-b7e9-06f59ca1ea3d/5c2e021f-c2d4-49e2-8c36-9a64f1f12001/40a61560-66df-4637-829b-67b6e4c25aea"
-					(reference "U85")
+					(reference "U3404")
 					(unit 1)
 				)
 				(path "/3f85abf4-0b95-4c4a-b7e9-06f59ca1ea3d/5c2e021f-c2d4-49e2-8c36-9a64f1f12001/bfb98524-ff97-426a-83b1-5a3236cd5c1c"
-					(reference "U90")
+					(reference "U304")
 					(unit 1)
 				)
@@
 			)
 		)
-		(property "Footprint" "5v rail sm-easyedapro:R0402"
+		(property "Footprint" "Resistor_SMD:R_0402_1005Metric"
 			(at 162.56 68.58 0)
 			(effects
@@
 			)
 		)
-		(property "Footprint" "JLCImport:EXB2HV102JV"
+		(property "Footprint" "Resistor_SMD:R_Array_Convex_8x0602"
 			(at 92.71 86.36 0)
 			(effects
@@
 			)
 		)
-		(property "Footprint" "JLCImport:EXB2HV102JV"
+		(property "Footprint" "Resistor_SMD:R_Array_Convex_8x0602"
 			(at 77.47 106.68 0)
 			(effects

Commit message: fixing inconsistencies in value convention
Parts:
- C142: value 100nF -> 100n
- R268, R269: value 10kΩ -> 10k
Changed lines of the file:
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@@
 			)
 		)
-		(property "Value" "100nF"
+		(property "Value" "100n"
 			(at 210.82 76.2 90)
 			(effects
@@
 			)
 		)
-		(property "Value" "10kΩ"
+		(property "Value" "10k"
 			(at 191.77 71.12 90)
 			(effects
@@
 			)
 		)
-		(property "Value" "10kΩ"
+		(property "Value" "10k"
 			(at 165.1 71.12 90)
 			(effects

Commit message: exported to schematic
Parts:
- C142: LCSC (none) -> C14663
- R268, R269: LCSC (none) -> C25744
Changed lines of the file:
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@@
+			)
+		)
+		(property "LCSC" "C14663"
+			(at 210.82 73.66 0)
+			(effects
+				(font
+					(size 1.27 1.27)
+				)
+				(hide yes)
 			)
 		)
@@
 		(property "LCSC Part Name" "10kΩ ±1% 62.5mW 厚膜电阻"
 			(at 189.23 68.58 0)
+			(effects
+				(font
+					(size 1.27 1.27)
+				)
+				(hide yes)
+			)
+		)
+		(property "LCSC" "C25744"
+			(at 191.77 68.58 0)
 			(effects
 				(font
@@
 			(effects
 				(font
+					(size 1.27 1.27)
+				)
+				(hide yes)
+			)
+		)
+		(property "LCSC" "C25744"
+			(at 165.1 68.58 0)
+			(effects
+				(font
