File: hardware/kicad/sheets/power/26_Power-3v3.kicad_sch (KiCad schematic)
At the start: 0 parts

Commit message: reorganized
Other:
- title: Power-3v3 -> 3V3 Rail
Changed lines of the file:
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@@
 	(paper "User" 37.1856 25.4)
 	(title_block
-		(title "Power-3v3")
+		(title "3V3 Rail")
 		(date "2026-02-16")
 	)
