File: hardware/kicad/sheets/power/16_Power-12v.kicad_sch (KiCad schematic)
At the start: 30 parts, among them CN11 5017, Q67 CSD17577Q5A, U115 LTM8055IY#PBF, U166 68uF, U168 MCP4725A0T-E/CH, U180 LM5050MKX-1/NOPB

Commit message: reorganized
Other:
- title: Power-12v -> 12V Rail
Changed lines of the file:
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@@
 	(paper "User" 437.51 244.47)
 	(title_block
-		(title "Power-12v")
+		(title "12V Rail")
 		(date "2026-02-16")
 	)

Commit message: before final cleanup
Parts:
- removed JP1: Jumper_2_Bridged, symbol Jumper:Jumper_2_Bridged
- removed JP2: Jumper_2_Open, symbol Jumper:Jumper_2_Open
- added R225, R226: 0, Resistor_SMD:R_0603_1608Metric, symbol Device:R
- renumbered C252 to C71, C289 to C72, C245 to C73, C290 to C74, C246 to C75, C249 to C76, C250 to C77, C247 to C78, C253 to C79, C273 to C80, C271 to C81, C272 to C82, CN11 to CN5, H2 to H4, Q67 to Q13, R467 to R125, R468 to R126, R460 to R127, R458 to R128, R459 to R129, R469 to R130, R512 to R131, R511 to R132, U168 to U42, U170 to U43, U115 to U44, U166 to U45, U180 to U46
Connections:
- net GND: now also R225.2; no longer U44.H2 (SYNC)
- net VCC: now also R226.1; no longer U44.L9 (IIN)
- new net: R226.2, U44.L9 (IIN)
- new net LTM8055-SYNC: R225.1, U44.H2 (SYNC)

Commit message: pre kicad footprints
Parts:
- H4: footprint 5v rail sm-easyedapro:HDR-TH_2P-P2.54-V-M -> Connector_PinHeader_2.54mm:PinHeader_2x01_P2.54mm_Vertical
Changed lines of the file:
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@@
 			)
 		)
-		(property "Footprint" "5v rail sm-easyedapro:HDR-TH_2P-P2.54-V-M"
+		(property "Footprint" "Connector_PinHeader_2.54mm:PinHeader_2x01_P2.54mm_Vertical"
 			(at 119.38 76.2 0)
 			(effects

Commit message: better sheet nesting for power rails
Connections:
- net +12V renamed 12V-BUCK-DIODED
- net VCC renamed 12V_BUCK_INPUT
Changed lines of the file:
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@@
 	)
 	(junction
+		(at 236.22 49.53)
+		(diameter 0)
+		(color 0 0 0 0)
+	)
+	(junction
 		(at 214.63 128.27)
 		(diameter 0)
@@
 	)
 	(junction
-		(at 38.1 33.02)
-		(diameter 0)
-		(color 0 0 0 0)
-	)
-	(junction
 		(at 210.82 67.31)
 		(diameter 0)
@@
 	(wire
 		(pts
-			(xy 236.22 46.99) (xy 236.22 52.07)
+			(xy 236.22 46.99) (xy 236.22 49.53)
 		)
 		(stroke
@@
 	(wire
 		(pts
+			(xy 233.68 49.53) (xy 236.22 49.53)
+		)
+		(stroke
+			(width 0)
+			(type default)
+		)
+	)
+	(wire
+		(pts
 			(xy 254 72.39) (xy 254 66.04)
 		)
@@
 	(wire
 		(pts
-			(xy 55.88 121.92) (xy 49.53 121.92)
+			(xy 82.55 127) (xy 76.2 127)
 		)
 		(stroke
@@
 	(wire
 		(pts
-			(xy 38.1 33.02) (xy 33.02 33.02)
+			(xy 55.88 121.92) (xy 49.53 121.92)
 		)
 		(stroke
@@
 	(wire
 		(pts
-			(xy 33.02 33.02) (xy 33.02 54.61)
-		)
-		(stroke
-			(width 0)
-			(type default)
-		)
-	)
-	(wire
-		(pts
 			(xy 210.82 97.79) (xy 210.82 100.33)
 		)
@@
 	(wire
 		(pts
+			(xy 82.55 129.54) (xy 82.55 127)
+		)
+		(stroke
+			(width 0)
+			(type default)
+		)
+	)
+	(wire
+		(pts
 			(xy 214.63 168.91) (xy 214.63 166.37)
 		)
@@
 	(wire
 		(pts
-			(xy 45.72 33.02) (xy 38.1 33.02)
+			(xy 33.02 33.02) (xy 45.72 33.02)
 		)
 		(stroke
@@
 	(wire
 		(pts
-			(xy 20.32 33.02) (xy 20.32 53.34)
+			(xy 143.51 66.04) (xy 143.51 68.58)
 		)
 		(stroke
@@
 	(wire
 		(pts
-			(xy 143.51 66.04) (xy 143.51 68.58)
+			(xy 134.62 60.96) (xy 160.02 60.96)
 		)
 		(stroke
@@
 	(wire
 		(pts
-			(xy 134.62 60.96) (xy 160.02 60.96)
+			(xy 381 33.02) (xy 381 30.48)
 		)
 		(stroke
@@
 	(wire
 		(pts
-			(xy 381 33.02) (xy 381 30.48)
+			(xy 143.51 154.94) (xy 143.51 157.48)
 		)
 		(stroke
@@
 	(wire
 		(pts
-			(xy 143.51 154.94) (xy 143.51 157.48)
+			(xy 143.51 48.26) (xy 143.51 58.42)
 		)
 		(stroke
@@
 	(wire
 		(pts
-			(xy 143.51 48.26) (xy 143.51 58.42)
+			(xy 128.27 53.34) (xy 160.02 53.34)
 		)
 		(stroke
@@
 	(wire
 		(pts
-			(xy 128.27 53.34) (xy 160.02 53.34)
+			(xy 33.02 33.02) (xy 20.32 33.02)
 		)
 		(stroke
@@
 	(wire
 		(pts
-			(xy 76.2 127) (xy 83.82 127)
+			(xy 82.55 129.54) (xy 85.09 129.54)
 		)
 		(stroke
@@
 	(wire
 		(pts
-			(xy 38.1 26.67) (xy 38.1 33.02)
+			(xy 214.63 138.43) (xy 198.12 138.43)
 		)
 		(stroke
@@
 	(wire
 		(pts
-			(xy 214.63 138.43) (xy 198.12 138.43)
+			(xy 214.63 143.51) (xy 214.63 140.97)
 		)
 		(stroke
@@
 	(wire
 		(pts
-			(xy 214.63 143.51) (xy 214.63 140.97)
+			(xy 214.63 85.09) (xy 214.63 102.87)
 		)
 		(stroke
@@
 	(wire
 		(pts
-			(xy 214.63 85.09) (xy 214.63 102.87)
+			(xy 198.12 57.15) (xy 214.63 57.15)
 		)
 		(stroke
@@
 	(wire
 		(pts
-			(xy 198.12 57.15) (xy 214.63 57.15)
+			(xy 210.82 95.25) (xy 198.12 95.25)
 		)
 		(stroke
@@
 	(wire
 		(pts
-			(xy 210.82 95.25) (xy 198.12 95.25)
+			(xy 33.02 82.55) (xy 20.32 82.55)
 		)
 		(stroke
@@
 	(wire
 		(pts
-			(xy 33.02 82.55) (xy 20.32 82.55)
+			(xy 337.82 36.83) (xy 337.82 33.02)
 		)
 		(stroke
@@
 	(wire
 		(pts
-			(xy 337.82 36.83) (xy 337.82 33.02)
+			(xy 33.02 30.48) (xy 33.02 33.02)
 		)
 		(stroke
@@
 	(wire
 		(pts
-			(xy 76.2 124.46) (xy 83.82 124.46)
+			(xy 76.2 124.46) (xy 85.09 124.46)
 		)
 		(stroke
@@
 	(wire
 		(pts
+			(xy 20.32 33.02) (xy 20.32 53.34)
+		)
+		(stroke
+			(width 0)
+			(type default)
+		)
+	)
+	(wire
+		(pts
 			(xy 134.62 35.56) (xy 134.62 60.96)
 		)
@@
 	(wire
 		(pts
-			(xy 143.51 149.86) (xy 143.51 152.4)
+			(xy 236.22 49.53) (xy 236.22 52.07)
 		)
 		(stroke
@@
 	(wire
 		(pts
-			(xy 156.21 172.72) (xy 156.21 175.26)
+			(xy 143.51 149.86) (xy 143.51 152.4)
 		)
 		(stroke
@@
 	(wire
 		(pts
-			(xy 309.88 33.02) (xy 309.88 45.72)
+			(xy 156.21 172.72) (xy 156.21 175.26)
 		)
 		(stroke
@@
 	(wire
 		(pts
-			(xy 33.02 33.02) (xy 20.32 33.02)
+			(xy 309.88 33.02) (xy 309.88 45.72)
 		)
 		(stroke
@@
 	(wire
 		(pts
+			(xy 33.02 33.02) (xy 33.02 54.61)
+		)
+		(stroke
+			(width 0)
+			(type default)
+		)
+	)
+	(wire
+		(pts
 			(xy 24.13 140.97) (xy 24.13 144.78)
 		)
@@
 	(global_label "SDA_SLOW"
 		(shape input)
-		(at 83.82 127 0)
+		(at 85.09 129.54 0)
 		(effects
 			(font
@@
 		)
 		(property "Intersheetrefs" "${INTERSHEET_REFS}"
-			(at 83.82 127 0)
+			(at 85.09 129.54 0)
 			(effects
 				(font
@@
 	(global_label "SCL_SLOW"
 		(shape input)
-		(at 83.82 124.46 0)
+		(at 85.09 124.46 0)
 		(effects
 			(font
@@
 		)
 		(property "Intersheetrefs" "${INTERSHEET_REFS}"
-			(at 83.82 124.46 0)
+			(at 85.09 124.46 0)
 			(effects
 				(font
@@
 	(global_label "12V-FB"
 		(shape output)
-		(at 236.22 49.53 180)
+		(at 233.68 49.53 180)
 		(effects
 			(font
@@
 		)
 		(property "Intersheetrefs" "${INTERSHEET_REFS}"
-			(at 236.22 49.53 0)
+			(at 233.68 49.53 0)
 			(effects
 				(font
@@
 		)
 	)
+	(hierarchical_label "12V_BUCK_INPUT"
+		(shape input)
+		(at 33.02 30.48 90)
+		(effects
+			(font
+				(size 1.27 1.27)
+			)
+			(justify left)
+		)
+	)
+	(hierarchical_label "12V-BUCK-DIODED"
+		(shape output)
+		(at 414.02 27.94 90)
+		(effects
+			(font
+				(size 1.27 1.27)
+			)
+			(justify left)
+		)
+	)
 	(symbol
 		(lib_id "5v rail sm-easyedapro:FRC0603F3652TS")
@@
 	)
 	(symbol
-		(lib_id "power:VCC")
-		(at 38.1 26.67 0)
-		(unit 1)
-		(exclude_from_sim no)
-		(in_bom yes)
-		(on_board yes)
-		(dnp no)
-		(property "Reference" "#PWR0206"
-			(at 38.1 26.67 0)
-			(effects
-				(font
-					(size 1.27 1.27)
-				)
-				(hide yes)
-			)
-		)
-		(property "Value" "VCC"
-			(at 38.1 22.86 0)
-			(effects
-				(font
-					(size 1.5748 1.5748)
-				)
-			)
-		)
-		(property "Footprint" ""
-			(at 38.1 26.67 0)
-			(effects
-				(font
-					(size 1.27 1.27)
-				)
-				(hide yes)
-			)
-		)
-		(property "Datasheet" ""
-			(at 38.1 26.67 0)
-			(effects
-				(font
-					(size 1.27 1.27)
-				)
-				(hide yes)
-			)
-		)
-		(property "Description" ""
-			(at 38.1 26.67 0)
-			(effects
-				(font
-					(size 1.27 1.27)
-				)
-				(hide yes)
-			)
-		)
-		(pin "1"
-		)
-		(instances
-			(project "svea_powerboard_rev3"
-				(path "/3f85abf4-0b95-4c4a-b7e9-06f59ca1ea3d/5c2e021f-c2d4-49e2-8c36-9a64f1f12002/8d05c3b8-20a4-4a7f-9b20-01f8d5d5be22"
-					(reference "#PWR0206")
-					(unit 1)
-				)
-			)
-		)
-	)
-	(symbol
 		(lib_id "5v rail sm-easyedapro:0603WAF1000T5E")
 		(at 414.02 39.37 90)
@@
 					(unit 1)
 				)
-			)
-		)
-	)
-	(symbol
-		(lib_id "power:+12V")
-		(at 414.02 27.94 0)
-		(unit 1)
-		(exclude_from_sim no)
-		(in_bom yes)
-		(on_board yes)
-		(dnp no)
-		(property "Reference" "#PWR0216"
-			(at 414.02 27.94 0)
-			(effects
-				(font
-					(size 1.27 1.27)
-				)
-				(hide yes)
-			)
-		)
-		(property "Value" "+12V"
-			(at 414.02 24.13 0)
-			(effects
-				(font
-					(size 1.27 1.27)
-				)
-			)
-		)
-		(property "Footprint" ""
-			(at 414.02 27.94 0)
-			(effects
-				(font
-					(size 1.27 1.27)
-				)
-				(hide yes)
-			)
-		)
-		(property "Datasheet" ""
-			(at 414.02 27.94 0)
-			(effects
-				(font
-					(size 1.27 1.27)
-				)
-				(hide yes)
-			)
-		)
-		(property "Description" "Power-5V"
-			(at 414.02 27.94 0)
-			(effects
-				(font
-					(size 1.27 1.27)
-				)
-				(hide yes)
-			)
-		)
-		(pin "1"
-		)
-		(instances
-			(project "svea_powerboard_rev3"
-				(path "/3f85abf4-0b95-4c4a-b7e9-06f59ca1ea3d/5c2e021f-c2d4-49e2-8c36-9a64f1f12002/8d05c3b8-20a4-4a7f-9b20-01f8d5d5be22"
-					(reference "#PWR0216")
-					(unit 1)
-				)
