File: hardware/kicad/sheets/power/5_Power-5v.kicad_sch (KiCad schematic)
At the start: 20 parts, among them Q32 DMN4800LSSL-13, U103 220uF, U47 LM74700QDBVRQ1, U49 8mΩ

Commit message: reorganized
Other:
- title: Power-5v -> 5V Rail
Changed lines of the file:
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@@
 	(paper "User" 297 210)
 	(title_block
-		(title "Power-5v")
+		(title "5V Rail")
 		(date "2026-02-16")
 	)

Commit message: before final cleanup
Parts:
- renumbered C141 to C55, C76 to C56, C74 to C57, C140 to C58, C138 to C59, C137 to C60, C71 to C61, C139 to C62, C142 to C63, L6 to L2, Q32 to Q12, R310 to R113, R278 to R114, R175 to R115, R176 to R116, U103 to U35, U47 to U36, U49 to U37, 5 to U38

Commit message: better sheet nesting for power rails
Parts:
- removed 5Vbuck-6A1: TPS566231RQFR, 5v rail sm-easyedapro:VQFN-HR-9_2.0-W1.5-P0.5-TL_TI_RQF0009A, symbol 5v rail sm-easyedapro:TPS566231RQFR
- removed C55, C58, C62, C63: 100nF, Capacitor_SMD:C_0402_1005Metric, symbol 5v rail sm-easyedapro:CL05B104KB54PNC
- removed C56: 47uF, Capacitor_SMD:C_1206_3216Metric, symbol 5v rail sm-easyedapro:HGC1206R5476M250NSPJ
- removed C57: 1uF, Capacitor_SMD:C_0603_1608Metric, symbol 5v rail sm-easyedapro:EMK107B7105KA-T
- removed C59: 10nF, Capacitor_SMD:C_0201_0603Metric, symbol 5v rail sm-easyedapro:TCC0201X7R103K500ZT
- removed C60: 33pF, Capacitor_SMD:C_0201_0603Metric, symbol 5v rail sm-easyedapro:GRM0335C1H330JA01D
- removed C61: 22uF, Capacitor_SMD:C_0805_2012Metric, symbol 5v rail sm-easyedapro:LMK212BJ226MG-T
- removed L2: 1.5uH, 5v rail sm-easyedapro:IND-SMD_L7.1-W6.5-P5.60, symbol 5v rail sm-easyedapro:SPM6530T-1R5M100
- removed Q12: DMN4800LSSL-13, Package_SO:SOIC-8_3.9x4.9mm_P1.27mm, symbol 5v rail sm-easyedapro:DMN4800LSSL-13
- removed R113: 47kΩ, Resistor_SMD:R_0201_0603Metric, symbol 5v rail sm-easyedapro:0201WMF4702TEE
- removed R114: 0Ω, Resistor_SMD:R_0402_1005Metric, symbol 5v rail sm-easyedapro:FRC0402P000 TS
- removed R115: 220kΩ, Resistor_SMD:R_0201_0603Metric, symbol 5v rail sm-easyedapro:0201WMF2203TEE
- removed R116: 30kΩ, Resistor_SMD:R_0201_0603Metric, symbol 5v rail sm-easyedapro:RC0201FR-0730KL
- removed U35: 220uF, 5v rail sm-easyedapro:CAP-SMD_BD6.3-L6.6-W6.6-LS7.0-FD, symbol 5v rail sm-easyedapro:HV1E227M0607PZ
- removed U36: LM74700QDBVRQ1, Package_TO_SOT_SMD:SOT-23-6, symbol 5v rail sm-easyedapro:LM74700QDBVRQ1
- removed U37: 8mΩ, Resistor_SMD:R_1206_3216Metric, symbol 5v rail sm-easyedapro:FRM121WFR008TM
- removed U38: ~, symbol 5v rail sm-easyedapro:Short-Symbol
