File: hardware/kicad/sheets/power/5vrail.kicad_sch (KiCad schematic)
At the start: 13 parts, among them Q12 L2N7002SLLT1G, U53 TPSM33625RDNR

Commit message: pre robot updating references
Parts:
- renumbered C96 to C94, C97 to C95, C98 to C96, C99 to C97, C100 to C98, C101 to C99, R118 to R125, R119 to R126, R120 to R127, R121 to R128, R122 to R129
Changed lines of the file:
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@@
 		(on_board yes)
 		(dnp no)
-		(property "Reference" "C101"
+		(property "Reference" "C99"
 			(at 215.9 68.58 90)
 			(effects
@@
 			(project "svea_powerboard_rev3"
 				(path "/3f85abf4-0b95-4c4a-b7e9-06f59ca1ea3d/5c2e021f-c2d4-49e2-8c36-9a64f1f12001/de8125f2-04ec-46c6-89d6-d0b5e89f6023"
-					(reference "C101")
+					(reference "C99")
 					(unit 1)
 				)
@@
 		(on_board yes)
 		(dnp no)
-		(property "Reference" "R118"
+		(property "Reference" "R125"
 			(at 114.3 119.38 90)
 			(effects
@@
 			(project "svea_powerboard_rev3"
 				(path "/3f85abf4-0b95-4c4a-b7e9-06f59ca1ea3d/5c2e021f-c2d4-49e2-8c36-9a64f1f12001/de8125f2-04ec-46c6-89d6-d0b5e89f6023"
-					(reference "R118")
+					(reference "R125")
 					(unit 1)
 				)
@@
 		(on_board yes)
 		(dnp no)
-		(property "Reference" "#PWR0165"
+		(property "Reference" "#PWR0152"
 			(at 212.09 78.74 0)
 			(effects
@@
 			(project "svea_powerboard_rev3"
 				(path "/3f85abf4-0b95-4c4a-b7e9-06f59ca1ea3d/5c2e021f-c2d4-49e2-8c36-9a64f1f12001/de8125f2-04ec-46c6-89d6-d0b5e89f6023"
-					(reference "#PWR0165")
+					(reference "#PWR0152")
 					(unit 1)
 				)
@@
 		(on_board yes)
 		(dnp no)
-		(property "Reference" "C96"
+		(property "Reference" "C94"
 			(at 53.34 93.98 90)
 			(effects
@@
 			(project "svea_powerboard_rev3"
 				(path "/3f85abf4-0b95-4c4a-b7e9-06f59ca1ea3d/5c2e021f-c2d4-49e2-8c36-9a64f1f12001/de8125f2-04ec-46c6-89d6-d0b5e89f6023"
-					(reference "C96")
+					(reference "C94")
 					(unit 1)
 				)
@@
 		(on_board yes)
 		(dnp no)
-		(property "Reference" "R121"
+		(property "Reference" "R128"
 			(at 182.88 71.12 90)
 			(effects
@@
 			(project "svea_powerboard_rev3"
 				(path "/3f85abf4-0b95-4c4a-b7e9-06f59ca1ea3d/5c2e021f-c2d4-49e2-8c36-9a64f1f12001/de8125f2-04ec-46c6-89d6-d0b5e89f6023"
-					(reference "R121")
+					(reference "R128")
 					(unit 1)
 				)
@@
 		(on_board yes)
 		(dnp no)
-		(property "Reference" "C99"
+		(property "Reference" "C97"
 			(at 161.29 99.06 90)
 			(effects
@@
 			(project "svea_powerboard_rev3"
 				(path "/3f85abf4-0b95-4c4a-b7e9-06f59ca1ea3d/5c2e021f-c2d4-49e2-8c36-9a64f1f12001/de8125f2-04ec-46c6-89d6-d0b5e89f6023"
-					(reference "C99")
+					(reference "C97")
 					(unit 1)
 				)
@@
 		(on_board yes)
 		(dnp no)
-		(property "Reference" "#PWR0164"
+		(property "Reference" "#PWR0151"
 			(at 180.34 119.38 0)
 			(effects
@@
 			(project "svea_powerboard_rev3"
 				(path "/3f85abf4-0b95-4c4a-b7e9-06f59ca1ea3d/5c2e021f-c2d4-49e2-8c36-9a64f1f12001/de8125f2-04ec-46c6-89d6-d0b5e89f6023"
-					(reference "#PWR0164")
+					(reference "#PWR0151")
 					(unit 1)
 				)
@@
 		(on_board yes)
 		(dnp no)
-		(property "Reference" "#PWR0163"
+		(property "Reference" "#PWR0150"
 			(at 121.92 129.54 0)
 			(effects
@@
 			(project "svea_powerboard_rev3"
 				(path "/3f85abf4-0b95-4c4a-b7e9-06f59ca1ea3d/5c2e021f-c2d4-49e2-8c36-9a64f1f12001/de8125f2-04ec-46c6-89d6-d0b5e89f6023"
-					(reference "#PWR0163")
+					(reference "#PWR0150")
 					(unit 1)
 				)
@@
 		(on_board yes)
 		(dnp no)
-		(property "Reference" "R120"
+		(property "Reference" "R127"
 			(at 160.02 73.66 0)
 			(effects
@@
 			(project "svea_powerboard_rev3"
 				(path "/3f85abf4-0b95-4c4a-b7e9-06f59ca1ea3d/5c2e021f-c2d4-49e2-8c36-9a64f1f12001/de8125f2-04ec-46c6-89d6-d0b5e89f6023"
-					(reference "R120")
+					(reference "R127")
 					(unit 1)
 				)
@@
 		(on_board yes)
 		(dnp no)
-		(property "Reference" "R119"
+		(property "Reference" "R126"
 			(at 111.76 78.74 0)
 			(effects
@@
 			(project "svea_powerboard_rev3"
 				(path "/3f85abf4-0b95-4c4a-b7e9-06f59ca1ea3d/5c2e021f-c2d4-49e2-8c36-9a64f1f12001/de8125f2-04ec-46c6-89d6-d0b5e89f6023"
-					(reference "R119")
+					(reference "R126")
 					(unit 1)
 				)
@@
 		(on_board yes)
 		(dnp no)
-		(property "Reference" "C100"
+		(property "Reference" "C98"
 			(at 201.93 68.58 90)
 			(effects
@@
 			(project "svea_powerboard_rev3"
 				(path "/3f85abf4-0b95-4c4a-b7e9-06f59ca1ea3d/5c2e021f-c2d4-49e2-8c36-9a64f1f12001/de8125f2-04ec-46c6-89d6-d0b5e89f6023"
-					(reference "C100")
+					(reference "C98")
 					(unit 1)
 				)
@@
 		(on_board yes)
 		(dnp no)
-		(property "Reference" "C97"
+		(property "Reference" "C95"
 			(at 68.58 95.25 90)
 			(effects
@@
 			(project "svea_powerboard_rev3"
 				(path "/3f85abf4-0b95-4c4a-b7e9-06f59ca1ea3d/5c2e021f-c2d4-49e2-8c36-9a64f1f12001/de8125f2-04ec-46c6-89d6-d0b5e89f6023"
-					(reference "C97")
+					(reference "C95")
 					(unit 1)
 				)
@@
 		(on_board yes)
 		(dnp no)
-		(property "Reference" "#PWR0162"
+		(property "Reference" "#PWR0149"
 			(at 64.77 110.49 0)
 			(effects
@@
 			(project "svea_powerboard_rev3"
 				(path "/3f85abf4-0b95-4c4a-b7e9-06f59ca1ea3d/5c2e021f-c2d4-49e2-8c36-9a64f1f12001/de8125f2-04ec-46c6-89d6-d0b5e89f6023"
-					(reference "#PWR0162")
+					(reference "#PWR0149")
 					(unit 1)
 				)
@@
 		(on_board yes)
 		(dnp no)
-		(property "Reference" "R122"
+		(property "Reference" "R129"
 			(at 182.88 95.25 90)
 			(effects
@@
 			(project "svea_powerboard_rev3"
 				(path "/3f85abf4-0b95-4c4a-b7e9-06f59ca1ea3d/5c2e021f-c2d4-49e2-8c36-9a64f1f12001/de8125f2-04ec-46c6-89d6-d0b5e89f6023"
-					(reference "R122")
+					(reference "R129")
 					(unit 1)
 				)
@@
 		(on_board yes)
 		(dnp no)
-		(property "Reference" "C98"
+		(property "Reference" "C96"
 			(at 82.55 93.98 90)
 			(effects
@@
 			(project "svea_powerboard_rev3"
 				(path "/3f85abf4-0b95-4c4a-b7e9-06f59ca1ea3d/5c2e021f-c2d4-49e2-8c36-9a64f1f12001/de8125f2-04ec-46c6-89d6-d0b5e89f6023"
-					(reference "C98")
+					(reference "C96")
 					(unit 1)
 				)

Commit message: various imprvements
Parts:
- renumbered C95 to C100, C96 to C101, C97 to C102, C98 to C103, C99 to C104, C94 to C99, R125 to R155, R126 to R156, R127 to R157, R128 to R158, R129 to R159, U53 to U59
Connections:
- net MCU-5V-BUCK-PGOOD renamed Power/5V-Buck/PGOOD
Changed lines of the file:
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@@
 		)
 	)
-	(global_label "MCU-5V-BUCK-PGOOD"
+	(global_label "Power/5V-Buck/PGOOD"
 		(shape output)
 		(at 119.38 72.39 180)
@@
 		(on_board yes)
 		(dnp no)
-		(property "Reference" "C99"
+		(property "Reference" "C104"
 			(at 215.9 68.58 90)
 			(effects
@@
 			(project "svea_powerboard_rev3"
 				(path "/3f85abf4-0b95-4c4a-b7e9-06f59ca1ea3d/5c2e021f-c2d4-49e2-8c36-9a64f1f12001/de8125f2-04ec-46c6-89d6-d0b5e89f6023"
-					(reference "C99")
+					(reference "C104")
 					(unit 1)
 				)
@@
 		(on_board yes)
 		(dnp no)
-		(property "Reference" "U53"
+		(property "Reference" "U59"
 			(at 129.54 74.93 0)
 			(effects
@@
 			(project "svea_powerboard_rev3"
 				(path "/3f85abf4-0b95-4c4a-b7e9-06f59ca1ea3d/5c2e021f-c2d4-49e2-8c36-9a64f1f12001/de8125f2-04ec-46c6-89d6-d0b5e89f6023"
-					(reference "U53")
+					(reference "U59")
 					(unit 1)
 				)
@@
 		(on_board yes)
 		(dnp no)
-		(property "Reference" "R125"
+		(property "Reference" "R155"
 			(at 114.3 119.38 90)
 			(effects
@@
 			(project "svea_powerboard_rev3"
 				(path "/3f85abf4-0b95-4c4a-b7e9-06f59ca1ea3d/5c2e021f-c2d4-49e2-8c36-9a64f1f12001/de8125f2-04ec-46c6-89d6-d0b5e89f6023"
-					(reference "R125")
+					(reference "R155")
 					(unit 1)
 				)
@@
 		(on_board yes)
 		(dnp no)
-		(property "Reference" "#PWR0152"
+		(property "Reference" "#PWR0165"
 			(at 212.09 78.74 0)
 			(effects
@@
 			(project "svea_powerboard_rev3"
 				(path "/3f85abf4-0b95-4c4a-b7e9-06f59ca1ea3d/5c2e021f-c2d4-49e2-8c36-9a64f1f12001/de8125f2-04ec-46c6-89d6-d0b5e89f6023"
-					(reference "#PWR0152")
+					(reference "#PWR0165")
 					(unit 1)
 				)
@@
 		(on_board yes)
 		(dnp no)
-		(property "Reference" "C94"
+		(property "Reference" "C99"
 			(at 53.34 93.98 90)
 			(effects
@@
 			(project "svea_powerboard_rev3"
 				(path "/3f85abf4-0b95-4c4a-b7e9-06f59ca1ea3d/5c2e021f-c2d4-49e2-8c36-9a64f1f12001/de8125f2-04ec-46c6-89d6-d0b5e89f6023"
-					(reference "C94")
+					(reference "C99")
 					(unit 1)
 				)
@@
 		(on_board yes)
 		(dnp no)
-		(property "Reference" "R128"
+		(property "Reference" "R158"
 			(at 182.88 71.12 90)
 			(effects
@@
 			(project "svea_powerboard_rev3"
 				(path "/3f85abf4-0b95-4c4a-b7e9-06f59ca1ea3d/5c2e021f-c2d4-49e2-8c36-9a64f1f12001/de8125f2-04ec-46c6-89d6-d0b5e89f6023"
-					(reference "R128")
+					(reference "R158")
 					(unit 1)
 				)
@@
 		(on_board yes)
 		(dnp no)
-		(property "Reference" "C97"
+		(property "Reference" "C102"
 			(at 161.29 99.06 90)
 			(effects
@@
 			(project "svea_powerboard_rev3"
 				(path "/3f85abf4-0b95-4c4a-b7e9-06f59ca1ea3d/5c2e021f-c2d4-49e2-8c36-9a64f1f12001/de8125f2-04ec-46c6-89d6-d0b5e89f6023"
-					(reference "C97")
+					(reference "C102")
 					(unit 1)
 				)
@@
 		(on_board yes)
 		(dnp no)
-		(property "Reference" "#PWR0151"
+		(property "Reference" "#PWR0164"
 			(at 180.34 119.38 0)
 			(effects
@@
 			(project "svea_powerboard_rev3"
 				(path "/3f85abf4-0b95-4c4a-b7e9-06f59ca1ea3d/5c2e021f-c2d4-49e2-8c36-9a64f1f12001/de8125f2-04ec-46c6-89d6-d0b5e89f6023"
-					(reference "#PWR0151")
+					(reference "#PWR0164")
 					(unit 1)
 				)
@@
 		(on_board yes)
 		(dnp no)
-		(property "Reference" "#PWR0150"
+		(property "Reference" "#PWR0163"
 			(at 121.92 129.54 0)
 			(effects
@@
 			(project "svea_powerboard_rev3"
 				(path "/3f85abf4-0b95-4c4a-b7e9-06f59ca1ea3d/5c2e021f-c2d4-49e2-8c36-9a64f1f12001/de8125f2-04ec-46c6-89d6-d0b5e89f6023"
-					(reference "#PWR0150")
+					(reference "#PWR0163")
 					(unit 1)
 				)
@@
 		(on_board yes)
 		(dnp no)
-		(property "Reference" "R127"
+		(property "Reference" "R157"
 			(at 160.02 73.66 0)
 			(effects
@@
 			(project "svea_powerboard_rev3"
 				(path "/3f85abf4-0b95-4c4a-b7e9-06f59ca1ea3d/5c2e021f-c2d4-49e2-8c36-9a64f1f12001/de8125f2-04ec-46c6-89d6-d0b5e89f6023"
-					(reference "R127")
+					(reference "R157")
 					(unit 1)
 				)
@@
 		(on_board yes)
 		(dnp no)
-		(property "Reference" "R126"
+		(property "Reference" "R156"
 			(at 111.76 78.74 0)
 			(effects
@@
 			(project "svea_powerboard_rev3"
 				(path "/3f85abf4-0b95-4c4a-b7e9-06f59ca1ea3d/5c2e021f-c2d4-49e2-8c36-9a64f1f12001/de8125f2-04ec-46c6-89d6-d0b5e89f6023"
-					(reference "R126")
+					(reference "R156")
 					(unit 1)
 				)
@@
 		(on_board yes)
 		(dnp no)
-		(property "Reference" "C98"
+		(property "Reference" "C103"
 			(at 201.93 68.58 90)
 			(effects
@@
 			(project "svea_powerboard_rev3"
 				(path "/3f85abf4-0b95-4c4a-b7e9-06f59ca1ea3d/5c2e021f-c2d4-49e2-8c36-9a64f1f12001/de8125f2-04ec-46c6-89d6-d0b5e89f6023"
-					(reference "C98")
+					(reference "C103")
 					(unit 1)
 				)
@@
 		(on_board yes)
 		(dnp no)
-		(property "Reference" "C95"
+		(property "Reference" "C100"
 			(at 68.58 95.25 90)
 			(effects
@@
 			(project "svea_powerboard_rev3"
 				(path "/3f85abf4-0b95-4c4a-b7e9-06f59ca1ea3d/5c2e021f-c2d4-49e2-8c36-9a64f1f12001/de8125f2-04ec-46c6-89d6-d0b5e89f6023"
-					(reference "C95")
+					(reference "C100")
 					(unit 1)
 				)
@@
 		(on_board yes)
 		(dnp no)
-		(property "Reference" "#PWR0149"
+		(property "Reference" "#PWR0162"
 			(at 64.77 110.49 0)
 			(effects
@@
 			(project "svea_powerboard_rev3"
 				(path "/3f85abf4-0b95-4c4a-b7e9-06f59ca1ea3d/5c2e021f-c2d4-49e2-8c36-9a64f1f12001/de8125f2-04ec-46c6-89d6-d0b5e89f6023"
-					(reference "#PWR0149")
+					(reference "#PWR0162")
 					(unit 1)
 				)
@@
 		(on_board yes)
 		(dnp no)
-		(property "Reference" "R129"
+		(property "Reference" "R159"
 			(at 182.88 95.25 90)
 			(effects
@@
 			(project "svea_powerboard_rev3"
 				(path "/3f85abf4-0b95-4c4a-b7e9-06f59ca1ea3d/5c2e021f-c2d4-49e2-8c36-9a64f1f12001/de8125f2-04ec-46c6-89d6-d0b5e89f6023"
-					(reference "R129")
+					(reference "R159")
 					(unit 1)
 				)
@@
 		(on_board yes)
 		(dnp no)
-		(property "Reference" "C96"
+		(property "Reference" "C101"
 			(at 82.55 93.98 90)
 			(effects
@@
 			(project "svea_powerboard_rev3"
 				(path "/3f85abf4-0b95-4c4a-b7e9-06f59ca1ea3d/5c2e021f-c2d4-49e2-8c36-9a64f1f12001/de8125f2-04ec-46c6-89d6-d0b5e89f6023"
-					(reference "C96")
+					(reference "C101")
 					(unit 1)
 				)
