File: hardware/kicad/sheets/power/Power-3v3.kicad_sch (KiCad schematic)
At the start: 12 parts, among them Q7 L2N7002SLLT1G, U7 TPSM33625RDNR

Commit message: resheeted bms and fixed links for the 12v buck
Parts:
- renumbered C19 to C59, C20 to C60, C24 to C61, C26 to C62, C27 to C63, Q7 to Q11, R36 to R69, R37 to R70, R39 to R71, R40 to R72, R41 to R73, U7 to U23
Connections:
- net MCU-3V3-EN renamed #EN
Changed lines of the file:
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@@
-		)
-	)
-	(global_label "MCU-3V3-EN"
-		(shape input)
-		(at 121.92 105.41 180)
-		(effects
-			(font
-				(size 1.5748 1.5748)
-			)
-			(justify right)
-		)
-		(property "Intersheetrefs" "${INTERSHEET_REFS}"
-			(at 121.92 105.41 0)
-			(effects
-				(font
-					(size 1.27 1.27)
-				)
-				(hide yes)
-			)
 		)
 	)
@@
 				(hide yes)
 			)
+		)
+	)
+	(hierarchical_label "#EN"
+		(shape input)
+		(at 121.92 105.41 180)
+		(effects
+			(font
+				(size 1.27 1.27)
+			)
+			(justify right)
 		)
 	)
@@
 		(on_board yes)
 		(dnp no)
-		(property "Reference" "#PWR0134"
+		(property "Reference" "#PWR076"
 			(at 71.12 106.68 0)
 			(effects
@@
 			(project "svea_powerboard_rev3"
 				(path "/3f85abf4-0b95-4c4a-b7e9-06f59ca1ea3d/5c2e021f-c2d4-49e2-8c36-9a64f1f12002/51095da8-7aff-4069-a0df-937720a4d2a2"
-					(reference "#PWR0134")
+					(reference "#PWR076")
 					(unit 1)
 				)
@@
 		(on_board yes)
 		(dnp no)
-		(property "Reference" "R39"
+		(property "Reference" "R71"
 			(at 172.72 69.85 0)
 			(effects
@@
 			(project "svea_powerboard_rev3"
 				(path "/3f85abf4-0b95-4c4a-b7e9-06f59ca1ea3d/5c2e021f-c2d4-49e2-8c36-9a64f1f12002/51095da8-7aff-4069-a0df-937720a4d2a2"
-					(reference "R39")
+					(reference "R71")
 					(unit 1)
 				)
@@
 		(on_board yes)
 		(dnp no)
-		(property "Reference" "R40"
+		(property "Reference" "R72"
 			(at 195.58 67.31 90)
 			(effects
@@
 			(project "svea_powerboard_rev3"
 				(path "/3f85abf4-0b95-4c4a-b7e9-06f59ca1ea3d/5c2e021f-c2d4-49e2-8c36-9a64f1f12002/51095da8-7aff-4069-a0df-937720a4d2a2"
-					(reference "R40")
+					(reference "R72")
 					(unit 1)
 				)
@@
 		(on_board yes)
 		(dnp no)
-		(property "Reference" "R37"
+		(property "Reference" "R70"
 			(at 123.19 74.93 0)
 			(effects
@@
 			(project "svea_powerboard_rev3"
 				(path "/3f85abf4-0b95-4c4a-b7e9-06f59ca1ea3d/5c2e021f-c2d4-49e2-8c36-9a64f1f12002/51095da8-7aff-4069-a0df-937720a4d2a2"
-					(reference "R37")
+					(reference "R70")
 					(unit 1)
 				)
@@
 		(on_board yes)
 		(dnp no)
-		(property "Reference" "R41"
+		(property "Reference" "R73"
 			(at 195.58 91.44 90)
 			(effects
@@
 			(project "svea_powerboard_rev3"
 				(path "/3f85abf4-0b95-4c4a-b7e9-06f59ca1ea3d/5c2e021f-c2d4-49e2-8c36-9a64f1f12002/51095da8-7aff-4069-a0df-937720a4d2a2"
-					(reference "R41")
+					(reference "R73")
 					(unit 1)
 				)
@@
 		(on_board yes)
 		(dnp no)
-		(property "Reference" "C24"
+		(property "Reference" "C61"
 			(at 173.99 95.25 90)
 			(effects
@@
 			(project "svea_powerboard_rev3"
 				(path "/3f85abf4-0b95-4c4a-b7e9-06f59ca1ea3d/5c2e021f-c2d4-49e2-8c36-9a64f1f12002/51095da8-7aff-4069-a0df-937720a4d2a2"
-					(reference "C24")
+					(reference "C61")
 					(unit 1)
 				)
@@
 		(on_board yes)
 		(dnp no)
-		(property "Reference" "Q7"
+		(property "Reference" "Q11"
 			(at 138.43 105.41 0)
 			(effects
@@
 			(project "svea_powerboard_rev3"
 				(path "/3f85abf4-0b95-4c4a-b7e9-06f59ca1ea3d/5c2e021f-c2d4-49e2-8c36-9a64f1f12002/51095da8-7aff-4069-a0df-937720a4d2a2"
-					(reference "Q7")
+					(reference "Q11")
 					(unit 1)
 				)
@@
 		(on_board yes)
 		(dnp no)
-		(property "Reference" "R36"
+		(property "Reference" "R69"
 			(at 125.73 115.57 90)
 			(effects
@@
 			(project "svea_powerboard_rev3"
 				(path "/3f85abf4-0b95-4c4a-b7e9-06f59ca1ea3d/5c2e021f-c2d4-49e2-8c36-9a64f1f12002/51095da8-7aff-4069-a0df-937720a4d2a2"
-					(reference "R36")
+					(reference "R69")
 					(unit 1)
 				)
@@
 		(on_board yes)
 		(dnp no)
-		(property "Reference" "#PWR0135"
+		(property "Reference" "#PWR078"
 			(at 133.35 125.73 0)
 			(effects
@@
 			(project "svea_powerboard_rev3"
 				(path "/3f85abf4-0b95-4c4a-b7e9-06f59ca1ea3d/5c2e021f-c2d4-49e2-8c36-9a64f1f12002/51095da8-7aff-4069-a0df-937720a4d2a2"
-					(reference "#PWR0135")
+					(reference "#PWR078")
 					(unit 1)
 				)
@@
 		(on_board yes)
 		(dnp no)
-		(property "Reference" "C20"
+		(property "Reference" "C60"
 			(at 82.55 91.44 90)
 			(effects
@@
 			(project "svea_powerboard_rev3"
 				(path "/3f85abf4-0b95-4c4a-b7e9-06f59ca1ea3d/5c2e021f-c2d4-49e2-8c36-9a64f1f12002/51095da8-7aff-4069-a0df-937720a4d2a2"
-					(reference "C20")
+					(reference "C60")
 					(unit 1)
 				)
@@
 		(on_board yes)
 		(dnp no)
-		(property "Reference" "#PWR0125"
+		(property "Reference" "#PWR079"
 			(at 193.04 119.38 0)
 			(effects
@@
 			(project "svea_powerboard_rev3"
 				(path "/3f85abf4-0b95-4c4a-b7e9-06f59ca1ea3d/5c2e021f-c2d4-49e2-8c36-9a64f1f12002/51095da8-7aff-4069-a0df-937720a4d2a2"
-					(reference "#PWR0125")
+					(reference "#PWR079")
 					(unit 1)
 				)
@@
 		(on_board yes)
 		(dnp no)
-		(property "Reference" "C27"
+		(property "Reference" "C63"
 			(at 228.6 63.5 0)
 			(effects
@@
 			(project "svea_powerboard_rev3"
 				(path "/3f85abf4-0b95-4c4a-b7e9-06f59ca1ea3d/5c2e021f-c2d4-49e2-8c36-9a64f1f12002/51095da8-7aff-4069-a0df-937720a4d2a2"
-					(reference "C27")
+					(reference "C63")
 					(unit 1)
 				)
@@
 		(on_board yes)
 		(dnp no)
-		(property "Reference" "C26"
+		(property "Reference" "C62"
 			(at 214.63 63.5 0)
 			(effects
@@
 			(project "svea_powerboard_rev3"
 				(path "/3f85abf4-0b95-4c4a-b7e9-06f59ca1ea3d/5c2e021f-c2d4-49e2-8c36-9a64f1f12002/51095da8-7aff-4069-a0df-937720a4d2a2"
-					(reference "C26")
+					(reference "C62")
 					(unit 1)
 				)
@@
 		(on_board yes)
 		(dnp no)
-		(property "Reference" "U7"
+		(property "Reference" "U23"
 			(at 142.24 71.12 0)
 			(effects
@@
 			(project "svea_powerboard_rev3"
 				(path "/3f85abf4-0b95-4c4a-b7e9-06f59ca1ea3d/5c2e021f-c2d4-49e2-8c36-9a64f1f12002/51095da8-7aff-4069-a0df-937720a4d2a2"
-					(reference "U7")
+					(reference "U23")
 					(unit 1)
 				)
@@
 		(on_board yes)
 		(dnp no)
-		(property "Reference" "#PWR0132"
+		(property "Reference" "#PWR080"
 			(at 224.79 74.93 0)
 			(effects
@@
 			(project "svea_powerboard_rev3"
 				(path "/3f85abf4-0b95-4c4a-b7e9-06f59ca1ea3d/5c2e021f-c2d4-49e2-8c36-9a64f1f12002/51095da8-7aff-4069-a0df-937720a4d2a2"
-					(reference "#PWR0132")
+					(reference "#PWR080")
 					(unit 1)
 				)
@@
 		(on_board yes)
 		(dnp no)
-		(property "Reference" "C19"
+		(property "Reference" "C59"
 			(at 67.31 90.17 90)
 			(effects
@@
 			(project "svea_powerboard_rev3"
 				(path "/3f85abf4-0b95-4c4a-b7e9-06f59ca1ea3d/5c2e021f-c2d4-49e2-8c36-9a64f1f12002/51095da8-7aff-4069-a0df-937720a4d2a2"
-					(reference "C19")
+					(reference "C59")
 					(unit 1)
 				)

Commit message: realized having 2 3v3 rails can cause issues
Parts:
- renumbered C59 to C53, C60 to C54, C61 to C55, C62 to C56, C63 to C57, Q11 to Q1, R69 to R1, R70 to R2, R71 to R3, R72 to R64, R73 to R65, U23 to U21
Changed lines of the file:
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@@
 		(on_board yes)
 		(dnp no)
-		(property "Reference" "#PWR076"
+		(property "Reference" "#PWR04"
 			(at 71.12 106.68 0)
 			(effects
@@
 		(instances
 			(project "svea_powerboard_rev3"
-				(path "/3f85abf4-0b95-4c4a-b7e9-06f59ca1ea3d/5c2e021f-c2d4-49e2-8c36-9a64f1f12002/51095da8-7aff-4069-a0df-937720a4d2a2"
-					(reference "#PWR076")
+				(path "/3f85abf4-0b95-4c4a-b7e9-06f59ca1ea3d/5c2e021f-c2d4-49e2-8c36-9a64f1f12001/ca6525fc-674d-4dae-a2f9-d25bb2ff7c72"
+					(reference "#PWR04")
 					(unit 1)
 				)
@@
 		(on_board yes)
 		(dnp no)
-		(property "Reference" "R71"
+		(property "Reference" "R3"
 			(at 172.72 69.85 0)
 			(effects
@@
 		(instances
 			(project "svea_powerboard_rev3"
-				(path "/3f85abf4-0b95-4c4a-b7e9-06f59ca1ea3d/5c2e021f-c2d4-49e2-8c36-9a64f1f12002/51095da8-7aff-4069-a0df-937720a4d2a2"
-					(reference "R71")
+				(path "/3f85abf4-0b95-4c4a-b7e9-06f59ca1ea3d/5c2e021f-c2d4-49e2-8c36-9a64f1f12001/ca6525fc-674d-4dae-a2f9-d25bb2ff7c72"
+					(reference "R3")
 					(unit 1)
 				)
@@
 		(on_board yes)
 		(dnp no)
-		(property "Reference" "R72"
+		(property "Reference" "R64"
 			(at 195.58 67.31 90)
 			(effects
@@
 		(instances
 			(project "svea_powerboard_rev3"
-				(path "/3f85abf4-0b95-4c4a-b7e9-06f59ca1ea3d/5c2e021f-c2d4-49e2-8c36-9a64f1f12002/51095da8-7aff-4069-a0df-937720a4d2a2"
-					(reference "R72")
+				(path "/3f85abf4-0b95-4c4a-b7e9-06f59ca1ea3d/5c2e021f-c2d4-49e2-8c36-9a64f1f12001/ca6525fc-674d-4dae-a2f9-d25bb2ff7c72"
+					(reference "R64")
 					(unit 1)
 				)
@@
 		(on_board yes)
 		(dnp no)
-		(property "Reference" "R70"
+		(property "Reference" "R2"
 			(at 123.19 74.93 0)
 			(effects
@@
 		(instances
 			(project "svea_powerboard_rev3"
-				(path "/3f85abf4-0b95-4c4a-b7e9-06f59ca1ea3d/5c2e021f-c2d4-49e2-8c36-9a64f1f12002/51095da8-7aff-4069-a0df-937720a4d2a2"
-					(reference "R70")
+				(path "/3f85abf4-0b95-4c4a-b7e9-06f59ca1ea3d/5c2e021f-c2d4-49e2-8c36-9a64f1f12001/ca6525fc-674d-4dae-a2f9-d25bb2ff7c72"
+					(reference "R2")
 					(unit 1)
 				)
@@
 		(on_board yes)
 		(dnp no)
-		(property "Reference" "R73"
+		(property "Reference" "R65"
 			(at 195.58 91.44 90)
 			(effects
@@
 		(instances
 			(project "svea_powerboard_rev3"
-				(path "/3f85abf4-0b95-4c4a-b7e9-06f59ca1ea3d/5c2e021f-c2d4-49e2-8c36-9a64f1f12002/51095da8-7aff-4069-a0df-937720a4d2a2"
-					(reference "R73")
+				(path "/3f85abf4-0b95-4c4a-b7e9-06f59ca1ea3d/5c2e021f-c2d4-49e2-8c36-9a64f1f12001/ca6525fc-674d-4dae-a2f9-d25bb2ff7c72"
+					(reference "R65")
 					(unit 1)
 				)
@@
 		(on_board yes)
 		(dnp no)
-		(property "Reference" "C61"
+		(property "Reference" "C55"
 			(at 173.99 95.25 90)
 			(effects
@@
 		(instances
 			(project "svea_powerboard_rev3"
-				(path "/3f85abf4-0b95-4c4a-b7e9-06f59ca1ea3d/5c2e021f-c2d4-49e2-8c36-9a64f1f12002/51095da8-7aff-4069-a0df-937720a4d2a2"
-					(reference "C61")
+				(path "/3f85abf4-0b95-4c4a-b7e9-06f59ca1ea3d/5c2e021f-c2d4-49e2-8c36-9a64f1f12001/ca6525fc-674d-4dae-a2f9-d25bb2ff7c72"
+					(reference "C55")
 					(unit 1)
 				)
@@
 		(on_board yes)
 		(dnp no)
-		(property "Reference" "Q11"
+		(property "Reference" "Q1"
 			(at 138.43 105.41 0)
 			(effects
@@
 		(instances
 			(project "svea_powerboard_rev3"
-				(path "/3f85abf4-0b95-4c4a-b7e9-06f59ca1ea3d/5c2e021f-c2d4-49e2-8c36-9a64f1f12002/51095da8-7aff-4069-a0df-937720a4d2a2"
-					(reference "Q11")
+				(path "/3f85abf4-0b95-4c4a-b7e9-06f59ca1ea3d/5c2e021f-c2d4-49e2-8c36-9a64f1f12001/ca6525fc-674d-4dae-a2f9-d25bb2ff7c72"
+					(reference "Q1")
 					(unit 1)
 				)
@@
 		(on_board yes)
 		(dnp no)
-		(property "Reference" "R69"
+		(property "Reference" "R1"
 			(at 125.73 115.57 90)
 			(effects
@@
 		(instances
 			(project "svea_powerboard_rev3"
-				(path "/3f85abf4-0b95-4c4a-b7e9-06f59ca1ea3d/5c2e021f-c2d4-49e2-8c36-9a64f1f12002/51095da8-7aff-4069-a0df-937720a4d2a2"
-					(reference "R69")
+				(path "/3f85abf4-0b95-4c4a-b7e9-06f59ca1ea3d/5c2e021f-c2d4-49e2-8c36-9a64f1f12001/ca6525fc-674d-4dae-a2f9-d25bb2ff7c72"
+					(reference "R1")
 					(unit 1)
 				)
@@
 		(on_board yes)
 		(dnp no)
-		(property "Reference" "#PWR078"
+		(property "Reference" "#PWR06"
 			(at 133.35 125.73 0)
 			(effects
@@
 		(instances
 			(project "svea_powerboard_rev3"
-				(path "/3f85abf4-0b95-4c4a-b7e9-06f59ca1ea3d/5c2e021f-c2d4-49e2-8c36-9a64f1f12002/51095da8-7aff-4069-a0df-937720a4d2a2"
-					(reference "#PWR078")
+				(path "/3f85abf4-0b95-4c4a-b7e9-06f59ca1ea3d/5c2e021f-c2d4-49e2-8c36-9a64f1f12001/ca6525fc-674d-4dae-a2f9-d25bb2ff7c72"
+					(reference "#PWR06")
 					(unit 1)
 				)
@@
 		(on_board yes)
 		(dnp no)
-		(property "Reference" "C60"
+		(property "Reference" "C54"
 			(at 82.55 91.44 90)
 			(effects
@@
 		(instances
 			(project "svea_powerboard_rev3"
-				(path "/3f85abf4-0b95-4c4a-b7e9-06f59ca1ea3d/5c2e021f-c2d4-49e2-8c36-9a64f1f12002/51095da8-7aff-4069-a0df-937720a4d2a2"
-					(reference "C60")
+				(path "/3f85abf4-0b95-4c4a-b7e9-06f59ca1ea3d/5c2e021f-c2d4-49e2-8c36-9a64f1f12001/ca6525fc-674d-4dae-a2f9-d25bb2ff7c72"
+					(reference "C54")
 					(unit 1)
 				)
@@
 		(on_board yes)
 		(dnp no)
-		(property "Reference" "#PWR079"
+		(property "Reference" "#PWR07"
 			(at 193.04 119.38 0)
 			(effects
@@
 		(instances
 			(project "svea_powerboard_rev3"
-				(path "/3f85abf4-0b95-4c4a-b7e9-06f59ca1ea3d/5c2e021f-c2d4-49e2-8c36-9a64f1f12002/51095da8-7aff-4069-a0df-937720a4d2a2"
-					(reference "#PWR079")
+				(path "/3f85abf4-0b95-4c4a-b7e9-06f59ca1ea3d/5c2e021f-c2d4-49e2-8c36-9a64f1f12001/ca6525fc-674d-4dae-a2f9-d25bb2ff7c72"
+					(reference "#PWR07")
 					(unit 1)
 				)
@@
 		(on_board yes)
 		(dnp no)
-		(property "Reference" "C63"
+		(property "Reference" "C57"
 			(at 228.6 63.5 0)
 			(effects
@@
 		(instances
 			(project "svea_powerboard_rev3"
-				(path "/3f85abf4-0b95-4c4a-b7e9-06f59ca1ea3d/5c2e021f-c2d4-49e2-8c36-9a64f1f12002/51095da8-7aff-4069-a0df-937720a4d2a2"
-					(reference "C63")
+				(path "/3f85abf4-0b95-4c4a-b7e9-06f59ca1ea3d/5c2e021f-c2d4-49e2-8c36-9a64f1f12001/ca6525fc-674d-4dae-a2f9-d25bb2ff7c72"
+					(reference "C57")
 					(unit 1)
 				)
@@
 		(on_board yes)
 		(dnp no)
-		(property "Reference" "C62"
+		(property "Reference" "C56"
 			(at 214.63 63.5 0)
 			(effects
@@
 		(instances
 			(project "svea_powerboard_rev3"
-				(path "/3f85abf4-0b95-4c4a-b7e9-06f59ca1ea3d/5c2e021f-c2d4-49e2-8c36-9a64f1f12002/51095da8-7aff-4069-a0df-937720a4d2a2"
-					(reference "C62")
+				(path "/3f85abf4-0b95-4c4a-b7e9-06f59ca1ea3d/5c2e021f-c2d4-49e2-8c36-9a64f1f12001/ca6525fc-674d-4dae-a2f9-d25bb2ff7c72"
+					(reference "C56")
 					(unit 1)
 				)
@@
 		(on_board yes)
 		(dnp no)
-		(property "Reference" "U23"
+		(property "Reference" "U21"
 			(at 142.24 71.12 0)
 			(effects
@@
 		(instances
 			(project "svea_powerboard_rev3"
-				(path "/3f85abf4-0b95-4c4a-b7e9-06f59ca1ea3d/5c2e021f-c2d4-49e2-8c36-9a64f1f12002/51095da8-7aff-4069-a0df-937720a4d2a2"
-					(reference "U23")
+				(path "/3f85abf4-0b95-4c4a-b7e9-06f59ca1ea3d/5c2e021f-c2d4-49e2-8c36-9a64f1f12001/ca6525fc-674d-4dae-a2f9-d25bb2ff7c72"
+					(reference "U21")
 					(unit 1)
 				)
@@
 		(on_board yes)
 		(dnp no)
-		(property "Reference" "#PWR080"
+		(property "Reference" "#PWR08"
 			(at 224.79 74.93 0)
 			(effects
@@
 		(instances
 			(project "svea_powerboard_rev3"
-				(path "/3f85abf4-0b95-4c4a-b7e9-06f59ca1ea3d/5c2e021f-c2d4-49e2-8c36-9a64f1f12002/51095da8-7aff-4069-a0df-937720a4d2a2"
-					(reference "#PWR080")
+				(path "/3f85abf4-0b95-4c4a-b7e9-06f59ca1ea3d/5c2e021f-c2d4-49e2-8c36-9a64f1f12001/ca6525fc-674d-4dae-a2f9-d25bb2ff7c72"
+					(reference "#PWR08")
 					(unit 1)
 				)
@@
 		(on_board yes)
 		(dnp no)
-		(property "Reference" "C59"
+		(property "Reference" "C53"
 			(at 67.31 90.17 90)
 			(effects
@@
 		(instances
 			(project "svea_powerboard_rev3"
-				(path "/3f85abf4-0b95-4c4a-b7e9-06f59ca1ea3d/5c2e021f-c2d4-49e2-8c36-9a64f1f12002/51095da8-7aff-4069-a0df-937720a4d2a2"
-					(reference "C59")
+				(path "/3f85abf4-0b95-4c4a-b7e9-06f59ca1ea3d/5c2e021f-c2d4-49e2-8c36-9a64f1f12001/ca6525fc-674d-4dae-a2f9-d25bb2ff7c72"
+					(reference "C53")
 					(unit 1)
 				)

Commit message: various improvements
Parts:
- renumbered C53 to C77, C54 to C78, C55 to C79, C56 to C80, C57 to C81, Q1 to Q15, R1 to R85, R2 to R86, R3 to R87, R64 to R88, R65 to R89, U21 to U43
Changed lines of the file:
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@@
 		(on_board yes)
 		(dnp no)
-		(property "Reference" "#PWR04"
+		(property "Reference" "#PWR0132"
 			(at 71.12 106.68 0)
 			(effects
@@
 			(project "svea_powerboard_rev3"
 				(path "/3f85abf4-0b95-4c4a-b7e9-06f59ca1ea3d/5c2e021f-c2d4-49e2-8c36-9a64f1f12001/ca6525fc-674d-4dae-a2f9-d25bb2ff7c72"
-					(reference "#PWR04")
+					(reference "#PWR0132")
 					(unit 1)
 				)
@@
 		(on_board yes)
 		(dnp no)
-		(property "Reference" "R3"
+		(property "Reference" "R87"
 			(at 172.72 69.85 0)
 			(effects
@@
 			(project "svea_powerboard_rev3"
 				(path "/3f85abf4-0b95-4c4a-b7e9-06f59ca1ea3d/5c2e021f-c2d4-49e2-8c36-9a64f1f12001/ca6525fc-674d-4dae-a2f9-d25bb2ff7c72"
-					(reference "R3")
+					(reference "R87")
 					(unit 1)
 				)
@@
 		(on_board yes)
 		(dnp no)
-		(property "Reference" "R64"
+		(property "Reference" "R88"
 			(at 195.58 67.31 90)
 			(effects
@@
 			(project "svea_powerboard_rev3"
 				(path "/3f85abf4-0b95-4c4a-b7e9-06f59ca1ea3d/5c2e021f-c2d4-49e2-8c36-9a64f1f12001/ca6525fc-674d-4dae-a2f9-d25bb2ff7c72"
-					(reference "R64")
+					(reference "R88")
 					(unit 1)
 				)
@@
 		(on_board yes)
 		(dnp no)
-		(property "Reference" "R2"
+		(property "Reference" "R86"
 			(at 123.19 74.93 0)
 			(effects
@@
 			(project "svea_powerboard_rev3"
 				(path "/3f85abf4-0b95-4c4a-b7e9-06f59ca1ea3d/5c2e021f-c2d4-49e2-8c36-9a64f1f12001/ca6525fc-674d-4dae-a2f9-d25bb2ff7c72"
-					(reference "R2")
+					(reference "R86")
 					(unit 1)
 				)
@@
 		(on_board yes)
 		(dnp no)
-		(property "Reference" "R65"
+		(property "Reference" "R89"
 			(at 195.58 91.44 90)
 			(effects
@@
 			(project "svea_powerboard_rev3"
 				(path "/3f85abf4-0b95-4c4a-b7e9-06f59ca1ea3d/5c2e021f-c2d4-49e2-8c36-9a64f1f12001/ca6525fc-674d-4dae-a2f9-d25bb2ff7c72"
-					(reference "R65")
+					(reference "R89")
 					(unit 1)
 				)
@@
 		(on_board yes)
 		(dnp no)
-		(property "Reference" "C55"
+		(property "Reference" "C79"
 			(at 173.99 95.25 90)
 			(effects
@@
 			(project "svea_powerboard_rev3"
 				(path "/3f85abf4-0b95-4c4a-b7e9-06f59ca1ea3d/5c2e021f-c2d4-49e2-8c36-9a64f1f12001/ca6525fc-674d-4dae-a2f9-d25bb2ff7c72"
-					(reference "C55")
+					(reference "C79")
 					(unit 1)
 				)
@@
 		(on_board yes)
 		(dnp no)
-		(property "Reference" "Q1"
+		(property "Reference" "Q15"
 			(at 138.43 105.41 0)
 			(effects
@@
 			(project "svea_powerboard_rev3"
 				(path "/3f85abf4-0b95-4c4a-b7e9-06f59ca1ea3d/5c2e021f-c2d4-49e2-8c36-9a64f1f12001/ca6525fc-674d-4dae-a2f9-d25bb2ff7c72"
-					(reference "Q1")
+					(reference "Q15")
 					(unit 1)
 				)
@@
 		(on_board yes)
 		(dnp no)
-		(property "Reference" "R1"
+		(property "Reference" "R85"
 			(at 125.73 115.57 90)
 			(effects
@@
 			(project "svea_powerboard_rev3"
 				(path "/3f85abf4-0b95-4c4a-b7e9-06f59ca1ea3d/5c2e021f-c2d4-49e2-8c36-9a64f1f12001/ca6525fc-674d-4dae-a2f9-d25bb2ff7c72"
-					(reference "R1")
+					(reference "R85")
 					(unit 1)
 				)
@@
 		(on_board yes)
 		(dnp no)
-		(property "Reference" "#PWR06"
+		(property "Reference" "#PWR0133"
 			(at 133.35 125.73 0)
 			(effects
@@
 			(project "svea_powerboard_rev3"
 				(path "/3f85abf4-0b95-4c4a-b7e9-06f59ca1ea3d/5c2e021f-c2d4-49e2-8c36-9a64f1f12001/ca6525fc-674d-4dae-a2f9-d25bb2ff7c72"
-					(reference "#PWR06")
+					(reference "#PWR0133")
 					(unit 1)
 				)
@@
 		(on_board yes)
 		(dnp no)
-		(property "Reference" "C54"
+		(property "Reference" "C78"
 			(at 82.55 91.44 90)
 			(effects
@@
 			(project "svea_powerboard_rev3"
 				(path "/3f85abf4-0b95-4c4a-b7e9-06f59ca1ea3d/5c2e021f-c2d4-49e2-8c36-9a64f1f12001/ca6525fc-674d-4dae-a2f9-d25bb2ff7c72"
-					(reference "C54")
+					(reference "C78")
 					(unit 1)
 				)
@@
 		(on_board yes)
 		(dnp no)
-		(property "Reference" "#PWR07"
+		(property "Reference" "#PWR0134"
 			(at 193.04 119.38 0)
 			(effects
@@
 			(project "svea_powerboard_rev3"
 				(path "/3f85abf4-0b95-4c4a-b7e9-06f59ca1ea3d/5c2e021f-c2d4-49e2-8c36-9a64f1f12001/ca6525fc-674d-4dae-a2f9-d25bb2ff7c72"
-					(reference "#PWR07")
+					(reference "#PWR0134")
 					(unit 1)
 				)
@@
 		(on_board yes)
 		(dnp no)
-		(property "Reference" "C57"
+		(property "Reference" "C81"
 			(at 228.6 63.5 0)
 			(effects
@@
 			(project "svea_powerboard_rev3"
 				(path "/3f85abf4-0b95-4c4a-b7e9-06f59ca1ea3d/5c2e021f-c2d4-49e2-8c36-9a64f1f12001/ca6525fc-674d-4dae-a2f9-d25bb2ff7c72"
-					(reference "C57")
+					(reference "C81")
 					(unit 1)
 				)
@@
 		(on_board yes)
 		(dnp no)
-		(property "Reference" "C56"
+		(property "Reference" "C80"
 			(at 214.63 63.5 0)
 			(effects
@@
 			(project "svea_powerboard_rev3"
 				(path "/3f85abf4-0b95-4c4a-b7e9-06f59ca1ea3d/5c2e021f-c2d4-49e2-8c36-9a64f1f12001/ca6525fc-674d-4dae-a2f9-d25bb2ff7c72"
-					(reference "C56")
+					(reference "C80")
 					(unit 1)
 				)
@@
 		(on_board yes)
 		(dnp no)
-		(property "Reference" "U21"
+		(property "Reference" "U43"
 			(at 142.24 71.12 0)
 			(effects
@@
 			(project "svea_powerboard_rev3"
 				(path "/3f85abf4-0b95-4c4a-b7e9-06f59ca1ea3d/5c2e021f-c2d4-49e2-8c36-9a64f1f12001/ca6525fc-674d-4dae-a2f9-d25bb2ff7c72"
-					(reference "U21")
+					(reference "U43")
 					(unit 1)
 				)
@@
 		(on_board yes)
 		(dnp no)
-		(property "Reference" "#PWR08"
+		(property "Reference" "#PWR0135"
 			(at 224.79 74.93 0)
 			(effects
@@
 			(project "svea_powerboard_rev3"
 				(path "/3f85abf4-0b95-4c4a-b7e9-06f59ca1ea3d/5c2e021f-c2d4-49e2-8c36-9a64f1f12001/ca6525fc-674d-4dae-a2f9-d25bb2ff7c72"
-					(reference "#PWR08")
+					(reference "#PWR0135")
 					(unit 1)
 				)
@@
 		(on_board yes)
 		(dnp no)
-		(property "Reference" "C53"
+		(property "Reference" "C77"
 			(at 67.31 90.17 90)
 			(effects
@@
 			(project "svea_powerboard_rev3"
 				(path "/3f85abf4-0b95-4c4a-b7e9-06f59ca1ea3d/5c2e021f-c2d4-49e2-8c36-9a64f1f12001/ca6525fc-674d-4dae-a2f9-d25bb2ff7c72"
-					(reference "C53")
+					(reference "C77")
 					(unit 1)
 				)

Commit message: various improvements
Parts:
- removed Q15: L2N7002SLLT1G, Package_TO_SOT_SMD:SOT-23, symbol 5v rail sm-easyedapro:L2N7002SLLT1G
- removed R85: 100kΩ, Resistor_SMD:R_0603_1608Metric, symbol 5v rail sm-easyedapro:FRC0603J104 TS
- renumbered C77 to C84, C78 to C85, C79 to C86, C80 to C87, C81 to C88, R86 to R94, R87 to R95, R88 to R96, R89 to R97
Connections:
- net GND: now also R94.2
- net VCC: no longer R94.2
- net EN: now reaches R94.1, U43.2 (EN)
Other:
- moved on the sheet: C84, C85, R94
