File: hardware/kicad/sheets/power/Power-3v3.kicad_sch (KiCad schematic)
At the start: 10 parts, among them U43 TPSM33625RDNR

Commit message: current sensing on the servos and cleaning up empty sheets
Parts:
- renumbered C84 to C89, C85 to C90, C86 to C91, C87 to C92, C88 to C93, R94 to R91, R95 to R92, R96 to R93, R97 to R94, U43 to U46
Changed lines of the file:
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@@
 		(on_board yes)
 		(dnp no)
-		(property "Reference" "#PWR0140"
+		(property "Reference" "#PWR0142"
 			(at 71.12 107.95 0)
 			(effects
@@
 			(project "svea_powerboard_rev3"
 				(path "/3f85abf4-0b95-4c4a-b7e9-06f59ca1ea3d/5c2e021f-c2d4-49e2-8c36-9a64f1f12001/ca6525fc-674d-4dae-a2f9-d25bb2ff7c72"
-					(reference "#PWR0140")
+					(reference "#PWR0142")
 					(unit 1)
 				)
@@
 		(on_board yes)
 		(dnp no)
-		(property "Reference" "R95"
+		(property "Reference" "R92"
 			(at 172.72 69.85 0)
 			(effects
@@
 			(project "svea_powerboard_rev3"
 				(path "/3f85abf4-0b95-4c4a-b7e9-06f59ca1ea3d/5c2e021f-c2d4-49e2-8c36-9a64f1f12001/ca6525fc-674d-4dae-a2f9-d25bb2ff7c72"
-					(reference "R95")
+					(reference "R92")
 					(unit 1)
 				)
@@
 		(on_board yes)
 		(dnp no)
-		(property "Reference" "R96"
+		(property "Reference" "R93"
 			(at 195.58 67.31 90)
 			(effects
@@
 			(project "svea_powerboard_rev3"
 				(path "/3f85abf4-0b95-4c4a-b7e9-06f59ca1ea3d/5c2e021f-c2d4-49e2-8c36-9a64f1f12001/ca6525fc-674d-4dae-a2f9-d25bb2ff7c72"
-					(reference "R96")
+					(reference "R93")
 					(unit 1)
 				)
@@
 		(on_board yes)
 		(dnp no)
-		(property "Reference" "R94"
+		(property "Reference" "R91"
 			(at 129.54 96.52 0)
 			(effects
@@
 			(project "svea_powerboard_rev3"
 				(path "/3f85abf4-0b95-4c4a-b7e9-06f59ca1ea3d/5c2e021f-c2d4-49e2-8c36-9a64f1f12001/ca6525fc-674d-4dae-a2f9-d25bb2ff7c72"
-					(reference "R94")
+					(reference "R91")
 					(unit 1)
 				)
@@
 		(on_board yes)
 		(dnp no)
-		(property "Reference" "R97"
+		(property "Reference" "R94"
 			(at 195.58 91.44 90)
 			(effects
@@
 			(project "svea_powerboard_rev3"
 				(path "/3f85abf4-0b95-4c4a-b7e9-06f59ca1ea3d/5c2e021f-c2d4-49e2-8c36-9a64f1f12001/ca6525fc-674d-4dae-a2f9-d25bb2ff7c72"
-					(reference "R97")
+					(reference "R94")
 					(unit 1)
 				)
@@
 		(on_board yes)
 		(dnp no)
-		(property "Reference" "C86"
+		(property "Reference" "C91"
 			(at 173.99 95.25 90)
 			(effects
@@
 			(project "svea_powerboard_rev3"
 				(path "/3f85abf4-0b95-4c4a-b7e9-06f59ca1ea3d/5c2e021f-c2d4-49e2-8c36-9a64f1f12001/ca6525fc-674d-4dae-a2f9-d25bb2ff7c72"
-					(reference "C86")
+					(reference "C91")
 					(unit 1)
 				)
@@
 		(on_board yes)
 		(dnp no)
-		(property "Reference" "#PWR0141"
+		(property "Reference" "#PWR0143"
 			(at 133.35 102.87 0)
 			(effects
@@
 			(project "svea_powerboard_rev3"
 				(path "/3f85abf4-0b95-4c4a-b7e9-06f59ca1ea3d/5c2e021f-c2d4-49e2-8c36-9a64f1f12001/ca6525fc-674d-4dae-a2f9-d25bb2ff7c72"
-					(reference "#PWR0141")
+					(reference "#PWR0143")
 					(unit 1)
 				)
@@
 		(on_board yes)
 		(dnp no)
-		(property "Reference" "C85"
+		(property "Reference" "C90"
 			(at 82.55 92.71 90)
 			(effects
@@
 			(project "svea_powerboard_rev3"
 				(path "/3f85abf4-0b95-4c4a-b7e9-06f59ca1ea3d/5c2e021f-c2d4-49e2-8c36-9a64f1f12001/ca6525fc-674d-4dae-a2f9-d25bb2ff7c72"
-					(reference "C85")
+					(reference "C90")
 					(unit 1)
 				)
@@
 		(on_board yes)
 		(dnp no)
-		(property "Reference" "#PWR0142"
+		(property "Reference" "#PWR0144"
 			(at 193.04 119.38 0)
 			(effects
@@
 			(project "svea_powerboard_rev3"
 				(path "/3f85abf4-0b95-4c4a-b7e9-06f59ca1ea3d/5c2e021f-c2d4-49e2-8c36-9a64f1f12001/ca6525fc-674d-4dae-a2f9-d25bb2ff7c72"
-					(reference "#PWR0142")
+					(reference "#PWR0144")
 					(unit 1)
 				)
@@
 		(on_board yes)
 		(dnp no)
-		(property "Reference" "C88"
+		(property "Reference" "C93"
 			(at 228.6 63.5 0)
 			(effects
@@
 			(project "svea_powerboard_rev3"
 				(path "/3f85abf4-0b95-4c4a-b7e9-06f59ca1ea3d/5c2e021f-c2d4-49e2-8c36-9a64f1f12001/ca6525fc-674d-4dae-a2f9-d25bb2ff7c72"
-					(reference "C88")
+					(reference "C93")
 					(unit 1)
 				)
@@
 		(on_board yes)
 		(dnp no)
-		(property "Reference" "C87"
+		(property "Reference" "C92"
 			(at 214.63 63.5 0)
 			(effects
@@
 			(project "svea_powerboard_rev3"
 				(path "/3f85abf4-0b95-4c4a-b7e9-06f59ca1ea3d/5c2e021f-c2d4-49e2-8c36-9a64f1f12001/ca6525fc-674d-4dae-a2f9-d25bb2ff7c72"
-					(reference "C87")
+					(reference "C92")
 					(unit 1)
 				)
@@
 		(on_board yes)
 		(dnp no)
-		(property "Reference" "U43"
+		(property "Reference" "U46"
 			(at 142.24 71.12 0)
 			(effects
@@
 			(project "svea_powerboard_rev3"
 				(path "/3f85abf4-0b95-4c4a-b7e9-06f59ca1ea3d/5c2e021f-c2d4-49e2-8c36-9a64f1f12001/ca6525fc-674d-4dae-a2f9-d25bb2ff7c72"
-					(reference "U43")
+					(reference "U46")
 					(unit 1)
 				)
@@
 		(on_board yes)
 		(dnp no)
-		(property "Reference" "#PWR0143"
+		(property "Reference" "#PWR0145"
 			(at 224.79 74.93 0)
 			(effects
@@
 			(project "svea_powerboard_rev3"
 				(path "/3f85abf4-0b95-4c4a-b7e9-06f59ca1ea3d/5c2e021f-c2d4-49e2-8c36-9a64f1f12001/ca6525fc-674d-4dae-a2f9-d25bb2ff7c72"
-					(reference "#PWR0143")
+					(reference "#PWR0145")
 					(unit 1)
 				)
@@
 		(on_board yes)
 		(dnp no)
-		(property "Reference" "C84"
+		(property "Reference" "C89"
 			(at 67.31 91.44 90)
 			(effects
@@
 			(project "svea_powerboard_rev3"
 				(path "/3f85abf4-0b95-4c4a-b7e9-06f59ca1ea3d/5c2e021f-c2d4-49e2-8c36-9a64f1f12001/ca6525fc-674d-4dae-a2f9-d25bb2ff7c72"
-					(reference "C84")
+					(reference "C89")
 					(unit 1)
 				)

Commit message: new references
Parts:
- renumbered C89 to C91, C90 to C92, C91 to C93, C92 to C94, C93 to C95, R91 to R114, R92 to R115, R93 to R116, R94 to R117, U46 to U52
Changed lines of the file:
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@@
 		(on_board yes)
 		(dnp no)
-		(property "Reference" "#PWR0142"
+		(property "Reference" "#PWR0158"
 			(at 71.12 107.95 0)
 			(effects
@@
 			(project "svea_powerboard_rev3"
 				(path "/3f85abf4-0b95-4c4a-b7e9-06f59ca1ea3d/5c2e021f-c2d4-49e2-8c36-9a64f1f12001/ca6525fc-674d-4dae-a2f9-d25bb2ff7c72"
-					(reference "#PWR0142")
+					(reference "#PWR0158")
 					(unit 1)
 				)
@@
 		(on_board yes)
 		(dnp no)
-		(property "Reference" "R92"
+		(property "Reference" "R115"
 			(at 172.72 69.85 0)
 			(effects
@@
 			(project "svea_powerboard_rev3"
 				(path "/3f85abf4-0b95-4c4a-b7e9-06f59ca1ea3d/5c2e021f-c2d4-49e2-8c36-9a64f1f12001/ca6525fc-674d-4dae-a2f9-d25bb2ff7c72"
-					(reference "R92")
+					(reference "R115")
 					(unit 1)
 				)
@@
 		(on_board yes)
 		(dnp no)
-		(property "Reference" "R93"
+		(property "Reference" "R116"
 			(at 195.58 67.31 90)
 			(effects
@@
 			(project "svea_powerboard_rev3"
 				(path "/3f85abf4-0b95-4c4a-b7e9-06f59ca1ea3d/5c2e021f-c2d4-49e2-8c36-9a64f1f12001/ca6525fc-674d-4dae-a2f9-d25bb2ff7c72"
-					(reference "R93")
+					(reference "R116")
 					(unit 1)
 				)
@@
 		(on_board yes)
 		(dnp no)
-		(property "Reference" "R91"
+		(property "Reference" "R114"
 			(at 129.54 96.52 0)
 			(effects
@@
 			(project "svea_powerboard_rev3"
 				(path "/3f85abf4-0b95-4c4a-b7e9-06f59ca1ea3d/5c2e021f-c2d4-49e2-8c36-9a64f1f12001/ca6525fc-674d-4dae-a2f9-d25bb2ff7c72"
-					(reference "R91")
+					(reference "R114")
 					(unit 1)
 				)
@@
 		(on_board yes)
 		(dnp no)
-		(property "Reference" "R94"
+		(property "Reference" "R117"
 			(at 195.58 91.44 90)
 			(effects
@@
 			(project "svea_powerboard_rev3"
 				(path "/3f85abf4-0b95-4c4a-b7e9-06f59ca1ea3d/5c2e021f-c2d4-49e2-8c36-9a64f1f12001/ca6525fc-674d-4dae-a2f9-d25bb2ff7c72"
-					(reference "R94")
+					(reference "R117")
 					(unit 1)
 				)
@@
 		(on_board yes)
 		(dnp no)
-		(property "Reference" "C91"
+		(property "Reference" "C93"
 			(at 173.99 95.25 90)
 			(effects
@@
 			(project "svea_powerboard_rev3"
 				(path "/3f85abf4-0b95-4c4a-b7e9-06f59ca1ea3d/5c2e021f-c2d4-49e2-8c36-9a64f1f12001/ca6525fc-674d-4dae-a2f9-d25bb2ff7c72"
-					(reference "C91")
+					(reference "C93")
 					(unit 1)
 				)
@@
 		(on_board yes)
 		(dnp no)
-		(property "Reference" "#PWR0143"
+		(property "Reference" "#PWR0159"
 			(at 133.35 102.87 0)
 			(effects
@@
 			(project "svea_powerboard_rev3"
 				(path "/3f85abf4-0b95-4c4a-b7e9-06f59ca1ea3d/5c2e021f-c2d4-49e2-8c36-9a64f1f12001/ca6525fc-674d-4dae-a2f9-d25bb2ff7c72"
-					(reference "#PWR0143")
+					(reference "#PWR0159")
 					(unit 1)
 				)
@@
 		(on_board yes)
 		(dnp no)
-		(property "Reference" "C90"
+		(property "Reference" "C92"
 			(at 82.55 92.71 90)
 			(effects
@@
 			(project "svea_powerboard_rev3"
 				(path "/3f85abf4-0b95-4c4a-b7e9-06f59ca1ea3d/5c2e021f-c2d4-49e2-8c36-9a64f1f12001/ca6525fc-674d-4dae-a2f9-d25bb2ff7c72"
-					(reference "C90")
+					(reference "C92")
 					(unit 1)
 				)
@@
 		(on_board yes)
 		(dnp no)
-		(property "Reference" "#PWR0144"
+		(property "Reference" "#PWR0160"
 			(at 193.04 119.38 0)
 			(effects
@@
 			(project "svea_powerboard_rev3"
 				(path "/3f85abf4-0b95-4c4a-b7e9-06f59ca1ea3d/5c2e021f-c2d4-49e2-8c36-9a64f1f12001/ca6525fc-674d-4dae-a2f9-d25bb2ff7c72"
-					(reference "#PWR0144")
+					(reference "#PWR0160")
 					(unit 1)
 				)
@@
 		(on_board yes)
 		(dnp no)
-		(property "Reference" "C93"
+		(property "Reference" "C95"
 			(at 228.6 63.5 0)
 			(effects
@@
 			(project "svea_powerboard_rev3"
 				(path "/3f85abf4-0b95-4c4a-b7e9-06f59ca1ea3d/5c2e021f-c2d4-49e2-8c36-9a64f1f12001/ca6525fc-674d-4dae-a2f9-d25bb2ff7c72"
-					(reference "C93")
+					(reference "C95")
 					(unit 1)
 				)
@@
 		(on_board yes)
 		(dnp no)
-		(property "Reference" "C92"
+		(property "Reference" "C94"
 			(at 214.63 63.5 0)
 			(effects
@@
 			(project "svea_powerboard_rev3"
 				(path "/3f85abf4-0b95-4c4a-b7e9-06f59ca1ea3d/5c2e021f-c2d4-49e2-8c36-9a64f1f12001/ca6525fc-674d-4dae-a2f9-d25bb2ff7c72"
-					(reference "C92")
+					(reference "C94")
 					(unit 1)
 				)
@@
 		(on_board yes)
 		(dnp no)
-		(property "Reference" "U46"
+		(property "Reference" "U52"
 			(at 142.24 71.12 0)
 			(effects
@@
 			(project "svea_powerboard_rev3"
 				(path "/3f85abf4-0b95-4c4a-b7e9-06f59ca1ea3d/5c2e021f-c2d4-49e2-8c36-9a64f1f12001/ca6525fc-674d-4dae-a2f9-d25bb2ff7c72"
-					(reference "U46")
+					(reference "U52")
 					(unit 1)
 				)
@@
 		(on_board yes)
 		(dnp no)
-		(property "Reference" "#PWR0145"
+		(property "Reference" "#PWR0161"
 			(at 224.79 74.93 0)
 			(effects
@@
 			(project "svea_powerboard_rev3"
 				(path "/3f85abf4-0b95-4c4a-b7e9-06f59ca1ea3d/5c2e021f-c2d4-49e2-8c36-9a64f1f12001/ca6525fc-674d-4dae-a2f9-d25bb2ff7c72"
-					(reference "#PWR0145")
+					(reference "#PWR0161")
 					(unit 1)
 				)
@@
 		(on_board yes)
 		(dnp no)
-		(property "Reference" "C89"
+		(property "Reference" "C91"
 			(at 67.31 91.44 90)
 			(effects
@@
 			(project "svea_powerboard_rev3"
 				(path "/3f85abf4-0b95-4c4a-b7e9-06f59ca1ea3d/5c2e021f-c2d4-49e2-8c36-9a64f1f12001/ca6525fc-674d-4dae-a2f9-d25bb2ff7c72"
-					(reference "C89")
+					(reference "C91")
 					(unit 1)
 				)

Commit message: pre robot updating references
Parts:
- renumbered C91 to C89, C92 to C90, C93 to C91, C94 to C92, C95 to C93, R114 to R121, R115 to R122, R116 to R123, R117 to R124
Changed lines of the file:
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@@
 		(on_board yes)
 		(dnp no)
-		(property "Reference" "#PWR0158"
+		(property "Reference" "#PWR0145"
 			(at 71.12 107.95 0)
 			(effects
@@
 			(project "svea_powerboard_rev3"
 				(path "/3f85abf4-0b95-4c4a-b7e9-06f59ca1ea3d/5c2e021f-c2d4-49e2-8c36-9a64f1f12001/ca6525fc-674d-4dae-a2f9-d25bb2ff7c72"
-					(reference "#PWR0158")
+					(reference "#PWR0145")
 					(unit 1)
 				)
@@
 		(on_board yes)
 		(dnp no)
-		(property "Reference" "R115"
+		(property "Reference" "R122"
 			(at 172.72 69.85 0)
 			(effects
@@
 			(project "svea_powerboard_rev3"
 				(path "/3f85abf4-0b95-4c4a-b7e9-06f59ca1ea3d/5c2e021f-c2d4-49e2-8c36-9a64f1f12001/ca6525fc-674d-4dae-a2f9-d25bb2ff7c72"
-					(reference "R115")
+					(reference "R122")
 					(unit 1)
 				)
@@
 		(on_board yes)
 		(dnp no)
-		(property "Reference" "R116"
+		(property "Reference" "R123"
 			(at 195.58 67.31 90)
 			(effects
@@
 			(project "svea_powerboard_rev3"
 				(path "/3f85abf4-0b95-4c4a-b7e9-06f59ca1ea3d/5c2e021f-c2d4-49e2-8c36-9a64f1f12001/ca6525fc-674d-4dae-a2f9-d25bb2ff7c72"
-					(reference "R116")
+					(reference "R123")
 					(unit 1)
 				)
@@
 		(on_board yes)
 		(dnp no)
-		(property "Reference" "R114"
+		(property "Reference" "R121"
 			(at 129.54 96.52 0)
 			(effects
@@
 			(project "svea_powerboard_rev3"
 				(path "/3f85abf4-0b95-4c4a-b7e9-06f59ca1ea3d/5c2e021f-c2d4-49e2-8c36-9a64f1f12001/ca6525fc-674d-4dae-a2f9-d25bb2ff7c72"
-					(reference "R114")
+					(reference "R121")
 					(unit 1)
 				)
@@
 		(on_board yes)
 		(dnp no)
-		(property "Reference" "R117"
+		(property "Reference" "R124"
 			(at 195.58 91.44 90)
 			(effects
@@
 			(project "svea_powerboard_rev3"
 				(path "/3f85abf4-0b95-4c4a-b7e9-06f59ca1ea3d/5c2e021f-c2d4-49e2-8c36-9a64f1f12001/ca6525fc-674d-4dae-a2f9-d25bb2ff7c72"
-					(reference "R117")
+					(reference "R124")
 					(unit 1)
 				)
@@
 		(on_board yes)
 		(dnp no)
-		(property "Reference" "C93"
+		(property "Reference" "C91"
 			(at 173.99 95.25 90)
 			(effects
@@
 			(project "svea_powerboard_rev3"
 				(path "/3f85abf4-0b95-4c4a-b7e9-06f59ca1ea3d/5c2e021f-c2d4-49e2-8c36-9a64f1f12001/ca6525fc-674d-4dae-a2f9-d25bb2ff7c72"
-					(reference "C93")
+					(reference "C91")
 					(unit 1)
 				)
@@
 		(on_board yes)
 		(dnp no)
-		(property "Reference" "#PWR0159"
+		(property "Reference" "#PWR0146"
 			(at 133.35 102.87 0)
 			(effects
@@
 			(project "svea_powerboard_rev3"
 				(path "/3f85abf4-0b95-4c4a-b7e9-06f59ca1ea3d/5c2e021f-c2d4-49e2-8c36-9a64f1f12001/ca6525fc-674d-4dae-a2f9-d25bb2ff7c72"
-					(reference "#PWR0159")
+					(reference "#PWR0146")
 					(unit 1)
 				)
@@
 		(on_board yes)
 		(dnp no)
-		(property "Reference" "C92"
+		(property "Reference" "C90"
 			(at 82.55 92.71 90)
 			(effects
@@
 			(project "svea_powerboard_rev3"
 				(path "/3f85abf4-0b95-4c4a-b7e9-06f59ca1ea3d/5c2e021f-c2d4-49e2-8c36-9a64f1f12001/ca6525fc-674d-4dae-a2f9-d25bb2ff7c72"
-					(reference "C92")
+					(reference "C90")
 					(unit 1)
 				)
@@
 		(on_board yes)
 		(dnp no)
-		(property "Reference" "#PWR0160"
+		(property "Reference" "#PWR0147"
 			(at 193.04 119.38 0)
 			(effects
@@
 			(project "svea_powerboard_rev3"
 				(path "/3f85abf4-0b95-4c4a-b7e9-06f59ca1ea3d/5c2e021f-c2d4-49e2-8c36-9a64f1f12001/ca6525fc-674d-4dae-a2f9-d25bb2ff7c72"
-					(reference "#PWR0160")
+					(reference "#PWR0147")
 					(unit 1)
 				)
@@
 		(on_board yes)
 		(dnp no)
-		(property "Reference" "C95"
+		(property "Reference" "C93"
 			(at 228.6 63.5 0)
 			(effects
@@
 			(project "svea_powerboard_rev3"
 				(path "/3f85abf4-0b95-4c4a-b7e9-06f59ca1ea3d/5c2e021f-c2d4-49e2-8c36-9a64f1f12001/ca6525fc-674d-4dae-a2f9-d25bb2ff7c72"
-					(reference "C95")
+					(reference "C93")
 					(unit 1)
 				)
@@
 		(on_board yes)
 		(dnp no)
-		(property "Reference" "C94"
+		(property "Reference" "C92"
 			(at 214.63 63.5 0)
 			(effects
@@
 			(project "svea_powerboard_rev3"
 				(path "/3f85abf4-0b95-4c4a-b7e9-06f59ca1ea3d/5c2e021f-c2d4-49e2-8c36-9a64f1f12001/ca6525fc-674d-4dae-a2f9-d25bb2ff7c72"
-					(reference "C94")
+					(reference "C92")
 					(unit 1)
 				)
@@
 		(on_board yes)
 		(dnp no)
-		(property "Reference" "#PWR0161"
+		(property "Reference" "#PWR0148"
 			(at 224.79 74.93 0)
 			(effects
@@
 			(project "svea_powerboard_rev3"
 				(path "/3f85abf4-0b95-4c4a-b7e9-06f59ca1ea3d/5c2e021f-c2d4-49e2-8c36-9a64f1f12001/ca6525fc-674d-4dae-a2f9-d25bb2ff7c72"
-					(reference "#PWR0161")
+					(reference "#PWR0148")
 					(unit 1)
 				)
@@
 		(on_board yes)
 		(dnp no)
-		(property "Reference" "C91"
+		(property "Reference" "C89"
 			(at 67.31 91.44 90)
 			(effects
@@
 			(project "svea_powerboard_rev3"
 				(path "/3f85abf4-0b95-4c4a-b7e9-06f59ca1ea3d/5c2e021f-c2d4-49e2-8c36-9a64f1f12001/ca6525fc-674d-4dae-a2f9-d25bb2ff7c72"
-					(reference "C91")
+					(reference "C89")
 					(unit 1)
 				)

Commit message: various imprvements
Parts:
- renumbered C89 to C94, C90 to C95, C91 to C96, C92 to C97, C93 to C98, R121 to R151, R122 to R152, R123 to R153, R124 to R154, U52 to U58
Connections:
- net MCU-3V3-PGOOD renamed Power/3V3/PGOOD
Changed lines of the file:
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@@
 		)
 	)
-	(global_label "MCU-3V3-PGOOD"
+	(global_label "Power/3V3/PGOOD"
 		(shape output)
 		(at 120.65 68.58 180)
@@
 		(on_board yes)
 		(dnp no)
-		(property "Reference" "#PWR0145"
+		(property "Reference" "#PWR0158"
 			(at 71.12 107.95 0)
 			(effects
@@
 			(project "svea_powerboard_rev3"
 				(path "/3f85abf4-0b95-4c4a-b7e9-06f59ca1ea3d/5c2e021f-c2d4-49e2-8c36-9a64f1f12001/ca6525fc-674d-4dae-a2f9-d25bb2ff7c72"
-					(reference "#PWR0145")
+					(reference "#PWR0158")
 					(unit 1)
 				)
@@
 		(on_board yes)
 		(dnp no)
-		(property "Reference" "R122"
+		(property "Reference" "R152"
 			(at 172.72 69.85 0)
 			(effects
@@
 			(project "svea_powerboard_rev3"
 				(path "/3f85abf4-0b95-4c4a-b7e9-06f59ca1ea3d/5c2e021f-c2d4-49e2-8c36-9a64f1f12001/ca6525fc-674d-4dae-a2f9-d25bb2ff7c72"
-					(reference "R122")
+					(reference "R152")
 					(unit 1)
 				)
@@
 		(on_board yes)
 		(dnp no)
-		(property "Reference" "R123"
+		(property "Reference" "R153"
 			(at 195.58 67.31 90)
 			(effects
@@
 			(project "svea_powerboard_rev3"
 				(path "/3f85abf4-0b95-4c4a-b7e9-06f59ca1ea3d/5c2e021f-c2d4-49e2-8c36-9a64f1f12001/ca6525fc-674d-4dae-a2f9-d25bb2ff7c72"
-					(reference "R123")
+					(reference "R153")
 					(unit 1)
 				)
@@
 		(on_board yes)
 		(dnp no)
-		(property "Reference" "R121"
+		(property "Reference" "R151"
 			(at 129.54 96.52 0)
 			(effects
@@
 			(project "svea_powerboard_rev3"
 				(path "/3f85abf4-0b95-4c4a-b7e9-06f59ca1ea3d/5c2e021f-c2d4-49e2-8c36-9a64f1f12001/ca6525fc-674d-4dae-a2f9-d25bb2ff7c72"
-					(reference "R121")
+					(reference "R151")
 					(unit 1)
 				)
@@
 		(on_board yes)
 		(dnp no)
-		(property "Reference" "R124"
+		(property "Reference" "R154"
 			(at 195.58 91.44 90)
 			(effects
@@
 			(project "svea_powerboard_rev3"
 				(path "/3f85abf4-0b95-4c4a-b7e9-06f59ca1ea3d/5c2e021f-c2d4-49e2-8c36-9a64f1f12001/ca6525fc-674d-4dae-a2f9-d25bb2ff7c72"
-					(reference "R124")
+					(reference "R154")
 					(unit 1)
 				)
@@
 		(on_board yes)
 		(dnp no)
-		(property "Reference" "C91"
+		(property "Reference" "C96"
 			(at 173.99 95.25 90)
 			(effects
@@
 			(project "svea_powerboard_rev3"
 				(path "/3f85abf4-0b95-4c4a-b7e9-06f59ca1ea3d/5c2e021f-c2d4-49e2-8c36-9a64f1f12001/ca6525fc-674d-4dae-a2f9-d25bb2ff7c72"
-					(reference "C91")
+					(reference "C96")
 					(unit 1)
 				)
@@
 		(on_board yes)
 		(dnp no)
-		(property "Reference" "#PWR0146"
+		(property "Reference" "#PWR0159"
 			(at 133.35 102.87 0)
 			(effects
@@
 			(project "svea_powerboard_rev3"
 				(path "/3f85abf4-0b95-4c4a-b7e9-06f59ca1ea3d/5c2e021f-c2d4-49e2-8c36-9a64f1f12001/ca6525fc-674d-4dae-a2f9-d25bb2ff7c72"
-					(reference "#PWR0146")
+					(reference "#PWR0159")
 					(unit 1)
 				)
@@
 		(on_board yes)
 		(dnp no)
-		(property "Reference" "C90"
+		(property "Reference" "C95"
 			(at 82.55 92.71 90)
 			(effects
@@
 			(project "svea_powerboard_rev3"
 				(path "/3f85abf4-0b95-4c4a-b7e9-06f59ca1ea3d/5c2e021f-c2d4-49e2-8c36-9a64f1f12001/ca6525fc-674d-4dae-a2f9-d25bb2ff7c72"
-					(reference "C90")
+					(reference "C95")
 					(unit 1)
 				)
@@
 		(on_board yes)
 		(dnp no)
-		(property "Reference" "#PWR0147"
+		(property "Reference" "#PWR0160"
 			(at 193.04 119.38 0)
 			(effects
@@
 			(project "svea_powerboard_rev3"
 				(path "/3f85abf4-0b95-4c4a-b7e9-06f59ca1ea3d/5c2e021f-c2d4-49e2-8c36-9a64f1f12001/ca6525fc-674d-4dae-a2f9-d25bb2ff7c72"
-					(reference "#PWR0147")
+					(reference "#PWR0160")
 					(unit 1)
 				)
@@
 		(on_board yes)
 		(dnp no)
-		(property "Reference" "C93"
+		(property "Reference" "C98"
 			(at 228.6 63.5 0)
 			(effects
@@
 			(project "svea_powerboard_rev3"
 				(path "/3f85abf4-0b95-4c4a-b7e9-06f59ca1ea3d/5c2e021f-c2d4-49e2-8c36-9a64f1f12001/ca6525fc-674d-4dae-a2f9-d25bb2ff7c72"
-					(reference "C93")
+					(reference "C98")
 					(unit 1)
 				)
@@
 		(on_board yes)
 		(dnp no)
-		(property "Reference" "C92"
+		(property "Reference" "C97"
 			(at 214.63 63.5 0)
 			(effects
@@
 			(project "svea_powerboard_rev3"
 				(path "/3f85abf4-0b95-4c4a-b7e9-06f59ca1ea3d/5c2e021f-c2d4-49e2-8c36-9a64f1f12001/ca6525fc-674d-4dae-a2f9-d25bb2ff7c72"
-					(reference "C92")
+					(reference "C97")
 					(unit 1)
 				)
@@
 		(on_board yes)
 		(dnp no)
-		(property "Reference" "U52"
+		(property "Reference" "U58"
 			(at 142.24 71.12 0)
 			(effects
@@
 			(project "svea_powerboard_rev3"
 				(path "/3f85abf4-0b95-4c4a-b7e9-06f59ca1ea3d/5c2e021f-c2d4-49e2-8c36-9a64f1f12001/ca6525fc-674d-4dae-a2f9-d25bb2ff7c72"
-					(reference "U52")
+					(reference "U58")
 					(unit 1)
 				)
@@
 		(on_board yes)
 		(dnp no)
-		(property "Reference" "#PWR0148"
+		(property "Reference" "#PWR0161"
 			(at 224.79 74.93 0)
 			(effects
@@
 			(project "svea_powerboard_rev3"
 				(path "/3f85abf4-0b95-4c4a-b7e9-06f59ca1ea3d/5c2e021f-c2d4-49e2-8c36-9a64f1f12001/ca6525fc-674d-4dae-a2f9-d25bb2ff7c72"
-					(reference "#PWR0148")
+					(reference "#PWR0161")
 					(unit 1)
 				)
@@
 		(on_board yes)
 		(dnp no)
-		(property "Reference" "C89"
+		(property "Reference" "C94"
 			(at 67.31 91.44 90)
 			(effects
@@
 			(project "svea_powerboard_rev3"
 				(path "/3f85abf4-0b95-4c4a-b7e9-06f59ca1ea3d/5c2e021f-c2d4-49e2-8c36-9a64f1f12001/ca6525fc-674d-4dae-a2f9-d25bb2ff7c72"
-					(reference "C89")
+					(reference "C94")
 					(unit 1)
 				)
