File: hardware/kicad/sheets/connectors/12V-VH-PORTS.kicad_sch (KiCad schematic)
At the start: 0 parts

Commit message: starting transition to single root
Other:
- removed sheet CUR1
- removed sheet JST-VH-12V-PIN
- removed sheet JST-VH-12V-PIN1
- removed sheet JST-VH-12V-PIN2
