File: hardware/kicad/sheets/connectors/MISC_IO_CURR_SENSING_1.kicad_sch (KiCad schematic)
At the start: 20 parts

Commit message: new references
Parts:
- renumbered C36 to C37, C37 to C38, C38 to C39, C39 to C40, C40 to C41, R35 to R57, R36 to R58, R37 to R59, R38 to R60, R39 to R61, R40 to R62, R41 to R63
Changed lines of the file:
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@@
 		(on_board yes)
 		(dnp no)
-		(property "Reference" "#PWR060"
+		(property "Reference" "#PWR072"
 			(at 63.5 142.24 0)
 			(effects
@@
 			(project "svea_powerboard_rev3"
 				(path "/3f85abf4-0b95-4c4a-b7e9-06f59ca1ea3d/5c2e021f-c2d4-49e2-8c36-9a64f1f12001/018d0221-df9b-4023-93f4-3996394924d7"
-					(reference "#PWR0151")
+					(reference "#PWR0167")
 					(unit 1)
 				)
 				(path "/3f85abf4-0b95-4c4a-b7e9-06f59ca1ea3d/5c2e021f-c2d4-49e2-8c36-9a64f1f12001/3defe835-7f3e-4186-81ed-0e8caa47e3eb"
-					(reference "#PWR060")
+					(reference "#PWR072")
 					(unit 1)
 				)
@@
 		(on_board yes)
 		(dnp no)
-		(property "Reference" "C38"
+		(property "Reference" "C39"
 			(at 118.11 105.41 90)
 			(effects
@@
 			(project "svea_powerboard_rev3"
 				(path "/3f85abf4-0b95-4c4a-b7e9-06f59ca1ea3d/5c2e021f-c2d4-49e2-8c36-9a64f1f12001/018d0221-df9b-4023-93f4-3996394924d7"
-					(reference "C102")
+					(reference "C104")
 					(unit 1)
 				)
 				(path "/3f85abf4-0b95-4c4a-b7e9-06f59ca1ea3d/5c2e021f-c2d4-49e2-8c36-9a64f1f12001/3defe835-7f3e-4186-81ed-0e8caa47e3eb"
-					(reference "C38")
+					(reference "C39")
 					(unit 1)
 				)
@@
 		(on_board yes)
 		(dnp no)
-		(property "Reference" "R41"
+		(property "Reference" "R63"
 			(at 228.6 110.49 0)
 			(effects
@@
 			(project "svea_powerboard_rev3"
 				(path "/3f85abf4-0b95-4c4a-b7e9-06f59ca1ea3d/5c2e021f-c2d4-49e2-8c36-9a64f1f12001/018d0221-df9b-4023-93f4-3996394924d7"
-					(reference "R106")
+					(reference "R129")
 					(unit 1)
 				)
 				(path "/3f85abf4-0b95-4c4a-b7e9-06f59ca1ea3d/5c2e021f-c2d4-49e2-8c36-9a64f1f12001/3defe835-7f3e-4186-81ed-0e8caa47e3eb"
-					(reference "R41")
+					(reference "R63")
 					(unit 1)
 				)
@@
 		(on_board yes)
 		(dnp no)
-		(property "Reference" "R37"
+		(property "Reference" "R59"
 			(at 139.7 137.16 0)
 			(effects
@@
 			(project "svea_powerboard_rev3"
 				(path "/3f85abf4-0b95-4c4a-b7e9-06f59ca1ea3d/5c2e021f-c2d4-49e2-8c36-9a64f1f12001/018d0221-df9b-4023-93f4-3996394924d7"
-					(reference "R102")
+					(reference "R125")
 					(unit 1)
 				)
 				(path "/3f85abf4-0b95-4c4a-b7e9-06f59ca1ea3d/5c2e021f-c2d4-49e2-8c36-9a64f1f12001/3defe835-7f3e-4186-81ed-0e8caa47e3eb"
-					(reference "R37")
+					(reference "R59")
 					(unit 1)
 				)
@@
 		(on_board yes)
 		(dnp no)
-		(property "Reference" "R39"
+		(property "Reference" "R61"
 			(at 171.4754 68.58 90)
 			(effects
@@
 			(project "svea_powerboard_rev3"
 				(path "/3f85abf4-0b95-4c4a-b7e9-06f59ca1ea3d/5c2e021f-c2d4-49e2-8c36-9a64f1f12001/018d0221-df9b-4023-93f4-3996394924d7"
-					(reference "R104")
+					(reference "R127")
 					(unit 1)
 				)
 				(path "/3f85abf4-0b95-4c4a-b7e9-06f59ca1ea3d/5c2e021f-c2d4-49e2-8c36-9a64f1f12001/3defe835-7f3e-4186-81ed-0e8caa47e3eb"
-					(reference "R39")
+					(reference "R61")
 					(unit 1)
 				)
@@
 		(on_board yes)
 		(dnp no)
-		(property "Reference" "C39"
+		(property "Reference" "C40"
 			(at 158.75 77.47 0)
 			(effects
@@
 			(project "svea_powerboard_rev3"
 				(path "/3f85abf4-0b95-4c4a-b7e9-06f59ca1ea3d/5c2e021f-c2d4-49e2-8c36-9a64f1f12001/018d0221-df9b-4023-93f4-3996394924d7"
-					(reference "C103")
+					(reference "C105")
 					(unit 1)
 				)
 				(path "/3f85abf4-0b95-4c4a-b7e9-06f59ca1ea3d/5c2e021f-c2d4-49e2-8c36-9a64f1f12001/3defe835-7f3e-4186-81ed-0e8caa47e3eb"
-					(reference "C39")
+					(reference "C40")
 					(unit 1)
 				)
@@
 		(on_board yes)
 		(dnp no)
-		(property "Reference" "C37"
+		(property "Reference" "C38"
 			(at 67.31 127 90)
 			(effects
@@
 			(project "svea_powerboard_rev3"
 				(path "/3f85abf4-0b95-4c4a-b7e9-06f59ca1ea3d/5c2e021f-c2d4-49e2-8c36-9a64f1f12001/018d0221-df9b-4023-93f4-3996394924d7"
-					(reference "C101")
+					(reference "C103")
 					(unit 1)
 				)
 				(path "/3f85abf4-0b95-4c4a-b7e9-06f59ca1ea3d/5c2e021f-c2d4-49e2-8c36-9a64f1f12001/3defe835-7f3e-4186-81ed-0e8caa47e3eb"
-					(reference "C37")
+					(reference "C38")
 					(unit 1)
 				)
@@
 		(on_board yes)
 		(dnp no)
-		(property "Reference" "#PWR061"
+		(property "Reference" "#PWR073"
 			(at 186.69 50.8 0)
 			(effects
@@
 			(project "svea_powerboard_rev3"
 				(path "/3f85abf4-0b95-4c4a-b7e9-06f59ca1ea3d/5c2e021f-c2d4-49e2-8c36-9a64f1f12001/018d0221-df9b-4023-93f4-3996394924d7"
-					(reference "#PWR0152")
+					(reference "#PWR0168")
 					(unit 1)
 				)
 				(path "/3f85abf4-0b95-4c4a-b7e9-06f59ca1ea3d/5c2e021f-c2d4-49e2-8c36-9a64f1f12001/3defe835-7f3e-4186-81ed-0e8caa47e3eb"
-					(reference "#PWR061")
+					(reference "#PWR073")
 					(unit 1)
 				)
@@
 		(on_board yes)
 		(dnp no)
-		(property "Reference" "#PWR059"
+		(property "Reference" "#PWR071"
 			(at 46.99 95.25 0)
 			(effects
@@
 			(project "svea_powerboard_rev3"
 				(path "/3f85abf4-0b95-4c4a-b7e9-06f59ca1ea3d/5c2e021f-c2d4-49e2-8c36-9a64f1f12001/018d0221-df9b-4023-93f4-3996394924d7"
-					(reference "#PWR0150")
+					(reference "#PWR0166")
 					(unit 1)
 				)
 				(path "/3f85abf4-0b95-4c4a-b7e9-06f59ca1ea3d/5c2e021f-c2d4-49e2-8c36-9a64f1f12001/3defe835-7f3e-4186-81ed-0e8caa47e3eb"
-					(reference "#PWR059")
+					(reference "#PWR071")
 					(unit 1)
 				)
@@
 		(on_board yes)
 		(dnp no)
-		(property "Reference" "R36"
+		(property "Reference" "R58"
 			(at 102.87 110.49 0)
 			(effects
@@
 			(project "svea_powerboard_rev3"
 				(path "/3f85abf4-0b95-4c4a-b7e9-06f59ca1ea3d/5c2e021f-c2d4-49e2-8c36-9a64f1f12001/018d0221-df9b-4023-93f4-3996394924d7"
-					(reference "R101")
+					(reference "R124")
 					(unit 1)
 				)
 				(path "/3f85abf4-0b95-4c4a-b7e9-06f59ca1ea3d/5c2e021f-c2d4-49e2-8c36-9a64f1f12001/3defe835-7f3e-4186-81ed-0e8caa47e3eb"
-					(reference "R36")
+					(reference "R58")
 					(unit 1)
 				)
@@
 		(on_board yes)
 		(dnp no)
-		(property "Reference" "R38"
+		(property "Reference" "R60"
 			(at 157.5054 68.58 90)
 			(effects
@@
 			(project "svea_powerboard_rev3"
 				(path "/3f85abf4-0b95-4c4a-b7e9-06f59ca1ea3d/5c2e021f-c2d4-49e2-8c36-9a64f1f12001/018d0221-df9b-4023-93f4-3996394924d7"
-					(reference "R103")
+					(reference "R126")
 					(unit 1)
 				)
 				(path "/3f85abf4-0b95-4c4a-b7e9-06f59ca1ea3d/5c2e021f-c2d4-49e2-8c36-9a64f1f12001/3defe835-7f3e-4186-81ed-0e8caa47e3eb"
-					(reference "R38")
+					(reference "R60")
 					(unit 1)
 				)
@@
 		(on_board yes)
 		(dnp no)
-		(property "Reference" "C36"
+		(property "Reference" "C37"
 			(at 50.8 127 90)
 			(effects
@@
 			(project "svea_powerboard_rev3"
 				(path "/3f85abf4-0b95-4c4a-b7e9-06f59ca1ea3d/5c2e021f-c2d4-49e2-8c36-9a64f1f12001/018d0221-df9b-4023-93f4-3996394924d7"
-					(reference "C100")
+					(reference "C102")
 					(unit 1)
 				)
 				(path "/3f85abf4-0b95-4c4a-b7e9-06f59ca1ea3d/5c2e021f-c2d4-49e2-8c36-9a64f1f12001/3defe835-7f3e-4186-81ed-0e8caa47e3eb"
-					(reference "C36")
+					(reference "C37")
 					(unit 1)
 				)
@@
 		(on_board yes)
 		(dnp no)
-		(property "Reference" "R40"
+		(property "Reference" "R62"
 			(at 228.6 96.52 0)
 			(effects
@@
 			(project "svea_powerboard_rev3"
 				(path "/3f85abf4-0b95-4c4a-b7e9-06f59ca1ea3d/5c2e021f-c2d4-49e2-8c36-9a64f1f12001/018d0221-df9b-4023-93f4-3996394924d7"
-					(reference "R105")
+					(reference "R128")
 					(unit 1)
 				)
 				(path "/3f85abf4-0b95-4c4a-b7e9-06f59ca1ea3d/5c2e021f-c2d4-49e2-8c36-9a64f1f12001/3defe835-7f3e-4186-81ed-0e8caa47e3eb"
-					(reference "R40")
+					(reference "R62")
 					(unit 1)
 				)
@@
 		(on_board yes)
 		(dnp no)
-		(property "Reference" "R35"
+		(property "Reference" "R57"
 			(at 102.87 96.52 0)
 			(effects
@@
 			(project "svea_powerboard_rev3"
 				(path "/3f85abf4-0b95-4c4a-b7e9-06f59ca1ea3d/5c2e021f-c2d4-49e2-8c36-9a64f1f12001/018d0221-df9b-4023-93f4-3996394924d7"
-					(reference "R100")
+					(reference "R123")
 					(unit 1)
 				)
 				(path "/3f85abf4-0b95-4c4a-b7e9-06f59ca1ea3d/5c2e021f-c2d4-49e2-8c36-9a64f1f12001/3defe835-7f3e-4186-81ed-0e8caa47e3eb"
-					(reference "R35")
+					(reference "R57")
 					(unit 1)
 				)
@@
 		(on_board yes)
 		(dnp no)
-		(property "Reference" "C40"
+		(property "Reference" "C41"
 			(at 228.6 105.41 90)
 			(effects
@@
 			(project "svea_powerboard_rev3"
 				(path "/3f85abf4-0b95-4c4a-b7e9-06f59ca1ea3d/5c2e021f-c2d4-49e2-8c36-9a64f1f12001/018d0221-df9b-4023-93f4-3996394924d7"
-					(reference "C104")
+					(reference "C106")
 					(unit 1)
 				)
 				(path "/3f85abf4-0b95-4c4a-b7e9-06f59ca1ea3d/5c2e021f-c2d4-49e2-8c36-9a64f1f12001/3defe835-7f3e-4186-81ed-0e8caa47e3eb"
-					(reference "C40")
-					(unit 1)
-				)
+					(reference "C41")
+					(unit 1)
+				)
