File: hardware/kicad/sheets/connectors/JST-VH-12V-PIN.kicad_sch (KiCad schematic)
At the start: 5 parts, among them U16 VH3_96-2P_WZ

Commit message: new references
Parts:
- renumbered C41 to C42, C42 to C43, D17 to D16, R42 to R64, U16 to U21
Changed lines of the file:
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@@
 		(on_board yes)
 		(dnp no)
-		(property "Reference" "U16"
+		(property "Reference" "U21"
 			(at 97.79 87.63 0)
 			(effects
@@
 			(project "svea_powerboard_rev3"
 				(path "/3f85abf4-0b95-4c4a-b7e9-06f59ca1ea3d/5c2e021f-c2d4-49e2-8c36-9a64f1f12001/03241f80-3125-4f5b-a1a0-add76ba31aaa"
-					(reference "U16")
+					(reference "U21")
 					(unit 1)
 				)
 				(path "/3f85abf4-0b95-4c4a-b7e9-06f59ca1ea3d/5c2e021f-c2d4-49e2-8c36-9a64f1f12001/782118f9-6c0b-4f5a-9c3b-1e5b8fc1f0ac"
-					(reference "U17")
+					(reference "U22")
 					(unit 1)
 				)
 				(path "/3f85abf4-0b95-4c4a-b7e9-06f59ca1ea3d/5c2e021f-c2d4-49e2-8c36-9a64f1f12001/beb9ceef-df3a-4e22-8974-012ce1407a41"
-					(reference "U18")
+					(reference "U23")
 					(unit 1)
 				)
@@
 		(on_board yes)
 		(dnp no)
-		(property "Reference" "D17"
+		(property "Reference" "D16"
 			(at 154.94 97.79 90)
 			(effects
@@
 			(project "svea_powerboard_rev3"
 				(path "/3f85abf4-0b95-4c4a-b7e9-06f59ca1ea3d/5c2e021f-c2d4-49e2-8c36-9a64f1f12001/03241f80-3125-4f5b-a1a0-add76ba31aaa"
+					(reference "D16")
+					(unit 1)
+				)
+				(path "/3f85abf4-0b95-4c4a-b7e9-06f59ca1ea3d/5c2e021f-c2d4-49e2-8c36-9a64f1f12001/782118f9-6c0b-4f5a-9c3b-1e5b8fc1f0ac"
 					(reference "D17")
 					(unit 1)
 				)
-				(path "/3f85abf4-0b95-4c4a-b7e9-06f59ca1ea3d/5c2e021f-c2d4-49e2-8c36-9a64f1f12001/782118f9-6c0b-4f5a-9c3b-1e5b8fc1f0ac"
+				(path "/3f85abf4-0b95-4c4a-b7e9-06f59ca1ea3d/5c2e021f-c2d4-49e2-8c36-9a64f1f12001/beb9ceef-df3a-4e22-8974-012ce1407a41"
 					(reference "D18")
-					(unit 1)
-				)
-				(path "/3f85abf4-0b95-4c4a-b7e9-06f59ca1ea3d/5c2e021f-c2d4-49e2-8c36-9a64f1f12001/beb9ceef-df3a-4e22-8974-012ce1407a41"
-					(reference "D19")
 					(unit 1)
 				)
@@
 		(on_board yes)
 		(dnp no)
-		(property "Reference" "C42"
+		(property "Reference" "C43"
 			(at 143.51 96.52 90)
 			(effects
@@
 			(project "svea_powerboard_rev3"
 				(path "/3f85abf4-0b95-4c4a-b7e9-06f59ca1ea3d/5c2e021f-c2d4-49e2-8c36-9a64f1f12001/03241f80-3125-4f5b-a1a0-add76ba31aaa"
-					(reference "C42")
+					(reference "C43")
 					(unit 1)
 				)
 				(path "/3f85abf4-0b95-4c4a-b7e9-06f59ca1ea3d/5c2e021f-c2d4-49e2-8c36-9a64f1f12001/782118f9-6c0b-4f5a-9c3b-1e5b8fc1f0ac"
-					(reference "C44")
+					(reference "C45")
 					(unit 1)
 				)
 				(path "/3f85abf4-0b95-4c4a-b7e9-06f59ca1ea3d/5c2e021f-c2d4-49e2-8c36-9a64f1f12001/beb9ceef-df3a-4e22-8974-012ce1407a41"
-					(reference "C46")
+					(reference "C47")
 					(unit 1)
 				)
@@
 		(on_board yes)
 		(dnp no)
-		(property "Reference" "#PWR062"
+		(property "Reference" "#PWR074"
 			(at 139.7 106.68 0)
 			(effects
@@
 			(project "svea_powerboard_rev3"
 				(path "/3f85abf4-0b95-4c4a-b7e9-06f59ca1ea3d/5c2e021f-c2d4-49e2-8c36-9a64f1f12001/03241f80-3125-4f5b-a1a0-add76ba31aaa"
-					(reference "#PWR062")
+					(reference "#PWR074")
 					(unit 1)
 				)
 				(path "/3f85abf4-0b95-4c4a-b7e9-06f59ca1ea3d/5c2e021f-c2d4-49e2-8c36-9a64f1f12001/782118f9-6c0b-4f5a-9c3b-1e5b8fc1f0ac"
-					(reference "#PWR063")
+					(reference "#PWR075")
 					(unit 1)
 				)
 				(path "/3f85abf4-0b95-4c4a-b7e9-06f59ca1ea3d/5c2e021f-c2d4-49e2-8c36-9a64f1f12001/beb9ceef-df3a-4e22-8974-012ce1407a41"
-					(reference "#PWR064")
+					(reference "#PWR076")
 					(unit 1)
 				)
@@
 		(on_board yes)
 		(dnp no)
-		(property "Reference" "C41"
+		(property "Reference" "C42"
 			(at 132.08 96.52 90)
 			(effects
@@
 			(project "svea_powerboard_rev3"
 				(path "/3f85abf4-0b95-4c4a-b7e9-06f59ca1ea3d/5c2e021f-c2d4-49e2-8c36-9a64f1f12001/03241f80-3125-4f5b-a1a0-add76ba31aaa"
-					(reference "C41")
+					(reference "C42")
 					(unit 1)
 				)
 				(path "/3f85abf4-0b95-4c4a-b7e9-06f59ca1ea3d/5c2e021f-c2d4-49e2-8c36-9a64f1f12001/782118f9-6c0b-4f5a-9c3b-1e5b8fc1f0ac"
-					(reference "C43")
+					(reference "C44")
 					(unit 1)
 				)
 				(path "/3f85abf4-0b95-4c4a-b7e9-06f59ca1ea3d/5c2e021f-c2d4-49e2-8c36-9a64f1f12001/beb9ceef-df3a-4e22-8974-012ce1407a41"
-					(reference "C45")
+					(reference "C46")
 					(unit 1)
 				)
@@
 		(on_board yes)
 		(dnp no)
-		(property "Reference" "R42"
+		(property "Reference" "R64"
 			(at 162.56 93.218 0)
 			(effects
@@
 			(project "svea_powerboard_rev3"
 				(path "/3f85abf4-0b95-4c4a-b7e9-06f59ca1ea3d/5c2e021f-c2d4-49e2-8c36-9a64f1f12001/03241f80-3125-4f5b-a1a0-add76ba31aaa"
-					(reference "R42")
+					(reference "R64")
 					(unit 1)
 				)
 				(path "/3f85abf4-0b95-4c4a-b7e9-06f59ca1ea3d/5c2e021f-c2d4-49e2-8c36-9a64f1f12001/782118f9-6c0b-4f5a-9c3b-1e5b8fc1f0ac"
-					(reference "R43")
+					(reference "R65")
 					(unit 1)
 				)
 				(path "/3f85abf4-0b95-4c4a-b7e9-06f59ca1ea3d/5c2e021f-c2d4-49e2-8c36-9a64f1f12001/beb9ceef-df3a-4e22-8974-012ce1407a41"
-					(reference "R44")
-					(unit 1)
-				)
+					(reference "R66")
+					(unit 1)
+				)

Commit message: pre robot updating references
Parts:
- renumbered C42 to C41, C43 to C42, R64 to R72, U21 to U22
Changed lines of the file:
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@@
 		(on_board yes)
 		(dnp no)
-		(property "Reference" "U21"
+		(property "Reference" "U22"
 			(at 97.79 87.63 0)
 			(effects
@@
 			(project "svea_powerboard_rev3"
 				(path "/3f85abf4-0b95-4c4a-b7e9-06f59ca1ea3d/5c2e021f-c2d4-49e2-8c36-9a64f1f12001/03241f80-3125-4f5b-a1a0-add76ba31aaa"
-					(reference "U21")
+					(reference "U22")
 					(unit 1)
 				)
 				(path "/3f85abf4-0b95-4c4a-b7e9-06f59ca1ea3d/5c2e021f-c2d4-49e2-8c36-9a64f1f12001/782118f9-6c0b-4f5a-9c3b-1e5b8fc1f0ac"
-					(reference "U22")
+					(reference "U23")
 					(unit 1)
 				)
 				(path "/3f85abf4-0b95-4c4a-b7e9-06f59ca1ea3d/5c2e021f-c2d4-49e2-8c36-9a64f1f12001/beb9ceef-df3a-4e22-8974-012ce1407a41"
-					(reference "U23")
+					(reference "U24")
 					(unit 1)
 				)
@@
 		(on_board yes)
 		(dnp no)
-		(property "Reference" "C43"
+		(property "Reference" "C42"
 			(at 143.51 96.52 90)
 			(effects
@@
 			(project "svea_powerboard_rev3"
 				(path "/3f85abf4-0b95-4c4a-b7e9-06f59ca1ea3d/5c2e021f-c2d4-49e2-8c36-9a64f1f12001/03241f80-3125-4f5b-a1a0-add76ba31aaa"
-					(reference "C43")
+					(reference "C42")
 					(unit 1)
 				)
 				(path "/3f85abf4-0b95-4c4a-b7e9-06f59ca1ea3d/5c2e021f-c2d4-49e2-8c36-9a64f1f12001/782118f9-6c0b-4f5a-9c3b-1e5b8fc1f0ac"
-					(reference "C45")
+					(reference "C44")
 					(unit 1)
 				)
 				(path "/3f85abf4-0b95-4c4a-b7e9-06f59ca1ea3d/5c2e021f-c2d4-49e2-8c36-9a64f1f12001/beb9ceef-df3a-4e22-8974-012ce1407a41"
-					(reference "C47")
+					(reference "C46")
 					(unit 1)
 				)
@@
 		(on_board yes)
 		(dnp no)
-		(property "Reference" "#PWR074"
+		(property "Reference" "#PWR079"
 			(at 139.7 106.68 0)
 			(effects
@@
 			(project "svea_powerboard_rev3"
 				(path "/3f85abf4-0b95-4c4a-b7e9-06f59ca1ea3d/5c2e021f-c2d4-49e2-8c36-9a64f1f12001/03241f80-3125-4f5b-a1a0-add76ba31aaa"
-					(reference "#PWR074")
+					(reference "#PWR079")
 					(unit 1)
 				)
 				(path "/3f85abf4-0b95-4c4a-b7e9-06f59ca1ea3d/5c2e021f-c2d4-49e2-8c36-9a64f1f12001/782118f9-6c0b-4f5a-9c3b-1e5b8fc1f0ac"
-					(reference "#PWR075")
+					(reference "#PWR080")
 					(unit 1)
 				)
 				(path "/3f85abf4-0b95-4c4a-b7e9-06f59ca1ea3d/5c2e021f-c2d4-49e2-8c36-9a64f1f12001/beb9ceef-df3a-4e22-8974-012ce1407a41"
-					(reference "#PWR076")
+					(reference "#PWR081")
 					(unit 1)
 				)
@@
 		(on_board yes)
 		(dnp no)
-		(property "Reference" "C42"
+		(property "Reference" "C41"
 			(at 132.08 96.52 90)
 			(effects
@@
 			(project "svea_powerboard_rev3"
 				(path "/3f85abf4-0b95-4c4a-b7e9-06f59ca1ea3d/5c2e021f-c2d4-49e2-8c36-9a64f1f12001/03241f80-3125-4f5b-a1a0-add76ba31aaa"
-					(reference "C42")
+					(reference "C41")
 					(unit 1)
 				)
 				(path "/3f85abf4-0b95-4c4a-b7e9-06f59ca1ea3d/5c2e021f-c2d4-49e2-8c36-9a64f1f12001/782118f9-6c0b-4f5a-9c3b-1e5b8fc1f0ac"
-					(reference "C44")
+					(reference "C43")
 					(unit 1)
 				)
 				(path "/3f85abf4-0b95-4c4a-b7e9-06f59ca1ea3d/5c2e021f-c2d4-49e2-8c36-9a64f1f12001/beb9ceef-df3a-4e22-8974-012ce1407a41"
-					(reference "C46")
+					(reference "C45")
 					(unit 1)
 				)
@@
 		(on_board yes)
 		(dnp no)
-		(property "Reference" "R64"
+		(property "Reference" "R72"
 			(at 162.56 93.218 0)
 			(effects
@@
 			(project "svea_powerboard_rev3"
 				(path "/3f85abf4-0b95-4c4a-b7e9-06f59ca1ea3d/5c2e021f-c2d4-49e2-8c36-9a64f1f12001/03241f80-3125-4f5b-a1a0-add76ba31aaa"
-					(reference "R64")
+					(reference "R72")
 					(unit 1)
 				)
 				(path "/3f85abf4-0b95-4c4a-b7e9-06f59ca1ea3d/5c2e021f-c2d4-49e2-8c36-9a64f1f12001/782118f9-6c0b-4f5a-9c3b-1e5b8fc1f0ac"
-					(reference "R65")
+					(reference "R73")
 					(unit 1)
 				)
 				(path "/3f85abf4-0b95-4c4a-b7e9-06f59ca1ea3d/5c2e021f-c2d4-49e2-8c36-9a64f1f12001/beb9ceef-df3a-4e22-8974-012ce1407a41"
-					(reference "R66")
-					(unit 1)
-				)
+					(reference "R74")
+					(unit 1)
+				)
