File: hardware/kicad/sheets/connectors/mt9700-efuse.kicad_sch (KiCad schematic)
At the start: 10 parts, among them U29 MT9700-N, U30 150uF

Commit message: various improvements
Parts:
- removed R101: 11.3kΩ, Resistor_SMD:R_0603_1608Metric, symbol 5v rail sm-easyedapro:0603WAF1132T5E
- gave numbers to parts that had none: 2
- renumbered C51 to C65, R98 to R78, R99 to R79, R100 to R80, U28 to U32, U29 to U33, U30 to U34
Connections:
- net SET: now reaches U33.3 (SET)
Other:
- note removed: "600mA"
Changed lines of the file:
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@@
 	(generator_version "9.0")
 	(paper "A4")
-	(text "600mA"
-		(exclude_from_sim no)
-		(at 151.13 90.17 0)
-		(effects
-			(font
-				(size 1.27 1.27)
-			)
-			(justify left bottom)
-		)
-	)
 	(junction
 		(at 69.85 76.2)
@@
 	)
 	(junction
-		(at 160.02 100.33)
-		(diameter 0)
-		(color 0 0 0 0)
-	)
-	(junction
 		(at 180.34 100.33)
 		(diameter 0)
@@
 	(wire
 		(pts
-			(xy 160.02 100.33) (xy 160.02 93.98)
-		)
-		(stroke
-			(width 0)
-			(type default)
-		)
-	)
-	(wire
-		(pts
 			(xy 194.31 76.2) (xy 227.33 76.2)
 		)
@@
 	(wire
 		(pts
-			(xy 160.02 83.82) (xy 160.02 81.28)
-		)
-		(stroke
-			(width 0)
-			(type default)
-		)
-	)
-	(wire
-		(pts
 			(xy 69.85 76.2) (xy 86.36 76.2)
 		)
@@
 			(width 0)
 			(type default)
+		)
+	)
+	(hierarchical_label "SET"
+		(shape input)
+		(at 160.02 81.28 0)
+		(effects
+			(font
+				(size 1.27 1.27)
+			)
+			(justify left)
 		)
 	)
@@
 		(on_board yes)
 		(dnp no)
-		(property "Reference" "#PWR092"
+		(property "Reference" "#PWR0110"
 			(at 160.02 102.87 0)
 			(effects
@@
 			(project "svea_powerboard_rev3"
 				(path "/3f85abf4-0b95-4c4a-b7e9-06f59ca1ea3d/5c2e021f-c2d4-49e2-8c36-9a64f1f12001/1d4a251e-4375-4aab-85e0-d11dfb5595c0"
-					(reference "#PWR092")
+					(reference "#PWR0110")
+					(unit 1)
+				)
+				(path "/3f85abf4-0b95-4c4a-b7e9-06f59ca1ea3d/5c2e021f-c2d4-49e2-8c36-9a64f1f12001/a553934f-48fa-4d71-a435-79ebd566d680"
+					(reference "#PWR0171")
 					(unit 1)
 				)
@@
 		(on_board yes)
 		(dnp no)
-		(property "Reference" "R98"
+		(property "Reference" "R78"
 			(at 106.68 101.6 0)
 			(effects
@@
 			(project "svea_powerboard_rev3"
 				(path "/3f85abf4-0b95-4c4a-b7e9-06f59ca1ea3d/5c2e021f-c2d4-49e2-8c36-9a64f1f12001/1d4a251e-4375-4aab-85e0-d11dfb5595c0"
-					(reference "R98")
+					(reference "R78")
+					(unit 1)
+				)
+				(path "/3f85abf4-0b95-4c4a-b7e9-06f59ca1ea3d/5c2e021f-c2d4-49e2-8c36-9a64f1f12001/a553934f-48fa-4d71-a435-79ebd566d680"
+					(reference "R189")
 					(unit 1)
 				)
@@
 		(on_board yes)
 		(dnp no)
-		(property "Reference" "U30"
+		(property "Reference" "U34"
 			(at 184.15 88.9 90)
 			(effects
@@
 			(project "svea_powerboard_rev3"
 				(path "/3f85abf4-0b95-4c4a-b7e9-06f59ca1ea3d/5c2e021f-c2d4-49e2-8c36-9a64f1f12001/1d4a251e-4375-4aab-85e0-d11dfb5595c0"
-					(reference "U30")
+					(reference "U34")
+					(unit 1)
+				)
+				(path "/3f85abf4-0b95-4c4a-b7e9-06f59ca1ea3d/5c2e021f-c2d4-49e2-8c36-9a64f1f12001/a553934f-48fa-4d71-a435-79ebd566d680"
+					(reference "U66")
 					(unit 1)
 				)
@@
 		(on_board yes)
 		(dnp no)
-		(property "Reference" "C?"
+		(property "Reference" "C63"
 			(at 73.66 88.9 90)
 			(effects
@@
 			(project "svea_powerboard_rev3"
 				(path "/3f85abf4-0b95-4c4a-b7e9-06f59ca1ea3d/5c2e021f-c2d4-49e2-8c36-9a64f1f12001/1d4a251e-4375-4aab-85e0-d11dfb5595c0"
-					(reference "C?")
+					(reference "C63")
+					(unit 1)
+				)
+				(path "/3f85abf4-0b95-4c4a-b7e9-06f59ca1ea3d/5c2e021f-c2d4-49e2-8c36-9a64f1f12001/a553934f-48fa-4d71-a435-79ebd566d680"
+					(reference "C97")
 					(unit 1)
 				)
@@
 		(on_board yes)
 		(dnp no)
-		(property "Reference" "#PWR088"
+		(property "Reference" "#PWR0109"
 			(at 116.84 125.73 0)
 			(effects
@@
 			(project "svea_powerboard_rev3"
 				(path "/3f85abf4-0b95-4c4a-b7e9-06f59ca1ea3d/5c2e021f-c2d4-49e2-8c36-9a64f1f12001/1d4a251e-4375-4aab-85e0-d11dfb5595c0"
-					(reference "#PWR088")
+					(reference "#PWR0109")
+					(unit 1)
+				)
+				(path "/3f85abf4-0b95-4c4a-b7e9-06f59ca1ea3d/5c2e021f-c2d4-49e2-8c36-9a64f1f12001/a553934f-48fa-4d71-a435-79ebd566d680"
+					(reference "#PWR0170")
 					(unit 1)
 				)
@@
 		(on_board yes)
 		(dnp no)
-		(property "Reference" "#PWR0136"
+		(property "Reference" "#PWR0108"
 			(at 78.74 105.41 0)
 			(effects
@@
 			(project "svea_powerboard_rev3"
 				(path "/3f85abf4-0b95-4c4a-b7e9-06f59ca1ea3d/5c2e021f-c2d4-49e2-8c36-9a64f1f12001/1d4a251e-4375-4aab-85e0-d11dfb5595c0"
-					(reference "#PWR0136")
+					(reference "#PWR0108")
+					(unit 1)
+				)
+				(path "/3f85abf4-0b95-4c4a-b7e9-06f59ca1ea3d/5c2e021f-c2d4-49e2-8c36-9a64f1f12001/a553934f-48fa-4d71-a435-79ebd566d680"
+					(reference "#PWR0169")
 					(unit 1)
 				)
@@
 		(on_board yes)
 		(dnp no)
-		(property "Reference" "U28"
+		(property "Reference" "U32"
 			(at 119.38 120.65 90)
 			(effects
@@
 			(project "svea_powerboard_rev3"
 				(path "/3f85abf4-0b95-4c4a-b7e9-06f59ca1ea3d/5c2e021f-c2d4-49e2-8c36-9a64f1f12001/1d4a251e-4375-4aab-85e0-d11dfb5595c0"
-					(reference "U28")
+					(reference "U32")
+					(unit 1)
+				)
+				(path "/3f85abf4-0b95-4c4a-b7e9-06f59ca1ea3d/5c2e021f-c2d4-49e2-8c36-9a64f1f12001/a553934f-48fa-4d71-a435-79ebd566d680"
+					(reference "U64")
 					(unit 1)
 				)
@@
 		(on_board yes)
 		(dnp no)
-		(property "Reference" "C51"
+		(property "Reference" "C65"
 			(at 198.12 88.9 90)
 			(effects
@@
 			(project "svea_powerboard_rev3"
 				(path "/3f85abf4-0b95-4c4a-b7e9-06f59ca1ea3d/5c2e021f-c2d4-49e2-8c36-9a64f1f12001/1d4a251e-4375-4aab-85e0-d11dfb5595c0"
-					(reference "C51")
+					(reference "C65")
+					(unit 1)
+				)
+				(path "/3f85abf4-0b95-4c4a-b7e9-06f59ca1ea3d/5c2e021f-c2d4-49e2-8c36-9a64f1f12001/a553934f-48fa-4d71-a435-79ebd566d680"
+					(reference "C99")
 					(unit 1)
 				)
@@
 		(on_board yes)
 		(dnp no)
-		(property "Reference" "R100"
+		(property "Reference" "R80"
 			(at 119.38 110.49 90)
 			(effects
@@
 			(project "svea_powerboard_rev3"
 				(path "/3f85abf4-0b95-4c4a-b7e9-06f59ca1ea3d/5c2e021f-c2d4-49e2-8c36-9a64f1f12001/1d4a251e-4375-4aab-85e0-d11dfb5595c0"
-					(reference "R100")
+					(reference "R80")
+					(unit 1)
+				)
+				(path "/3f85abf4-0b95-4c4a-b7e9-06f59ca1ea3d/5c2e021f-c2d4-49e2-8c36-9a64f1f12001/a553934f-48fa-4d71-a435-79ebd566d680"
+					(reference "R191")
 					(unit 1)
 				)
@@
 		(on_board yes)
 		(dnp no)
-		(property "Reference" "R99"
+		(property "Reference" "R79"
 			(at 119.38 83.82 90)
 			(effects
@@
 			(project "svea_powerboard_rev3"
 				(path "/3f85abf4-0b95-4c4a-b7e9-06f59ca1ea3d/5c2e021f-c2d4-49e2-8c36-9a64f1f12001/1d4a251e-4375-4aab-85e0-d11dfb5595c0"
-					(reference "R99")
+					(reference "R79")
+					(unit 1)
+				)
+				(path "/3f85abf4-0b95-4c4a-b7e9-06f59ca1ea3d/5c2e021f-c2d4-49e2-8c36-9a64f1f12001/a553934f-48fa-4d71-a435-79ebd566d680"
+					(reference "R190")
 					(unit 1)
 				)
@@
 		(on_board yes)
 		(dnp no)
-		(property "Reference" "U29"
+		(property "Reference" "U33"
 			(at 135.89 73.66 0)
 			(effects
@@
 			(project "svea_powerboard_rev3"
 				(path "/3f85abf4-0b95-4c4a-b7e9-06f59ca1ea3d/5c2e021f-c2d4-49e2-8c36-9a64f1f12001/1d4a251e-4375-4aab-85e0-d11dfb5595c0"
-					(reference "U29")
-					(unit 1)
-				)
-			)
-		)
-	)
-	(symbol
-		(lib_id "5v rail sm-easyedapro:0603WAF1132T5E")
-		(at 160.02 88.9 90)
-		(unit 1)
-		(exclude_from_sim no)
-		(in_bom yes)
-		(on_board yes)
-		(dnp no)
-		(property "Reference" "R101"
-			(at 162.56 88.9 90)
-			(effects
-				(font
-					(size 1.27 1.27)
-				)
-				(justify right top)
-			)
-		)
-		(property "Value" "11.3kΩ"
-			(at 162.56 91.44 90)
-			(effects
-				(font
-					(size 1.27 1.27)
-				)
-				(justify right top)
-			)
-		)
-		(property "Footprint" "Resistor_SMD:R_0603_1608Metric"
-			(at 160.02 88.9 0)
-			(effects
-				(font
-					(size 1.27 1.27)
-				)
-				(hide yes)
-			)
-		)
-		(property "Datasheet" "https://item.szlcsc.com/datasheet/0603WAF1132T5E/23587.html"
-			(at 160.02 88.9 0)
-			(effects
-				(font
-					(size 1.27 1.27)
-				)
-				(hide yes)
-			)
-		)
-		(property "Description" "Type:Thick Film Resistor Resistance:11.3kΩ Tolerance:±1% Tolerance:±1% Power(Watts):100mW Voltage-Supply(Max):75V Temperature Coefficient:±100ppm/°C Temperature Coefficient:±100ppm/°C Operating Temperature:-55°C~+155°C Operating Temperature:-55°C~+155°C"
-			(at 160.02 88.9 0)
-			(effects
-				(font
-					(size 1.27 1.27)
-				)
-				(hide yes)
-			)
-		)
-		(property "Manufacturer Part" "0603WAF1132T5E"
-			(at 160.02 88.9 0)
-			(effects
-				(font
-					(size 1.27 1.27)
-				)
-				(hide yes)
-			)
-		)
-		(property "Manufacturer" "UNI-ROYAL(厚声)"
-			(at 160.02 88.9 0)
-			(effects
-				(font
-					(size 1.27 1.27)
-				)
-				(hide yes)
-			)
-		)
-		(property "Supplier Part" "C22860"
-			(at 160.02 88.9 0)
-			(effects
-				(font
-					(size 1.27 1.27)
-				)
-				(hide yes)
-			)
-		)
-		(property "Supplier" "LCSC"
-			(at 160.02 88.9 0)
-			(effects
-				(font
-					(size 1.27 1.27)
-				)
-				(hide yes)
-			)
-		)
-		(property "LCSC Part Name" "11.3kΩ ±1% 100mW 厚膜电阻"
-			(at 160.02 88.9 0)
-			(effects
-				(font
-					(size 1.27 1.27)
-				)
-				(hide yes)
-			)
-		)
-		(pin "1"
-		)
-		(pin "2"
-		)
-		(instances
-			(project "svea_powerboard_rev3"
-				(path "/3f85abf4-0b95-4c4a-b7e9-06f59ca1ea3d/5c2e021f-c2d4-49e2-8c36-9a64f1f12001/1d4a251e-4375-4aab-85e0-d11dfb5595c0"
-					(reference "R101")
+					(reference "U33")
+					(unit 1)
+				)
+				(path "/3f85abf4-0b95-4c4a-b7e9-06f59ca1ea3d/5c2e021f-c2d4-49e2-8c36-9a64f1f12001/a553934f-48fa-4d71-a435-79ebd566d680"
+					(reference "U65")
 					(unit 1)
 				)
@@
 		(on_board yes)
 		(dnp no)
-		(property "Reference" "C?"
+		(property "Reference" "C64"
 			(at 90.17 88.9 90)
 			(effects
@@
 			(project "svea_powerboard_rev3"
 				(path "/3f85abf4-0b95-4c4a-b7e9-06f59ca1ea3d/5c2e021f-c2d4-49e2-8c36-9a64f1f12001/1d4a251e-4375-4aab-85e0-d11dfb5595c0"
-					(reference "C?")
-					(unit 1)
-				)
+					(reference "C64")
+					(unit 1)
+				)
+				(path "/3f85abf4-0b95-4c4a-b7e9-06f59ca1ea3d/5c2e021f-c2d4-49e2-8c36-9a64f1f12001/a553934f-48fa-4d71-a435-79ebd566d680"
+					(reference "C98")
+					(unit 1)
+				)

Commit message: various improvements
Parts:
- renumbered C63 to C70, C64 to C71, C65 to C72, R78 to R87, R79 to R88, R80 to R89
Changed lines of the file:
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@@
 		(on_board yes)
 		(dnp no)
-		(property "Reference" "#PWR0110"
+		(property "Reference" "#PWR0118"
 			(at 160.02 102.87 0)
 			(effects
@@
 			(project "svea_powerboard_rev3"
 				(path "/3f85abf4-0b95-4c4a-b7e9-06f59ca1ea3d/5c2e021f-c2d4-49e2-8c36-9a64f1f12001/1d4a251e-4375-4aab-85e0-d11dfb5595c0"
-					(reference "#PWR0110")
+					(reference "#PWR0118")
 					(unit 1)
 				)
 				(path "/3f85abf4-0b95-4c4a-b7e9-06f59ca1ea3d/5c2e021f-c2d4-49e2-8c36-9a64f1f12001/a553934f-48fa-4d71-a435-79ebd566d680"
-					(reference "#PWR0171")
+					(reference "#PWR0153")
 					(unit 1)
 				)
@@
 		(on_board yes)
 		(dnp no)
-		(property "Reference" "R78"
+		(property "Reference" "R87"
 			(at 106.68 101.6 0)
 			(effects
@@
 			(project "svea_powerboard_rev3"
 				(path "/3f85abf4-0b95-4c4a-b7e9-06f59ca1ea3d/5c2e021f-c2d4-49e2-8c36-9a64f1f12001/1d4a251e-4375-4aab-85e0-d11dfb5595c0"
-					(reference "R78")
+					(reference "R87")
 					(unit 1)
 				)
 				(path "/3f85abf4-0b95-4c4a-b7e9-06f59ca1ea3d/5c2e021f-c2d4-49e2-8c36-9a64f1f12001/a553934f-48fa-4d71-a435-79ebd566d680"
-					(reference "R189")
+					(reference "R110")
 					(unit 1)
 				)
@@
 				)
 				(path "/3f85abf4-0b95-4c4a-b7e9-06f59ca1ea3d/5c2e021f-c2d4-49e2-8c36-9a64f1f12001/a553934f-48fa-4d71-a435-79ebd566d680"
-					(reference "U66")
+					(reference "U47")
 					(unit 1)
 				)
@@
 		(on_board yes)
 		(dnp no)
-		(property "Reference" "C63"
+		(property "Reference" "C70"
 			(at 73.66 88.9 90)
 			(effects
@@
 			(project "svea_powerboard_rev3"
 				(path "/3f85abf4-0b95-4c4a-b7e9-06f59ca1ea3d/5c2e021f-c2d4-49e2-8c36-9a64f1f12001/1d4a251e-4375-4aab-85e0-d11dfb5595c0"
-					(reference "C63")
+					(reference "C70")
 					(unit 1)
 				)
 				(path "/3f85abf4-0b95-4c4a-b7e9-06f59ca1ea3d/5c2e021f-c2d4-49e2-8c36-9a64f1f12001/a553934f-48fa-4d71-a435-79ebd566d680"
-					(reference "C97")
+					(reference "C100")
 					(unit 1)
 				)
@@
 		(on_board yes)
 		(dnp no)
-		(property "Reference" "#PWR0109"
+		(property "Reference" "#PWR0117"
 			(at 116.84 125.73 0)
 			(effects
@@
 			(project "svea_powerboard_rev3"
 				(path "/3f85abf4-0b95-4c4a-b7e9-06f59ca1ea3d/5c2e021f-c2d4-49e2-8c36-9a64f1f12001/1d4a251e-4375-4aab-85e0-d11dfb5595c0"
-					(reference "#PWR0109")
+					(reference "#PWR0117")
 					(unit 1)
 				)
 				(path "/3f85abf4-0b95-4c4a-b7e9-06f59ca1ea3d/5c2e021f-c2d4-49e2-8c36-9a64f1f12001/a553934f-48fa-4d71-a435-79ebd566d680"
-					(reference "#PWR0170")
+					(reference "#PWR0152")
 					(unit 1)
 				)
@@
 		(on_board yes)
 		(dnp no)
-		(property "Reference" "#PWR0108"
+		(property "Reference" "#PWR0116"
 			(at 78.74 105.41 0)
 			(effects
@@
 			(project "svea_powerboard_rev3"
 				(path "/3f85abf4-0b95-4c4a-b7e9-06f59ca1ea3d/5c2e021f-c2d4-49e2-8c36-9a64f1f12001/1d4a251e-4375-4aab-85e0-d11dfb5595c0"
-					(reference "#PWR0108")
+					(reference "#PWR0116")
 					(unit 1)
 				)
 				(path "/3f85abf4-0b95-4c4a-b7e9-06f59ca1ea3d/5c2e021f-c2d4-49e2-8c36-9a64f1f12001/a553934f-48fa-4d71-a435-79ebd566d680"
-					(reference "#PWR0169")
+					(reference "#PWR0151")
 					(unit 1)
 				)
@@
 				)
 				(path "/3f85abf4-0b95-4c4a-b7e9-06f59ca1ea3d/5c2e021f-c2d4-49e2-8c36-9a64f1f12001/a553934f-48fa-4d71-a435-79ebd566d680"
-					(reference "U64")
+					(reference "U45")
 					(unit 1)
 				)
@@
 		(on_board yes)
 		(dnp no)
-		(property "Reference" "C65"
+		(property "Reference" "C72"
 			(at 198.12 88.9 90)
 			(effects
@@
 			(project "svea_powerboard_rev3"
 				(path "/3f85abf4-0b95-4c4a-b7e9-06f59ca1ea3d/5c2e021f-c2d4-49e2-8c36-9a64f1f12001/1d4a251e-4375-4aab-85e0-d11dfb5595c0"
-					(reference "C65")
+					(reference "C72")
 					(unit 1)
 				)
 				(path "/3f85abf4-0b95-4c4a-b7e9-06f59ca1ea3d/5c2e021f-c2d4-49e2-8c36-9a64f1f12001/a553934f-48fa-4d71-a435-79ebd566d680"
-					(reference "C99")
+					(reference "C102")
 					(unit 1)
 				)
@@
 		(on_board yes)
 		(dnp no)
-		(property "Reference" "R80"
+		(property "Reference" "R89"
 			(at 119.38 110.49 90)
 			(effects
@@
 			(project "svea_powerboard_rev3"
 				(path "/3f85abf4-0b95-4c4a-b7e9-06f59ca1ea3d/5c2e021f-c2d4-49e2-8c36-9a64f1f12001/1d4a251e-4375-4aab-85e0-d11dfb5595c0"
-					(reference "R80")
+					(reference "R89")
 					(unit 1)
 				)
 				(path "/3f85abf4-0b95-4c4a-b7e9-06f59ca1ea3d/5c2e021f-c2d4-49e2-8c36-9a64f1f12001/a553934f-48fa-4d71-a435-79ebd566d680"
-					(reference "R191")
+					(reference "R112")
 					(unit 1)
 				)
@@
 		(on_board yes)
 		(dnp no)
-		(property "Reference" "R79"
+		(property "Reference" "R88"
 			(at 119.38 83.82 90)
 			(effects
@@
 			(project "svea_powerboard_rev3"
 				(path "/3f85abf4-0b95-4c4a-b7e9-06f59ca1ea3d/5c2e021f-c2d4-49e2-8c36-9a64f1f12001/1d4a251e-4375-4aab-85e0-d11dfb5595c0"
-					(reference "R79")
+					(reference "R88")
 					(unit 1)
 				)
 				(path "/3f85abf4-0b95-4c4a-b7e9-06f59ca1ea3d/5c2e021f-c2d4-49e2-8c36-9a64f1f12001/a553934f-48fa-4d71-a435-79ebd566d680"
-					(reference "R190")
+					(reference "R111")
 					(unit 1)
 				)
@@
 				)
 				(path "/3f85abf4-0b95-4c4a-b7e9-06f59ca1ea3d/5c2e021f-c2d4-49e2-8c36-9a64f1f12001/a553934f-48fa-4d71-a435-79ebd566d680"
-					(reference "U65")
+					(reference "U46")
 					(unit 1)
 				)
@@
 		(on_board yes)
 		(dnp no)
-		(property "Reference" "C64"
+		(property "Reference" "C71"
 			(at 90.17 88.9 90)
 			(effects
@@
 			(project "svea_powerboard_rev3"
 				(path "/3f85abf4-0b95-4c4a-b7e9-06f59ca1ea3d/5c2e021f-c2d4-49e2-8c36-9a64f1f12001/1d4a251e-4375-4aab-85e0-d11dfb5595c0"
-					(reference "C64")
+					(reference "C71")
 					(unit 1)
 				)
 				(path "/3f85abf4-0b95-4c4a-b7e9-06f59ca1ea3d/5c2e021f-c2d4-49e2-8c36-9a64f1f12001/a553934f-48fa-4d71-a435-79ebd566d680"
-					(reference "C98")
-					(unit 1)
-				)
+					(reference "C101")
+					(unit 1)
+				)

Commit message: current sensing on the servos and cleaning up empty sheets
Parts:
- renumbered C70 to C75, C71 to C76, C72 to C77, R87 to R85, R88 to R86, R89 to R87, U32 to U35, U33 to U36, U34 to U37
Changed lines of the file:
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@@
 		(on_board yes)
 		(dnp no)
-		(property "Reference" "#PWR0118"
+		(property "Reference" "#PWR0120"
 			(at 160.02 102.87 0)
 			(effects
@@
 			(project "svea_powerboard_rev3"
 				(path "/3f85abf4-0b95-4c4a-b7e9-06f59ca1ea3d/5c2e021f-c2d4-49e2-8c36-9a64f1f12001/1d4a251e-4375-4aab-85e0-d11dfb5595c0"
-					(reference "#PWR0118")
+					(reference "#PWR0120")
 					(unit 1)
 				)
 				(path "/3f85abf4-0b95-4c4a-b7e9-06f59ca1ea3d/5c2e021f-c2d4-49e2-8c36-9a64f1f12001/a553934f-48fa-4d71-a435-79ebd566d680"
-					(reference "#PWR0153")
+					(reference "#PWR0155")
 					(unit 1)
 				)
@@
 		(on_board yes)
 		(dnp no)
-		(property "Reference" "R87"
+		(property "Reference" "R85"
 			(at 106.68 101.6 0)
 			(effects
@@
 			(project "svea_powerboard_rev3"
 				(path "/3f85abf4-0b95-4c4a-b7e9-06f59ca1ea3d/5c2e021f-c2d4-49e2-8c36-9a64f1f12001/1d4a251e-4375-4aab-85e0-d11dfb5595c0"
-					(reference "R87")
+					(reference "R85")
 					(unit 1)
 				)
 				(path "/3f85abf4-0b95-4c4a-b7e9-06f59ca1ea3d/5c2e021f-c2d4-49e2-8c36-9a64f1f12001/a553934f-48fa-4d71-a435-79ebd566d680"
-					(reference "R110")
+					(reference "R107")
 					(unit 1)
 				)
@@
 		(on_board yes)
 		(dnp no)
-		(property "Reference" "U34"
+		(property "Reference" "U37"
 			(at 184.15 88.9 90)
 			(effects
@@
 			(project "svea_powerboard_rev3"
 				(path "/3f85abf4-0b95-4c4a-b7e9-06f59ca1ea3d/5c2e021f-c2d4-49e2-8c36-9a64f1f12001/1d4a251e-4375-4aab-85e0-d11dfb5595c0"
-					(reference "U34")
+					(reference "U37")
 					(unit 1)
 				)
 				(path "/3f85abf4-0b95-4c4a-b7e9-06f59ca1ea3d/5c2e021f-c2d4-49e2-8c36-9a64f1f12001/a553934f-48fa-4d71-a435-79ebd566d680"
-					(reference "U47")
+					(reference "U50")
 					(unit 1)
 				)
@@
 		(on_board yes)
 		(dnp no)
-		(property "Reference" "C70"
+		(property "Reference" "C75"
 			(at 73.66 88.9 90)
 			(effects
@@
 			(project "svea_powerboard_rev3"
 				(path "/3f85abf4-0b95-4c4a-b7e9-06f59ca1ea3d/5c2e021f-c2d4-49e2-8c36-9a64f1f12001/1d4a251e-4375-4aab-85e0-d11dfb5595c0"
-					(reference "C70")
+					(reference "C75")
 					(unit 1)
 				)
 				(path "/3f85abf4-0b95-4c4a-b7e9-06f59ca1ea3d/5c2e021f-c2d4-49e2-8c36-9a64f1f12001/a553934f-48fa-4d71-a435-79ebd566d680"
-					(reference "C100")
+					(reference "C105")
 					(unit 1)
 				)
@@
 		(on_board yes)
 		(dnp no)
-		(property "Reference" "#PWR0117"
+		(property "Reference" "#PWR0119"
 			(at 116.84 125.73 0)
 			(effects
@@
 			(project "svea_powerboard_rev3"
 				(path "/3f85abf4-0b95-4c4a-b7e9-06f59ca1ea3d/5c2e021f-c2d4-49e2-8c36-9a64f1f12001/1d4a251e-4375-4aab-85e0-d11dfb5595c0"
-					(reference "#PWR0117")
+					(reference "#PWR0119")
 					(unit 1)
 				)
 				(path "/3f85abf4-0b95-4c4a-b7e9-06f59ca1ea3d/5c2e021f-c2d4-49e2-8c36-9a64f1f12001/a553934f-48fa-4d71-a435-79ebd566d680"
-					(reference "#PWR0152")
+					(reference "#PWR0154")
 					(unit 1)
 				)
@@
 		(on_board yes)
 		(dnp no)
-		(property "Reference" "#PWR0116"
+		(property "Reference" "#PWR0118"
 			(at 78.74 105.41 0)
 			(effects
@@
 			(project "svea_powerboard_rev3"
 				(path "/3f85abf4-0b95-4c4a-b7e9-06f59ca1ea3d/5c2e021f-c2d4-49e2-8c36-9a64f1f12001/1d4a251e-4375-4aab-85e0-d11dfb5595c0"
-					(reference "#PWR0116")
+					(reference "#PWR0118")
 					(unit 1)
 				)
 				(path "/3f85abf4-0b95-4c4a-b7e9-06f59ca1ea3d/5c2e021f-c2d4-49e2-8c36-9a64f1f12001/a553934f-48fa-4d71-a435-79ebd566d680"
-					(reference "#PWR0151")
+					(reference "#PWR0153")
 					(unit 1)
 				)
@@
 		(on_board yes)
 		(dnp no)
-		(property "Reference" "U32"
+		(property "Reference" "U35"
 			(at 119.38 120.65 90)
 			(effects
@@
 			(project "svea_powerboard_rev3"
 				(path "/3f85abf4-0b95-4c4a-b7e9-06f59ca1ea3d/5c2e021f-c2d4-49e2-8c36-9a64f1f12001/1d4a251e-4375-4aab-85e0-d11dfb5595c0"
-					(reference "U32")
+					(reference "U35")
 					(unit 1)
 				)
 				(path "/3f85abf4-0b95-4c4a-b7e9-06f59ca1ea3d/5c2e021f-c2d4-49e2-8c36-9a64f1f12001/a553934f-48fa-4d71-a435-79ebd566d680"
-					(reference "U45")
+					(reference "U48")
 					(unit 1)
 				)
@@
 		(on_board yes)
 		(dnp no)
-		(property "Reference" "C72"
+		(property "Reference" "C77"
 			(at 198.12 88.9 90)
 			(effects
@@
 			(project "svea_powerboard_rev3"
 				(path "/3f85abf4-0b95-4c4a-b7e9-06f59ca1ea3d/5c2e021f-c2d4-49e2-8c36-9a64f1f12001/1d4a251e-4375-4aab-85e0-d11dfb5595c0"
-					(reference "C72")
+					(reference "C77")
 					(unit 1)
 				)
 				(path "/3f85abf4-0b95-4c4a-b7e9-06f59ca1ea3d/5c2e021f-c2d4-49e2-8c36-9a64f1f12001/a553934f-48fa-4d71-a435-79ebd566d680"
-					(reference "C102")
+					(reference "C107")
 					(unit 1)
 				)
@@
 		(on_board yes)
 		(dnp no)
-		(property "Reference" "R89"
+		(property "Reference" "R87"
 			(at 119.38 110.49 90)
 			(effects
@@
 			(project "svea_powerboard_rev3"
 				(path "/3f85abf4-0b95-4c4a-b7e9-06f59ca1ea3d/5c2e021f-c2d4-49e2-8c36-9a64f1f12001/1d4a251e-4375-4aab-85e0-d11dfb5595c0"
-					(reference "R89")
+					(reference "R87")
 					(unit 1)
 				)
 				(path "/3f85abf4-0b95-4c4a-b7e9-06f59ca1ea3d/5c2e021f-c2d4-49e2-8c36-9a64f1f12001/a553934f-48fa-4d71-a435-79ebd566d680"
-					(reference "R112")
+					(reference "R109")
 					(unit 1)
 				)
@@
 		(on_board yes)
 		(dnp no)
-		(property "Reference" "R88"
+		(property "Reference" "R86"
 			(at 119.38 83.82 90)
 			(effects
@@
 			(project "svea_powerboard_rev3"
 				(path "/3f85abf4-0b95-4c4a-b7e9-06f59ca1ea3d/5c2e021f-c2d4-49e2-8c36-9a64f1f12001/1d4a251e-4375-4aab-85e0-d11dfb5595c0"
-					(reference "R88")
+					(reference "R86")
 					(unit 1)
 				)
 				(path "/3f85abf4-0b95-4c4a-b7e9-06f59ca1ea3d/5c2e021f-c2d4-49e2-8c36-9a64f1f12001/a553934f-48fa-4d71-a435-79ebd566d680"
-					(reference "R111")
+					(reference "R108")
 					(unit 1)
 				)
@@
 		(on_board yes)
 		(dnp no)
-		(property "Reference" "U33"
+		(property "Reference" "U36"
 			(at 135.89 73.66 0)
 			(effects
@@
 			(project "svea_powerboard_rev3"
 				(path "/3f85abf4-0b95-4c4a-b7e9-06f59ca1ea3d/5c2e021f-c2d4-49e2-8c36-9a64f1f12001/1d4a251e-4375-4aab-85e0-d11dfb5595c0"
-					(reference "U33")
+					(reference "U36")
 					(unit 1)
 				)
 				(path "/3f85abf4-0b95-4c4a-b7e9-06f59ca1ea3d/5c2e021f-c2d4-49e2-8c36-9a64f1f12001/a553934f-48fa-4d71-a435-79ebd566d680"
-					(reference "U46")
+					(reference "U49")
 					(unit 1)
 				)
@@
 		(on_board yes)
 		(dnp no)
-		(property "Reference" "C71"
+		(property "Reference" "C76"
 			(at 90.17 88.9 90)
 			(effects
@@
 			(project "svea_powerboard_rev3"
 				(path "/3f85abf4-0b95-4c4a-b7e9-06f59ca1ea3d/5c2e021f-c2d4-49e2-8c36-9a64f1f12001/1d4a251e-4375-4aab-85e0-d11dfb5595c0"
-					(reference "C71")
+					(reference "C76")
 					(unit 1)
 				)
 				(path "/3f85abf4-0b95-4c4a-b7e9-06f59ca1ea3d/5c2e021f-c2d4-49e2-8c36-9a64f1f12001/a553934f-48fa-4d71-a435-79ebd566d680"
-					(reference "C101")
-					(unit 1)
-				)
+					(reference "C106")
+					(unit 1)
+				)
