File: hardware/kicad/sheets/connectors/mt9700-efuse.kicad_sch (KiCad schematic)
At the start: 9 parts, among them U36 MT9700-N, U37 150uF

Commit message: new references
Parts:
- renumbered C75 to C77, C76 to C78, C77 to C79, R85 to R108, R86 to R109, R87 to R110, U35 to U41, U36 to U42, U37 to U43
Changed lines of the file:
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@@
 		(on_board yes)
 		(dnp no)
-		(property "Reference" "#PWR0120"
+		(property "Reference" "#PWR0136"
 			(at 160.02 102.87 0)
 			(effects
@@
 			(project "svea_powerboard_rev3"
 				(path "/3f85abf4-0b95-4c4a-b7e9-06f59ca1ea3d/5c2e021f-c2d4-49e2-8c36-9a64f1f12001/1d4a251e-4375-4aab-85e0-d11dfb5595c0"
-					(reference "#PWR0120")
+					(reference "#PWR0136")
 					(unit 1)
 				)
 				(path "/3f85abf4-0b95-4c4a-b7e9-06f59ca1ea3d/5c2e021f-c2d4-49e2-8c36-9a64f1f12001/a553934f-48fa-4d71-a435-79ebd566d680"
-					(reference "#PWR0155")
+					(reference "#PWR0171")
 					(unit 1)
 				)
@@
 		(on_board yes)
 		(dnp no)
-		(property "Reference" "R85"
+		(property "Reference" "R108"
 			(at 106.68 101.6 0)
 			(effects
@@
 			(project "svea_powerboard_rev3"
 				(path "/3f85abf4-0b95-4c4a-b7e9-06f59ca1ea3d/5c2e021f-c2d4-49e2-8c36-9a64f1f12001/1d4a251e-4375-4aab-85e0-d11dfb5595c0"
-					(reference "R85")
+					(reference "R108")
 					(unit 1)
 				)
 				(path "/3f85abf4-0b95-4c4a-b7e9-06f59ca1ea3d/5c2e021f-c2d4-49e2-8c36-9a64f1f12001/a553934f-48fa-4d71-a435-79ebd566d680"
-					(reference "R107")
+					(reference "R130")
 					(unit 1)
 				)
@@
 		(on_board yes)
 		(dnp no)
-		(property "Reference" "U37"
+		(property "Reference" "U43"
 			(at 184.15 88.9 90)
 			(effects
@@
 			(project "svea_powerboard_rev3"
 				(path "/3f85abf4-0b95-4c4a-b7e9-06f59ca1ea3d/5c2e021f-c2d4-49e2-8c36-9a64f1f12001/1d4a251e-4375-4aab-85e0-d11dfb5595c0"
-					(reference "U37")
+					(reference "U43")
 					(unit 1)
 				)
 				(path "/3f85abf4-0b95-4c4a-b7e9-06f59ca1ea3d/5c2e021f-c2d4-49e2-8c36-9a64f1f12001/a553934f-48fa-4d71-a435-79ebd566d680"
-					(reference "U50")
+					(reference "U56")
 					(unit 1)
 				)
@@
 		(on_board yes)
 		(dnp no)
-		(property "Reference" "C75"
+		(property "Reference" "C77"
 			(at 73.66 88.9 90)
 			(effects
@@
 			(project "svea_powerboard_rev3"
 				(path "/3f85abf4-0b95-4c4a-b7e9-06f59ca1ea3d/5c2e021f-c2d4-49e2-8c36-9a64f1f12001/1d4a251e-4375-4aab-85e0-d11dfb5595c0"
-					(reference "C75")
+					(reference "C77")
 					(unit 1)
 				)
 				(path "/3f85abf4-0b95-4c4a-b7e9-06f59ca1ea3d/5c2e021f-c2d4-49e2-8c36-9a64f1f12001/a553934f-48fa-4d71-a435-79ebd566d680"
-					(reference "C105")
+					(reference "C107")
 					(unit 1)
 				)
@@
 		(on_board yes)
 		(dnp no)
-		(property "Reference" "#PWR0119"
+		(property "Reference" "#PWR0135"
 			(at 116.84 125.73 0)
 			(effects
@@
 			(project "svea_powerboard_rev3"
 				(path "/3f85abf4-0b95-4c4a-b7e9-06f59ca1ea3d/5c2e021f-c2d4-49e2-8c36-9a64f1f12001/1d4a251e-4375-4aab-85e0-d11dfb5595c0"
-					(reference "#PWR0119")
+					(reference "#PWR0135")
 					(unit 1)
 				)
 				(path "/3f85abf4-0b95-4c4a-b7e9-06f59ca1ea3d/5c2e021f-c2d4-49e2-8c36-9a64f1f12001/a553934f-48fa-4d71-a435-79ebd566d680"
-					(reference "#PWR0154")
+					(reference "#PWR0170")
 					(unit 1)
 				)
@@
 		(on_board yes)
 		(dnp no)
-		(property "Reference" "#PWR0118"
+		(property "Reference" "#PWR0134"
 			(at 78.74 105.41 0)
 			(effects
@@
 			(project "svea_powerboard_rev3"
 				(path "/3f85abf4-0b95-4c4a-b7e9-06f59ca1ea3d/5c2e021f-c2d4-49e2-8c36-9a64f1f12001/1d4a251e-4375-4aab-85e0-d11dfb5595c0"
-					(reference "#PWR0118")
+					(reference "#PWR0134")
 					(unit 1)
 				)
 				(path "/3f85abf4-0b95-4c4a-b7e9-06f59ca1ea3d/5c2e021f-c2d4-49e2-8c36-9a64f1f12001/a553934f-48fa-4d71-a435-79ebd566d680"
-					(reference "#PWR0153")
+					(reference "#PWR0169")
 					(unit 1)
 				)
@@
 		(on_board yes)
 		(dnp no)
-		(property "Reference" "U35"
+		(property "Reference" "U41"
 			(at 119.38 120.65 90)
 			(effects
@@
 			(project "svea_powerboard_rev3"
 				(path "/3f85abf4-0b95-4c4a-b7e9-06f59ca1ea3d/5c2e021f-c2d4-49e2-8c36-9a64f1f12001/1d4a251e-4375-4aab-85e0-d11dfb5595c0"
-					(reference "U35")
+					(reference "U41")
 					(unit 1)
 				)
 				(path "/3f85abf4-0b95-4c4a-b7e9-06f59ca1ea3d/5c2e021f-c2d4-49e2-8c36-9a64f1f12001/a553934f-48fa-4d71-a435-79ebd566d680"
-					(reference "U48")
+					(reference "U54")
 					(unit 1)
 				)
@@
 		(on_board yes)
 		(dnp no)
-		(property "Reference" "C77"
+		(property "Reference" "C79"
 			(at 198.12 88.9 90)
 			(effects
@@
 			(project "svea_powerboard_rev3"
 				(path "/3f85abf4-0b95-4c4a-b7e9-06f59ca1ea3d/5c2e021f-c2d4-49e2-8c36-9a64f1f12001/1d4a251e-4375-4aab-85e0-d11dfb5595c0"
-					(reference "C77")
+					(reference "C79")
 					(unit 1)
 				)
 				(path "/3f85abf4-0b95-4c4a-b7e9-06f59ca1ea3d/5c2e021f-c2d4-49e2-8c36-9a64f1f12001/a553934f-48fa-4d71-a435-79ebd566d680"
-					(reference "C107")
+					(reference "C109")
 					(unit 1)
 				)
@@
 		(on_board yes)
 		(dnp no)
-		(property "Reference" "R87"
+		(property "Reference" "R110"
 			(at 119.38 110.49 90)
 			(effects
@@
 			(project "svea_powerboard_rev3"
 				(path "/3f85abf4-0b95-4c4a-b7e9-06f59ca1ea3d/5c2e021f-c2d4-49e2-8c36-9a64f1f12001/1d4a251e-4375-4aab-85e0-d11dfb5595c0"
-					(reference "R87")
+					(reference "R110")
 					(unit 1)
 				)
 				(path "/3f85abf4-0b95-4c4a-b7e9-06f59ca1ea3d/5c2e021f-c2d4-49e2-8c36-9a64f1f12001/a553934f-48fa-4d71-a435-79ebd566d680"
-					(reference "R109")
+					(reference "R132")
 					(unit 1)
 				)
@@
 		(on_board yes)
 		(dnp no)
-		(property "Reference" "R86"
+		(property "Reference" "R109"
 			(at 119.38 83.82 90)
 			(effects
@@
 			(project "svea_powerboard_rev3"
 				(path "/3f85abf4-0b95-4c4a-b7e9-06f59ca1ea3d/5c2e021f-c2d4-49e2-8c36-9a64f1f12001/1d4a251e-4375-4aab-85e0-d11dfb5595c0"
-					(reference "R86")
+					(reference "R109")
 					(unit 1)
 				)
 				(path "/3f85abf4-0b95-4c4a-b7e9-06f59ca1ea3d/5c2e021f-c2d4-49e2-8c36-9a64f1f12001/a553934f-48fa-4d71-a435-79ebd566d680"
-					(reference "R108")
+					(reference "R131")
 					(unit 1)
 				)
@@
 		(on_board yes)
 		(dnp no)
-		(property "Reference" "U36"
+		(property "Reference" "U42"
 			(at 135.89 73.66 0)
 			(effects
@@
 			(project "svea_powerboard_rev3"
 				(path "/3f85abf4-0b95-4c4a-b7e9-06f59ca1ea3d/5c2e021f-c2d4-49e2-8c36-9a64f1f12001/1d4a251e-4375-4aab-85e0-d11dfb5595c0"
-					(reference "U36")
+					(reference "U42")
 					(unit 1)
 				)
 				(path "/3f85abf4-0b95-4c4a-b7e9-06f59ca1ea3d/5c2e021f-c2d4-49e2-8c36-9a64f1f12001/a553934f-48fa-4d71-a435-79ebd566d680"
-					(reference "U49")
+					(reference "U55")
 					(unit 1)
 				)
@@
 		(on_board yes)
 		(dnp no)
-		(property "Reference" "C76"
+		(property "Reference" "C78"
 			(at 90.17 88.9 90)
 			(effects
@@
 			(project "svea_powerboard_rev3"
 				(path "/3f85abf4-0b95-4c4a-b7e9-06f59ca1ea3d/5c2e021f-c2d4-49e2-8c36-9a64f1f12001/1d4a251e-4375-4aab-85e0-d11dfb5595c0"
-					(reference "C76")
+					(reference "C78")
 					(unit 1)
 				)
 				(path "/3f85abf4-0b95-4c4a-b7e9-06f59ca1ea3d/5c2e021f-c2d4-49e2-8c36-9a64f1f12001/a553934f-48fa-4d71-a435-79ebd566d680"
-					(reference "C106")
-					(unit 1)
-				)
+					(reference "C108")
+					(unit 1)
+				)

Commit message: pre robot updating references
Parts:
- renumbered C77 to C75, C78 to C76, C79 to C77, R108 to R115, R109 to R116, R110 to R117
Changed lines of the file:
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@@
 		(on_board yes)
 		(dnp no)
-		(property "Reference" "#PWR0136"
+		(property "Reference" "#PWR0123"
 			(at 160.02 102.87 0)
 			(effects
@@
 			(project "svea_powerboard_rev3"
 				(path "/3f85abf4-0b95-4c4a-b7e9-06f59ca1ea3d/5c2e021f-c2d4-49e2-8c36-9a64f1f12001/1d4a251e-4375-4aab-85e0-d11dfb5595c0"
-					(reference "#PWR0136")
+					(reference "#PWR0123")
 					(unit 1)
 				)
 				(path "/3f85abf4-0b95-4c4a-b7e9-06f59ca1ea3d/5c2e021f-c2d4-49e2-8c36-9a64f1f12001/a553934f-48fa-4d71-a435-79ebd566d680"
-					(reference "#PWR0171")
+					(reference "#PWR0158")
 					(unit 1)
 				)
@@
 		(on_board yes)
 		(dnp no)
-		(property "Reference" "R108"
+		(property "Reference" "R115"
 			(at 106.68 101.6 0)
 			(effects
@@
 			(project "svea_powerboard_rev3"
 				(path "/3f85abf4-0b95-4c4a-b7e9-06f59ca1ea3d/5c2e021f-c2d4-49e2-8c36-9a64f1f12001/1d4a251e-4375-4aab-85e0-d11dfb5595c0"
-					(reference "R108")
+					(reference "R115")
 					(unit 1)
 				)
 				(path "/3f85abf4-0b95-4c4a-b7e9-06f59ca1ea3d/5c2e021f-c2d4-49e2-8c36-9a64f1f12001/a553934f-48fa-4d71-a435-79ebd566d680"
-					(reference "R130")
+					(reference "R137")
 					(unit 1)
 				)
@@
 		(on_board yes)
 		(dnp no)
-		(property "Reference" "C77"
+		(property "Reference" "C75"
 			(at 73.66 88.9 90)
 			(effects
@@
 			(project "svea_powerboard_rev3"
 				(path "/3f85abf4-0b95-4c4a-b7e9-06f59ca1ea3d/5c2e021f-c2d4-49e2-8c36-9a64f1f12001/1d4a251e-4375-4aab-85e0-d11dfb5595c0"
-					(reference "C77")
+					(reference "C75")
 					(unit 1)
 				)
 				(path "/3f85abf4-0b95-4c4a-b7e9-06f59ca1ea3d/5c2e021f-c2d4-49e2-8c36-9a64f1f12001/a553934f-48fa-4d71-a435-79ebd566d680"
-					(reference "C107")
+					(reference "C105")
 					(unit 1)
 				)
@@
 		(on_board yes)
 		(dnp no)
-		(property "Reference" "#PWR0135"
+		(property "Reference" "#PWR0122"
 			(at 116.84 125.73 0)
 			(effects
@@
 			(project "svea_powerboard_rev3"
 				(path "/3f85abf4-0b95-4c4a-b7e9-06f59ca1ea3d/5c2e021f-c2d4-49e2-8c36-9a64f1f12001/1d4a251e-4375-4aab-85e0-d11dfb5595c0"
-					(reference "#PWR0135")
+					(reference "#PWR0122")
 					(unit 1)
 				)
 				(path "/3f85abf4-0b95-4c4a-b7e9-06f59ca1ea3d/5c2e021f-c2d4-49e2-8c36-9a64f1f12001/a553934f-48fa-4d71-a435-79ebd566d680"
-					(reference "#PWR0170")
+					(reference "#PWR0157")
 					(unit 1)
 				)
@@
 		(on_board yes)
 		(dnp no)
-		(property "Reference" "#PWR0134"
+		(property "Reference" "#PWR0121"
 			(at 78.74 105.41 0)
 			(effects
@@
 			(project "svea_powerboard_rev3"
 				(path "/3f85abf4-0b95-4c4a-b7e9-06f59ca1ea3d/5c2e021f-c2d4-49e2-8c36-9a64f1f12001/1d4a251e-4375-4aab-85e0-d11dfb5595c0"
-					(reference "#PWR0134")
+					(reference "#PWR0121")
 					(unit 1)
 				)
 				(path "/3f85abf4-0b95-4c4a-b7e9-06f59ca1ea3d/5c2e021f-c2d4-49e2-8c36-9a64f1f12001/a553934f-48fa-4d71-a435-79ebd566d680"
-					(reference "#PWR0169")
+					(reference "#PWR0156")
 					(unit 1)
 				)
@@
 		(on_board yes)
 		(dnp no)
-		(property "Reference" "C79"
+		(property "Reference" "C77"
 			(at 198.12 88.9 90)
 			(effects
@@
 			(project "svea_powerboard_rev3"
 				(path "/3f85abf4-0b95-4c4a-b7e9-06f59ca1ea3d/5c2e021f-c2d4-49e2-8c36-9a64f1f12001/1d4a251e-4375-4aab-85e0-d11dfb5595c0"
-					(reference "C79")
+					(reference "C77")
 					(unit 1)
 				)
 				(path "/3f85abf4-0b95-4c4a-b7e9-06f59ca1ea3d/5c2e021f-c2d4-49e2-8c36-9a64f1f12001/a553934f-48fa-4d71-a435-79ebd566d680"
-					(reference "C109")
+					(reference "C107")
 					(unit 1)
 				)
@@
 		(on_board yes)
 		(dnp no)
-		(property "Reference" "R110"
+		(property "Reference" "R117"
 			(at 119.38 110.49 90)
 			(effects
@@
 			(project "svea_powerboard_rev3"
 				(path "/3f85abf4-0b95-4c4a-b7e9-06f59ca1ea3d/5c2e021f-c2d4-49e2-8c36-9a64f1f12001/1d4a251e-4375-4aab-85e0-d11dfb5595c0"
-					(reference "R110")
+					(reference "R117")
 					(unit 1)
 				)
 				(path "/3f85abf4-0b95-4c4a-b7e9-06f59ca1ea3d/5c2e021f-c2d4-49e2-8c36-9a64f1f12001/a553934f-48fa-4d71-a435-79ebd566d680"
-					(reference "R132")
+					(reference "R139")
 					(unit 1)
 				)
@@
 		(on_board yes)
 		(dnp no)
-		(property "Reference" "R109"
+		(property "Reference" "R116"
 			(at 119.38 83.82 90)
 			(effects
@@
 			(project "svea_powerboard_rev3"
 				(path "/3f85abf4-0b95-4c4a-b7e9-06f59ca1ea3d/5c2e021f-c2d4-49e2-8c36-9a64f1f12001/1d4a251e-4375-4aab-85e0-d11dfb5595c0"
-					(reference "R109")
+					(reference "R116")
 					(unit 1)
 				)
 				(path "/3f85abf4-0b95-4c4a-b7e9-06f59ca1ea3d/5c2e021f-c2d4-49e2-8c36-9a64f1f12001/a553934f-48fa-4d71-a435-79ebd566d680"
-					(reference "R131")
+					(reference "R138")
 					(unit 1)
 				)
@@
 		(on_board yes)
 		(dnp no)
-		(property "Reference" "C78"
+		(property "Reference" "C76"
 			(at 90.17 88.9 90)
 			(effects
@@
 			(project "svea_powerboard_rev3"
 				(path "/3f85abf4-0b95-4c4a-b7e9-06f59ca1ea3d/5c2e021f-c2d4-49e2-8c36-9a64f1f12001/1d4a251e-4375-4aab-85e0-d11dfb5595c0"
-					(reference "C78")
+					(reference "C76")
 					(unit 1)
 				)
 				(path "/3f85abf4-0b95-4c4a-b7e9-06f59ca1ea3d/5c2e021f-c2d4-49e2-8c36-9a64f1f12001/a553934f-48fa-4d71-a435-79ebd566d680"
-					(reference "C108")
-					(unit 1)
-				)
+					(reference "C106")
+					(unit 1)
+				)
