File: hardware/kicad/sheets/analog/11_Frontend.kicad_sch (KiCad schematic)
At the start: 12 parts, among them SW2 DSHP04TS-S

Commit message: resheeted bms and fixed links for the 12v buck
Parts:
- renumbered R93 to R130, R94 to R131, R95 to R132, R96 to R133, R97 to R134, R99 to R135, SW2 to SW1
Changed lines of the file:
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@@
 		(on_board yes)
 		(dnp no)
-		(property "Reference" "#PWR0167"
+		(property "Reference" "#PWR0122"
 			(at 240.03 34.29 0)
 			(effects
@@
 			(project "svea_powerboard_rev3"
 				(path "/3f85abf4-0b95-4c4a-b7e9-06f59ca1ea3d/5c2e021f-c2d4-49e2-8c36-9a64f1f12004/8d05c3b8-20a4-4a7f-9b20-01f8d5d5be48"
-					(reference "#PWR0167")
+					(reference "#PWR0122")
 					(unit 1)
 				)
@@
 		(on_board yes)
 		(dnp no)
-		(property "Reference" "#PWR0163"
+		(property "Reference" "#PWR0118"
 			(at 62.23 106.68 0)
 			(effects
@@
 			(project "svea_powerboard_rev3"
 				(path "/3f85abf4-0b95-4c4a-b7e9-06f59ca1ea3d/5c2e021f-c2d4-49e2-8c36-9a64f1f12004/8d05c3b8-20a4-4a7f-9b20-01f8d5d5be48"
-					(reference "#PWR0163")
+					(reference "#PWR0118")
 					(unit 1)
 				)
@@
 		(on_board yes)
 		(dnp no)
-		(property "Reference" "#PWR0164"
+		(property "Reference" "#PWR0119"
 			(at 68.58 106.68 0)
 			(effects
@@
 			(project "svea_powerboard_rev3"
 				(path "/3f85abf4-0b95-4c4a-b7e9-06f59ca1ea3d/5c2e021f-c2d4-49e2-8c36-9a64f1f12004/8d05c3b8-20a4-4a7f-9b20-01f8d5d5be48"
-					(reference "#PWR0164")
+					(reference "#PWR0119")
 					(unit 1)
 				)
@@
 		(on_board yes)
 		(dnp no)
-		(property "Reference" "#PWR0161"
+		(property "Reference" "#PWR0120"
 			(at 76.2 106.68 0)
 			(effects
@@
 			(project "svea_powerboard_rev3"
 				(path "/3f85abf4-0b95-4c4a-b7e9-06f59ca1ea3d/5c2e021f-c2d4-49e2-8c36-9a64f1f12004/8d05c3b8-20a4-4a7f-9b20-01f8d5d5be48"
-					(reference "#PWR0161")
+					(reference "#PWR0120")
 					(unit 1)
 				)
@@
 		(on_board yes)
 		(dnp no)
-		(property "Reference" "R95"
+		(property "Reference" "R132"
 			(at 115.57 153.67 0)
 			(effects
@@
 			(project "svea_powerboard_rev3"
 				(path "/3f85abf4-0b95-4c4a-b7e9-06f59ca1ea3d/5c2e021f-c2d4-49e2-8c36-9a64f1f12004/8d05c3b8-20a4-4a7f-9b20-01f8d5d5be48"
-					(reference "R95")
+					(reference "R132")
 					(unit 1)
 				)
@@
 		(on_board yes)
 		(dnp no)
-		(property "Reference" "R94"
+		(property "Reference" "R131"
 			(at 115.57 140.97 0)
 			(effects
@@
 			(project "svea_powerboard_rev3"
 				(path "/3f85abf4-0b95-4c4a-b7e9-06f59ca1ea3d/5c2e021f-c2d4-49e2-8c36-9a64f1f12004/8d05c3b8-20a4-4a7f-9b20-01f8d5d5be48"
-					(reference "R94")
+					(reference "R131")
 					(unit 1)
 				)
@@
 		(on_board yes)
 		(dnp no)
-		(property "Reference" "R93"
+		(property "Reference" "R130"
 			(at 115.57 128.27 0)
 			(effects
@@
 			(project "svea_powerboard_rev3"
 				(path "/3f85abf4-0b95-4c4a-b7e9-06f59ca1ea3d/5c2e021f-c2d4-49e2-8c36-9a64f1f12004/8d05c3b8-20a4-4a7f-9b20-01f8d5d5be48"
-					(reference "R93")
+					(reference "R130")
 					(unit 1)
 				)
@@
 		(on_board yes)
 		(dnp no)
-		(property "Reference" "#PWR0168"
+		(property "Reference" "#PWR0121"
 			(at 123.19 190.5 0)
 			(effects
@@
 			(project "svea_powerboard_rev3"
 				(path "/3f85abf4-0b95-4c4a-b7e9-06f59ca1ea3d/5c2e021f-c2d4-49e2-8c36-9a64f1f12004/8d05c3b8-20a4-4a7f-9b20-01f8d5d5be48"
-					(reference "#PWR0168")
+					(reference "#PWR0121")
 					(unit 1)
 				)
@@
 		(on_board yes)
 		(dnp no)
-		(property "Reference" "#PWR0162"
+		(property "Reference" "#PWR0117"
 			(at 55.88 106.68 0)
 			(effects
@@
 			(project "svea_powerboard_rev3"
 				(path "/3f85abf4-0b95-4c4a-b7e9-06f59ca1ea3d/5c2e021f-c2d4-49e2-8c36-9a64f1f12004/8d05c3b8-20a4-4a7f-9b20-01f8d5d5be48"
-					(reference "#PWR0162")
+					(reference "#PWR0117")
 					(unit 1)
 				)
@@
 		(on_board yes)
 		(dnp no)
-		(property "Reference" "SW2"
+		(property "Reference" "SW1"
 			(at 165.1 29.21 0)
 			(effects
@@
 			(project "svea_powerboard_rev3"
 				(path "/3f85abf4-0b95-4c4a-b7e9-06f59ca1ea3d/5c2e021f-c2d4-49e2-8c36-9a64f1f12004/8d05c3b8-20a4-4a7f-9b20-01f8d5d5be48"
-					(reference "SW2")
+					(reference "SW1")
 					(unit 1)
 				)
@@
 		(on_board yes)
 		(dnp no)
-		(property "Reference" "R99"
+		(property "Reference" "R135"
 			(at 226.06 30.48 0)
 			(effects
@@
 			(project "svea_powerboard_rev3"
 				(path "/3f85abf4-0b95-4c4a-b7e9-06f59ca1ea3d/5c2e021f-c2d4-49e2-8c36-9a64f1f12004/8d05c3b8-20a4-4a7f-9b20-01f8d5d5be48"
-					(reference "R99")
+					(reference "R135")
 					(unit 1)
 				)
@@
 		(on_board yes)
 		(dnp no)
-		(property "Reference" "#PWR0165"
+		(property "Reference" "#PWR0116"
 			(at 46.99 106.68 0)
 			(effects
@@
 			(project "svea_powerboard_rev3"
 				(path "/3f85abf4-0b95-4c4a-b7e9-06f59ca1ea3d/5c2e021f-c2d4-49e2-8c36-9a64f1f12004/8d05c3b8-20a4-4a7f-9b20-01f8d5d5be48"
-					(reference "#PWR0165")
+					(reference "#PWR0116")
 					(unit 1)
 				)
@@
 		(on_board yes)
 		(dnp no)
-		(property "Reference" "R96"
+		(property "Reference" "R133"
 			(at 115.57 166.37 0)
 			(effects
@@
 			(project "svea_powerboard_rev3"
 				(path "/3f85abf4-0b95-4c4a-b7e9-06f59ca1ea3d/5c2e021f-c2d4-49e2-8c36-9a64f1f12004/8d05c3b8-20a4-4a7f-9b20-01f8d5d5be48"
-					(reference "R96")
+					(reference "R133")
 					(unit 1)
 				)
@@
 		(on_board yes)
 		(dnp no)
-		(property "Reference" "R97"
+		(property "Reference" "R134"
 			(at 115.57 179.07 0)
 			(effects
@@
 			(project "svea_powerboard_rev3"
 				(path "/3f85abf4-0b95-4c4a-b7e9-06f59ca1ea3d/5c2e021f-c2d4-49e2-8c36-9a64f1f12004/8d05c3b8-20a4-4a7f-9b20-01f8d5d5be48"
-					(reference "R97")
-					(unit 1)
-				)
+					(reference "R134")
+					(unit 1)
+				)

Commit message: various improvements
Parts:
- renumbered R130 to R127, R131 to R128, R132 to R129, R133 to R130, R134 to R131, R135 to R132
Changed lines of the file:
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@@
 		(on_board yes)
 		(dnp no)
-		(property "Reference" "#PWR0122"
+		(property "Reference" "#PWR0161"
 			(at 240.03 34.29 0)
 			(effects
@@
 			(project "svea_powerboard_rev3"
 				(path "/3f85abf4-0b95-4c4a-b7e9-06f59ca1ea3d/5c2e021f-c2d4-49e2-8c36-9a64f1f12004/8d05c3b8-20a4-4a7f-9b20-01f8d5d5be48"
-					(reference "#PWR0122")
+					(reference "#PWR0161")
 					(unit 1)
 				)
@@
 		(on_board yes)
 		(dnp no)
-		(property "Reference" "#PWR0118"
+		(property "Reference" "#PWR0157"
 			(at 62.23 106.68 0)
 			(effects
@@
 			(project "svea_powerboard_rev3"
 				(path "/3f85abf4-0b95-4c4a-b7e9-06f59ca1ea3d/5c2e021f-c2d4-49e2-8c36-9a64f1f12004/8d05c3b8-20a4-4a7f-9b20-01f8d5d5be48"
-					(reference "#PWR0118")
+					(reference "#PWR0157")
 					(unit 1)
 				)
@@
 		(on_board yes)
 		(dnp no)
-		(property "Reference" "#PWR0119"
+		(property "Reference" "#PWR0158"
 			(at 68.58 106.68 0)
 			(effects
@@
 			(project "svea_powerboard_rev3"
 				(path "/3f85abf4-0b95-4c4a-b7e9-06f59ca1ea3d/5c2e021f-c2d4-49e2-8c36-9a64f1f12004/8d05c3b8-20a4-4a7f-9b20-01f8d5d5be48"
-					(reference "#PWR0119")
+					(reference "#PWR0158")
 					(unit 1)
 				)
@@
 		(on_board yes)
 		(dnp no)
-		(property "Reference" "#PWR0120"
+		(property "Reference" "#PWR0159"
 			(at 76.2 106.68 0)
 			(effects
@@
 			(project "svea_powerboard_rev3"
 				(path "/3f85abf4-0b95-4c4a-b7e9-06f59ca1ea3d/5c2e021f-c2d4-49e2-8c36-9a64f1f12004/8d05c3b8-20a4-4a7f-9b20-01f8d5d5be48"
-					(reference "#PWR0120")
+					(reference "#PWR0159")
 					(unit 1)
 				)
@@
 		(on_board yes)
 		(dnp no)
-		(property "Reference" "R132"
+		(property "Reference" "R129"
 			(at 115.57 153.67 0)
 			(effects
@@
 			(project "svea_powerboard_rev3"
 				(path "/3f85abf4-0b95-4c4a-b7e9-06f59ca1ea3d/5c2e021f-c2d4-49e2-8c36-9a64f1f12004/8d05c3b8-20a4-4a7f-9b20-01f8d5d5be48"
-					(reference "R132")
+					(reference "R129")
 					(unit 1)
 				)
@@
 		(on_board yes)
 		(dnp no)
-		(property "Reference" "R131"
+		(property "Reference" "R128"
 			(at 115.57 140.97 0)
 			(effects
@@
 			(project "svea_powerboard_rev3"
 				(path "/3f85abf4-0b95-4c4a-b7e9-06f59ca1ea3d/5c2e021f-c2d4-49e2-8c36-9a64f1f12004/8d05c3b8-20a4-4a7f-9b20-01f8d5d5be48"
-					(reference "R131")
+					(reference "R128")
 					(unit 1)
 				)
@@
 		(on_board yes)
 		(dnp no)
-		(property "Reference" "R130"
+		(property "Reference" "R127"
 			(at 115.57 128.27 0)
 			(effects
@@
 			(project "svea_powerboard_rev3"
 				(path "/3f85abf4-0b95-4c4a-b7e9-06f59ca1ea3d/5c2e021f-c2d4-49e2-8c36-9a64f1f12004/8d05c3b8-20a4-4a7f-9b20-01f8d5d5be48"
-					(reference "R130")
+					(reference "R127")
 					(unit 1)
 				)
@@
 		(on_board yes)
 		(dnp no)
-		(property "Reference" "#PWR0121"
+		(property "Reference" "#PWR0160"
 			(at 123.19 190.5 0)
 			(effects
@@
 			(project "svea_powerboard_rev3"
 				(path "/3f85abf4-0b95-4c4a-b7e9-06f59ca1ea3d/5c2e021f-c2d4-49e2-8c36-9a64f1f12004/8d05c3b8-20a4-4a7f-9b20-01f8d5d5be48"
-					(reference "#PWR0121")
+					(reference "#PWR0160")
 					(unit 1)
 				)
@@
 		(on_board yes)
 		(dnp no)
-		(property "Reference" "#PWR0117"
+		(property "Reference" "#PWR0156"
 			(at 55.88 106.68 0)
 			(effects
@@
 			(project "svea_powerboard_rev3"
 				(path "/3f85abf4-0b95-4c4a-b7e9-06f59ca1ea3d/5c2e021f-c2d4-49e2-8c36-9a64f1f12004/8d05c3b8-20a4-4a7f-9b20-01f8d5d5be48"
-					(reference "#PWR0117")
+					(reference "#PWR0156")
 					(unit 1)
 				)
@@
 		(on_board yes)
 		(dnp no)
-		(property "Reference" "R135"
+		(property "Reference" "R132"
 			(at 226.06 30.48 0)
 			(effects
@@
 			(project "svea_powerboard_rev3"
 				(path "/3f85abf4-0b95-4c4a-b7e9-06f59ca1ea3d/5c2e021f-c2d4-49e2-8c36-9a64f1f12004/8d05c3b8-20a4-4a7f-9b20-01f8d5d5be48"
-					(reference "R135")
+					(reference "R132")
 					(unit 1)
 				)
@@
 		(on_board yes)
 		(dnp no)
-		(property "Reference" "#PWR0116"
+		(property "Reference" "#PWR0155"
 			(at 46.99 106.68 0)
 			(effects
@@
 			(project "svea_powerboard_rev3"
 				(path "/3f85abf4-0b95-4c4a-b7e9-06f59ca1ea3d/5c2e021f-c2d4-49e2-8c36-9a64f1f12004/8d05c3b8-20a4-4a7f-9b20-01f8d5d5be48"
-					(reference "#PWR0116")
+					(reference "#PWR0155")
 					(unit 1)
 				)
@@
 		(on_board yes)
 		(dnp no)
-		(property "Reference" "R133"
+		(property "Reference" "R130"
 			(at 115.57 166.37 0)
 			(effects
@@
 			(project "svea_powerboard_rev3"
 				(path "/3f85abf4-0b95-4c4a-b7e9-06f59ca1ea3d/5c2e021f-c2d4-49e2-8c36-9a64f1f12004/8d05c3b8-20a4-4a7f-9b20-01f8d5d5be48"
-					(reference "R133")
+					(reference "R130")
 					(unit 1)
 				)
@@
 		(on_board yes)
 		(dnp no)
-		(property "Reference" "R134"
+		(property "Reference" "R131"
 			(at 115.57 179.07 0)
 			(effects
@@
 			(project "svea_powerboard_rev3"
 				(path "/3f85abf4-0b95-4c4a-b7e9-06f59ca1ea3d/5c2e021f-c2d4-49e2-8c36-9a64f1f12004/8d05c3b8-20a4-4a7f-9b20-01f8d5d5be48"
-					(reference "R134")
-					(unit 1)
-				)
+					(reference "R131")
+					(unit 1)
+				)

Commit message: various improvements
Parts:
- renumbered R127 to R138, R128 to R139, R129 to R140, R130 to R141, R131 to R142, R132 to R143
Changed lines of the file:
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@@
 		(on_board yes)
 		(dnp no)
-		(property "Reference" "#PWR0161"
+		(property "Reference" "#PWR0172"
 			(at 240.03 34.29 0)
 			(effects
@@
 			(project "svea_powerboard_rev3"
 				(path "/3f85abf4-0b95-4c4a-b7e9-06f59ca1ea3d/5c2e021f-c2d4-49e2-8c36-9a64f1f12004/8d05c3b8-20a4-4a7f-9b20-01f8d5d5be48"
-					(reference "#PWR0161")
+					(reference "#PWR0172")
 					(unit 1)
 				)
@@
 		(on_board yes)
 		(dnp no)
-		(property "Reference" "#PWR0157"
+		(property "Reference" "#PWR0168"
 			(at 62.23 106.68 0)
 			(effects
@@
 			(project "svea_powerboard_rev3"
 				(path "/3f85abf4-0b95-4c4a-b7e9-06f59ca1ea3d/5c2e021f-c2d4-49e2-8c36-9a64f1f12004/8d05c3b8-20a4-4a7f-9b20-01f8d5d5be48"
-					(reference "#PWR0157")
+					(reference "#PWR0168")
 					(unit 1)
 				)
@@
 		(on_board yes)
 		(dnp no)
-		(property "Reference" "#PWR0158"
+		(property "Reference" "#PWR0169"
 			(at 68.58 106.68 0)
 			(effects
@@
 			(project "svea_powerboard_rev3"
 				(path "/3f85abf4-0b95-4c4a-b7e9-06f59ca1ea3d/5c2e021f-c2d4-49e2-8c36-9a64f1f12004/8d05c3b8-20a4-4a7f-9b20-01f8d5d5be48"
-					(reference "#PWR0158")
+					(reference "#PWR0169")
 					(unit 1)
 				)
@@
 		(on_board yes)
 		(dnp no)
-		(property "Reference" "#PWR0159"
+		(property "Reference" "#PWR0170"
 			(at 76.2 106.68 0)
 			(effects
@@
 			(project "svea_powerboard_rev3"
 				(path "/3f85abf4-0b95-4c4a-b7e9-06f59ca1ea3d/5c2e021f-c2d4-49e2-8c36-9a64f1f12004/8d05c3b8-20a4-4a7f-9b20-01f8d5d5be48"
-					(reference "#PWR0159")
+					(reference "#PWR0170")
 					(unit 1)
 				)
@@
 		(on_board yes)
 		(dnp no)
-		(property "Reference" "R129"
+		(property "Reference" "R140"
 			(at 115.57 153.67 0)
 			(effects
@@
 			(project "svea_powerboard_rev3"
 				(path "/3f85abf4-0b95-4c4a-b7e9-06f59ca1ea3d/5c2e021f-c2d4-49e2-8c36-9a64f1f12004/8d05c3b8-20a4-4a7f-9b20-01f8d5d5be48"
-					(reference "R129")
+					(reference "R140")
 					(unit 1)
 				)
@@
 		(on_board yes)
 		(dnp no)
-		(property "Reference" "R128"
+		(property "Reference" "R139"
 			(at 115.57 140.97 0)
 			(effects
@@
 			(project "svea_powerboard_rev3"
 				(path "/3f85abf4-0b95-4c4a-b7e9-06f59ca1ea3d/5c2e021f-c2d4-49e2-8c36-9a64f1f12004/8d05c3b8-20a4-4a7f-9b20-01f8d5d5be48"
-					(reference "R128")
+					(reference "R139")
 					(unit 1)
 				)
@@
 		(on_board yes)
 		(dnp no)
-		(property "Reference" "R127"
+		(property "Reference" "R138"
 			(at 115.57 128.27 0)
 			(effects
@@
 			(project "svea_powerboard_rev3"
 				(path "/3f85abf4-0b95-4c4a-b7e9-06f59ca1ea3d/5c2e021f-c2d4-49e2-8c36-9a64f1f12004/8d05c3b8-20a4-4a7f-9b20-01f8d5d5be48"
-					(reference "R127")
+					(reference "R138")
 					(unit 1)
 				)
@@
 		(on_board yes)
 		(dnp no)
-		(property "Reference" "#PWR0160"
+		(property "Reference" "#PWR0171"
 			(at 123.19 190.5 0)
 			(effects
@@
 			(project "svea_powerboard_rev3"
 				(path "/3f85abf4-0b95-4c4a-b7e9-06f59ca1ea3d/5c2e021f-c2d4-49e2-8c36-9a64f1f12004/8d05c3b8-20a4-4a7f-9b20-01f8d5d5be48"
-					(reference "#PWR0160")
+					(reference "#PWR0171")
 					(unit 1)
 				)
@@
 		(on_board yes)
 		(dnp no)
-		(property "Reference" "#PWR0156"
+		(property "Reference" "#PWR0167"
 			(at 55.88 106.68 0)
 			(effects
@@
 			(project "svea_powerboard_rev3"
 				(path "/3f85abf4-0b95-4c4a-b7e9-06f59ca1ea3d/5c2e021f-c2d4-49e2-8c36-9a64f1f12004/8d05c3b8-20a4-4a7f-9b20-01f8d5d5be48"
-					(reference "#PWR0156")
+					(reference "#PWR0167")
 					(unit 1)
 				)
@@
 		(on_board yes)
 		(dnp no)
-		(property "Reference" "R132"
+		(property "Reference" "R143"
 			(at 226.06 30.48 0)
 			(effects
@@
 			(project "svea_powerboard_rev3"
 				(path "/3f85abf4-0b95-4c4a-b7e9-06f59ca1ea3d/5c2e021f-c2d4-49e2-8c36-9a64f1f12004/8d05c3b8-20a4-4a7f-9b20-01f8d5d5be48"
-					(reference "R132")
+					(reference "R143")
 					(unit 1)
 				)
@@
 		(on_board yes)
 		(dnp no)
-		(property "Reference" "#PWR0155"
+		(property "Reference" "#PWR0166"
 			(at 46.99 106.68 0)
 			(effects
@@
 			(project "svea_powerboard_rev3"
 				(path "/3f85abf4-0b95-4c4a-b7e9-06f59ca1ea3d/5c2e021f-c2d4-49e2-8c36-9a64f1f12004/8d05c3b8-20a4-4a7f-9b20-01f8d5d5be48"
-					(reference "#PWR0155")
+					(reference "#PWR0166")
 					(unit 1)
 				)
@@
 		(on_board yes)
 		(dnp no)
-		(property "Reference" "R130"
+		(property "Reference" "R141"
 			(at 115.57 166.37 0)
 			(effects
@@
 			(project "svea_powerboard_rev3"
 				(path "/3f85abf4-0b95-4c4a-b7e9-06f59ca1ea3d/5c2e021f-c2d4-49e2-8c36-9a64f1f12004/8d05c3b8-20a4-4a7f-9b20-01f8d5d5be48"
-					(reference "R130")
+					(reference "R141")
 					(unit 1)
 				)
@@
 		(on_board yes)
 		(dnp no)
-		(property "Reference" "R131"
+		(property "Reference" "R142"
 			(at 115.57 179.07 0)
 			(effects
@@
 			(project "svea_powerboard_rev3"
 				(path "/3f85abf4-0b95-4c4a-b7e9-06f59ca1ea3d/5c2e021f-c2d4-49e2-8c36-9a64f1f12004/8d05c3b8-20a4-4a7f-9b20-01f8d5d5be48"
-					(reference "R131")
-					(unit 1)
-				)
+					(reference "R142")
+					(unit 1)
+				)
