File: hardware/kicad/sheets/mcu/27_Microcontroller-PIN-IC.kicad_sch (KiCad schematic)
At the start: 19 parts, among them U37 PCAL6524HEAZ

Commit message: various improvements
Parts:
- renumbered C85 to C94, R117 to R114, R118 to R115, R119 to R116, R120 to R117, R121 to R118, R122 to R119, R123 to R120, R124 to R121, R125 to R122, R126 to R123, R127 to R124, R128 to R125, R129 to R126, U37 to U47, U38 to U48, U39 to U49, U40 to U50, U41 to U51
Changed lines of the file:
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@@
 		(on_board yes)
 		(dnp no)
-		(property "Reference" "R122"
+		(property "Reference" "R119"
 			(at 69.85 99.06 0)
 			(effects
@@
 			(project "svea_powerboard_rev3"
 				(path "/3f85abf4-0b95-4c4a-b7e9-06f59ca1ea3d/5c2e021f-c2d4-49e2-8c36-9a64f1f12004/8d05c3b8-20a4-4a7f-9b20-01f8d5d5be42"
-					(reference "R122")
+					(reference "R119")
 					(unit 1)
 				)
@@
 		(on_board yes)
 		(dnp no)
-		(property "Reference" "R121"
+		(property "Reference" "R118"
 			(at 69.85 91.44 0)
 			(effects
@@
 			(project "svea_powerboard_rev3"
 				(path "/3f85abf4-0b95-4c4a-b7e9-06f59ca1ea3d/5c2e021f-c2d4-49e2-8c36-9a64f1f12004/8d05c3b8-20a4-4a7f-9b20-01f8d5d5be42"
-					(reference "R121")
+					(reference "R118")
 					(unit 1)
 				)
@@
 		(on_board yes)
 		(dnp no)
-		(property "Reference" "U40"
+		(property "Reference" "U50"
 			(at 182.88 62.23 0)
 			(effects
@@
 			(project "svea_powerboard_rev3"
 				(path "/3f85abf4-0b95-4c4a-b7e9-06f59ca1ea3d/5c2e021f-c2d4-49e2-8c36-9a64f1f12004/8d05c3b8-20a4-4a7f-9b20-01f8d5d5be42"
-					(reference "U40")
+					(reference "U50")
 					(unit 1)
 				)
@@
 		(on_board yes)
 		(dnp no)
-		(property "Reference" "C85"
+		(property "Reference" "C94"
 			(at 227.33 52.07 90)
 			(effects
@@
 			(project "svea_powerboard_rev3"
 				(path "/3f85abf4-0b95-4c4a-b7e9-06f59ca1ea3d/5c2e021f-c2d4-49e2-8c36-9a64f1f12004/8d05c3b8-20a4-4a7f-9b20-01f8d5d5be42"
-					(reference "C85")
+					(reference "C94")
 					(unit 1)
 				)
@@
 		(on_board yes)
 		(dnp no)
-		(property "Reference" "#PWR0115"
+		(property "Reference" "#PWR0154"
 			(at 223.52 57.15 0)
 			(effects
@@
 			(project "svea_powerboard_rev3"
 				(path "/3f85abf4-0b95-4c4a-b7e9-06f59ca1ea3d/5c2e021f-c2d4-49e2-8c36-9a64f1f12004/8d05c3b8-20a4-4a7f-9b20-01f8d5d5be42"
-					(reference "#PWR0115")
+					(reference "#PWR0154")
 					(unit 1)
 				)
@@
 		(on_board yes)
 		(dnp no)
-		(property "Reference" "R120"
+		(property "Reference" "R117"
 			(at 69.85 83.82 0)
 			(effects
@@
 			(project "svea_powerboard_rev3"
 				(path "/3f85abf4-0b95-4c4a-b7e9-06f59ca1ea3d/5c2e021f-c2d4-49e2-8c36-9a64f1f12004/8d05c3b8-20a4-4a7f-9b20-01f8d5d5be42"
-					(reference "R120")
+					(reference "R117")
 					(unit 1)
 				)
@@
 		(on_board yes)
 		(dnp no)
-		(property "Reference" "U39"
+		(property "Reference" "U49"
 			(at 180.34 57.15 0)
 			(effects
@@
 			(project "svea_powerboard_rev3"
 				(path "/3f85abf4-0b95-4c4a-b7e9-06f59ca1ea3d/5c2e021f-c2d4-49e2-8c36-9a64f1f12004/8d05c3b8-20a4-4a7f-9b20-01f8d5d5be42"
-					(reference "U39")
+					(reference "U49")
 					(unit 1)
 				)
@@
 		(on_board yes)
 		(dnp no)
-		(property "Reference" "R118"
+		(property "Reference" "R115"
 			(at 69.85 68.58 0)
 			(effects
@@
 			(project "svea_powerboard_rev3"
 				(path "/3f85abf4-0b95-4c4a-b7e9-06f59ca1ea3d/5c2e021f-c2d4-49e2-8c36-9a64f1f12004/8d05c3b8-20a4-4a7f-9b20-01f8d5d5be42"
-					(reference "R118")
+					(reference "R115")
 					(unit 1)
 				)
@@
 		(on_board yes)
 		(dnp no)
-		(property "Reference" "R125"
+		(property "Reference" "R122"
 			(at 69.85 123.19 0)
 			(effects
@@
 			(project "svea_powerboard_rev3"
 				(path "/3f85abf4-0b95-4c4a-b7e9-06f59ca1ea3d/5c2e021f-c2d4-49e2-8c36-9a64f1f12004/8d05c3b8-20a4-4a7f-9b20-01f8d5d5be42"
-					(reference "R125")
+					(reference "R122")
 					(unit 1)
 				)
@@
 		(on_board yes)
 		(dnp no)
-		(property "Reference" "U37"
+		(property "Reference" "U47"
 			(at 127 49.53 0)
 			(effects
@@
 			(project "svea_powerboard_rev3"
 				(path "/3f85abf4-0b95-4c4a-b7e9-06f59ca1ea3d/5c2e021f-c2d4-49e2-8c36-9a64f1f12004/8d05c3b8-20a4-4a7f-9b20-01f8d5d5be42"
-					(reference "U37")
+					(reference "U47")
 					(unit 1)
 				)
@@
 		(on_board yes)
 		(dnp no)
-		(property "Reference" "R123"
+		(property "Reference" "R120"
 			(at 69.85 106.68 0)
 			(effects
@@
 			(project "svea_powerboard_rev3"
 				(path "/3f85abf4-0b95-4c4a-b7e9-06f59ca1ea3d/5c2e021f-c2d4-49e2-8c36-9a64f1f12004/8d05c3b8-20a4-4a7f-9b20-01f8d5d5be42"
-					(reference "R123")
+					(reference "R120")
 					(unit 1)
 				)
@@
 		(on_board yes)
 		(dnp no)
-		(property "Reference" "U38"
+		(property "Reference" "U48"
 			(at 180.34 54.61 0)
 			(effects
@@
 			(project "svea_powerboard_rev3"
 				(path "/3f85abf4-0b95-4c4a-b7e9-06f59ca1ea3d/5c2e021f-c2d4-49e2-8c36-9a64f1f12004/8d05c3b8-20a4-4a7f-9b20-01f8d5d5be42"
-					(reference "U38")
+					(reference "U48")
 					(unit 1)
 				)
@@
 		(on_board yes)
 		(dnp no)
-		(property "Reference" "R119"
+		(property "Reference" "R116"
 			(at 69.85 76.2 0)
 			(effects
@@
 			(project "svea_powerboard_rev3"
 				(path "/3f85abf4-0b95-4c4a-b7e9-06f59ca1ea3d/5c2e021f-c2d4-49e2-8c36-9a64f1f12004/8d05c3b8-20a4-4a7f-9b20-01f8d5d5be42"
-					(reference "R119")
+					(reference "R116")
 					(unit 1)
 				)
@@
 		(on_board yes)
 		(dnp no)
-		(property "Reference" "R129"
+		(property "Reference" "R126"
 			(at 185.42 46.99 90)
 			(effects
@@
 			(project "svea_powerboard_rev3"
 				(path "/3f85abf4-0b95-4c4a-b7e9-06f59ca1ea3d/5c2e021f-c2d4-49e2-8c36-9a64f1f12004/8d05c3b8-20a4-4a7f-9b20-01f8d5d5be42"
-					(reference "R129")
+					(reference "R126")
 					(unit 1)
 				)
@@
 		(on_board yes)
 		(dnp no)
-		(property "Reference" "R128"
+		(property "Reference" "R125"
 			(at 69.85 146.05 0)
 			(effects
@@
 			(project "svea_powerboard_rev3"
 				(path "/3f85abf4-0b95-4c4a-b7e9-06f59ca1ea3d/5c2e021f-c2d4-49e2-8c36-9a64f1f12004/8d05c3b8-20a4-4a7f-9b20-01f8d5d5be42"
-					(reference "R128")
+					(reference "R125")
 					(unit 1)
 				)
@@
 		(on_board yes)
 		(dnp no)
-		(property "Reference" "R127"
+		(property "Reference" "R124"
 			(at 69.85 138.43 0)
 			(effects
@@
 			(project "svea_powerboard_rev3"
 				(path "/3f85abf4-0b95-4c4a-b7e9-06f59ca1ea3d/5c2e021f-c2d4-49e2-8c36-9a64f1f12004/8d05c3b8-20a4-4a7f-9b20-01f8d5d5be42"
-					(reference "R127")
+					(reference "R124")
 					(unit 1)
 				)
@@
 		(on_board yes)
 		(dnp no)
-		(property "Reference" "U41"
+		(property "Reference" "U51"
 			(at 182.88 64.77 0)
 			(effects
@@
 			(project "svea_powerboard_rev3"
 				(path "/3f85abf4-0b95-4c4a-b7e9-06f59ca1ea3d/5c2e021f-c2d4-49e2-8c36-9a64f1f12004/8d05c3b8-20a4-4a7f-9b20-01f8d5d5be42"
-					(reference "U41")
+					(reference "U51")
 					(unit 1)
 				)
@@
 		(on_board yes)
 		(dnp no)
-		(property "Reference" "#PWR0114"
+		(property "Reference" "#PWR0153"
 			(at 182.88 39.37 0)
 			(effects
@@
 			(project "svea_powerboard_rev3"
 				(path "/3f85abf4-0b95-4c4a-b7e9-06f59ca1ea3d/5c2e021f-c2d4-49e2-8c36-9a64f1f12004/8d05c3b8-20a4-4a7f-9b20-01f8d5d5be42"
-					(reference "#PWR0114")
+					(reference "#PWR0153")
 					(unit 1)
 				)
@@
 		(on_board yes)
 		(dnp no)
-		(property "Reference" "R117"
+		(property "Reference" "R114"
 			(at 69.85 60.96 0)
 			(effects
@@
 			(project "svea_powerboard_rev3"
 				(path "/3f85abf4-0b95-4c4a-b7e9-06f59ca1ea3d/5c2e021f-c2d4-49e2-8c36-9a64f1f12004/8d05c3b8-20a4-4a7f-9b20-01f8d5d5be42"
-					(reference "R117")
+					(reference "R114")
 					(unit 1)
 				)
@@
 		(on_board yes)
 		(dnp no)
-		(property "Reference" "R124"
+		(property "Reference" "R121"
 			(at 69.85 115.57 0)
 			(effects
@@
 			(project "svea_powerboard_rev3"
 				(path "/3f85abf4-0b95-4c4a-b7e9-06f59ca1ea3d/5c2e021f-c2d4-49e2-8c36-9a64f1f12004/8d05c3b8-20a4-4a7f-9b20-01f8d5d5be42"
-					(reference "R124")
+					(reference "R121")
 					(unit 1)
 				)
@@
 		(on_board yes)
 		(dnp no)
-		(property "Reference" "R126"
+		(property "Reference" "R123"
 			(at 69.85 130.81 0)
 			(effects
@@
 			(project "svea_powerboard_rev3"
 				(path "/3f85abf4-0b95-4c4a-b7e9-06f59ca1ea3d/5c2e021f-c2d4-49e2-8c36-9a64f1f12004/8d05c3b8-20a4-4a7f-9b20-01f8d5d5be42"
-					(reference "R126")
+					(reference "R123")
 					(unit 1)
 				)
@@
 		(on_board yes)
 		(dnp no)
-		(property "Reference" "#PWR0113"
+		(property "Reference" "#PWR0152"
 			(at 170.18 101.6 0)
 			(effects
@@
 			(project "svea_powerboard_rev3"
 				(path "/3f85abf4-0b95-4c4a-b7e9-06f59ca1ea3d/5c2e021f-c2d4-49e2-8c36-9a64f1f12004/8d05c3b8-20a4-4a7f-9b20-01f8d5d5be42"
-					(reference "#PWR0113")
+					(reference "#PWR0152")
 					(unit 1)
 				)

Commit message: various improvements
Parts:
- renumbered C94 to C104, R114 to R125, R115 to R126, R116 to R127, R117 to R128, R118 to R129, R119 to R130, R120 to R131, R121 to R132, R122 to R133, R123 to R134, R124 to R135, R125 to R136, R126 to R137, U47 to U50, U48 to U51, U49 to U52, U50 to U53, U51 to U54
Changed lines of the file:
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@@
 		(on_board yes)
 		(dnp no)
-		(property "Reference" "R119"
+		(property "Reference" "R130"
 			(at 69.85 99.06 0)
 			(effects
@@
 			(project "svea_powerboard_rev3"
 				(path "/3f85abf4-0b95-4c4a-b7e9-06f59ca1ea3d/5c2e021f-c2d4-49e2-8c36-9a64f1f12004/8d05c3b8-20a4-4a7f-9b20-01f8d5d5be42"
-					(reference "R119")
+					(reference "R130")
 					(unit 1)
 				)
@@
 		(on_board yes)
 		(dnp no)
-		(property "Reference" "R118"
+		(property "Reference" "R129"
 			(at 69.85 91.44 0)
 			(effects
@@
 			(project "svea_powerboard_rev3"
 				(path "/3f85abf4-0b95-4c4a-b7e9-06f59ca1ea3d/5c2e021f-c2d4-49e2-8c36-9a64f1f12004/8d05c3b8-20a4-4a7f-9b20-01f8d5d5be42"
-					(reference "R118")
+					(reference "R129")
 					(unit 1)
 				)
@@
 		(on_board yes)
 		(dnp no)
-		(property "Reference" "U50"
+		(property "Reference" "U53"
 			(at 182.88 62.23 0)
 			(effects
@@
 			(project "svea_powerboard_rev3"
 				(path "/3f85abf4-0b95-4c4a-b7e9-06f59ca1ea3d/5c2e021f-c2d4-49e2-8c36-9a64f1f12004/8d05c3b8-20a4-4a7f-9b20-01f8d5d5be42"
-					(reference "U50")
+					(reference "U53")
 					(unit 1)
 				)
@@
 		(on_board yes)
 		(dnp no)
-		(property "Reference" "C94"
+		(property "Reference" "C104"
 			(at 227.33 52.07 90)
 			(effects
@@
 			(project "svea_powerboard_rev3"
 				(path "/3f85abf4-0b95-4c4a-b7e9-06f59ca1ea3d/5c2e021f-c2d4-49e2-8c36-9a64f1f12004/8d05c3b8-20a4-4a7f-9b20-01f8d5d5be42"
-					(reference "C94")
+					(reference "C104")
 					(unit 1)
 				)
@@
 		(on_board yes)
 		(dnp no)
-		(property "Reference" "#PWR0154"
+		(property "Reference" "#PWR0165"
 			(at 223.52 57.15 0)
 			(effects
@@
 			(project "svea_powerboard_rev3"
 				(path "/3f85abf4-0b95-4c4a-b7e9-06f59ca1ea3d/5c2e021f-c2d4-49e2-8c36-9a64f1f12004/8d05c3b8-20a4-4a7f-9b20-01f8d5d5be42"
-					(reference "#PWR0154")
+					(reference "#PWR0165")
 					(unit 1)
 				)
@@
 		(on_board yes)
 		(dnp no)
-		(property "Reference" "R117"
+		(property "Reference" "R128"
 			(at 69.85 83.82 0)
 			(effects
@@
 			(project "svea_powerboard_rev3"
 				(path "/3f85abf4-0b95-4c4a-b7e9-06f59ca1ea3d/5c2e021f-c2d4-49e2-8c36-9a64f1f12004/8d05c3b8-20a4-4a7f-9b20-01f8d5d5be42"
-					(reference "R117")
+					(reference "R128")
 					(unit 1)
 				)
@@
 		(on_board yes)
 		(dnp no)
-		(property "Reference" "U49"
+		(property "Reference" "U52"
 			(at 180.34 57.15 0)
 			(effects
@@
 			(project "svea_powerboard_rev3"
 				(path "/3f85abf4-0b95-4c4a-b7e9-06f59ca1ea3d/5c2e021f-c2d4-49e2-8c36-9a64f1f12004/8d05c3b8-20a4-4a7f-9b20-01f8d5d5be42"
-					(reference "U49")
+					(reference "U52")
 					(unit 1)
 				)
@@
 		(on_board yes)
 		(dnp no)
-		(property "Reference" "R115"
+		(property "Reference" "R126"
 			(at 69.85 68.58 0)
 			(effects
@@
 			(project "svea_powerboard_rev3"
 				(path "/3f85abf4-0b95-4c4a-b7e9-06f59ca1ea3d/5c2e021f-c2d4-49e2-8c36-9a64f1f12004/8d05c3b8-20a4-4a7f-9b20-01f8d5d5be42"
-					(reference "R115")
+					(reference "R126")
 					(unit 1)
 				)
@@
 		(on_board yes)
 		(dnp no)
-		(property "Reference" "R122"
+		(property "Reference" "R133"
 			(at 69.85 123.19 0)
 			(effects
@@
 			(project "svea_powerboard_rev3"
 				(path "/3f85abf4-0b95-4c4a-b7e9-06f59ca1ea3d/5c2e021f-c2d4-49e2-8c36-9a64f1f12004/8d05c3b8-20a4-4a7f-9b20-01f8d5d5be42"
-					(reference "R122")
+					(reference "R133")
 					(unit 1)
 				)
@@
 		(on_board yes)
 		(dnp no)
-		(property "Reference" "U47"
+		(property "Reference" "U50"
 			(at 127 49.53 0)
 			(effects
@@
 			(project "svea_powerboard_rev3"
 				(path "/3f85abf4-0b95-4c4a-b7e9-06f59ca1ea3d/5c2e021f-c2d4-49e2-8c36-9a64f1f12004/8d05c3b8-20a4-4a7f-9b20-01f8d5d5be42"
-					(reference "U47")
+					(reference "U50")
 					(unit 1)
 				)
@@
 		(on_board yes)
 		(dnp no)
-		(property "Reference" "R120"
+		(property "Reference" "R131"
 			(at 69.85 106.68 0)
 			(effects
@@
 			(project "svea_powerboard_rev3"
 				(path "/3f85abf4-0b95-4c4a-b7e9-06f59ca1ea3d/5c2e021f-c2d4-49e2-8c36-9a64f1f12004/8d05c3b8-20a4-4a7f-9b20-01f8d5d5be42"
-					(reference "R120")
+					(reference "R131")
 					(unit 1)
 				)
@@
 		(on_board yes)
 		(dnp no)
-		(property "Reference" "U48"
+		(property "Reference" "U51"
 			(at 180.34 54.61 0)
 			(effects
@@
 			(project "svea_powerboard_rev3"
 				(path "/3f85abf4-0b95-4c4a-b7e9-06f59ca1ea3d/5c2e021f-c2d4-49e2-8c36-9a64f1f12004/8d05c3b8-20a4-4a7f-9b20-01f8d5d5be42"
-					(reference "U48")
+					(reference "U51")
 					(unit 1)
 				)
@@
 		(on_board yes)
 		(dnp no)
-		(property "Reference" "R116"
+		(property "Reference" "R127"
 			(at 69.85 76.2 0)
 			(effects
@@
 			(project "svea_powerboard_rev3"
 				(path "/3f85abf4-0b95-4c4a-b7e9-06f59ca1ea3d/5c2e021f-c2d4-49e2-8c36-9a64f1f12004/8d05c3b8-20a4-4a7f-9b20-01f8d5d5be42"
-					(reference "R116")
+					(reference "R127")
 					(unit 1)
 				)
@@
 		(on_board yes)
 		(dnp no)
-		(property "Reference" "R126"
+		(property "Reference" "R137"
 			(at 185.42 46.99 90)
 			(effects
@@
 			(project "svea_powerboard_rev3"
 				(path "/3f85abf4-0b95-4c4a-b7e9-06f59ca1ea3d/5c2e021f-c2d4-49e2-8c36-9a64f1f12004/8d05c3b8-20a4-4a7f-9b20-01f8d5d5be42"
-					(reference "R126")
+					(reference "R137")
 					(unit 1)
 				)
@@
 		(on_board yes)
 		(dnp no)
-		(property "Reference" "R125"
+		(property "Reference" "R136"
 			(at 69.85 146.05 0)
 			(effects
@@
 			(project "svea_powerboard_rev3"
 				(path "/3f85abf4-0b95-4c4a-b7e9-06f59ca1ea3d/5c2e021f-c2d4-49e2-8c36-9a64f1f12004/8d05c3b8-20a4-4a7f-9b20-01f8d5d5be42"
-					(reference "R125")
+					(reference "R136")
 					(unit 1)
 				)
@@
 		(on_board yes)
 		(dnp no)
-		(property "Reference" "R124"
+		(property "Reference" "R135"
 			(at 69.85 138.43 0)
 			(effects
@@
 			(project "svea_powerboard_rev3"
 				(path "/3f85abf4-0b95-4c4a-b7e9-06f59ca1ea3d/5c2e021f-c2d4-49e2-8c36-9a64f1f12004/8d05c3b8-20a4-4a7f-9b20-01f8d5d5be42"
-					(reference "R124")
+					(reference "R135")
 					(unit 1)
 				)
@@
 		(on_board yes)
 		(dnp no)
-		(property "Reference" "U51"
+		(property "Reference" "U54"
 			(at 182.88 64.77 0)
 			(effects
@@
 			(project "svea_powerboard_rev3"
 				(path "/3f85abf4-0b95-4c4a-b7e9-06f59ca1ea3d/5c2e021f-c2d4-49e2-8c36-9a64f1f12004/8d05c3b8-20a4-4a7f-9b20-01f8d5d5be42"
-					(reference "U51")
+					(reference "U54")
 					(unit 1)
 				)
@@
 		(on_board yes)
 		(dnp no)
-		(property "Reference" "#PWR0153"
+		(property "Reference" "#PWR0164"
 			(at 182.88 39.37 0)
 			(effects
@@
 			(project "svea_powerboard_rev3"
 				(path "/3f85abf4-0b95-4c4a-b7e9-06f59ca1ea3d/5c2e021f-c2d4-49e2-8c36-9a64f1f12004/8d05c3b8-20a4-4a7f-9b20-01f8d5d5be42"
-					(reference "#PWR0153")
+					(reference "#PWR0164")
 					(unit 1)
 				)
@@
 		(on_board yes)
 		(dnp no)
-		(property "Reference" "R114"
+		(property "Reference" "R125"
 			(at 69.85 60.96 0)
 			(effects
@@
 			(project "svea_powerboard_rev3"
 				(path "/3f85abf4-0b95-4c4a-b7e9-06f59ca1ea3d/5c2e021f-c2d4-49e2-8c36-9a64f1f12004/8d05c3b8-20a4-4a7f-9b20-01f8d5d5be42"
-					(reference "R114")
+					(reference "R125")
 					(unit 1)
 				)
@@
 		(on_board yes)
 		(dnp no)
-		(property "Reference" "R121"
+		(property "Reference" "R132"
 			(at 69.85 115.57 0)
 			(effects
@@
 			(project "svea_powerboard_rev3"
 				(path "/3f85abf4-0b95-4c4a-b7e9-06f59ca1ea3d/5c2e021f-c2d4-49e2-8c36-9a64f1f12004/8d05c3b8-20a4-4a7f-9b20-01f8d5d5be42"
-					(reference "R121")
+					(reference "R132")
 					(unit 1)
 				)
@@
 		(on_board yes)
 		(dnp no)
-		(property "Reference" "R123"
+		(property "Reference" "R134"
 			(at 69.85 130.81 0)
 			(effects
@@
 			(project "svea_powerboard_rev3"
 				(path "/3f85abf4-0b95-4c4a-b7e9-06f59ca1ea3d/5c2e021f-c2d4-49e2-8c36-9a64f1f12004/8d05c3b8-20a4-4a7f-9b20-01f8d5d5be42"
-					(reference "R123")
+					(reference "R134")
 					(unit 1)
 				)
@@
 		(on_board yes)
 		(dnp no)
-		(property "Reference" "#PWR0152"
+		(property "Reference" "#PWR0163"
 			(at 170.18 101.6 0)
 			(effects
@@
 			(project "svea_powerboard_rev3"
 				(path "/3f85abf4-0b95-4c4a-b7e9-06f59ca1ea3d/5c2e021f-c2d4-49e2-8c36-9a64f1f12004/8d05c3b8-20a4-4a7f-9b20-01f8d5d5be42"
-					(reference "#PWR0152")
+					(reference "#PWR0163")
 					(unit 1)
 				)
