File: hardware/kicad/sheets/mcu/25_Microcontroller-PWM-IC.kicad_sch (KiCad schematic)
At the start: 18 parts, among them U140 PCA9685PW,118

Commit message: reorganized
Other:
- title: Microcontroller-PWM-IC -> PWM Driver
Changed lines of the file:
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@@
 	(paper "User" 297 210)
 	(title_block
-		(title "Microcontroller-PWM-IC")
+		(title "PWM Driver")
 		(date "2026-02-16")
 	)

Commit message: before final cleanup
Parts:
- renumbered C202 to C47, C251 to C48, R438 to R100, R439 to R101, R440 to R102, R441 to R103, R442 to R104, R435 to R105, R432 to R106, R433 to R107, R434 to R108, R436 to R109, R437 to R110, U140 to U22, U145 to U23, U146 to U24, U144 to U25, U143 to U26

Commit message: resheeted bms and fixed links for the 12v buck
Parts:
- renumbered C47 to C86, C48 to C87, R100 to R136, R101 to R137, R102 to R138, R103 to R139, R104 to R140, R105 to R141, R106 to R142, R107 to R143, R108 to R144, R109 to R145, R110 to R146, U22 to U42, U23 to U43, U24 to U44, U25 to U45, U26 to U46
Changed lines of the file:
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@@
 		(on_board yes)
 		(dnp no)
-		(property "Reference" "R106"
+		(property "Reference" "R142"
 			(at 128.27 71.12 0)
 			(effects
@@
 			(project "svea_powerboard_rev3"
 				(path "/3f85abf4-0b95-4c4a-b7e9-06f59ca1ea3d/5c2e021f-c2d4-49e2-8c36-9a64f1f12004/8d05c3b8-20a4-4a7f-9b20-01f8d5d5be43"
-					(reference "R106")
+					(reference "R142")
 					(unit 1)
 				)
@@
 		(on_board yes)
 		(dnp no)
-		(property "Reference" "#PWR0173"
+		(property "Reference" "#PWR0125"
 			(at 243.84 60.96 0)
 			(effects
@@
 			(project "svea_powerboard_rev3"
 				(path "/3f85abf4-0b95-4c4a-b7e9-06f59ca1ea3d/5c2e021f-c2d4-49e2-8c36-9a64f1f12004/8d05c3b8-20a4-4a7f-9b20-01f8d5d5be43"
-					(reference "#PWR0173")
+					(reference "#PWR0125")
 					(unit 1)
 				)
@@
 		(on_board yes)
 		(dnp no)
-		(property "Reference" "R100"
+		(property "Reference" "R136"
 			(at 45.72 111.76 0)
 			(effects
@@
 			(project "svea_powerboard_rev3"
 				(path "/3f85abf4-0b95-4c4a-b7e9-06f59ca1ea3d/5c2e021f-c2d4-49e2-8c36-9a64f1f12004/8d05c3b8-20a4-4a7f-9b20-01f8d5d5be43"
-					(reference "R100")
+					(reference "R136")
 					(unit 1)
 				)
@@
 		(on_board yes)
 		(dnp no)
-		(property "Reference" "R104"
+		(property "Reference" "R140"
 			(at 86.36 121.92 0)
 			(effects
@@
 			(project "svea_powerboard_rev3"
 				(path "/3f85abf4-0b95-4c4a-b7e9-06f59ca1ea3d/5c2e021f-c2d4-49e2-8c36-9a64f1f12004/8d05c3b8-20a4-4a7f-9b20-01f8d5d5be43"
-					(reference "R104")
+					(reference "R140")
 					(unit 1)
 				)
@@
 		(on_board yes)
 		(dnp no)
-		(property "Reference" "U26"
+		(property "Reference" "U46"
 			(at 201.93 100.33 0)
 			(effects
@@
 			(project "svea_powerboard_rev3"
 				(path "/3f85abf4-0b95-4c4a-b7e9-06f59ca1ea3d/5c2e021f-c2d4-49e2-8c36-9a64f1f12004/8d05c3b8-20a4-4a7f-9b20-01f8d5d5be43"
-					(reference "U26")
+					(reference "U46")
 					(unit 1)
 				)
@@
 		(on_board yes)
 		(dnp no)
-		(property "Reference" "R110"
+		(property "Reference" "R146"
 			(at 194.31 106.68 0)
 			(effects
@@
 			(project "svea_powerboard_rev3"
 				(path "/3f85abf4-0b95-4c4a-b7e9-06f59ca1ea3d/5c2e021f-c2d4-49e2-8c36-9a64f1f12004/8d05c3b8-20a4-4a7f-9b20-01f8d5d5be43"
-					(reference "R110")
+					(reference "R146")
 					(unit 1)
 				)
@@
 		(on_board yes)
 		(dnp no)
-		(property "Reference" "R101"
+		(property "Reference" "R137"
 			(at 55.88 114.3 0)
 			(effects
@@
 			(project "svea_powerboard_rev3"
 				(path "/3f85abf4-0b95-4c4a-b7e9-06f59ca1ea3d/5c2e021f-c2d4-49e2-8c36-9a64f1f12004/8d05c3b8-20a4-4a7f-9b20-01f8d5d5be43"
-					(reference "R101")
+					(reference "R137")
 					(unit 1)
 				)
@@
 		(on_board yes)
 		(dnp no)
-		(property "Reference" "R102"
+		(property "Reference" "R138"
 			(at 66.04 116.84 0)
 			(effects
@@
 			(project "svea_powerboard_rev3"
 				(path "/3f85abf4-0b95-4c4a-b7e9-06f59ca1ea3d/5c2e021f-c2d4-49e2-8c36-9a64f1f12004/8d05c3b8-20a4-4a7f-9b20-01f8d5d5be43"
-					(reference "R102")
+					(reference "R138")
 					(unit 1)
 				)
@@
 		(on_board yes)
 		(dnp no)
-		(property "Reference" "R103"
+		(property "Reference" "R139"
 			(at 76.2 119.38 0)
 			(effects
@@
 			(project "svea_powerboard_rev3"
 				(path "/3f85abf4-0b95-4c4a-b7e9-06f59ca1ea3d/5c2e021f-c2d4-49e2-8c36-9a64f1f12004/8d05c3b8-20a4-4a7f-9b20-01f8d5d5be43"
-					(reference "R103")
+					(reference "R139")
 					(unit 1)
 				)
@@
 		(on_board yes)
 		(dnp no)
-		(property "Reference" "C48"
+		(property "Reference" "C87"
 			(at 255.27 74.93 90)
 			(effects
@@
 			(project "svea_powerboard_rev3"
 				(path "/3f85abf4-0b95-4c4a-b7e9-06f59ca1ea3d/5c2e021f-c2d4-49e2-8c36-9a64f1f12004/8d05c3b8-20a4-4a7f-9b20-01f8d5d5be43"
-					(reference "C48")
+					(reference "C87")
 					(unit 1)
 				)
@@
 		(on_board yes)
 		(dnp no)
-		(property "Reference" "U25"
+		(property "Reference" "U45"
 			(at 201.93 97.79 0)
 			(effects
@@
 			(project "svea_powerboard_rev3"
 				(path "/3f85abf4-0b95-4c4a-b7e9-06f59ca1ea3d/5c2e021f-c2d4-49e2-8c36-9a64f1f12004/8d05c3b8-20a4-4a7f-9b20-01f8d5d5be43"
-					(reference "U25")
+					(reference "U45")
 					(unit 1)
 				)
@@
 		(on_board yes)
 		(dnp no)
-		(property "Reference" "R109"
+		(property "Reference" "R145"
 			(at 163.83 63.5 0)
 			(effects
@@
 			(project "svea_powerboard_rev3"
 				(path "/3f85abf4-0b95-4c4a-b7e9-06f59ca1ea3d/5c2e021f-c2d4-49e2-8c36-9a64f1f12004/8d05c3b8-20a4-4a7f-9b20-01f8d5d5be43"
-					(reference "R109")
+					(reference "R145")
 					(unit 1)
 				)
@@
 		(on_board yes)
 		(dnp no)
-		(property "Reference" "#PWR0172"
+		(property "Reference" "#PWR0126"
 			(at 243.84 87.63 0)
 			(effects
@@
 			(project "svea_powerboard_rev3"
 				(path "/3f85abf4-0b95-4c4a-b7e9-06f59ca1ea3d/5c2e021f-c2d4-49e2-8c36-9a64f1f12004/8d05c3b8-20a4-4a7f-9b20-01f8d5d5be43"
-					(reference "#PWR0172")
+					(reference "#PWR0126")
 					(unit 1)
 				)
@@
 		(on_board yes)
 		(dnp no)
-		(property "Reference" "#PWR0171"
+		(property "Reference" "#PWR0123"
 			(at 121.92 92.71 0)
 			(effects
@@
 			(project "svea_powerboard_rev3"
 				(path "/3f85abf4-0b95-4c4a-b7e9-06f59ca1ea3d/5c2e021f-c2d4-49e2-8c36-9a64f1f12004/8d05c3b8-20a4-4a7f-9b20-01f8d5d5be43"
-					(reference "#PWR0171")
+					(reference "#PWR0123")
 					(unit 1)
 				)
@@
 		(on_board yes)
 		(dnp no)
-		(property "Reference" "U23"
+		(property "Reference" "U43"
 			(at 199.39 90.17 0)
 			(effects
@@
 			(project "svea_powerboard_rev3"
 				(path "/3f85abf4-0b95-4c4a-b7e9-06f59ca1ea3d/5c2e021f-c2d4-49e2-8c36-9a64f1f12004/8d05c3b8-20a4-4a7f-9b20-01f8d5d5be43"
-					(reference "U23")
+					(reference "U43")
 					(unit 1)
 				)
@@
 		(on_board yes)
 		(dnp no)
-		(property "Reference" "U24"
+		(property "Reference" "U44"
 			(at 199.39 92.71 0)
 			(effects
@@
 			(project "svea_powerboard_rev3"
 				(path "/3f85abf4-0b95-4c4a-b7e9-06f59ca1ea3d/5c2e021f-c2d4-49e2-8c36-9a64f1f12004/8d05c3b8-20a4-4a7f-9b20-01f8d5d5be43"
-					(reference "U24")
+					(reference "U44")
 					(unit 1)
 				)
@@
 		(on_board yes)
 		(dnp no)
-		(property "Reference" "R108"
+		(property "Reference" "R144"
 			(at 128.27 86.36 0)
 			(effects
@@
 			(project "svea_powerboard_rev3"
 				(path "/3f85abf4-0b95-4c4a-b7e9-06f59ca1ea3d/5c2e021f-c2d4-49e2-8c36-9a64f1f12004/8d05c3b8-20a4-4a7f-9b20-01f8d5d5be43"
-					(reference "R108")
+					(reference "R144")
 					(unit 1)
 				)
@@
 		(on_board yes)
 		(dnp no)
-		(property "Reference" "R105"
+		(property "Reference" "R141"
 			(at 128.27 63.5 0)
 			(effects
@@
 			(project "svea_powerboard_rev3"
 				(path "/3f85abf4-0b95-4c4a-b7e9-06f59ca1ea3d/5c2e021f-c2d4-49e2-8c36-9a64f1f12004/8d05c3b8-20a4-4a7f-9b20-01f8d5d5be43"
-					(reference "R105")
+					(reference "R141")
 					(unit 1)
 				)
@@
 		(on_board yes)
 		(dnp no)
-		(property "Reference" "#PWR0170"
+		(property "Reference" "#PWR0124"
 			(at 172.72 146.05 0)
 			(effects
@@
 			(project "svea_powerboard_rev3"
 				(path "/3f85abf4-0b95-4c4a-b7e9-06f59ca1ea3d/5c2e021f-c2d4-49e2-8c36-9a64f1f12004/8d05c3b8-20a4-4a7f-9b20-01f8d5d5be43"
-					(reference "#PWR0170")
+					(reference "#PWR0124")
 					(unit 1)
 				)
@@
 		(on_board yes)
 		(dnp no)
-		(property "Reference" "C47"
+		(property "Reference" "C86"
 			(at 240.03 74.93 90)
 			(effects
@@
 			(project "svea_powerboard_rev3"
 				(path "/3f85abf4-0b95-4c4a-b7e9-06f59ca1ea3d/5c2e021f-c2d4-49e2-8c36-9a64f1f12004/8d05c3b8-20a4-4a7f-9b20-01f8d5d5be43"
-					(reference "C47")
+					(reference "C86")
 					(unit 1)
 				)
@@
 		(on_board yes)
 		(dnp no)
-		(property "Reference" "U22"
+		(property "Reference" "U42"
 			(at 161.29 88.9 0)
 			(effects
@@
 			(project "svea_powerboard_rev3"
 				(path "/3f85abf4-0b95-4c4a-b7e9-06f59ca1ea3d/5c2e021f-c2d4-49e2-8c36-9a64f1f12004/8d05c3b8-20a4-4a7f-9b20-01f8d5d5be43"
-					(reference "U22")
+					(reference "U42")
 					(unit 1)
 				)
@@
 		(on_board yes)
 		(dnp no)
-		(property "Reference" "R107"
+		(property "Reference" "R143"
 			(at 128.27 78.74 0)
 			(effects
@@
 			(project "svea_powerboard_rev3"
 				(path "/3f85abf4-0b95-4c4a-b7e9-06f59ca1ea3d/5c2e021f-c2d4-49e2-8c36-9a64f1f12004/8d05c3b8-20a4-4a7f-9b20-01f8d5d5be43"
-					(reference "R107")
+					(reference "R143")
 					(unit 1)
 				)

Commit message: various improvements
Parts:
- renumbered C86 to C95, C87 to C96, R136 to R133, R137 to R134, R138 to R135, R139 to R136, R140 to R137, R141 to R138, R142 to R139, R143 to R140, R144 to R141, R145 to R142, R146 to R143, U42 to U52, U43 to U53, U44 to U54, U45 to U55, U46 to U56
Changed lines of the file:
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@@
 		(on_board yes)
 		(dnp no)
-		(property "Reference" "R142"
+		(property "Reference" "R139"
 			(at 128.27 71.12 0)
 			(effects
@@
 			(project "svea_powerboard_rev3"
 				(path "/3f85abf4-0b95-4c4a-b7e9-06f59ca1ea3d/5c2e021f-c2d4-49e2-8c36-9a64f1f12004/8d05c3b8-20a4-4a7f-9b20-01f8d5d5be43"
-					(reference "R142")
+					(reference "R139")
 					(unit 1)
 				)
@@
 		(on_board yes)
 		(dnp no)
-		(property "Reference" "#PWR0125"
+		(property "Reference" "#PWR0164"
 			(at 243.84 60.96 0)
 			(effects
@@
 			(project "svea_powerboard_rev3"
 				(path "/3f85abf4-0b95-4c4a-b7e9-06f59ca1ea3d/5c2e021f-c2d4-49e2-8c36-9a64f1f12004/8d05c3b8-20a4-4a7f-9b20-01f8d5d5be43"
-					(reference "#PWR0125")
+					(reference "#PWR0164")
 					(unit 1)
 				)
@@
 		(on_board yes)
 		(dnp no)
-		(property "Reference" "R136"
+		(property "Reference" "R133"
 			(at 45.72 111.76 0)
 			(effects
@@
 			(project "svea_powerboard_rev3"
 				(path "/3f85abf4-0b95-4c4a-b7e9-06f59ca1ea3d/5c2e021f-c2d4-49e2-8c36-9a64f1f12004/8d05c3b8-20a4-4a7f-9b20-01f8d5d5be43"
-					(reference "R136")
+					(reference "R133")
 					(unit 1)
 				)
@@
 		(on_board yes)
 		(dnp no)
-		(property "Reference" "R140"
+		(property "Reference" "R137"
 			(at 86.36 121.92 0)
 			(effects
@@
 			(project "svea_powerboard_rev3"
 				(path "/3f85abf4-0b95-4c4a-b7e9-06f59ca1ea3d/5c2e021f-c2d4-49e2-8c36-9a64f1f12004/8d05c3b8-20a4-4a7f-9b20-01f8d5d5be43"
-					(reference "R140")
+					(reference "R137")
 					(unit 1)
 				)
@@
 		(on_board yes)
 		(dnp no)
-		(property "Reference" "U46"
+		(property "Reference" "U56"
 			(at 201.93 100.33 0)
 			(effects
@@
 			(project "svea_powerboard_rev3"
 				(path "/3f85abf4-0b95-4c4a-b7e9-06f59ca1ea3d/5c2e021f-c2d4-49e2-8c36-9a64f1f12004/8d05c3b8-20a4-4a7f-9b20-01f8d5d5be43"
-					(reference "U46")
+					(reference "U56")
 					(unit 1)
 				)
@@
 		(on_board yes)
 		(dnp no)
-		(property "Reference" "R146"
+		(property "Reference" "R143"
 			(at 194.31 106.68 0)
 			(effects
@@
 			(project "svea_powerboard_rev3"
 				(path "/3f85abf4-0b95-4c4a-b7e9-06f59ca1ea3d/5c2e021f-c2d4-49e2-8c36-9a64f1f12004/8d05c3b8-20a4-4a7f-9b20-01f8d5d5be43"
-					(reference "R146")
+					(reference "R143")
 					(unit 1)
 				)
@@
 		(on_board yes)
 		(dnp no)
-		(property "Reference" "R137"
+		(property "Reference" "R134"
 			(at 55.88 114.3 0)
 			(effects
@@
 			(project "svea_powerboard_rev3"
 				(path "/3f85abf4-0b95-4c4a-b7e9-06f59ca1ea3d/5c2e021f-c2d4-49e2-8c36-9a64f1f12004/8d05c3b8-20a4-4a7f-9b20-01f8d5d5be43"
-					(reference "R137")
+					(reference "R134")
 					(unit 1)
 				)
@@
 		(on_board yes)
 		(dnp no)
-		(property "Reference" "R138"
+		(property "Reference" "R135"
 			(at 66.04 116.84 0)
 			(effects
@@
 			(project "svea_powerboard_rev3"
 				(path "/3f85abf4-0b95-4c4a-b7e9-06f59ca1ea3d/5c2e021f-c2d4-49e2-8c36-9a64f1f12004/8d05c3b8-20a4-4a7f-9b20-01f8d5d5be43"
-					(reference "R138")
+					(reference "R135")
 					(unit 1)
 				)
@@
 		(on_board yes)
 		(dnp no)
-		(property "Reference" "R139"
+		(property "Reference" "R136"
 			(at 76.2 119.38 0)
 			(effects
@@
 			(project "svea_powerboard_rev3"
 				(path "/3f85abf4-0b95-4c4a-b7e9-06f59ca1ea3d/5c2e021f-c2d4-49e2-8c36-9a64f1f12004/8d05c3b8-20a4-4a7f-9b20-01f8d5d5be43"
-					(reference "R139")
+					(reference "R136")
 					(unit 1)
 				)
@@
 		(on_board yes)
 		(dnp no)
-		(property "Reference" "C87"
+		(property "Reference" "C96"
 			(at 255.27 74.93 90)
 			(effects
@@
 			(project "svea_powerboard_rev3"
 				(path "/3f85abf4-0b95-4c4a-b7e9-06f59ca1ea3d/5c2e021f-c2d4-49e2-8c36-9a64f1f12004/8d05c3b8-20a4-4a7f-9b20-01f8d5d5be43"
-					(reference "C87")
+					(reference "C96")
 					(unit 1)
 				)
@@
 		(on_board yes)
 		(dnp no)
-		(property "Reference" "U45"
+		(property "Reference" "U55"
 			(at 201.93 97.79 0)
 			(effects
@@
 			(project "svea_powerboard_rev3"
 				(path "/3f85abf4-0b95-4c4a-b7e9-06f59ca1ea3d/5c2e021f-c2d4-49e2-8c36-9a64f1f12004/8d05c3b8-20a4-4a7f-9b20-01f8d5d5be43"
-					(reference "U45")
+					(reference "U55")
 					(unit 1)
 				)
@@
 		(on_board yes)
 		(dnp no)
-		(property "Reference" "R145"
+		(property "Reference" "R142"
 			(at 163.83 63.5 0)
 			(effects
@@
 			(project "svea_powerboard_rev3"
 				(path "/3f85abf4-0b95-4c4a-b7e9-06f59ca1ea3d/5c2e021f-c2d4-49e2-8c36-9a64f1f12004/8d05c3b8-20a4-4a7f-9b20-01f8d5d5be43"
-					(reference "R145")
+					(reference "R142")
 					(unit 1)
 				)
@@
 		(on_board yes)
 		(dnp no)
-		(property "Reference" "#PWR0126"
+		(property "Reference" "#PWR0165"
 			(at 243.84 87.63 0)
 			(effects
@@
 			(project "svea_powerboard_rev3"
 				(path "/3f85abf4-0b95-4c4a-b7e9-06f59ca1ea3d/5c2e021f-c2d4-49e2-8c36-9a64f1f12004/8d05c3b8-20a4-4a7f-9b20-01f8d5d5be43"
-					(reference "#PWR0126")
+					(reference "#PWR0165")
 					(unit 1)
 				)
@@
 		(on_board yes)
 		(dnp no)
-		(property "Reference" "#PWR0123"
+		(property "Reference" "#PWR0162"
 			(at 121.92 92.71 0)
 			(effects
@@
 			(project "svea_powerboard_rev3"
 				(path "/3f85abf4-0b95-4c4a-b7e9-06f59ca1ea3d/5c2e021f-c2d4-49e2-8c36-9a64f1f12004/8d05c3b8-20a4-4a7f-9b20-01f8d5d5be43"
-					(reference "#PWR0123")
+					(reference "#PWR0162")
 					(unit 1)
 				)
@@
 		(on_board yes)
 		(dnp no)
-		(property "Reference" "U43"
+		(property "Reference" "U53"
 			(at 199.39 90.17 0)
 			(effects
@@
 			(project "svea_powerboard_rev3"
 				(path "/3f85abf4-0b95-4c4a-b7e9-06f59ca1ea3d/5c2e021f-c2d4-49e2-8c36-9a64f1f12004/8d05c3b8-20a4-4a7f-9b20-01f8d5d5be43"
-					(reference "U43")
+					(reference "U53")
 					(unit 1)
 				)
@@
 		(on_board yes)
 		(dnp no)
-		(property "Reference" "U44"
+		(property "Reference" "U54"
 			(at 199.39 92.71 0)
 			(effects
@@
 			(project "svea_powerboard_rev3"
 				(path "/3f85abf4-0b95-4c4a-b7e9-06f59ca1ea3d/5c2e021f-c2d4-49e2-8c36-9a64f1f12004/8d05c3b8-20a4-4a7f-9b20-01f8d5d5be43"
-					(reference "U44")
+					(reference "U54")
 					(unit 1)
 				)
@@
 		(on_board yes)
 		(dnp no)
-		(property "Reference" "R144"
+		(property "Reference" "R141"
 			(at 128.27 86.36 0)
 			(effects
@@
 			(project "svea_powerboard_rev3"
 				(path "/3f85abf4-0b95-4c4a-b7e9-06f59ca1ea3d/5c2e021f-c2d4-49e2-8c36-9a64f1f12004/8d05c3b8-20a4-4a7f-9b20-01f8d5d5be43"
-					(reference "R144")
+					(reference "R141")
 					(unit 1)
 				)
@@
 		(on_board yes)
 		(dnp no)
-		(property "Reference" "R141"
+		(property "Reference" "R138"
 			(at 128.27 63.5 0)
 			(effects
@@
 			(project "svea_powerboard_rev3"
 				(path "/3f85abf4-0b95-4c4a-b7e9-06f59ca1ea3d/5c2e021f-c2d4-49e2-8c36-9a64f1f12004/8d05c3b8-20a4-4a7f-9b20-01f8d5d5be43"
-					(reference "R141")
+					(reference "R138")
 					(unit 1)
 				)
@@
 		(on_board yes)
 		(dnp no)
-		(property "Reference" "#PWR0124"
+		(property "Reference" "#PWR0163"
 			(at 172.72 146.05 0)
 			(effects
@@
 			(project "svea_powerboard_rev3"
 				(path "/3f85abf4-0b95-4c4a-b7e9-06f59ca1ea3d/5c2e021f-c2d4-49e2-8c36-9a64f1f12004/8d05c3b8-20a4-4a7f-9b20-01f8d5d5be43"
-					(reference "#PWR0124")
+					(reference "#PWR0163")
 					(unit 1)
 				)
@@
 		(on_board yes)
 		(dnp no)
-		(property "Reference" "C86"
+		(property "Reference" "C95"
 			(at 240.03 74.93 90)
 			(effects
@@
 			(project "svea_powerboard_rev3"
 				(path "/3f85abf4-0b95-4c4a-b7e9-06f59ca1ea3d/5c2e021f-c2d4-49e2-8c36-9a64f1f12004/8d05c3b8-20a4-4a7f-9b20-01f8d5d5be43"
-					(reference "C86")
+					(reference "C95")
 					(unit 1)
 				)
@@
 		(on_board yes)
 		(dnp no)
-		(property "Reference" "U42"
+		(property "Reference" "U52"
 			(at 161.29 88.9 0)
 			(effects
@@
 			(project "svea_powerboard_rev3"
 				(path "/3f85abf4-0b95-4c4a-b7e9-06f59ca1ea3d/5c2e021f-c2d4-49e2-8c36-9a64f1f12004/8d05c3b8-20a4-4a7f-9b20-01f8d5d5be43"
-					(reference "U42")
+					(reference "U52")
 					(unit 1)
 				)
@@
 		(on_board yes)
 		(dnp no)
-		(property "Reference" "R143"
+		(property "Reference" "R140"
 			(at 128.27 78.74 0)
 			(effects
@@
 			(project "svea_powerboard_rev3"
 				(path "/3f85abf4-0b95-4c4a-b7e9-06f59ca1ea3d/5c2e021f-c2d4-49e2-8c36-9a64f1f12004/8d05c3b8-20a4-4a7f-9b20-01f8d5d5be43"
-					(reference "R143")
+					(reference "R140")
 					(unit 1)
 				)

Commit message: various improvements
Parts:
- removed U53, U54: ~, Jumper:SolderJumper-2_P1.3mm_Open_Pad1.0x1.5mm, symbol Jumper:Jumper_2_Open
- removed U55, U56: ~, Jumper:SolderJumper-2_P1.3mm_Bridged_Pad1.0x1.5mm, symbol Jumper:Jumper_2_Bridged
- added R151, R152: 47Ω, Resistor_SMD:R_0603_1608Metric, symbol 5v rail sm-easyedapro:RS-03K47R0FT
- renumbered C95 to C105, C96 to C106, R133 to R10, R134 to R11, R135 to R12, R137 to R144, R138 to R145, R139 to R146, R140 to R147, R141 to R148, R142 to R149, R143 to R150, R136 to R93, U52 to U55
Connections:
- net SCL: now reaches U55.26 (SCL)
- net SDA: now reaches U55.27 (SDA)
- net at U55.11 (LED5): now also R151.2
- net at U55.12 (LED6): now also R152.2
- net DIFF_FRONT_PWM renamed OUT3
- net DIFF_REAR_PWM renamed OUT4
- net SPEED_PWM renamed OUT2
- net STEER_PWM renamed OUT1
- net THROTTLE_PWM renamed OUT0
- new net OUT5: R151.1
- new net OUT6: R152.1
