File: hardware/kicad/sheets/mcu/25_Microcontroller-PWM-IC.kicad_sch (KiCad schematic)
At the start: 16 parts, among them U59 PCA9685PW,118

Commit message: pre robot updating references
Parts:
- renumbered C123 to C121, C124 to C122, R146 to R153, R147 to R154, R148 to R155, R149 to R156, R150 to R157, R152 to R159, R155 to R162, R157 to R164, R158 to R165, R159 to R166, R160 to R167, R168 to R175, R171 to R178
Changed lines of the file:
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@@
 		(on_board yes)
 		(dnp no)
-		(property "Reference" "R158"
+		(property "Reference" "R165"
 			(at 128.27 71.12 0)
 			(effects
@@
 			(project "svea_powerboard_rev3"
 				(path "/3f85abf4-0b95-4c4a-b7e9-06f59ca1ea3d/5c2e021f-c2d4-49e2-8c36-9a64f1f12001/8281c4bd-f2fa-451b-b37c-f7eda375ddce"
-					(reference "R158")
+					(reference "R165")
 					(unit 1)
 				)
@@
 		(on_board yes)
 		(dnp no)
-		(property "Reference" "#PWR0175"
+		(property "Reference" "#PWR0162"
 			(at 243.84 60.96 0)
 			(effects
@@
 			(project "svea_powerboard_rev3"
 				(path "/3f85abf4-0b95-4c4a-b7e9-06f59ca1ea3d/5c2e021f-c2d4-49e2-8c36-9a64f1f12001/8281c4bd-f2fa-451b-b37c-f7eda375ddce"
-					(reference "#PWR0175")
+					(reference "#PWR0162")
 					(unit 1)
 				)
@@
 		(on_board yes)
 		(dnp no)
-		(property "Reference" "R146"
+		(property "Reference" "R153"
 			(at 45.72 111.76 0)
 			(effects
@@
 			(project "svea_powerboard_rev3"
 				(path "/3f85abf4-0b95-4c4a-b7e9-06f59ca1ea3d/5c2e021f-c2d4-49e2-8c36-9a64f1f12001/8281c4bd-f2fa-451b-b37c-f7eda375ddce"
-					(reference "R146")
+					(reference "R153")
 					(unit 1)
 				)
@@
 		(on_board yes)
 		(dnp no)
-		(property "Reference" "R150"
+		(property "Reference" "R157"
 			(at 86.36 121.92 0)
 			(effects
@@
 			(project "svea_powerboard_rev3"
 				(path "/3f85abf4-0b95-4c4a-b7e9-06f59ca1ea3d/5c2e021f-c2d4-49e2-8c36-9a64f1f12001/8281c4bd-f2fa-451b-b37c-f7eda375ddce"
-					(reference "R150")
+					(reference "R157")
 					(unit 1)
 				)
@@
 		(on_board yes)
 		(dnp no)
-		(property "Reference" "R171"
+		(property "Reference" "R178"
 			(at 194.31 106.68 0)
 			(effects
@@
 			(project "svea_powerboard_rev3"
 				(path "/3f85abf4-0b95-4c4a-b7e9-06f59ca1ea3d/5c2e021f-c2d4-49e2-8c36-9a64f1f12001/8281c4bd-f2fa-451b-b37c-f7eda375ddce"
-					(reference "R171")
+					(reference "R178")
 					(unit 1)
 				)
@@
 		(on_board yes)
 		(dnp no)
-		(property "Reference" "R147"
+		(property "Reference" "R154"
 			(at 55.88 114.3 0)
 			(effects
@@
 			(project "svea_powerboard_rev3"
 				(path "/3f85abf4-0b95-4c4a-b7e9-06f59ca1ea3d/5c2e021f-c2d4-49e2-8c36-9a64f1f12001/8281c4bd-f2fa-451b-b37c-f7eda375ddce"
-					(reference "R147")
+					(reference "R154")
 					(unit 1)
 				)
@@
 		(on_board yes)
 		(dnp no)
-		(property "Reference" "R148"
+		(property "Reference" "R155"
 			(at 66.04 116.84 0)
 			(effects
@@
 			(project "svea_powerboard_rev3"
 				(path "/3f85abf4-0b95-4c4a-b7e9-06f59ca1ea3d/5c2e021f-c2d4-49e2-8c36-9a64f1f12001/8281c4bd-f2fa-451b-b37c-f7eda375ddce"
-					(reference "R148")
+					(reference "R155")
 					(unit 1)
 				)
@@
 		(on_board yes)
 		(dnp no)
-		(property "Reference" "R149"
+		(property "Reference" "R156"
 			(at 76.2 119.38 0)
 			(effects
@@
 			(project "svea_powerboard_rev3"
 				(path "/3f85abf4-0b95-4c4a-b7e9-06f59ca1ea3d/5c2e021f-c2d4-49e2-8c36-9a64f1f12001/8281c4bd-f2fa-451b-b37c-f7eda375ddce"
-					(reference "R149")
+					(reference "R156")
 					(unit 1)
 				)
@@
 		(on_board yes)
 		(dnp no)
-		(property "Reference" "C124"
+		(property "Reference" "C122"
 			(at 255.27 74.93 90)
 			(effects
@@
 			(project "svea_powerboard_rev3"
 				(path "/3f85abf4-0b95-4c4a-b7e9-06f59ca1ea3d/5c2e021f-c2d4-49e2-8c36-9a64f1f12001/8281c4bd-f2fa-451b-b37c-f7eda375ddce"
-					(reference "C124")
+					(reference "C122")
 					(unit 1)
 				)
@@
 		(on_board yes)
 		(dnp no)
-		(property "Reference" "R168"
+		(property "Reference" "R175"
 			(at 163.83 63.5 0)
 			(effects
@@
 			(project "svea_powerboard_rev3"
 				(path "/3f85abf4-0b95-4c4a-b7e9-06f59ca1ea3d/5c2e021f-c2d4-49e2-8c36-9a64f1f12001/8281c4bd-f2fa-451b-b37c-f7eda375ddce"
-					(reference "R168")
+					(reference "R175")
 					(unit 1)
 				)
@@
 		(on_board yes)
 		(dnp no)
-		(property "Reference" "#PWR0176"
+		(property "Reference" "#PWR0163"
 			(at 243.84 87.63 0)
 			(effects
@@
 			(project "svea_powerboard_rev3"
 				(path "/3f85abf4-0b95-4c4a-b7e9-06f59ca1ea3d/5c2e021f-c2d4-49e2-8c36-9a64f1f12001/8281c4bd-f2fa-451b-b37c-f7eda375ddce"
-					(reference "#PWR0176")
+					(reference "#PWR0163")
 					(unit 1)
 				)
@@
 		(on_board yes)
 		(dnp no)
-		(property "Reference" "#PWR0173"
+		(property "Reference" "#PWR0160"
 			(at 121.92 92.71 0)
 			(effects
@@
 			(project "svea_powerboard_rev3"
 				(path "/3f85abf4-0b95-4c4a-b7e9-06f59ca1ea3d/5c2e021f-c2d4-49e2-8c36-9a64f1f12001/8281c4bd-f2fa-451b-b37c-f7eda375ddce"
-					(reference "#PWR0173")
+					(reference "#PWR0160")
 					(unit 1)
 				)
@@
 		(on_board yes)
 		(dnp no)
-		(property "Reference" "R160"
+		(property "Reference" "R167"
 			(at 128.27 86.36 0)
 			(effects
@@
 			(project "svea_powerboard_rev3"
 				(path "/3f85abf4-0b95-4c4a-b7e9-06f59ca1ea3d/5c2e021f-c2d4-49e2-8c36-9a64f1f12001/8281c4bd-f2fa-451b-b37c-f7eda375ddce"
-					(reference "R160")
+					(reference "R167")
 					(unit 1)
 				)
@@
 		(on_board yes)
 		(dnp no)
-		(property "Reference" "R157"
+		(property "Reference" "R164"
 			(at 128.27 63.5 0)
 			(effects
@@
 			(project "svea_powerboard_rev3"
 				(path "/3f85abf4-0b95-4c4a-b7e9-06f59ca1ea3d/5c2e021f-c2d4-49e2-8c36-9a64f1f12001/8281c4bd-f2fa-451b-b37c-f7eda375ddce"
-					(reference "R157")
+					(reference "R164")
 					(unit 1)
 				)
@@
 		(on_board yes)
 		(dnp no)
-		(property "Reference" "R155"
+		(property "Reference" "R162"
 			(at 106.68 127 0)
 			(effects
@@
 			(project "svea_powerboard_rev3"
 				(path "/3f85abf4-0b95-4c4a-b7e9-06f59ca1ea3d/5c2e021f-c2d4-49e2-8c36-9a64f1f12001/8281c4bd-f2fa-451b-b37c-f7eda375ddce"
-					(reference "R155")
+					(reference "R162")
 					(unit 1)
 				)
@@
 		(on_board yes)
 		(dnp no)
-		(property "Reference" "#PWR0174"
+		(property "Reference" "#PWR0161"
 			(at 172.72 146.05 0)
 			(effects
@@
 			(project "svea_powerboard_rev3"
 				(path "/3f85abf4-0b95-4c4a-b7e9-06f59ca1ea3d/5c2e021f-c2d4-49e2-8c36-9a64f1f12001/8281c4bd-f2fa-451b-b37c-f7eda375ddce"
-					(reference "#PWR0174")
+					(reference "#PWR0161")
 					(unit 1)
 				)
@@
 		(on_board yes)
 		(dnp no)
-		(property "Reference" "C123"
+		(property "Reference" "C121"
 			(at 240.03 74.93 90)
 			(effects
@@
 			(project "svea_powerboard_rev3"
 				(path "/3f85abf4-0b95-4c4a-b7e9-06f59ca1ea3d/5c2e021f-c2d4-49e2-8c36-9a64f1f12001/8281c4bd-f2fa-451b-b37c-f7eda375ddce"
-					(reference "C123")
+					(reference "C121")
 					(unit 1)
 				)
@@
 		(on_board yes)
 		(dnp no)
-		(property "Reference" "R159"
+		(property "Reference" "R166"
 			(at 128.27 78.74 0)
 			(effects
@@
 			(project "svea_powerboard_rev3"
 				(path "/3f85abf4-0b95-4c4a-b7e9-06f59ca1ea3d/5c2e021f-c2d4-49e2-8c36-9a64f1f12001/8281c4bd-f2fa-451b-b37c-f7eda375ddce"
-					(reference "R159")
+					(reference "R166")
 					(unit 1)
 				)
@@
 		(on_board yes)
 		(dnp no)
-		(property "Reference" "R152"
+		(property "Reference" "R159"
 			(at 96.52 124.46 0)
 			(effects
@@
 			(project "svea_powerboard_rev3"
 				(path "/3f85abf4-0b95-4c4a-b7e9-06f59ca1ea3d/5c2e021f-c2d4-49e2-8c36-9a64f1f12001/8281c4bd-f2fa-451b-b37c-f7eda375ddce"
-					(reference "R152")
+					(reference "R159")
 					(unit 1)
 				)
