File: hardware/kicad/sheets/charging/23_Charging-USB-C-Port.kicad_sch (KiCad schematic)
At the start: 25 parts, among them Q56 DMP3028LK3-13, U176 TCA9517DGKRQ1, U43 HUSB238A-BB001-QN16R

Commit message: reorganized
Other:
- title: Charging-USB-C-Port -> USB-C Input
Changed lines of the file:
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@@
 	(paper "User" 398.14 217.8)
 	(title_block
-		(title "Charging-USB-C-Port")
+		(title "USB-C Input")
 		(date "2026-02-16")
 	)

Commit message: before final cleanup
Parts:
- renumbered C270 to C125, C200 to C126, C196 to C127, D83 to D38, D62 to D40, Q56 to Q19, R493 to R181, R477 to R182, R389 to R183, R180 to R184, R494 to R185, R182 to R186, R391 to R187, R101 to R188, R392 to R189, R539 to R190, R484 to R191, U176 to U54, U178 to U55, U179 to U56, U43 to U57

Commit message: resheeted bms and fixed links for the 12v buck
Parts:
- renumbered C125 to C50, C126 to C51, C127 to C52, D38 to D16, D39 to D17, D40 to D18, Q19 to Q9, R181 to R53, R182 to R54, R183 to R55, R184 to R56, R185 to R57, R186 to R58, R187 to R59, R188 to R60, R189 to R61, R190 to R62, R191 to R63, U54 to U17, U55 to U18, U56 to U19, U57 to U20
Connections:
- net IN-CHARGING-VCC-USBC renamed OUT

Commit message: starting transition to single root
Parts:
- renumbered C50 to C16, C51 to C17, C52 to C18, D17 to D10, D18 to D11, D16 to D9, Q9 to Q5, R53 to R55, R54 to R56, R55 to R57, R56 to R58, R57 to R59, R58 to R60, R59 to R61, R60 to R62, R61 to R63, R62 to R94, R63 to R95

Commit message: various improvements
Parts:
- renumbered C16 to C60, C17 to C61, C18 to C62, D9 to D21, D10 to D22, D11 to D23, Q5 to Q11, R55 to R67, R56 to R68, R57 to R69, R58 to R70, R59 to R71, R60 to R72, R61 to R73, R62 to R74, R63 to R75, R94 to R76, R95 to R77, U17 to U28, U18 to U29, U19 to U30, U20 to U31

Commit message: various improvements
Parts:
- renumbered C60 to C67, C61 to C68, C62 to C69, D21 to D24, D22 to D25, D23 to D26, R67 to R76, R68 to R77, R69 to R78, R70 to R79, R71 to R80, R72 to R81, R73 to R82, R74 to R83, R75 to R84, R76 to R85, R77 to R86

Commit message: current sensing on the servos and cleaning up empty sheets
Parts:
- renumbered C67 to C72, C68 to C73, C69 to C74, D24 to D23, D25 to D24, D26 to D25, Q11 to Q9, R76 to R74, R77 to R75, R78 to R76, R79 to R77, R80 to R78, R81 to R79, R82 to R80, R83 to R81, R84 to R82, R85 to R83, R86 to R84, U28 to U31, U29 to U32, U30 to U33, U31 to U34

Commit message: new references
Parts:
- renumbered C72 to C74, C73 to C75, C74 to C76, D23 to D22, D24 to D23, D25 to D24, R77 to R100, R78 to R101, R79 to R102, R80 to R103, R81 to R104, R82 to R105, R83 to R106, R84 to R107, R74 to R97, R75 to R98, R76 to R99, U31 to U37, U32 to U38, U33 to U39, U34 to U40
