File: hardware/kicad/sheets/charging/highcurrendiodeor.kicad_sch (KiCad schematic)
At the start: 8 parts, among them CN6 5017, Q3 CSD17577Q5A, U13 LM5050MKX-1/NOPB

Commit message: new references
Parts:
- renumbered C30 to C31, C31 to C32, D14 to D13, R29 to R51, R30 to R52, U13 to U18

Commit message: pre robot updating references
Parts:
- renumbered C31 to C30, C32 to C31, R51 to R59, R52 to R60, U18 to U19
Changed lines of the file:
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@@
 		(on_board yes)
 		(dnp no)
-		(property "Reference" "R51"
+		(property "Reference" "R59"
 			(at 153.67 123.19 90)
 			(effects
@@
 			(project "svea_powerboard_rev3"
 				(path "/3f85abf4-0b95-4c4a-b7e9-06f59ca1ea3d/5c2e021f-c2d4-49e2-8c36-9a64f1f12001/8eee6623-4878-45b2-bdab-0e37d3220c38"
-					(reference "R77")
+					(reference "R85")
 					(unit 1)
 				)
 				(path "/3f85abf4-0b95-4c4a-b7e9-06f59ca1ea3d/5c2e021f-c2d4-49e2-8c36-9a64f1f12001/a048a8c1-de8c-4417-9e40-d40a18f390ce"
-					(reference "R51")
+					(reference "R59")
 					(unit 1)
 				)
 				(path "/3f85abf4-0b95-4c4a-b7e9-06f59ca1ea3d/5c2e021f-c2d4-49e2-8c36-9a64f1f12001/ad660ab0-1da6-44b7-9096-9ee4c3bc2383"
-					(reference "R53")
+					(reference "R61")
 					(unit 1)
 				)
 				(path "/3f85abf4-0b95-4c4a-b7e9-06f59ca1ea3d/5c2e021f-c2d4-49e2-8c36-9a64f1f12001/ca919776-c91b-4883-8f90-f75d19396b00"
-					(reference "R55")
+					(reference "R63")
 					(unit 1)
 				)
 				(path "/3f85abf4-0b95-4c4a-b7e9-06f59ca1ea3d/5c2e021f-c2d4-49e2-8c36-9a64f1f12001/d932e0fc-7b09-4e74-a033-a342c08a0a15"
-					(reference "R87")
+					(reference "R95")
 					(unit 1)
 				)
 				(path "/3f85abf4-0b95-4c4a-b7e9-06f59ca1ea3d/5c2e021f-c2d4-49e2-8c36-9a64f1f12001/dbcfb661-1d23-45dc-813f-0febc1515a98"
-					(reference "R75")
+					(reference "R83")
 					(unit 1)
 				)
@@
 		(on_board yes)
 		(dnp no)
-		(property "Reference" "R52"
+		(property "Reference" "R60"
 			(at 213.36 83.82 90)
 			(effects
@@
 			(project "svea_powerboard_rev3"
 				(path "/3f85abf4-0b95-4c4a-b7e9-06f59ca1ea3d/5c2e021f-c2d4-49e2-8c36-9a64f1f12001/8eee6623-4878-45b2-bdab-0e37d3220c38"
-					(reference "R78")
+					(reference "R86")
 					(unit 1)
 				)
 				(path "/3f85abf4-0b95-4c4a-b7e9-06f59ca1ea3d/5c2e021f-c2d4-49e2-8c36-9a64f1f12001/a048a8c1-de8c-4417-9e40-d40a18f390ce"
-					(reference "R52")
+					(reference "R60")
 					(unit 1)
 				)
 				(path "/3f85abf4-0b95-4c4a-b7e9-06f59ca1ea3d/5c2e021f-c2d4-49e2-8c36-9a64f1f12001/ad660ab0-1da6-44b7-9096-9ee4c3bc2383"
-					(reference "R54")
+					(reference "R62")
 					(unit 1)
 				)
 				(path "/3f85abf4-0b95-4c4a-b7e9-06f59ca1ea3d/5c2e021f-c2d4-49e2-8c36-9a64f1f12001/ca919776-c91b-4883-8f90-f75d19396b00"
-					(reference "R56")
+					(reference "R64")
 					(unit 1)
 				)
 				(path "/3f85abf4-0b95-4c4a-b7e9-06f59ca1ea3d/5c2e021f-c2d4-49e2-8c36-9a64f1f12001/d932e0fc-7b09-4e74-a033-a342c08a0a15"
-					(reference "R88")
+					(reference "R96")
 					(unit 1)
 				)
 				(path "/3f85abf4-0b95-4c4a-b7e9-06f59ca1ea3d/5c2e021f-c2d4-49e2-8c36-9a64f1f12001/dbcfb661-1d23-45dc-813f-0febc1515a98"
-					(reference "R76")
+					(reference "R84")
 					(unit 1)
 				)
@@
 		(on_board yes)
 		(dnp no)
-		(property "Reference" "C31"
+		(property "Reference" "C30"
 			(at 139.7 86.36 90)
 			(effects
@@
 			(project "svea_powerboard_rev3"
 				(path "/3f85abf4-0b95-4c4a-b7e9-06f59ca1ea3d/5c2e021f-c2d4-49e2-8c36-9a64f1f12001/8eee6623-4878-45b2-bdab-0e37d3220c38"
-					(reference "C61")
+					(reference "C60")
 					(unit 1)
 				)
 				(path "/3f85abf4-0b95-4c4a-b7e9-06f59ca1ea3d/5c2e021f-c2d4-49e2-8c36-9a64f1f12001/a048a8c1-de8c-4417-9e40-d40a18f390ce"
-					(reference "C31")
+					(reference "C30")
 					(unit 1)
 				)
 				(path "/3f85abf4-0b95-4c4a-b7e9-06f59ca1ea3d/5c2e021f-c2d4-49e2-8c36-9a64f1f12001/ad660ab0-1da6-44b7-9096-9ee4c3bc2383"
-					(reference "C33")
+					(reference "C32")
 					(unit 1)
 				)
 				(path "/3f85abf4-0b95-4c4a-b7e9-06f59ca1ea3d/5c2e021f-c2d4-49e2-8c36-9a64f1f12001/ca919776-c91b-4883-8f90-f75d19396b00"
-					(reference "C35")
+					(reference "C34")
 					(unit 1)
 				)
 				(path "/3f85abf4-0b95-4c4a-b7e9-06f59ca1ea3d/5c2e021f-c2d4-49e2-8c36-9a64f1f12001/d932e0fc-7b09-4e74-a033-a342c08a0a15"
-					(reference "C70")
+					(reference "C69")
 					(unit 1)
 				)
 				(path "/3f85abf4-0b95-4c4a-b7e9-06f59ca1ea3d/5c2e021f-c2d4-49e2-8c36-9a64f1f12001/dbcfb661-1d23-45dc-813f-0febc1515a98"
-					(reference "C59")
+					(reference "C58")
 					(unit 1)
 				)
@@
 		(on_board yes)
 		(dnp no)
-		(property "Reference" "#PWR063"
+		(property "Reference" "#PWR073"
 			(at 151.13 129.54 0)
 			(effects
@@
 			(project "svea_powerboard_rev3"
 				(path "/3f85abf4-0b95-4c4a-b7e9-06f59ca1ea3d/5c2e021f-c2d4-49e2-8c36-9a64f1f12001/8eee6623-4878-45b2-bdab-0e37d3220c38"
-					(reference "#PWR094")
+					(reference "#PWR096")
 					(unit 1)
 				)
 				(path "/3f85abf4-0b95-4c4a-b7e9-06f59ca1ea3d/5c2e021f-c2d4-49e2-8c36-9a64f1f12001/a048a8c1-de8c-4417-9e40-d40a18f390ce"
-					(reference "#PWR063")
+					(reference "#PWR073")
 					(unit 1)
 				)
 				(path "/3f85abf4-0b95-4c4a-b7e9-06f59ca1ea3d/5c2e021f-c2d4-49e2-8c36-9a64f1f12001/ad660ab0-1da6-44b7-9096-9ee4c3bc2383"
-					(reference "#PWR066")
+					(reference "#PWR074")
 					(unit 1)
 				)
 				(path "/3f85abf4-0b95-4c4a-b7e9-06f59ca1ea3d/5c2e021f-c2d4-49e2-8c36-9a64f1f12001/ca919776-c91b-4883-8f90-f75d19396b00"
-					(reference "#PWR069")
+					(reference "#PWR075")
 					(unit 1)
 				)
 				(path "/3f85abf4-0b95-4c4a-b7e9-06f59ca1ea3d/5c2e021f-c2d4-49e2-8c36-9a64f1f12001/d932e0fc-7b09-4e74-a033-a342c08a0a15"
-					(reference "#PWR0108")
+					(reference "#PWR0105")
 					(unit 1)
 				)
 				(path "/3f85abf4-0b95-4c4a-b7e9-06f59ca1ea3d/5c2e021f-c2d4-49e2-8c36-9a64f1f12001/dbcfb661-1d23-45dc-813f-0febc1515a98"
-					(reference "#PWR091")
+					(reference "#PWR095")
 					(unit 1)
 				)
@@
 		(on_board yes)
 		(dnp no)
-		(property "Reference" "U18"
+		(property "Reference" "U19"
 			(at 157.48 92.71 0)
 			(effects
@@
 			(project "svea_powerboard_rev3"
 				(path "/3f85abf4-0b95-4c4a-b7e9-06f59ca1ea3d/5c2e021f-c2d4-49e2-8c36-9a64f1f12001/8eee6623-4878-45b2-bdab-0e37d3220c38"
+					(reference "U31")
+					(unit 1)
+				)
+				(path "/3f85abf4-0b95-4c4a-b7e9-06f59ca1ea3d/5c2e021f-c2d4-49e2-8c36-9a64f1f12001/a048a8c1-de8c-4417-9e40-d40a18f390ce"
+					(reference "U19")
+					(unit 1)
+				)
+				(path "/3f85abf4-0b95-4c4a-b7e9-06f59ca1ea3d/5c2e021f-c2d4-49e2-8c36-9a64f1f12001/ad660ab0-1da6-44b7-9096-9ee4c3bc2383"
+					(reference "U20")
+					(unit 1)
+				)
+				(path "/3f85abf4-0b95-4c4a-b7e9-06f59ca1ea3d/5c2e021f-c2d4-49e2-8c36-9a64f1f12001/ca919776-c91b-4883-8f90-f75d19396b00"
+					(reference "U21")
+					(unit 1)
+				)
+				(path "/3f85abf4-0b95-4c4a-b7e9-06f59ca1ea3d/5c2e021f-c2d4-49e2-8c36-9a64f1f12001/d932e0fc-7b09-4e74-a033-a342c08a0a15"
+					(reference "U34")
+					(unit 1)
+				)
+				(path "/3f85abf4-0b95-4c4a-b7e9-06f59ca1ea3d/5c2e021f-c2d4-49e2-8c36-9a64f1f12001/dbcfb661-1d23-45dc-813f-0febc1515a98"
 					(reference "U30")
-					(unit 1)
-				)
-				(path "/3f85abf4-0b95-4c4a-b7e9-06f59ca1ea3d/5c2e021f-c2d4-49e2-8c36-9a64f1f12001/a048a8c1-de8c-4417-9e40-d40a18f390ce"
-					(reference "U18")
-					(unit 1)
-				)
-				(path "/3f85abf4-0b95-4c4a-b7e9-06f59ca1ea3d/5c2e021f-c2d4-49e2-8c36-9a64f1f12001/ad660ab0-1da6-44b7-9096-9ee4c3bc2383"
-					(reference "U19")
-					(unit 1)
-				)
-				(path "/3f85abf4-0b95-4c4a-b7e9-06f59ca1ea3d/5c2e021f-c2d4-49e2-8c36-9a64f1f12001/ca919776-c91b-4883-8f90-f75d19396b00"
-					(reference "U20")
-					(unit 1)
-				)
-				(path "/3f85abf4-0b95-4c4a-b7e9-06f59ca1ea3d/5c2e021f-c2d4-49e2-8c36-9a64f1f12001/d932e0fc-7b09-4e74-a033-a342c08a0a15"
-					(reference "U33")
-					(unit 1)
-				)
-				(path "/3f85abf4-0b95-4c4a-b7e9-06f59ca1ea3d/5c2e021f-c2d4-49e2-8c36-9a64f1f12001/dbcfb661-1d23-45dc-813f-0febc1515a98"
-					(reference "U29")
 					(unit 1)
 				)
@@
 		(on_board yes)
 		(dnp no)
-		(property "Reference" "C32"
+		(property "Reference" "C31"
 			(at 214.63 96.52 90)
 			(effects
@@
 			(project "svea_powerboard_rev3"
 				(path "/3f85abf4-0b95-4c4a-b7e9-06f59ca1ea3d/5c2e021f-c2d4-49e2-8c36-9a64f1f12001/8eee6623-4878-45b2-bdab-0e37d3220c38"
-					(reference "C62")
+					(reference "C61")
 					(unit 1)
 				)
 				(path "/3f85abf4-0b95-4c4a-b7e9-06f59ca1ea3d/5c2e021f-c2d4-49e2-8c36-9a64f1f12001/a048a8c1-de8c-4417-9e40-d40a18f390ce"
-					(reference "C32")
+					(reference "C31")
 					(unit 1)
 				)
 				(path "/3f85abf4-0b95-4c4a-b7e9-06f59ca1ea3d/5c2e021f-c2d4-49e2-8c36-9a64f1f12001/ad660ab0-1da6-44b7-9096-9ee4c3bc2383"
-					(reference "C34")
+					(reference "C33")
 					(unit 1)
 				)
 				(path "/3f85abf4-0b95-4c4a-b7e9-06f59ca1ea3d/5c2e021f-c2d4-49e2-8c36-9a64f1f12001/ca919776-c91b-4883-8f90-f75d19396b00"
-					(reference "C36")
+					(reference "C35")
 					(unit 1)
 				)
 				(path "/3f85abf4-0b95-4c4a-b7e9-06f59ca1ea3d/5c2e021f-c2d4-49e2-8c36-9a64f1f12001/d932e0fc-7b09-4e74-a033-a342c08a0a15"
-					(reference "C71")
+					(reference "C70")
 					(unit 1)
 				)
 				(path "/3f85abf4-0b95-4c4a-b7e9-06f59ca1ea3d/5c2e021f-c2d4-49e2-8c36-9a64f1f12001/dbcfb661-1d23-45dc-813f-0febc1515a98"
-					(reference "C60")
-					(unit 1)
-				)
+					(reference "C59")
+					(unit 1)
+				)

Commit message: various imprvements
Parts:
- D13: value SS16T3G -> ~; footprint Diode_SMD:SMA -> 5v rail sm-easyedapro:SMA_L4.4-W2.8-LS5.4-RD
- renumbered C30 to C35, C31 to C36, R59 to R89, R60 to R90, U19 to U25

Commit message: updated some footprints, fixed board
Parts:
- renumbered C35 to C33, C36 to C34, R89 to R90, R90 to R91, U25 to U24
Changed lines of the file:
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@@
 		(on_board yes)
 		(dnp no)
-		(property "Reference" "R89"
+		(property "Reference" "R90"
 			(at 153.67 123.19 90)
 			(effects
@@
 			(project "svea_powerboard_rev3"
 				(path "/3f85abf4-0b95-4c4a-b7e9-06f59ca1ea3d/5c2e021f-c2d4-49e2-8c36-9a64f1f12001/8eee6623-4878-45b2-bdab-0e37d3220c38"
-					(reference "R115")
+					(reference "R116")
 					(unit 1)
 				)
 				(path "/3f85abf4-0b95-4c4a-b7e9-06f59ca1ea3d/5c2e021f-c2d4-49e2-8c36-9a64f1f12001/a048a8c1-de8c-4417-9e40-d40a18f390ce"
-					(reference "R89")
+					(reference "R90")
 					(unit 1)
 				)
 				(path "/3f85abf4-0b95-4c4a-b7e9-06f59ca1ea3d/5c2e021f-c2d4-49e2-8c36-9a64f1f12001/ad660ab0-1da6-44b7-9096-9ee4c3bc2383"
-					(reference "R91")
+					(reference "R92")
 					(unit 1)
 				)
 				(path "/3f85abf4-0b95-4c4a-b7e9-06f59ca1ea3d/5c2e021f-c2d4-49e2-8c36-9a64f1f12001/ca919776-c91b-4883-8f90-f75d19396b00"
-					(reference "R93")
+					(reference "R94")
 					(unit 1)
 				)
 				(path "/3f85abf4-0b95-4c4a-b7e9-06f59ca1ea3d/5c2e021f-c2d4-49e2-8c36-9a64f1f12001/d932e0fc-7b09-4e74-a033-a342c08a0a15"
-					(reference "R125")
+					(reference "R126")
 					(unit 1)
 				)
 				(path "/3f85abf4-0b95-4c4a-b7e9-06f59ca1ea3d/5c2e021f-c2d4-49e2-8c36-9a64f1f12001/dbcfb661-1d23-45dc-813f-0febc1515a98"
-					(reference "R113")
+					(reference "R114")
 					(unit 1)
 				)
@@
 		(on_board yes)
 		(dnp no)
-		(property "Reference" "R90"
+		(property "Reference" "R91"
 			(at 213.36 83.82 90)
 			(effects
@@
 			(project "svea_powerboard_rev3"
 				(path "/3f85abf4-0b95-4c4a-b7e9-06f59ca1ea3d/5c2e021f-c2d4-49e2-8c36-9a64f1f12001/8eee6623-4878-45b2-bdab-0e37d3220c38"
-					(reference "R116")
+					(reference "R117")
 					(unit 1)
 				)
 				(path "/3f85abf4-0b95-4c4a-b7e9-06f59ca1ea3d/5c2e021f-c2d4-49e2-8c36-9a64f1f12001/a048a8c1-de8c-4417-9e40-d40a18f390ce"
-					(reference "R90")
+					(reference "R91")
 					(unit 1)
 				)
 				(path "/3f85abf4-0b95-4c4a-b7e9-06f59ca1ea3d/5c2e021f-c2d4-49e2-8c36-9a64f1f12001/ad660ab0-1da6-44b7-9096-9ee4c3bc2383"
-					(reference "R92")
+					(reference "R93")
 					(unit 1)
 				)
 				(path "/3f85abf4-0b95-4c4a-b7e9-06f59ca1ea3d/5c2e021f-c2d4-49e2-8c36-9a64f1f12001/ca919776-c91b-4883-8f90-f75d19396b00"
-					(reference "R94")
+					(reference "R95")
 					(unit 1)
 				)
 				(path "/3f85abf4-0b95-4c4a-b7e9-06f59ca1ea3d/5c2e021f-c2d4-49e2-8c36-9a64f1f12001/d932e0fc-7b09-4e74-a033-a342c08a0a15"
-					(reference "R126")
+					(reference "R127")
 					(unit 1)
 				)
 				(path "/3f85abf4-0b95-4c4a-b7e9-06f59ca1ea3d/5c2e021f-c2d4-49e2-8c36-9a64f1f12001/dbcfb661-1d23-45dc-813f-0febc1515a98"
-					(reference "R114")
+					(reference "R115")
 					(unit 1)
 				)
@@
 		(on_board yes)
 		(dnp no)
-		(property "Reference" "C35"
+		(property "Reference" "C33"
 			(at 139.7 86.36 90)
 			(effects
@@
 			(project "svea_powerboard_rev3"
 				(path "/3f85abf4-0b95-4c4a-b7e9-06f59ca1ea3d/5c2e021f-c2d4-49e2-8c36-9a64f1f12001/8eee6623-4878-45b2-bdab-0e37d3220c38"
-					(reference "C65")
+					(reference "C63")
 					(unit 1)
 				)
 				(path "/3f85abf4-0b95-4c4a-b7e9-06f59ca1ea3d/5c2e021f-c2d4-49e2-8c36-9a64f1f12001/a048a8c1-de8c-4417-9e40-d40a18f390ce"
+					(reference "C33")
+					(unit 1)
+				)
+				(path "/3f85abf4-0b95-4c4a-b7e9-06f59ca1ea3d/5c2e021f-c2d4-49e2-8c36-9a64f1f12001/ad660ab0-1da6-44b7-9096-9ee4c3bc2383"
 					(reference "C35")
 					(unit 1)
 				)
-				(path "/3f85abf4-0b95-4c4a-b7e9-06f59ca1ea3d/5c2e021f-c2d4-49e2-8c36-9a64f1f12001/ad660ab0-1da6-44b7-9096-9ee4c3bc2383"
+				(path "/3f85abf4-0b95-4c4a-b7e9-06f59ca1ea3d/5c2e021f-c2d4-49e2-8c36-9a64f1f12001/ca919776-c91b-4883-8f90-f75d19396b00"
 					(reference "C37")
 					(unit 1)
 				)
-				(path "/3f85abf4-0b95-4c4a-b7e9-06f59ca1ea3d/5c2e021f-c2d4-49e2-8c36-9a64f1f12001/ca919776-c91b-4883-8f90-f75d19396b00"
-					(reference "C39")
-					(unit 1)
-				)
 				(path "/3f85abf4-0b95-4c4a-b7e9-06f59ca1ea3d/5c2e021f-c2d4-49e2-8c36-9a64f1f12001/d932e0fc-7b09-4e74-a033-a342c08a0a15"
-					(reference "C74")
+					(reference "C72")
 					(unit 1)
 				)
 				(path "/3f85abf4-0b95-4c4a-b7e9-06f59ca1ea3d/5c2e021f-c2d4-49e2-8c36-9a64f1f12001/dbcfb661-1d23-45dc-813f-0febc1515a98"
-					(reference "C63")
+					(reference "C61")
 					(unit 1)
 				)
@@
 		(on_board yes)
 		(dnp no)
-		(property "Reference" "#PWR086"
+		(property "Reference" "#PWR082"
 			(at 151.13 129.54 0)
 			(effects
@@
 			(project "svea_powerboard_rev3"
 				(path "/3f85abf4-0b95-4c4a-b7e9-06f59ca1ea3d/5c2e021f-c2d4-49e2-8c36-9a64f1f12001/8eee6623-4878-45b2-bdab-0e37d3220c38"
-					(reference "#PWR0109")
+					(reference "#PWR0105")
 					(unit 1)
 				)
 				(path "/3f85abf4-0b95-4c4a-b7e9-06f59ca1ea3d/5c2e021f-c2d4-49e2-8c36-9a64f1f12001/a048a8c1-de8c-4417-9e40-d40a18f390ce"
-					(reference "#PWR086")
+					(reference "#PWR082")
 					(unit 1)
 				)
 				(path "/3f85abf4-0b95-4c4a-b7e9-06f59ca1ea3d/5c2e021f-c2d4-49e2-8c36-9a64f1f12001/ad660ab0-1da6-44b7-9096-9ee4c3bc2383"
-					(reference "#PWR087")
+					(reference "#PWR083")
 					(unit 1)
 				)
 				(path "/3f85abf4-0b95-4c4a-b7e9-06f59ca1ea3d/5c2e021f-c2d4-49e2-8c36-9a64f1f12001/ca919776-c91b-4883-8f90-f75d19396b00"
-					(reference "#PWR088")
+					(reference "#PWR084")
 					(unit 1)
 				)
 				(path "/3f85abf4-0b95-4c4a-b7e9-06f59ca1ea3d/5c2e021f-c2d4-49e2-8c36-9a64f1f12001/d932e0fc-7b09-4e74-a033-a342c08a0a15"
-					(reference "#PWR0118")
+					(reference "#PWR0114")
 					(unit 1)
 				)
 				(path "/3f85abf4-0b95-4c4a-b7e9-06f59ca1ea3d/5c2e021f-c2d4-49e2-8c36-9a64f1f12001/dbcfb661-1d23-45dc-813f-0febc1515a98"
-					(reference "#PWR0108")
+					(reference "#PWR0104")
 					(unit 1)
 				)
@@
 		(on_board yes)
 		(dnp no)
-		(property "Reference" "U25"
+		(property "Reference" "U24"
 			(at 157.48 92.71 0)
 			(effects
@@
 			(project "svea_powerboard_rev3"
 				(path "/3f85abf4-0b95-4c4a-b7e9-06f59ca1ea3d/5c2e021f-c2d4-49e2-8c36-9a64f1f12001/8eee6623-4878-45b2-bdab-0e37d3220c38"
-					(reference "U37")
+					(reference "U36")
 					(unit 1)
 				)
 				(path "/3f85abf4-0b95-4c4a-b7e9-06f59ca1ea3d/5c2e021f-c2d4-49e2-8c36-9a64f1f12001/a048a8c1-de8c-4417-9e40-d40a18f390ce"
+					(reference "U24")
+					(unit 1)
+				)
+				(path "/3f85abf4-0b95-4c4a-b7e9-06f59ca1ea3d/5c2e021f-c2d4-49e2-8c36-9a64f1f12001/ad660ab0-1da6-44b7-9096-9ee4c3bc2383"
 					(reference "U25")
 					(unit 1)
 				)
-				(path "/3f85abf4-0b95-4c4a-b7e9-06f59ca1ea3d/5c2e021f-c2d4-49e2-8c36-9a64f1f12001/ad660ab0-1da6-44b7-9096-9ee4c3bc2383"
+				(path "/3f85abf4-0b95-4c4a-b7e9-06f59ca1ea3d/5c2e021f-c2d4-49e2-8c36-9a64f1f12001/ca919776-c91b-4883-8f90-f75d19396b00"
 					(reference "U26")
 					(unit 1)
 				)
-				(path "/3f85abf4-0b95-4c4a-b7e9-06f59ca1ea3d/5c2e021f-c2d4-49e2-8c36-9a64f1f12001/ca919776-c91b-4883-8f90-f75d19396b00"
-					(reference "U27")
-					(unit 1)
-				)
 				(path "/3f85abf4-0b95-4c4a-b7e9-06f59ca1ea3d/5c2e021f-c2d4-49e2-8c36-9a64f1f12001/d932e0fc-7b09-4e74-a033-a342c08a0a15"
-					(reference "U40")
+					(reference "U39")
 					(unit 1)
 				)
 				(path "/3f85abf4-0b95-4c4a-b7e9-06f59ca1ea3d/5c2e021f-c2d4-49e2-8c36-9a64f1f12001/dbcfb661-1d23-45dc-813f-0febc1515a98"
-					(reference "U36")
+					(reference "U35")
 					(unit 1)
 				)
@@
 		(on_board yes)
 		(dnp no)
-		(property "Reference" "C36"
+		(property "Reference" "C34"
 			(at 214.63 96.52 90)
 			(effects
@@
 			(project "svea_powerboard_rev3"
 				(path "/3f85abf4-0b95-4c4a-b7e9-06f59ca1ea3d/5c2e021f-c2d4-49e2-8c36-9a64f1f12001/8eee6623-4878-45b2-bdab-0e37d3220c38"
-					(reference "C66")
+					(reference "C64")
 					(unit 1)
 				)
 				(path "/3f85abf4-0b95-4c4a-b7e9-06f59ca1ea3d/5c2e021f-c2d4-49e2-8c36-9a64f1f12001/a048a8c1-de8c-4417-9e40-d40a18f390ce"
+					(reference "C34")
+					(unit 1)
+				)
+				(path "/3f85abf4-0b95-4c4a-b7e9-06f59ca1ea3d/5c2e021f-c2d4-49e2-8c36-9a64f1f12001/ad660ab0-1da6-44b7-9096-9ee4c3bc2383"
 					(reference "C36")
 					(unit 1)
 				)
-				(path "/3f85abf4-0b95-4c4a-b7e9-06f59ca1ea3d/5c2e021f-c2d4-49e2-8c36-9a64f1f12001/ad660ab0-1da6-44b7-9096-9ee4c3bc2383"
+				(path "/3f85abf4-0b95-4c4a-b7e9-06f59ca1ea3d/5c2e021f-c2d4-49e2-8c36-9a64f1f12001/ca919776-c91b-4883-8f90-f75d19396b00"
 					(reference "C38")
 					(unit 1)
 				)
-				(path "/3f85abf4-0b95-4c4a-b7e9-06f59ca1ea3d/5c2e021f-c2d4-49e2-8c36-9a64f1f12001/ca919776-c91b-4883-8f90-f75d19396b00"
-					(reference "C40")
-					(unit 1)
-				)
 				(path "/3f85abf4-0b95-4c4a-b7e9-06f59ca1ea3d/5c2e021f-c2d4-49e2-8c36-9a64f1f12001/d932e0fc-7b09-4e74-a033-a342c08a0a15"
-					(reference "C75")
+					(reference "C73")
 					(unit 1)
 				)
 				(path "/3f85abf4-0b95-4c4a-b7e9-06f59ca1ea3d/5c2e021f-c2d4-49e2-8c36-9a64f1f12001/dbcfb661-1d23-45dc-813f-0febc1515a98"
-					(reference "C64")
-					(unit 1)
-				)
+					(reference "C62")
+					(unit 1)
+				)
