File: hardware/kicad/sheets/modules/bms_button_logic.kicad_sch (KiCad schematic)
At the start: 13 parts, among them Q18 L2N7002SLLT1G, SW1 TL3305AF160QG, U61 NCP718ASN330T1G, U63 PMEG10030ELPX

Commit message: pre robot updating references
Parts:
- renumbered C129 to C127, C131 to C129, C133 to C131, R177 to R184, R178 to R185, R179 to R186, R180 to R187
Changed lines of the file:
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@@
 	(wire
 		(pts
-			(xy 113.03 78.74) (xy 113.03 80.01)
+			(xy 113.03 73.66) (xy 113.03 80.01)
 		)
 		(stroke
@@
 	(hierarchical_label "3v3"
 		(shape output)
-		(at 113.03 78.74 90)
+		(at 113.03 73.66 90)
 		(effects
 			(font
@@
 		(on_board yes)
 		(dnp no)
-		(property "Reference" "R178"
+		(property "Reference" "R185"
 			(at 161.29 124.46 90)
 			(effects
@@
 			(project "svea_powerboard_rev3"
 				(path "/3f85abf4-0b95-4c4a-b7e9-06f59ca1ea3d/5c2e021f-c2d4-49e2-8c36-9a64f1f12001/261b4c59-ebc7-47a2-bb10-0e71ece0f9bf"
-					(reference "R178")
+					(reference "R185")
 					(unit 1)
 				)
@@
 		(on_board yes)
 		(dnp no)
-		(property "Reference" "R180"
+		(property "Reference" "R187"
 			(at 209.55 124.46 90)
 			(effects
@@
 			(project "svea_powerboard_rev3"
 				(path "/3f85abf4-0b95-4c4a-b7e9-06f59ca1ea3d/5c2e021f-c2d4-49e2-8c36-9a64f1f12001/261b4c59-ebc7-47a2-bb10-0e71ece0f9bf"
-					(reference "R180")
+					(reference "R187")
 					(unit 1)
 				)
@@
 		(on_board yes)
 		(dnp no)
-		(property "Reference" "C129"
+		(property "Reference" "C127"
 			(at 64.77 96.52 90)
 			(effects
@@
 			(project "svea_powerboard_rev3"
 				(path "/3f85abf4-0b95-4c4a-b7e9-06f59ca1ea3d/5c2e021f-c2d4-49e2-8c36-9a64f1f12001/261b4c59-ebc7-47a2-bb10-0e71ece0f9bf"
-					(reference "C129")
+					(reference "C127")
 					(unit 1)
 				)
@@
 		(on_board yes)
 		(dnp no)
-		(property "Reference" "R177"
+		(property "Reference" "R184"
 			(at 78.74 97.79 90)
 			(effects
@@
 			(project "svea_powerboard_rev3"
 				(path "/3f85abf4-0b95-4c4a-b7e9-06f59ca1ea3d/5c2e021f-c2d4-49e2-8c36-9a64f1f12001/261b4c59-ebc7-47a2-bb10-0e71ece0f9bf"
-					(reference "R177")
+					(reference "R184")
 					(unit 1)
 				)
@@
 		(on_board yes)
 		(dnp no)
-		(property "Reference" "C133"
+		(property "Reference" "C131"
 			(at 190.5 124.46 90)
 			(effects
@@
 			(project "svea_powerboard_rev3"
 				(path "/3f85abf4-0b95-4c4a-b7e9-06f59ca1ea3d/5c2e021f-c2d4-49e2-8c36-9a64f1f12001/261b4c59-ebc7-47a2-bb10-0e71ece0f9bf"
-					(reference "C133")
+					(reference "C131")
 					(unit 1)
 				)
@@
 		(on_board yes)
 		(dnp no)
-		(property "Reference" "R179"
+		(property "Reference" "R186"
 			(at 209.55 68.58 90)
 			(effects
@@
 			(project "svea_powerboard_rev3"
 				(path "/3f85abf4-0b95-4c4a-b7e9-06f59ca1ea3d/5c2e021f-c2d4-49e2-8c36-9a64f1f12001/261b4c59-ebc7-47a2-bb10-0e71ece0f9bf"
-					(reference "R179")
+					(reference "R186")
 					(unit 1)
 				)
@@
 		(on_board yes)
 		(dnp no)
-		(property "Reference" "C131"
+		(property "Reference" "C129"
 			(at 116.84 93.98 90)
 			(effects
@@
 			(project "svea_powerboard_rev3"
 				(path "/3f85abf4-0b95-4c4a-b7e9-06f59ca1ea3d/5c2e021f-c2d4-49e2-8c36-9a64f1f12001/261b4c59-ebc7-47a2-bb10-0e71ece0f9bf"
-					(reference "C131")
+					(reference "C129")
 					(unit 1)
 				)

Commit message: various imprvements
Parts:
- renumbered C127 to C133, C129 to C135, C131 to C137, D38 to D39, Q18 to Q19, R184 to R220, R185 to R221, R186 to R222, R187 to R223, U61 to U68, U63 to U70
Connections:
- net BTN_HIGH renamed Button/HIGH
- net BTN_LOW renamed Button/LOW
- net MCU-BTN-DIGITAL renamed Button/DIGITAL
Changed lines of the file:
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@@
 		)
 	)
-	(global_label "MCU-BTN-DIGITAL"
-		(shape input)
+	(global_label "Button/DIGITAL"
+		(shape output)
 		(at 153.67 95.25 180)
 		(effects
@@
 		(property "Intersheetrefs" "${INTERSHEET_REFS}"
 			(at 153.67 95.25 0)
+			(effects
+				(font
+					(size 1.27 1.27)
+				)
+				(hide yes)
+			)
+		)
+	)
+	(global_label "Button/LOW"
+		(shape output)
+		(at 186.69 110.49 0)
+		(effects
+			(font
+				(size 1.5748 1.5748)
+			)
+			(justify left)
+		)
+		(property "Intersheetrefs" "${INTERSHEET_REFS}"
+			(at 186.69 110.49 0)
 			(effects
 				(font
@@
 		)
 	)
-	(hierarchical_label "BTN_HIGH"
+	(hierarchical_label "Button/HIGH"
 		(shape passive)
 		(at 210.82 80.01 0)
@@
 		)
 	)
-	(hierarchical_label "BTN_LOW"
+	(hierarchical_label "Button/LOW"
 		(shape passive)
 		(at 210.82 110.49 0)
@@
 		(on_board yes)
 		(dnp no)
-		(property "Reference" "R185"
+		(property "Reference" "R221"
 			(at 161.29 124.46 90)
 			(effects
@@
 			(project "svea_powerboard_rev3"
 				(path "/3f85abf4-0b95-4c4a-b7e9-06f59ca1ea3d/5c2e021f-c2d4-49e2-8c36-9a64f1f12001/261b4c59-ebc7-47a2-bb10-0e71ece0f9bf"
-					(reference "R185")
+					(reference "R221")
 					(unit 1)
 				)
@@
 		(on_board yes)
 		(dnp no)
-		(property "Reference" "D38"
+		(property "Reference" "D39"
 			(at 175.26 124.46 90)
 			(effects
@@
 			(project "svea_powerboard_rev3"
 				(path "/3f85abf4-0b95-4c4a-b7e9-06f59ca1ea3d/5c2e021f-c2d4-49e2-8c36-9a64f1f12001/261b4c59-ebc7-47a2-bb10-0e71ece0f9bf"
-					(reference "D38")
+					(reference "D39")
 					(unit 1)
 				)
@@
 		(on_board yes)
 		(dnp no)
-		(property "Reference" "R187"
+		(property "Reference" "R223"
 			(at 209.55 124.46 90)
 			(effects
@@
 			(project "svea_powerboard_rev3"
 				(path "/3f85abf4-0b95-4c4a-b7e9-06f59ca1ea3d/5c2e021f-c2d4-49e2-8c36-9a64f1f12001/261b4c59-ebc7-47a2-bb10-0e71ece0f9bf"
-					(reference "R187")
+					(reference "R223")
 					(unit 1)
 				)
@@
 		(on_board yes)
 		(dnp no)
-		(property "Reference" "C127"
+		(property "Reference" "C133"
 			(at 64.77 96.52 90)
 			(effects
@@
 			(project "svea_powerboard_rev3"
 				(path "/3f85abf4-0b95-4c4a-b7e9-06f59ca1ea3d/5c2e021f-c2d4-49e2-8c36-9a64f1f12001/261b4c59-ebc7-47a2-bb10-0e71ece0f9bf"
-					(reference "C127")
+					(reference "C133")
 					(unit 1)
 				)
@@
 		(on_board yes)
 		(dnp no)
-		(property "Reference" "U61"
+		(property "Reference" "U68"
 			(at 81.28 76.2 0)
 			(effects
@@
 			(project "svea_powerboard_rev3"
 				(path "/3f85abf4-0b95-4c4a-b7e9-06f59ca1ea3d/5c2e021f-c2d4-49e2-8c36-9a64f1f12001/261b4c59-ebc7-47a2-bb10-0e71ece0f9bf"
-					(reference "U61")
+					(reference "U68")
 					(unit 1)
 				)
@@
 		(on_board yes)
 		(dnp no)
-		(property "Reference" "R184"
+		(property "Reference" "R220"
 			(at 78.74 97.79 90)
 			(effects
@@
 			(project "svea_powerboard_rev3"
 				(path "/3f85abf4-0b95-4c4a-b7e9-06f59ca1ea3d/5c2e021f-c2d4-49e2-8c36-9a64f1f12001/261b4c59-ebc7-47a2-bb10-0e71ece0f9bf"
-					(reference "R184")
+					(reference "R220")
 					(unit 1)
 				)
@@
 		(on_board yes)
 		(dnp no)
-		(property "Reference" "C131"
+		(property "Reference" "C137"
 			(at 190.5 124.46 90)
 			(effects
@@
 			(project "svea_powerboard_rev3"
 				(path "/3f85abf4-0b95-4c4a-b7e9-06f59ca1ea3d/5c2e021f-c2d4-49e2-8c36-9a64f1f12001/261b4c59-ebc7-47a2-bb10-0e71ece0f9bf"
-					(reference "C131")
+					(reference "C137")
 					(unit 1)
 				)
@@
 		(on_board yes)
 		(dnp no)
-		(property "Reference" "U63"
+		(property "Reference" "U70"
 			(at 144.78 74.93 0)
 			(effects
@@
 			(project "svea_powerboard_rev3"
 				(path "/3f85abf4-0b95-4c4a-b7e9-06f59ca1ea3d/5c2e021f-c2d4-49e2-8c36-9a64f1f12001/261b4c59-ebc7-47a2-bb10-0e71ece0f9bf"
-					(reference "U63")
+					(reference "U70")
 					(unit 1)
 				)
@@
 		(on_board yes)
 		(dnp no)
-		(property "Reference" "R186"
+		(property "Reference" "R222"
 			(at 209.55 68.58 90)
 			(effects
@@
 			(project "svea_powerboard_rev3"
 				(path "/3f85abf4-0b95-4c4a-b7e9-06f59ca1ea3d/5c2e021f-c2d4-49e2-8c36-9a64f1f12001/261b4c59-ebc7-47a2-bb10-0e71ece0f9bf"
-					(reference "R186")
+					(reference "R222")
 					(unit 1)
 				)
@@
 		(on_board yes)
 		(dnp no)
-		(property "Reference" "C129"
+		(property "Reference" "C135"
 			(at 116.84 93.98 90)
 			(effects
@@
 			(project "svea_powerboard_rev3"
 				(path "/3f85abf4-0b95-4c4a-b7e9-06f59ca1ea3d/5c2e021f-c2d4-49e2-8c36-9a64f1f12001/261b4c59-ebc7-47a2-bb10-0e71ece0f9bf"
-					(reference "C129")
+					(reference "C135")
 					(unit 1)
 				)
@@
 		(on_board yes)
 		(dnp no)
-		(property "Reference" "Q18"
+		(property "Reference" "Q19"
 			(at 179.07 90.17 0)
 			(effects
@@
 			(project "svea_powerboard_rev3"
 				(path "/3f85abf4-0b95-4c4a-b7e9-06f59ca1ea3d/5c2e021f-c2d4-49e2-8c36-9a64f1f12001/261b4c59-ebc7-47a2-bb10-0e71ece0f9bf"
-					(reference "Q18")
+					(reference "Q19")
 					(unit 1)
 				)

Commit message: updated some footprints, fixed board
Parts:
- renumbered C133 to C130, C135 to C132, C137 to C134, D39 to D38, Q19 to Q18, R220 to R215, R221 to R216, R222 to R217, R223 to R218, U68 to U66, U70 to U68
Changed lines of the file:
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@@
+	)
+	(junction
+		(at 207.01 101.6)
+		(diameter 0)
+		(color 0 0 0 0)
 	)
 	(junction
@@
 	(wire
 		(pts
-			(xy 207.01 110.49) (xy 207.01 99.06)
+			(xy 207.01 99.06) (xy 207.01 101.6)
 		)
 		(stroke
@@
 	(wire
 		(pts
-			(xy 207.01 110.49) (xy 186.69 110.49)
+			(xy 186.69 110.49) (xy 207.01 110.49)
 		)
 		(stroke
@@
 	(wire
 		(pts
+			(xy 207.01 101.6) (xy 207.01 110.49)
+		)
+		(stroke
+			(width 0)
+			(type default)
+		)
+	)
+	(wire
+		(pts
 			(xy 71.12 110.49) (xy 76.2 110.49)
+		)
+		(stroke
+			(width 0)
+			(type default)
+		)
+	)
+	(wire
+		(pts
+			(xy 210.82 101.6) (xy 207.01 101.6)
 		)
 		(stroke
@@
 	(global_label "Button/LOW"
 		(shape output)
-		(at 186.69 110.49 0)
+		(at 210.82 101.6 0)
 		(effects
 			(font
@@
 		)
 		(property "Intersheetrefs" "${INTERSHEET_REFS}"
-			(at 186.69 110.49 0)
+			(at 210.82 101.6 0)
 			(effects
 				(font
@@
 		(on_board yes)
 		(dnp no)
-		(property "Reference" "R221"
+		(property "Reference" "R216"
 			(at 161.29 124.46 90)
 			(effects
@@
 			(project "svea_powerboard_rev3"
 				(path "/3f85abf4-0b95-4c4a-b7e9-06f59ca1ea3d/5c2e021f-c2d4-49e2-8c36-9a64f1f12001/261b4c59-ebc7-47a2-bb10-0e71ece0f9bf"
-					(reference "R221")
+					(reference "R216")
 					(unit 1)
 				)
@@
 		(on_board yes)
 		(dnp no)
-		(property "Reference" "D39"
+		(property "Reference" "D38"
 			(at 175.26 124.46 90)
 			(effects
@@
 			(project "svea_powerboard_rev3"
 				(path "/3f85abf4-0b95-4c4a-b7e9-06f59ca1ea3d/5c2e021f-c2d4-49e2-8c36-9a64f1f12001/261b4c59-ebc7-47a2-bb10-0e71ece0f9bf"
-					(reference "D39")
+					(reference "D38")
 					(unit 1)
 				)
@@
 		(on_board yes)
 		(dnp no)
-		(property "Reference" "R223"
+		(property "Reference" "R218"
 			(at 209.55 124.46 90)
 			(effects
@@
 			(project "svea_powerboard_rev3"
 				(path "/3f85abf4-0b95-4c4a-b7e9-06f59ca1ea3d/5c2e021f-c2d4-49e2-8c36-9a64f1f12001/261b4c59-ebc7-47a2-bb10-0e71ece0f9bf"
-					(reference "R223")
+					(reference "R218")
 					(unit 1)
 				)
@@
 		(on_board yes)
 		(dnp no)
-		(property "Reference" "C133"
+		(property "Reference" "C130"
 			(at 64.77 96.52 90)
 			(effects
@@
 			(project "svea_powerboard_rev3"
 				(path "/3f85abf4-0b95-4c4a-b7e9-06f59ca1ea3d/5c2e021f-c2d4-49e2-8c36-9a64f1f12001/261b4c59-ebc7-47a2-bb10-0e71ece0f9bf"
-					(reference "C133")
+					(reference "C130")
 					(unit 1)
 				)
@@
 		(on_board yes)
 		(dnp no)
-		(property "Reference" "U68"
+		(property "Reference" "U66"
 			(at 81.28 76.2 0)
 			(effects
@@
 			(project "svea_powerboard_rev3"
 				(path "/3f85abf4-0b95-4c4a-b7e9-06f59ca1ea3d/5c2e021f-c2d4-49e2-8c36-9a64f1f12001/261b4c59-ebc7-47a2-bb10-0e71ece0f9bf"
-					(reference "U68")
+					(reference "U66")
 					(unit 1)
 				)
@@
 		(on_board yes)
 		(dnp no)
-		(property "Reference" "R220"
+		(property "Reference" "R215"
 			(at 78.74 97.79 90)
 			(effects
@@
 			(project "svea_powerboard_rev3"
 				(path "/3f85abf4-0b95-4c4a-b7e9-06f59ca1ea3d/5c2e021f-c2d4-49e2-8c36-9a64f1f12001/261b4c59-ebc7-47a2-bb10-0e71ece0f9bf"
-					(reference "R220")
+					(reference "R215")
 					(unit 1)
 				)
@@
 		(on_board yes)
 		(dnp no)
-		(property "Reference" "C137"
+		(property "Reference" "C134"
 			(at 190.5 124.46 90)
 			(effects
@@
 			(project "svea_powerboard_rev3"
 				(path "/3f85abf4-0b95-4c4a-b7e9-06f59ca1ea3d/5c2e021f-c2d4-49e2-8c36-9a64f1f12001/261b4c59-ebc7-47a2-bb10-0e71ece0f9bf"
-					(reference "C137")
+					(reference "C134")
 					(unit 1)
 				)
@@
 		(on_board yes)
 		(dnp no)
-		(property "Reference" "U70"
+		(property "Reference" "U68"
 			(at 144.78 74.93 0)
 			(effects
@@
 			(project "svea_powerboard_rev3"
 				(path "/3f85abf4-0b95-4c4a-b7e9-06f59ca1ea3d/5c2e021f-c2d4-49e2-8c36-9a64f1f12001/261b4c59-ebc7-47a2-bb10-0e71ece0f9bf"
-					(reference "U70")
+					(reference "U68")
 					(unit 1)
 				)
@@
 		(on_board yes)
 		(dnp no)
-		(property "Reference" "R222"
+		(property "Reference" "R217"
 			(at 209.55 68.58 90)
 			(effects
@@
 			(project "svea_powerboard_rev3"
 				(path "/3f85abf4-0b95-4c4a-b7e9-06f59ca1ea3d/5c2e021f-c2d4-49e2-8c36-9a64f1f12001/261b4c59-ebc7-47a2-bb10-0e71ece0f9bf"
-					(reference "R222")
+					(reference "R217")
 					(unit 1)
 				)
@@
 		(on_board yes)
 		(dnp no)
-		(property "Reference" "C135"
+		(property "Reference" "C132"
 			(at 116.84 93.98 90)
 			(effects
@@
 			(project "svea_powerboard_rev3"
 				(path "/3f85abf4-0b95-4c4a-b7e9-06f59ca1ea3d/5c2e021f-c2d4-49e2-8c36-9a64f1f12001/261b4c59-ebc7-47a2-bb10-0e71ece0f9bf"
-					(reference "C135")
+					(reference "C132")
 					(unit 1)
 				)
@@
 		(on_board yes)
 		(dnp no)
-		(property "Reference" "Q19"
+		(property "Reference" "Q18"
 			(at 179.07 90.17 0)
 			(effects
@@
 			(project "svea_powerboard_rev3"
 				(path "/3f85abf4-0b95-4c4a-b7e9-06f59ca1ea3d/5c2e021f-c2d4-49e2-8c36-9a64f1f12001/261b4c59-ebc7-47a2-bb10-0e71ece0f9bf"
-					(reference "Q19")
+					(reference "Q18")
 					(unit 1)
 				)
